File: BluetoothClassD/_autosave-BluetoothClassD.kicad_pcb (KiCad board)
At the start: 2 copper layers, 81 x 72.7 mm, 111 parts, among them IC1 ESP32-WROOM-32UE-N8R2, IC2 RESET, IC3 BOOT, IC4 TPS7A2033, J1 POWER, J2 LOW OUT, J3 HI OUT, U1 TLV9362, U2 LD1117, U3 PCM5121, U5 MCP6H01, U6 LMR51430, U7 TPA3130D2DAPR

Commit message: work
Parts:
- U7: value TPA3130D2DAPR -> TPA3130
Connections:
- U7 pad 1: unconnected-(U7-MODSEL-Pad1) -> GND
- U7 pad 12: unconnected-(U7-MUTE-Pad12) -> GND
- U7 pad 13: unconnected-(U7-AM2-Pad13) -> GND
- U7 pad 14: unconnected-(U7-AM1-Pad14) -> GND
- U7 pad 15: unconnected-(U7-AM0-Pad15) -> GND
Routing:
- net /Amp/AMP-POWER: track 124.2 -> 121.8 mm
Changed lines of the file:
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@@
 	(net 96 "/Amp/FAULT")
 	(net 97 "unconnected-(U7-SDZ-Pad2)")
-	(net 98 "unconnected-(U7-AM1-Pad14)")
-	(net 99 "unconnected-(U7-PVCC-Pad32)")
-	(net 100 "unconnected-(U7-PVCC-Pad19)")
-	(net 101 "unconnected-(U7-AM0-Pad15)")
-	(net 102 "unconnected-(U7-GVDD-Pad7)")
-	(net 103 "unconnected-(U7-MODSEL-Pad1)")
-	(net 104 "unconnected-(U7-GAIN_SLV-Pad8)")
-	(net 105 "unconnected-(U7-FAULTZ-Pad3)")
-	(net 106 "unconnected-(U7-AM2-Pad13)")
-	(net 107 "unconnected-(U7-PLIMIT-Pad6)")
-	(net 108 "unconnected-(U7-SYNC-Pad16)")
-	(net 109 "unconnected-(U7-PVCC-Pad31)")
-	(net 110 "unconnected-(U7-MUTE-Pad12)")
-	(net 111 "unconnected-(U7-AVCC-Pad17)")
-	(net 112 "unconnected-(U7-PVCC-Pad18)")
+	(net 98 "unconnected-(U7-PVCC-Pad32)")
+	(net 99 "unconnected-(U7-PVCC-Pad19)")
+	(net 100 "unconnected-(U7-GVDD-Pad7)")
+	(net 101 "unconnected-(U7-GAIN_SLV-Pad8)")
+	(net 102 "unconnected-(U7-FAULTZ-Pad3)")
+	(net 103 "unconnected-(U7-PLIMIT-Pad6)")
+	(net 104 "unconnected-(U7-SYNC-Pad16)")
+	(net 105 "unconnected-(U7-PVCC-Pad31)")
+	(net 106 "unconnected-(U7-AVCC-Pad17)")
+	(net 107 "unconnected-(U7-PVCC-Pad18)")
 	(footprint "Capacitor_SMD:C_0805_2012Metric_Pad1.18x1.45mm_HandSolder"
 		(layer "F.Cu")
@@
 			)
 		)
-		(property "Value" "TPA3130D2DAPR"
-			(at 0 0 180)
+		(property "Value" "TPA3130"
+			(at 0 6.107696 0)
 			(unlocked yes)
-			(layer "F.Fab")
+			(layer "F.SilkS")
 			(effects
 				(font
-					(size 1 1)
-					(thickness 0.15)
+					(size 0.5 0.5)
+					(thickness 0.0625)
 				)
 			)
@@
 			(size 1.27 0.3048)
 			(layers "F.Cu" "F.Mask" "F.Paste")
-			(net 103 "unconnected-(U7-MODSEL-Pad1)")
+			(net 1 "GND")
 			(pinfunction "MODSEL")
 			(pintype "input")
@@
 			(size 1.27 0.3048)
 			(layers "F.Cu" "F.Mask" "F.Paste")
-			(net 105 "unconnected-(U7-FAULTZ-Pad3)")
+			(net 102 "unconnected-(U7-FAULTZ-Pad3)")
 			(pinfunction "FAULTZ")
 			(pintype "open_collector")
@@
 			(size 1.27 0.3048)
 			(layers "F.Cu" "F.Mask" "F.Paste")
-			(net 107 "unconnected-(U7-PLIMIT-Pad6)")
+			(net 103 "unconnected-(U7-PLIMIT-Pad6)")
 			(pinfunction "PLIMIT")
 			(pintype "input")
@@
 			(size 1.27 0.3048)
 			(layers "F.Cu" "F.Mask" "F.Paste")
-			(net 102 "unconnected-(U7-GVDD-Pad7)")
+			(net 100 "unconnected-(U7-GVDD-Pad7)")
 			(pinfunction "GVDD")
 			(pintype "unspecified")
@@
 			(size 1.27 0.3048)
 			(layers "F.Cu" "F.Mask" "F.Paste")
-			(net 104 "unconnected-(U7-GAIN_SLV-Pad8)")
+			(net 101 "unconnected-(U7-GAIN_SLV-Pad8)")
 			(pinfunction "GAIN_SLV")
 			(pintype "input")
@@
 			(size 1.27 0.3048)
 			(layers "F.Cu" "F.Mask" "F.Paste")
-			(net 110 "unconnected-(U7-MUTE-Pad12)")
+			(net 1 "GND")
 			(pinfunction "MUTE")
 			(pintype "input")
@@
 			(size 1.27 0.3048)
 			(layers "F.Cu" "F.Mask" "F.Paste")
-			(net 106 "unconnected-(U7-AM2-Pad13)")
+			(net 1 "GND")
 			(pinfunction "AM2")
 			(pintype "input")
@@
 			(size 1.27 0.3048)
 			(layers "F.Cu" "F.Mask" "F.Paste")
-			(net 98 "unconnected-(U7-AM1-Pad14)")
+			(net 1 "GND")
 			(pinfunction "AM1")
 			(pintype "input")
@@
 			(size 1.27 0.3048)
 			(layers "F.Cu" "F.Mask" "F.Paste")
-			(net 101 "unconnected-(U7-AM0-Pad15)")
+			(net 1 "GND")
 			(pinfunction "AM0")
 			(pintype "input")
@@
 			(size 1.27 0.3048)
 			(layers "F.Cu" "F.Mask" "F.Paste")
-			(net 108 "unconnected-(U7-SYNC-Pad16)")
+			(net 104 "unconnected-(U7-SYNC-Pad16)")
 			(pinfunction "SYNC")
 			(pintype "bidirectional")
@@
 			(size 1.27 0.3048)
 			(layers "F.Cu" "F.Mask" "F.Paste")
-			(net 111 "unconnected-(U7-AVCC-Pad17)")
+			(net 106 "unconnected-(U7-AVCC-Pad17)")
 			(pinfunction "AVCC")
 			(pintype "power_in")
@@
 			(size 1.27 0.3048)
 			(layers "F.Cu" "F.Mask" "F.Paste")
-			(net 112 "unconnected-(U7-PVCC-Pad18)")
+			(net 107 "unconnected-(U7-PVCC-Pad18)")
 			(pinfunction "PVCC")
 			(pintype "power_in")
@@
 			(size 1.27 0.3048)
 			(layers "F.Cu" "F.Mask" "F.Paste")
-			(net 100 "unconnected-(U7-PVCC-Pad19)")
+			(net 99 "unconnected-(U7-PVCC-Pad19)")
 			(pinfunction "PVCC")
 			(pintype "power_in")
@@
 			(size 1.27 0.3048)
 			(layers "F.Cu" "F.Mask" "F.Paste")
-			(net 109 "unconnected-(U7-PVCC-Pad31)")
+			(net 105 "unconnected-(U7-PVCC-Pad31)")
 			(pinfunction "PVCC")
 			(pintype "power_in")
@@
 			(size 1.27 0.3048)
 			(layers "F.Cu" "F.Mask" "F.Paste")
-			(net 99 "unconnected-(U7-PVCC-Pad32)")
+			(net 98 "unconnected-(U7-PVCC-Pad32)")
 			(pinfunction "PVCC")
 			(pintype "power_in")
@@
 		)
 		(embedded_fonts no)
+		(model "/Users/tomwatson/Downloads/TPA3130D2DAPR (1)/DAP0032B.stp"
+			(offset
+				(xyz 0 0 0)
+			)
+			(scale
+				(xyz 1 1 1)
+			)
+			(rotate
+				(xyz 0 0 0)
+			)
+		)
 	)
 	(footprint "Custom:ESP32WROOM32UEN8R2"
@@
 	)
 	(segment
-		(start 103.378 133.858)
-		(end 105.029 132.207)
-		(width 0.2)
-		(layer "B.Cu")
-		(net 68)
-	)
-	(segment
 		(start 86.487 111.252)
 		(end 86.487 109.728)
@@
 			)
 		)
-	)
-	(zone
-		(net 1)
-		(net_name "GND")
-		(layer "B.Cu")
-		(hatch edge 0.5)
-		(priority 4)
-		(connect_pads yes
-			(clearance 0.2)
-		)
-		(min_thickness 0.2)
-		(filled_areas_thickness no)
-		(fill yes
-			(thermal_gap 0.2)
-			(thermal_bridge_width 0.2)
-			(island_removal_mode 1)
-			(island_area_min 10)
-		)
-		(polygon
-			(pts
-				(xy 97.409 132.461) (xy 97.409 122.682) (xy 93.853 122.682) (xy 93.853 132.461)
-			)
-		)
