File: BluetoothClassD/Power.kicad_sch (KiCad schematic)
At the start: 13 parts, among them J1 POWER, U6 LMR51430

Commit message: loads
Parts:
- removed J1: POWER, Connector_JST:JST_XH_B2B-XH-A_1x02_P2.50mm_Vertical, symbol Connector:Conn_01x02_Socket
- added C56: 100nF, Capacitor_SMD:C_1206_3216Metric_Pad1.33x1.80mm_HandSolder, symbol Device:C
- added Q1: DMP4015, Custom:DMP4015SK313, symbol Custom:DMP4015SK3-13
- added R40: 4K7, Resistor_SMD:R_0805_2012Metric_Pad1.20x1.40mm_HandSolder, symbol Device:R
- added R41: 100K, Resistor_SMD:R_0805_2012Metric_Pad1.20x1.40mm_HandSolder, symbol Device:R
- added R42: 1K, Resistor_SMD:R_0805_2012Metric_Pad1.20x1.40mm_HandSolder, symbol Device:R
Connections:
- net 5V: now also R40.1
- net AMP-POWER: now also Q1.2; no longer F1.2
- net POWER-IN: now reaches F1.1
- new net: C56.1, F1.2, Q1.3, R41.1
- new net: C56.2, Q1.1, R41.2, R42.2
- new net POWER-LED: R40.2
- new net POWER-SW-1: R42.1
Other:
- moved on the sheet: C16, C46, C47, C48, C49, C51, C52, L1, R38, R39, U6
