File: BluetoothClassD/BluetoothClassD.kicad_sch (KiCad schematic)
At the start: 4 parts

Commit message: solarcontroller
Changed lines of the file:
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@@
 	(paper "A4")
+	(junction
+		(at 101.6 25.4)
+		(diameter 0)
+		(color 0 0 0 0)
+	)
 	(junction
 		(at 54.61 66.04)
@@
 		(color 0 0 0 0)
 	)
-	(junction
-		(at 101.6 24.13)
-		(diameter 0)
-		(color 0 0 0 0)
-	)
 	(wire
 		(pts
@@
 	(wire
 		(pts
+			(xy 101.6 13.97) (xy 101.6 25.4)
+		)
+		(stroke
+			(width 0)
+			(type default)
+		)
+	)
+	(wire
+		(pts
 			(xy 107.95 44.45) (xy 101.6 44.45)
 		)
@@
 	(wire
 		(pts
-			(xy 101.6 25.4) (xy 101.6 24.13)
-		)
-		(stroke
-			(width 0)
-			(type default)
-		)
-	)
-	(wire
-		(pts
 			(xy 52.07 36.83) (xy 107.95 36.83)
 		)
@@
 	(wire
 		(pts
-			(xy 101.6 24.13) (xy 107.95 24.13)
+			(xy 101.6 25.4) (xy 107.95 25.4)
 		)
 		(stroke
@@
 		(pts
 			(xy 139.7 109.22) (xy 167.64 109.22)
-		)
-		(stroke
-			(width 0)
-			(type default)
-		)
-	)
-	(wire
-		(pts
-			(xy 101.6 13.97) (xy 101.6 24.13)
 		)
 		(stroke
@@
 	(sheet
 		(at 167.64 85.09)
-		(size 58.42 41.91)
+		(size 42.545 38.1)
 		(exclude_from_sim no)
 		(in_bom yes)
@@
 		)
 		(property "Sheetfile" "dac.kicad_sch"
-			(at 167.64 127.5846 0)
+			(at 167.64 123.7746 0)
 			(effects
 				(font
@@
 		)
 		(pin "5V" input
-			(at 107.95 24.13 180)
-			(effects
-				(font
+			(at 107.95 25.4 180)
+			(effects
+				(font

Commit message: loads
Parts:
- added C40: 100nF, Capacitor_SMD:C_1206_3216Metric_Pad1.33x1.80mm_HandSolder, symbol Device:C
- added J1: SYSTEM CONNECTOR 1, Connector_JST:JST_XH_B6B-XH-A_1x06_P2.50mm_Vertical, symbol Connector:Conn_01x06_Socket
- added J6: SYSTEM CONNECTOR 2, Connector_JST:JST_XH_B8B-XH-A_1x08_P2.50mm_Vertical, symbol Connector:Conn_01x08_Socket
- added R28: 1K, Resistor_SMD:R_0805_2012Metric_Pad1.20x1.40mm_HandSolder, symbol Device:R
Connections:
- new net: J6.2 (Pin_2), R28.2
- new net BT-LED: J6.7 (Pin_7)
- new net ENC-A: J6.3 (Pin_3)
- new net ENC-B: J6.4 (Pin_4)
- new net ENC-BTN: J6.5 (Pin_5)
- new net ESP-3V3: J6.1 (Pin_1)
- new net GND: C40.2, J1.2 (Pin_2), J1.4 (Pin_4), J1.6 (Pin_6), J6.6 (Pin_6), J6.8 (Pin_8)
- new net POWER-IN: J1.1 (Pin_1)
- new net POWER-LED: J1.5 (Pin_5)
- new net POWER-SW1: J1.3 (Pin_3)
- new net VOL-ADC: C40.1, R28.1
Other:
- sheet ESP32 ports: added BT-LED, ENC-A, ENC-B, ENC-BTN, VOL-ADC; removed none
- sheet Power ports: added POWER-IN, POWER-LED, POWER-SW-1; removed none

Commit message: more
Parts:
- added R31, R32, R33: 10K, Resistor_SMD:R_0603_1608Metric_Pad0.98x0.95mm_HandSolder, symbol Device:R
Connections:
- net ENC-A: now also R31.2
- net ENC-B: now also R32.2
- net ENC-BTN: now also R33.2
- net ESP-3V3: now also R31.1, R32.1, R33.1
Other:
- sheet Amp ports: added L-OUT-DAC, R-OUT-DAC; removed none
- sheet DAC ports: added L-OUT-DAC, R-OUT-DAC; removed none
