File: BluetoothClassD/Crossover.kicad_sch (KiCad schematic)
At the start: 33 parts, among them U1 TLV9362, U5 MCP6H01

Commit message: more work
Parts:
- removed C44: 100nF, Capacitor_SMD:C_1206_3216Metric_Pad1.33x1.80mm_HandSolder, symbol Device:C
- removed C72: 10uF, Capacitor_THT:CP_Radial_D4.0mm_P1.50mm, symbol Device:C_Polarized
- removed R46: 100R, Resistor_SMD:R_0805_2012Metric_Pad1.20x1.40mm_HandSolder, symbol Device:R
Connections:
- net VREF: now also C42.1, C61.1, R25.2

Commit message: more
Parts:
- C12, C13, C14, C15: value 10nF -> 10nF*
- C22, C41, C42, C45, C50: value 100nF -> 100nF*
- C37: value 47uF -> 47uF*
- C38: value 1uF -> 1uF*
- C6, C7: value 470pF -> 470pF*
- C61, C9: value 10uF -> 10uF*
- R1: value 1M -> 1M*
- R12, R8: value 10K -> 10K*
- R18, R19, R24: value 100R -> 100R*
- R2, R3, R4, R5: value RX -> RX*
- R21: value 10R -> 10R*
- R25: value 22R -> 22R*
- R27: value 100K -> 100K*
- U1: value TLV9362 -> TLV9362*
- U5: value MCP6H01 -> MCP6H01*
Changed lines of the file:
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@@
 			)
 		)
-		(property "Value" "470pF"
+		(property "Value" "470pF*"
 			(at 149.86 142.2399 0)
 			(show_name no)
@@
 			)
 		)
-		(property "Value" "100nF"
+		(property "Value" "100nF*"
 			(at 127 97.7899 0)
 			(show_name no)
@@
 			)
 		)
-		(property "Value" "22R"
+		(property "Value" "22R*"
 			(at 99.06 44.45 90)
 			(show_name no)
@@
 			)
 		)
-		(property "Value" "10nF"
+		(property "Value" "10nF*"
 			(at 99.06 142.2399 0)
 			(show_name no)
@@
 			)
 		)
-		(property "Value" "100R"
+		(property "Value" "100R*"
 			(at 137.16 180.34 90)
 			(show_name no)
@@
 			)
 		)
-		(property "Value" "47uF"
+		(property "Value" "47uF*"
 			(at 238.76 57.5309 0)
 			(show_name no)
@@
 			)
 		)
-		(property "Value" "MCP6H01"
+		(property "Value" "MCP6H01*"
 			(at 88.646 39.116 0)
 			(show_name no)
@@
 			)
 		)
-		(property "Value" "10uF"
+		(property "Value" "10uF*"
 			(at 60.198 51.816 0)
 			(show_name no)
@@
 			)
 		)
-		(property "Value" "10K"
+		(property "Value" "10K*"
 			(at 31.75 36.322 90)
 			(show_name no)
@@
 			)
 		)
-		(property "Value" "10R"
+		(property "Value" "10R*"
 			(at 247.65 49.53 90)
 			(show_name no)
@@
 			)
 		)
-		(property "Value" "100nF"
+		(property "Value" "100nF*"
 			(at 42.672 51.816 0)
 			(show_name no)
@@
 			)
 		)
-		(property "Value" "TLV9362"
+		(property "Value" "TLV9362*"
 			(at 116.84 127 0)
 			(show_name no)
@@
 			)
 		)
-		(property "Value" "100R"
+		(property "Value" "100R*"
 			(at 137.16 134.62 90)
 			(show_name no)
@@
 			)
 		)
-		(property "Value" "10nF"
+		(property "Value" "10nF*"
 			(at 95.25 172.72 90)
 			(show_name no)
@@
 			)
 		)
-		(property "Value" "RX"
+		(property "Value" "RX*"
 			(at 146.05 170.18 90)
 			(show_name no)
@@
 		(fields_autoplaced yes)
 		(property "Reference" "C61"
-			(at 121.92 52.4509 0)
+			(at 120.65 52.4509 0)
 			(show_name no)
 			(do_not_autoplace no)
@@
 			)
 		)
-		(property "Value" "10uF"
-			(at 121.92 54.9909 0)
+		(property "Value" "10uF*"
+			(at 120.65 54.9909 0)
 			(show_name no)
 			(do_not_autoplace no)
@@
 			)
 		)
-		(property "Value" "100nF"
+		(property "Value" "100nF*"
 			(at 227.33 58.4199 0)
 			(show_name no)
@@
 			)
 		)
-		(property "Value" "100nF"
+		(property "Value" "100nF*"
 			(at 109.22 39.3699 0)
 			(show_name no)
@@
 			)
 		)
-		(property "Value" "RX"
+		(property "Value" "RX*"
 			(at 73.66 132.08 90)
 			(show_name no)
@@
 			)
 		)
-		(property "Value" "1uF"
+		(property "Value" "1uF*"
 			(at 35.814 130.81 90)
 			(show_name no)
@@
 			)
 		)
-		(property "Value" "100nF"
+		(property "Value" "100nF*"
 			(at 134.62 55.8799 0)
 			(show_name no)
@@
 			)
 		)
-		(property "Value" "TLV9362"
+		(property "Value" "TLV9362*"
 			(at 116.84 172.72 0)
 			(show_name no)
@@
 			)
 		)
-		(property "Value" "1M"
+		(property "Value" "1M*"
 			(at 144.78 125.73 90)
 			(show_name no)
@@
 			)
 		)
-		(property "Value" "10nF"
+		(property "Value" "10nF*"
 			(at 95.25 113.03 90)
 			(show_name no)
@@
 			)
 		)
-		(property "Value" "RX"
+		(property "Value" "RX*"
 			(at 88.9 132.08 90)
 			(show_name no)
@@
 			)
 		)
-		(property "Value" "100R"
+		(property "Value" "100R*"
 			(at 62.23 41.91 90)
 			(show_name no)
@@
 			)
 		)
-		(property "Value" "10nF"
+		(property "Value" "10nF*"
 			(at 72.39 172.72 90)
 			(show_name no)
@@
 			)
 		)
-		(property "Value" "TLV9362"
+		(property "Value" "TLV9362*"
 			(at 107.442 97.79 90)
 			(show_name no)
@@
 			)
 		)
-		(property "Value" "100K"
+		(property "Value" "100K*"
 			(at 62.23 124.46 90)
 			(show_name no)
@@
 			)
 		)
-		(property "Value" "470pF"
+		(property "Value" "470pF*"
 			(at 149.86 187.9599 0)
 			(show_name no)
@@
 			)
 		)
-		(property "Value" "10K"
+		(property "Value" "10K*"
 			(at 31.75 51.308 90)
 			(show_name no)
@@
 			)
 		)
-		(property "Value" "RX"
+		(property "Value" "RX*"
 			(at 96.52 163.83 90)
 			(show_name no)
