File: BluetoothClassD/ESP32.kicad_sch (KiCad schematic)
At the start: 15 parts, among them IC1 ESP32-WROOM-32UE-N8R2, IC2 RESET, IC3 BOOT, U2 LD1117

Commit message: work
Changed lines of the file:
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@@
+		)
+	)
+	(hierarchical_label "FAULT"
+		(shape output)
+		(at 227.33 44.45 0)
+		(effects
+			(font
+				(size 1.27 1.27)
+			)
+			(justify left)
 		)
 	)
@@
 		)
 	)
+	(hierarchical_label "SDZ"
+		(shape output)
+		(at 227.33 46.99 0)
+		(effects
+			(font
+				(size 1.27 1.27)
+			)
+			(justify left)
+		)
+	)

Commit message: solarcontroller
Connections:
- net FAULT: now also IC1.6 (IO34)
- net SDZ: now also IC1.12 (IO27)
Changed lines of the file:
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@@
+	(wire
+		(pts
+			(xy 107.95 92.71) (xy 128.27 92.71)
+		)
+		(stroke
+			(width 0)
+			(type default)
+		)
+	)
 	(wire
 		(pts
@@
 		(pts
 			(xy 260.35 80.01) (xy 260.35 66.04)
+		)
+		(stroke
+			(width 0)
+			(type default)
+		)
+	)
+	(wire
+		(pts
+			(xy 107.95 77.47) (xy 128.27 77.47)
 		)
 		(stroke
@@
 	(hierarchical_label "FAULT"
 		(shape output)
-		(at 227.33 44.45 0)
-		(effects
-			(font
-				(size 1.27 1.27)
-			)
-			(justify left)
+		(at 107.95 77.47 180)
+		(effects
+			(font
+				(size 1.27 1.27)
+			)
+			(justify right)
 		)
 	)
@@
 	(hierarchical_label "SDZ"
 		(shape output)
-		(at 227.33 46.99 0)
-		(effects
-			(font
-				(size 1.27 1.27)
-			)
-			(justify left)
-		)
-	)
+		(at 107.95 92.71 180)
+		(effects
+			(font
+				(size 1.27 1.27)
+			)
+			(justify right)
+		)
+	)

Commit message: signalpoweron
Parts:
- added J4: PROG, Connector_PinHeader_2.54mm:PinHeader_1x04_P2.54mm_Vertical, symbol Connector:Conn_01x04_Socket
Connections:
- net 3.3V: now also J4.3 (Pin_3)
- net GND: now also J4.4 (Pin_4)
- net RX: now also J4.2 (Pin_2)
- net TX: now also J4.1 (Pin_1)

Commit message: loads
Connections:
- net ENC-BTN: now reaches IC1.30 (IO18)
- net BT-LED: now reaches IC1.31 (IO19)
- net VOL-ADC: now reaches IC1.7 (IO35)
- net ENC-A: now reaches IC1.8 (IO32)
- net ENC-B: now reaches IC1.9 (IO33)
Changed lines of the file:
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@@
+	(wire
+		(pts
+			(xy 107.95 82.55) (xy 128.27 82.55)
+		)
+		(stroke
+			(width 0)
+			(type default)
+		)
+	)
 	(wire
 		(pts
@@
 	(wire
 		(pts
+			(xy 166.37 77.47) (xy 199.39 77.47)
+		)
+		(stroke
+			(width 0)
+			(type default)
+		)
+	)
+	(wire
+		(pts
 			(xy 227.33 85.09) (xy 227.33 86.36)
 		)
@@
 	(wire
 		(pts
+			(xy 166.37 80.01) (xy 199.39 80.01)
+		)
+		(stroke
+			(width 0)
+			(type default)
+		)
+	)
+	(wire
+		(pts
 			(xy 186.69 118.11) (xy 186.69 120.65)
 		)
@@
 	(wire
 		(pts
+			(xy 107.95 85.09) (xy 128.27 85.09)
+		)
+		(stroke
+			(width 0)
+			(type default)
+		)
+	)
+	(wire
+		(pts
 			(xy 186.69 59.69) (xy 186.69 64.77)
 		)
@@
 		(pts
 			(xy 107.95 39.37) (xy 107.95 44.45)
+		)
+		(stroke
+			(width 0)
+			(type default)
+		)
+	)
+	(wire
+		(pts
+			(xy 107.95 80.01) (xy 128.27 80.01)
 		)
 		(stroke
@@
 			)
 			(justify left bottom)
+		)
+	)
+	(hierarchical_label "ENC-B"
+		(shape input)
+		(at 107.95 85.09 180)
+		(effects
+			(font
+				(size 1.27 1.27)
+			)
+			(justify right)
+		)
+	)
+	(hierarchical_label "ENC-BTN"
+		(shape input)
+		(at 199.39 77.47 0)
+		(effects
+			(font
+				(size 1.27 1.27)
+			)
+			(justify left)
+		)
+	)
+	(hierarchical_label "ENC-A"
+		(shape input)
+		(at 107.95 82.55 180)
+		(effects
+			(font
+				(size 1.27 1.27)
+			)
+			(justify right)
 		)
 	)
@@
 		)
 	)
+	(hierarchical_label "BT-LED"
+		(shape input)
+		(at 199.39 80.01 0)
+		(effects
+			(font
+				(size 1.27 1.27)
+			)
+			(justify left)
+		)
+	)
 	(hierarchical_label "SDZ"
 		(shape output)
@@
 		(effects
 			(font
+				(size 1.27 1.27)
+			)
+			(justify right)
+		)
+	)
+	(hierarchical_label "VOL-ADC"
+		(shape input)
+		(at 107.95 80.01 180)
+		(effects
+			(font

Commit message: more
Parts:
- removed R6, R7: 4K7, Resistor_SMD:R_0805_2012Metric_Pad1.20x1.40mm_HandSolder, symbol Device:R
- added C59: 220nF, Capacitor_SMD:C_0805_2012Metric_Pad1.18x1.45mm_HandSolder, symbol Device:C
- added R34: 4K7, Resistor_SMD:R_0805_2012Metric_Pad1.20x1.40mm_HandSolder, symbol Device:R
Connections:
- net GND: now also C59.2
- net SDZ: now also C59.1, R34.2; no longer IC1.12 (IO27)
- new net: IC1.12 (IO27), R34.1
