File: BluetoothClassD/dac.kicad_sch (KiCad schematic)
At the start: 11 parts, among them IC4 TPS7A2033, U3 PCM5121

Commit message: more work
Parts:
- added C43, C53, C55, C58: 100nF, Capacitor_SMD:C_1206_3216Metric_Pad1.33x1.80mm_HandSolder, symbol Device:C
- added C44: 47uF, Capacitor_THT:CP_Radial_D8.0mm_P2.50mm, symbol Device:C_Polarized
- added C54: 10uF, Capacitor_THT:CP_Radial_D4.0mm_P2.00mm, symbol Device:C_Polarized
- added C57: 2.2uF, Capacitor_SMD:C_0805_2012Metric_Pad1.18x1.45mm_HandSolder, symbol Device:C
Connections:
- net DAC-3V3: now also C43.1, C44.1, C53.1, C55.1
- net GND: now also C43.2, C44.2, C53.2, C54.2, C55.2, C57.2, C58.2
- net at U3.26 (LDOO): now also C54.1, C58.1
- net at U3.5 (VNEG): now also C57.1

Commit message: more
Parts:
- added J5: LINE IN, Connector_JST:JST_XH_B2B-XH-A_1x02_P2.50mm_Vertical, symbol Connector:Conn_01x02_Socket
- added R35, R36: 4K7, Resistor_SMD:R_0805_2012Metric_Pad1.20x1.40mm_HandSolder, symbol Device:R
- added R37, R43: 0R*, Resistor_SMD:R_0805_2012Metric_Pad1.20x1.40mm_HandSolder, symbol Device:R
- added R63: DAC, Resistor_SMD:R_0805_2012Metric_Pad1.20x1.40mm_HandSolder, symbol Device:R
- added R64: L-IN, Resistor_SMD:R_0805_2012Metric_Pad1.20x1.40mm_HandSolder, symbol Device:R
- R17, R20: value 15K -> 15K*
Connections:
- net DAC-3V3: now also U3.25 (XSMT), R35.2, R36.2
- net GND: now also U3.20 (SCK), J5.2 (Pin_2)
- net MONO-AUDIO: now also R63.2, R64.1; no longer R17.2, R20.2
- net SCL: now also R35.1
- net SDA: now also R36.1
- net at C19.1, R16.2, R20.1: now also R43.1
- net at C20.1, R15.2, R17.1: now also R37.1
- new net: J5.1 (Pin_1), R64.2
- new net: R17.2, R20.2, R63.1
- new net L-OUT-DAC: R37.2
- new net R-OUT-DAC: R43.2
Other:
- moved on the sheet: R17, R20
