File: BluetoothClassD/BluetoothClassD.kicad_pcb (KiCad board)
At the start: 2 copper layers, 81 x 72.7 mm, 111 parts, among them IC1 ESP32-WROOM-32UE-N8R2, IC2 RESET, IC3 BOOT, IC4 TPS7A2033, J1 POWER, J2 LOW OUT, J3 HI OUT, U1 TLV9362, U2 LD1117, U3 PCM5121, U5 MCP6H01, U6 LMR51430, U7 TPA3130D2DAPR

Commit message: solarcontroller
Parts:
- removed C40: 1uF, Capacitor_SMD:C_1206_3216Metric_Pad1.33x1.80mm_HandSolder
- added C39: 1uF, Capacitor_SMD:C_1206_3216Metric_Pad1.33x1.80mm_HandSolder, F.Cu at (102.1, 128.7)
- R22: value 1K -> 5K6
- R23: value 100K -> 10K
- R26: value 10K -> 100K
- U7: value TPA3130D2DAPR -> TPA3130
- moved R26 3.95 mm to (96.9, 135.5), turned to 180 degrees
- moved R22 2.03 mm to (96.9, 137.5), turned to 180 degrees
- moved R23 2.03 mm to (96.9, 139.6), turned to 180 degrees
Connections:
- C16 pad 1: /Amp/AMP-POWER -> /Amp/PVCC
- C31 pad 1: /Amp/AMP-POWER -> /Amp/PVCC
- C32 pad 1: /Amp/AMP-POWER -> /Amp/PVCC
- C33 pad 1: /Amp/AMP-POWER -> /Amp/PVCC
- C34 pad 1: /Amp/AMP-POWER -> /Amp/PVCC
- C35 pad 1: /Amp/AMP-POWER -> /Amp/PVCC
- C36 pad 1: /Amp/AMP-POWER -> /Amp/PVCC
- C46 pad 1: /Amp/AMP-POWER -> /Amp/PVCC
- C47 pad 1: /Amp/AMP-POWER -> /Amp/PVCC
- F1 pad 2: /Amp/AMP-POWER -> /Amp/PVCC
- IC1 pad 12: unconnected-(IC1-IO27-Pad12) -> /Amp/SDZ
- IC1 pad 6: unconnected-(IC1-IO34-Pad6) -> /Amp/FAULTZ
- R21 pad 2: /Amp/AMP-POWER -> /Amp/PVCC
- R22 pad 1: /Amp/STBY -> GND
- R22 pad 2: Net-(U4-~{SD}) -> Net-(U7-GAIN_SLV)
- R23 pad 1: GND -> /ESP32/3V3-ESP
- R23 pad 2: Net-(U4-~{SD}) -> /Amp/FAULTZ
- R26 pad 1: /Amp/FAULT -> GND
- R26 pad 2: /ESP32/3V3-ESP -> /Amp/SDZ
- U6 pad 3: /Amp/AMP-POWER -> /Amp/PVCC
- U6 pad 5: /Amp/AMP-POWER -> /Amp/PVCC
- U7 pad 1: unconnected-(U7-MODSEL-Pad1) -> GND
- U7 pad 12: unconnected-(U7-MUTE-Pad12) -> GND
- U7 pad 13: unconnected-(U7-AM2-Pad13) -> GND
- U7 pad 14: unconnected-(U7-AM1-Pad14) -> GND
- U7 pad 15: unconnected-(U7-AM0-Pad15) -> GND
- U7 pad 17: unconnected-(U7-AVCC-Pad17) -> /Amp/PVCC
- U7 pad 18: unconnected-(U7-PVCC-Pad18) -> /Amp/PVCC
- U7 pad 19: unconnected-(U7-PVCC-Pad19) -> /Amp/PVCC
- U7 pad 2: unconnected-(U7-SDZ-Pad2) -> /Amp/SDZ
- U7 pad 3: unconnected-(U7-FAULTZ-Pad3) -> /Amp/FAULTZ
- U7 pad 31: unconnected-(U7-PVCC-Pad31) -> /Amp/PVCC
- U7 pad 32: unconnected-(U7-PVCC-Pad32) -> /Amp/PVCC
- U7 pad 6: unconnected-(U7-PLIMIT-Pad6) -> Net-(U7-GVDD)
- U7 pad 7: unconnected-(U7-GVDD-Pad7) -> Net-(U7-GVDD)
- U7 pad 8: unconnected-(U7-GAIN_SLV-Pad8) -> Net-(U7-GAIN_SLV)
Routing:
- net /Amp/AMP-POWER: track 124.2 -> 0.00 mm, vias 3 -> 0
- net /Amp/PVCC: track 0.00 -> 121.7 mm, vias 0 -> 9
- net /Amp/FAULTZ: track 0.00 -> 68.1 mm, vias 0 -> 2
- net /Amp/SDZ: track 0.00 -> 43.8 mm, vias 0 -> 2
- net Net-(U7-GAIN_SLV): track 0.00 -> 12.7 mm
- net /ESP32/3V3-ESP: track 231.6 -> 223.8 mm
- net Net-(U7-GVDD): track 0.00 -> 2.28 mm
- net Net-(J3-Pin_1): track 12.5 -> 11.0 mm
- net Net-(J2-Pin_2): track 10.6 -> 9.61 mm
- net /Crossover/VREF: track 34.2 -> 33.3 mm
- net /DAC/5V: track 62.4 -> 61.5 mm
- net /Crossover/XOVERPOWER: track 58.6 -> 57.9 mm
- net Net-(U7-OUTNL): track 7.89 -> 7.26 mm
- net /DAC/SDA: track 27.1 -> 26.5 mm
- net GND: track 2.65 -> 2.63 mm, vias 260 -> 289
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- added copper zone on B.Cu, net /Amp/PVCC
- added copper zone on F.Cu, net /Amp/PVCC

Commit message: signalpoweron
Parts:
- added J4: PROG, Connector_PinHeader_2.54mm:PinHeader_1x04_P2.54mm_Vertical, F.Cu at (129.3, 109.7)
Routing:
- net /ESP32/3V3-ESP: track 223.8 -> 292.4 mm, vias 7 -> 8
- net /ESP32/RX: track 0.00 -> 27.3 mm
- net /ESP32/TX: track 0.00 -> 25.8 mm
- net /Amp/FAULTZ: track 68.1 -> 64.6 mm
- net /DAC/SDA: track 26.5 -> 28.5 mm
- net /DAC/SCL: track 41.0 -> 39.4 mm
- net GND: vias 289 -> 302
Other:
- board text added: "+ -"
- board text added: "ESP32 Bluetooth - PCM5121 - TPA3130 Active Crossover Tom Watson Audio - 2026"
- board text added: "POWER 10-15V"
- board text added: "TX RX 3V3 GND"
- board text removed: "10-18V MAX"
- board text removed: "ESP32 Bluetooth - PCM5121 - TPA3110 Active Crossover Tom Watson Audio - 2026"

Commit message: m0re
Routing:
- net Net-(J2-Pin_1): track 11.3 -> 12.7 mm
- net Net-(J3-Pin_1): track 11.0 -> 12.0 mm
- net /Crossover/VREF: track 33.5 -> 34.2 mm
- net /Crossover/MONO-AUDIO: vias 1 -> 0

Commit message: loads
Parts:
- added C40: 100nF, Capacitor_SMD:C_1206_3216Metric_Pad1.33x1.80mm_HandSolder, F.Cu at (111.8, 73.8)
- added C56: 100nF, Capacitor_SMD:C_1206_3216Metric_Pad1.33x1.80mm_HandSolder, F.Cu at (82.8, 80.8)
- added J6: SYSTEM CONNECTOR 2, Connector_JST:JST_XH_B8B-XH-A_1x08_P2.50mm_Vertical, F.Cu at (105.7, 66.8)
- added Q1: DMP4015, Custom:DMP4015SK313, F.Cu at (74.9, 80.8)
- added R28: 1K, Resistor_SMD:R_0805_2012Metric_Pad1.20x1.40mm_HandSolder, F.Cu at (107.3, 73.7)
- added R40: 4K7, Resistor_SMD:R_0805_2012Metric_Pad1.20x1.40mm_HandSolder, F.Cu at (88.6, 77.0)
- added R41: 100K, Resistor_SMD:R_0805_2012Metric_Pad1.20x1.40mm_HandSolder, F.Cu at (85.1, 80.8)
- added R42: 1K, Resistor_SMD:R_0805_2012Metric_Pad1.20x1.40mm_HandSolder, F.Cu at (83.6, 77.0)
- J1: value POWER -> SYSTEM CONNECTOR 1; footprint Connector_JST:JST_XH_B2B-XH-A_1x02_P2.50mm_Vertical -> Connector_JST:JST_XH_B6B-XH-A_1x06_P2.50mm_Vertical
- moved J1 13.2 mm to (78.4, 66.8), turned to 0 degrees
- moved F1 12.2 mm to (72.2, 73.2), turned to 0 degrees
- moved H3 10.9 mm to (141.0, 66.5)
- moved H1 10.9 mm to (70.2, 66.5)
- moved C48 2.28 mm to (96.8, 87.1)
- moved C16 1.02 mm to (71.7, 96.8)
- moved G*** 0.64 mm to (102.6, 116.1)
- moved C3 0.38 mm to (101.0, 91.4), turned to 90 degrees
Connections:
- net /ESP32/3V3-ESP renamed /ESP-3V3
- F1 pad 1: Net-(J1-Pin_2) -> /POWER-IN
- F1 pad 2: /Amp/PVCC -> Net-(C56-Pad1)
- IC1 pad 30: unconnected-(IC1-IO18-Pad30) -> /ENC-BTN
- IC1 pad 31: unconnected-(IC1-IO19-Pad31) -> /BT-LED
- IC1 pad 7: unconnected-(IC1-IO35-Pad7) -> /VOL-ADC
- IC1 pad 8: unconnected-(IC1-IO32-Pad8) -> /ENC-A
- IC1 pad 9: unconnected-(IC1-IO33-Pad9) -> /ENC-B
- J1 pad 1: GND -> /POWER-IN
- J1 pad 2: Net-(J1-Pin_2) -> GND
Routing:
- net /ESP-3V3: track 292.4 -> 242.8 mm
- net /ENC-BTN: track 0.00 -> 38.0 mm, vias 0 -> 1
- net /ENC-B: track 0.00 -> 36.3 mm, vias 0 -> 1
- net /ENC-A: track 0.00 -> 35.6 mm, vias 0 -> 1
- net /BT-LED: track 0.00 -> 34.0 mm, vias 0 -> 1
- net /VOL-ADC: track 0.00 -> 28.9 mm, vias 0 -> 2
- net Net-(C56-Pad2): track 0.00 -> 15.0 mm
- net Net-(C56-Pad1): track 0.00 -> 14.2 mm
- net /POWER-IN: track 0.00 -> 12.1 mm
- net /POWER-SW1: track 0.00 -> 10.5 mm
- net GND: track 2.63 -> 13.0 mm, vias 302 -> 317
- net /POWER-LED: track 0.00 -> 9.28 mm
- net Net-(J1-Pin_2): track 9.00 -> 0.00 mm
- net /DAC/5V: track 61.5 -> 69.5 mm
- net Net-(J6-Pin_2): track 0.00 -> 6.93 mm
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Other:
- board size 81 x 72.7 mm -> 81 x 85 mm
- board text added: "3V3"
- board text added: "BT LED +"
- board text added: "BT LED -"
- board text added: "ENC A"
- board text added: "ENC B"
- board text added: "END BTN"
- board text added: "GND"
- board text added: "POWER IN +"
- board text added: "POWER IN -"
- board text added: "POWER LED +"
- board text added: "POWER LED -"
- board text added: "POWER RATING 10-15V"
- board text added: "POWER SWITCH"
- board text added: "VOL ADC"
- board text removed: "+ -"
- board text removed: "POWER 10-15V"

Commit message: more
Parts:
- removed R6, R7: 4K7, Resistor_SMD:R_0805_2012Metric_Pad1.20x1.40mm_HandSolder
- added C59: 220nF, Capacitor_SMD:C_0805_2012Metric_Pad1.18x1.45mm_HandSolder, F.Cu at (104.9, 109.2)
- added J5: LINE IN, Connector_JST:JST_XH_B2B-XH-A_1x02_P2.50mm_Vertical, F.Cu at (140.9, 131.8)
- added R29: 100R, Resistor_SMD:R_0805_2012Metric_Pad1.20x1.40mm_HandSolder, F.Cu at (115.8, 132.1)
- added R30: 100R, Resistor_SMD:R_0805_2012Metric_Pad1.20x1.40mm_HandSolder, F.Cu at (115.8, 116.6)
- added R31: 10K, Resistor_SMD:R_0603_1608Metric_Pad0.98x0.95mm_HandSolder, F.Cu at (101.6, 67.4)
- added R32: 10K, Resistor_SMD:R_0603_1608Metric_Pad0.98x0.95mm_HandSolder, F.Cu at (99.8, 67.4)
- added R33: 10K, Resistor_SMD:R_0603_1608Metric_Pad0.98x0.95mm_HandSolder, F.Cu at (98.0, 67.4)
- added R34: 4K7, Resistor_SMD:R_0805_2012Metric_Pad1.20x1.40mm_HandSolder, F.Cu at (101.1, 103.1)
- added R35: 4K7, Resistor_SMD:R_0805_2012Metric_Pad1.20x1.40mm_HandSolder, F.Cu at (141.5, 97.8)
- added R36: 4K7, Resistor_SMD:R_0805_2012Metric_Pad1.20x1.40mm_HandSolder, F.Cu at (141.5, 95.8)
- added R37: 0R*, Resistor_SMD:R_0805_2012Metric_Pad1.20x1.40mm_HandSolder, F.Cu at (122.0, 118.6)
- added R43: 0R*, Resistor_SMD:R_0805_2012Metric_Pad1.20x1.40mm_HandSolder, F.Cu at (116.0, 124.8)
- added R63: DAC, Resistor_SMD:R_0805_2012Metric_Pad1.20x1.40mm_HandSolder, F.Cu at (140.2, 104.9)
- added R64: L-IN, Resistor_SMD:R_0805_2012Metric_Pad1.20x1.40mm_HandSolder, F.Cu at (140.2, 125.0)
- C12, C13, C14, C15: value 10nF -> 10nF*
- C22, C41, C42, C45, C50: value 100nF -> 100nF*
- C31, C32: footprint Capacitor_SMD:C_0805_2012Metric_Pad1.18x1.45mm_HandSolder -> Capacitor_SMD:C_0603_1608Metric_Pad1.08x0.95mm_HandSolder
- C37: value 47uF -> 47uF*
- C38: value 1uF -> 1uF*
- C6, C7: value 470pF -> 470pF*
- C61, C9: value 10uF -> 10uF*
- J2: value LOW OUT -> LOW/R OUT
- J3: value HI OUT -> HI/L OUT
- R1: value 1M -> 1M*
- R12, R8: value 10K -> 10K*
- R17, R20: value 15K -> 15K*
- R18, R19, R24: value 100R -> 100R*
- R2, R3, R4, R5: value RX -> RX*
- R21: value 10R -> 10R*
- R25: value 22R -> 22R*
- R27: value 100K -> 100K*
- U1: value TLV9362 -> TLV9362*
- U5: value MCP6H01 -> MCP6H01*
- moved C19 2.15 mm to (138.2, 104.9), turned to -90 degrees
- moved R17 2.15 mm to (130.0, 104.9), turned to 90 degrees
- moved C20 1.92 mm to (128.0, 104.9), turned to -90 degrees
- moved R20 1.92 mm to (136.1, 104.9), turned to 90 degrees
- moved C23 1.09 mm to (86.6, 123.2)
- moved C26 1.02 mm to (86.6, 132.3)
- moved C25 0.90 mm to (86.6, 129.0)
- moved C24 0.87 mm to (86.6, 126.4)
- moved C32 0.36 mm to (90.7, 118.6)
- moved C38 0.15 mm to (136.2, 124.7)
- moved R15 0.12 mm to (132.1, 104.9)
- moved R16 0.12 mm to (134.1, 104.9)
Connections:
- C10 pad 1: GND -> Net-(C10-Pad1)
- C5 pad 1: GND -> Net-(C5-Pad1)
- IC1 pad 12: /Amp/SDZ -> Net-(IC1-IO27)
- R17 pad 2: /Crossover/MONO-AUDIO -> Net-(R17-Pad2)
- R20 pad 2: /Crossover/MONO-AUDIO -> Net-(R17-Pad2)
- U3 pad 20: unconnected-(U3-SCK-Pad20) -> GND
- U3 pad 25: unconnected-(U3-XSMT-Pad25) -> /DAC/DAC-3V3
Routing:
- net /ESP-3V3: track 242.8 -> 341.9 mm, vias 8 -> 5
- net Net-(C19-Pad1): track 4.78 -> 33.6 mm, vias 0 -> 2
- net /Crossover/XOVERPOWER: track 57.9 -> 79.3 mm, vias 3 -> 4
- net /ENC-BTN: track 38.0 -> 57.4 mm
- net Net-(C20-Pad1): track 4.89 -> 23.1 mm, vias 0 -> 2
- net /DAC/DAC-3V3: track 68.3 -> 83.5 mm, vias 3 -> 5
- net /ENC-B: track 36.3 -> 51.1 mm
- net /Crossover/MONO-AUDIO: track 37.2 -> 22.5 mm
- net /DAC/SCL: track 39.4 -> 27.0 mm
- net Net-(R17-Pad2): track 0.00 -> 11.9 mm
- net /ENC-A: track 35.6 -> 45.6 mm
- net Net-(J5-Pin_1): track 0.00 -> 6.98 mm
- net Net-(IC1-IO27): track 0.00 -> 3.27 mm
- net Net-(C10-Pad1): track 0.00 -> 2.91 mm
- net /Amp/SDZ: track 43.8 -> 41.2 mm
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Other:
- board text added: "FIT XOVER AND 15K* FOR ACTIVE XOVER DNP 0R* DNP XOVER(*)/15K* AND FIT 0R* FOR ESP XOVER"
- board text added: "GND SIG"
- board text added: "TWEETER - LEFT WOOFER - RIGHT"

Commit message: more
Parts:
- added R44: 47K, Resistor_SMD:R_0805_2012Metric_Pad1.20x1.40mm_HandSolder, F.Cu at (116.1, 122.6)
- added R45: 47K, Resistor_SMD:R_0805_2012Metric_Pad1.20x1.40mm_HandSolder, F.Cu at (116.0, 130.3)
- moved R29 2.27 mm to (116.0, 134.4), turned to 90 degrees
- moved H4 2.13 mm to (141.5, 141.9)
- moved H2 1.94 mm to (69.7, 141.9)
- moved R43 1.21 mm to (117.0, 125.5), turned to 0 degrees
- moved H1 0.63 mm to (69.7, 66.2)
- moved H3 0.54 mm to (141.4, 66.2)
Routing:
- net /Amp/LOW-AUDIO: track 10.3 -> 12.2 mm
- net /Amp/HI-AUDIO: track 10.3 -> 11.7 mm
- net /ESP-3V3: track 341.9 -> 342.8 mm
- net GND: vias 321 -> 329
Other:
- board text added: "ENC BTN"
- board text removed: "END BTN"
