File: SolarLights/Buck.kicad_sch (KiCad schematic)
At the start: 9 parts

Commit message: solar lights
Parts:
- added 1K13: 47K, Resistor_SMD:R_0805_2012Metric_Pad1.20x1.40mm_HandSolder, symbol Device:R
- added D3: CH4, LED_THT:LED_D5.0mm, symbol Device:LED
- added Q1: AO3400A, Package_TO_SOT_SMD:SOT-23, symbol Transistor_FET:AO3400A
- added R2: 100R, Resistor_SMD:R_0805_2012Metric_Pad1.20x1.40mm_HandSolder, symbol Device:R
- added R3: 100K, Resistor_SMD:R_0805_2012Metric_Pad1.20x1.40mm_HandSolder, symbol Device:R
- added R4: 2K2, Resistor_SMD:R_0805_2012Metric_Pad1.20x1.40mm_HandSolder, symbol Device:R
- R1: renamed from 1K1; footprint Resistor_THT:R_Axial_DIN0207_L6.3mm_D2.5mm_P10.16mm_Horizontal -> Resistor_SMD:R_0805_2012Metric_Pad1.20x1.40mm_HandSolder
Connections:
- net CONTROL: now also 1K13.2
- net GND: now also Q1.2 (S), R3.2; no longer -   +3.2 (Pin_2)
- net 3V: now reaches -   +3.1 (Pin_1), 100uH1.2, 220uF1.1, 5K1.1
- net 3V: now also D3.2 (A)
- new net: Q1.1 (G), R2.2, R3.1
- new net: D3.1 (K), R4.1
- new net: -   +3.2 (Pin_2), Q1.3 (D), R4.2
- new net 5V: 1K13.1
- new net PWM-DRIVE: R2.1
Other:
- moved on the sheet: - +3

Commit message: loads
Changed lines of the file:
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@@
 	(wire
 		(pts
-			(xy 182.88 72.39) (xy 182.88 77.47)
+			(xy 182.88 62.23) (xy 182.88 77.47)
 		)
 		(stroke
@@
 	)
 	(label "3V"
-		(at 182.88 72.39 90)
+		(at 182.88 62.23 90)
 		(effects
 			(font
@@
 		(dnp no)
 		(property "Reference" "R2"
-			(at 193.04 105.41 90)
+			(at 191.516 105.41 90)
 			(show_name no)
 			(do_not_autoplace no)
@@
 		(dnp no)
 		(property "Reference" "R3"
-			(at 199.39 111.252 0)
-			(show_name no)
-			(do_not_autoplace no)
+			(at 199.136 109.474 0)
+			(show_name no)
+			(do_not_autoplace no)
