File: SignalPowerOn/SignalPowerOn.kicad_pcb (KiCad board)
At the start: 2 copper layers, 81.3 x 82 mm, 43 parts, among them J1 LIVE IN, J2 NEUTRAL IN, J3 AUDIO IN, J4 NEUTRAL OUT, J5 SWITCHED LIVE, K1 SDT-S-112DMR, Q1 2N7000, Q2 BC549, T1 Block AVB 2,3/2/6, U1 LM358

Commit message: work
Parts:
- moved G*** 88.3 mm to (151.5, 121.4)
- moved R8 83.7 mm to (155.7, 78.9), turned to -90 degrees
- moved R3 71.8 mm to (153.4, 78.9), turned to -90 degrees
- moved R7 68.6 mm to (158.8, 91.6), turned to 90 degrees
- moved H2 67.3 mm to (163.1, 63.2)
- moved C7 66.3 mm to (146.0, 68.2)
- moved C4 63.8 mm to (139.1, 103.4), turned to -90 degrees
- moved R6 61.1 mm to (143.4, 95.2), turned to 180 degrees
- moved R10 60.6 mm to (159.4, 69.7)
- moved R12 59.5 mm to (155.7, 83.7), turned to -90 degrees
- moved R11 59.2 mm to (163.6, 69.7)
- moved R13 58.2 mm to (158.9, 83.7), turned to 90 degrees
- moved H3 57.4 mm to (162.9, 122.0)
- moved C5 57.0 mm to (144.8, 106.2), turned to -90 degrees
- moved R14 55.9 mm to (155.4, 99.4)
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Routing:
- net Net-(D4-K): track 0.00 -> 32.3 mm, vias 0 -> 1
- net Net-(Q1-G): track 0.00 -> 18.5 mm
- net Net-(U1A--): track 0.00 -> 17.7 mm
- net Net-(C7-Pad2): track 0.00 -> 17.5 mm
- net GND: track 30.3 -> 42.4 mm, vias 0 -> 9
- net Net-(C5-Pad1): track 0.00 -> 11.9 mm, vias 0 -> 1
- net Net-(D5-K): track 0.00 -> 11.5 mm
- net GNDD: track 0.00 -> 9.82 mm
- net Net-(U1B--): track 9.72 -> 19.1 mm
- net Net-(D2-A): track 0.00 -> 8.50 mm
- net Net-(U1A-+): track 0.00 -> 6.83 mm
- net Net-(U1B-+): track 0.00 -> 6.47 mm
- net /VCC: track 81.1 -> 86.6 mm, vias 0 -> 1
- net Net-(J3-Pin_3): track 5.12 -> 10.3 mm
- net Net-(J3-Pin_1): track 5.16 -> 10.1 mm
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Other:
- board size 81.3 x 82 mm -> 74.8 x 67.7 mm
