File: SignalPowerOn/SignalPowerOn.kicad_sch (KiCad schematic)
At the start: 42 parts, among them J1 LIVE IN, J2 NEUTRAL IN, J3 AUDIO IN, J4 NEUTRAL OUT, J5 SWITCHED LIVE, K1 SDT-S-112DMR, Q1 2N7000, Q2 BC549, T1 Block AVB 2,3/2/6, U1 LM358

Commit message: m0re
Other:
- moved on the sheet: C1, D1, F1, J1, J2, J4, T1
