File: MOSFETAmp/MOSFETAmp.kicad_pcb (KiCad board)
At the start: 2 copper layers, 100.8 x 67.3 mm, 48 parts, among them J1 IN, J2 OUT, J3 VEE, J4 VCC, J5 PGND, Q1 MPSA42, Q2 BC559, Q3 BC559, Q4 MPSA42, Q5 MPSA42, Q6 BC549, Q7 ECX10P20, Q8 ECX10N20, Q9 MJE350

Commit message: work
Other:
- board text added: "D"
- board text added: "G"
- board text added: "S"
Changed lines of the file:
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@@
 			(plot_on_all_layers_selection 0x00000000_00000000_00000000_00000000)
 			(disableapertmacros no)
-			(usegerberextensions no)
+			(usegerberextensions yes)
 			(usegerberattributes yes)
 			(usegerberadvancedattributes yes)
@@
 			(sketchdnponfab yes)
 			(crossoutdnponfab yes)
-			(subtractmaskfromsilk no)
+			(subtractmaskfromsilk yes)
 			(outputformat 1)
 			(mirror no)
-			(drillshape 1)
+			(drillshape 0)
 			(scaleselection 1)
-			(outputdirectory "")
+			(outputdirectory "/Users/tomwatson/Desktop/Gerber files/MOSFETAmp/")
 		)
 	)
@@
 		(layer "Edge.Cuts")
 	)
+	(gr_text "D"
+		(at 163.957 84.582 0)
+		(layer "F.SilkS")
+		(effects
+			(font
+				(size 1.5 1.5)
+				(thickness 0.3)
+				(bold yes)
+			)
+			(justify left bottom)
+		)
+	)
+	(gr_text "S"
+		(at 164.084 90.17 0)
+		(layer "F.SilkS")
+		(effects
+			(font
+				(size 1.5 1.5)
+				(thickness 0.3)
+				(bold yes)
+			)
+			(justify left bottom)
+		)
+	)
+	(gr_text "S"
+		(at 149.733 131.064 0)
+		(layer "F.SilkS")
+		(effects
+			(font
+				(size 1.5 1.5)
+				(thickness 0.3)
+				(bold yes)
+			)
+			(justify left bottom)
+		)
+	)
 	(gr_text "SIG   GND"
 		(at 95.885 86.36 90)
@@
 		)
 	)
+	(gr_text "G"
+		(at 163.957 95.631 0)
+		(layer "F.SilkS")
+		(effects
+			(font
+				(size 1.5 1.5)
+				(thickness 0.3)
+				(bold yes)
+			)
+			(justify left bottom)
+		)
+	)
 	(gr_text "MOSFET Class AB Amplifier\nTom Watson Audio 2026"
 		(at 156.464 102.362 0)
@@
 		)
 	)
+	(gr_text "G"
+		(at 149.733 125.603 0)
+		(layer "F.SilkS")
+		(effects
+			(font
+				(size 1.5 1.5)
+				(thickness 0.3)
+				(bold yes)
+			)
+			(justify left bottom)
+		)
+	)
 	(gr_text "Use Lateral MOSFETS only"
 		(at 157.48 120.65 0)
@@
 		)
 	)
+	(gr_text "D"
+		(at 149.733 136.398 0)
+		(layer "F.SilkS")
+		(effects
+			(font
+				(size 1.5 1.5)
+				(thickness 0.3)
+				(bold yes)
+			)
+			(justify left bottom)
+		)
+	)

Commit message: loads
Parts:
- F1, F2: footprint Fuse:Fuseholder_Cylinder-5x20mm_Stelvio-Kontek_PTF78_Horizontal_Open -> Fuse:Fuseholder_Cylinder-5x20mm_Schurter_0031_8201_Horizontal_Open

Commit message: more
Parts:
- moved R7 13.5 mm to (138.4, 124.0), turned to -90 degrees
- moved C9 4.99 mm to (116.4, 126.7), turned to 180 degrees
- moved C12 4.43 mm to (135.4, 129.0)
- moved R8 2.79 mm to (173.7, 82.5)
Connections:
- C9 pad 1: Net-(Q1-B) -> Net-(C9-Pad1)
- C9 pad 2: Net-(C9-Pad2) -> Net-(Q1-B)
- R10 pad 1: Net-(C9-Pad2) -> Net-(C9-Pad1)
Routing:
- net Net-(C9-Pad2): track 33.3 -> 0.00 mm
- net Net-(C9-Pad1): track 0.00 -> 33.3 mm
- net Net-(D4-K): track 37.5 -> 52.7 mm
- net Net-(Q8-G): track 24.2 -> 12.9 mm
- net Net-(D5-A): track 80.7 -> 71.4 mm
- net Net-(D2-A): track 35.4 -> 38.2 mm
- net Net-(Q7-G): track 8.70 -> 5.90 mm
- net Net-(Q1-B): track 37.2 -> 37.8 mm
