File: MOSFETAmp/MOSFETAmp.kicad_sch (KiCad schematic)
At the start: 47 parts, among them J1 IN, J2 OUT, J3 VEE, J4 VCC, J5 PGND, Q1 MPSA42, Q2 BC559, Q3 BC559, Q4 MPSA42, Q5 MPSA42, Q6 BC549, Q7 ECX10P20, Q8 ECX10N20, Q9 MJE350

Commit message: m0re
Parts:
- J2, J3, J4, J5: footprint Spade connector:TE_62409-1 -> (none)

Commit message: loads
Parts:
- F1, F2: footprint Fuse:Fuseholder_Cylinder-5x20mm_Stelvio-Kontek_PTF78_Horizontal_Open -> Fuse:Fuseholder_Cylinder-5x20mm_Schurter_0031_8201_Horizontal_Open
Changed lines of the file:
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@@
 			)
 		)
-		(property "Footprint" "Fuse:Fuseholder_Cylinder-5x20mm_Stelvio-Kontek_PTF78_Horizontal_Open"
+		(property "Footprint" "Fuse:Fuseholder_Cylinder-5x20mm_Schurter_0031_8201_Horizontal_Open"
 			(at 257.81 17.018 90)
 			(hide yes)
@@
 			)
 		)
-		(property "Footprint" "Fuse:Fuseholder_Cylinder-5x20mm_Stelvio-Kontek_PTF78_Horizontal_Open"
+		(property "Footprint" "Fuse:Fuseholder_Cylinder-5x20mm_Schurter_0031_8201_Horizontal_Open"
 			(at 261.62 157.988 90)
 			(hide yes)

Commit message: more
Connections:
- net at R10.1: now also C9.1; no longer C9.2
- net at Q1.2 (B), R6.2: now also C9.2; no longer C9.1
Other:
- moved on the sheet: C9
Changed lines of the file:
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@@
 	(symbol
 		(lib_id "Device:C_Polarized")
-		(at 132.08 91.44 0)
+		(at 132.08 91.44 180)
 		(unit 1)
 		(body_style 1)
@@
 		(fields_autoplaced yes)
 		(property "Reference" "C9"
-			(at 135.89 89.2809 0)
+			(at 135.89 91.0589 0)
 			(show_name no)
 			(do_not_autoplace no)
@@
 					(size 1.27 1.27)
 				)
-				(justify left)
+				(justify right)
 			)
 		)
 		(property "Value" "220uF"
-			(at 135.89 91.8209 0)
+			(at 135.89 93.5989 0)
 			(show_name no)
 			(do_not_autoplace no)
@@
 					(size 1.27 1.27)
 				)
-				(justify left)
+				(justify right)
 			)
 		)
 		(property "Footprint" "Capacitor_THT:CP_Radial_D10.0mm_P5.00mm"
-			(at 133.0452 95.25 0)
+			(at 131.1148 87.63 0)
 			(hide yes)
 			(show_name no)
