File: PCM2706TestAmp/PCM2706TestAmp.kicad_pcb (KiCad board)
At the start: 2 copper layers, 68.3 x 82.3 mm, 59 parts, among them IC1 PCM2706, IC2 USBLC6, J1 TWEETER/RIGHT, J10 POWER -, J2 WOOFER/LEFT, J3 USB-B CONNECTOR, J4 LINE OUT, J5 62409-1, J6 62409-1, J7 62409-1, J8 62409-1, J9 POWER +, U1 TPS22917, U2 LM317, Y1 12MHz

Commit message: more
Routing:
- net /AMPVCC: track 85.0 -> 83.9 mm
- net Net-(IC1-V_OUTR): track 14.1 -> 13.5 mm
Other:
- board text added: "TWEETER +"
- board text added: "TWEETER -"
Changed lines of the file:
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@@
 		)
 	)
-	(gr_text "WOOFER +"
+	(gr_text "TWEETER +"
 		(at 147.828 86.106 0)
 		(layer "F.SilkS")
@@
 		)
 	)
-	(gr_text "WOOFER -"
+	(gr_text "TWEETER -"
 		(at 159.004 90.678 0)
 		(layer "F.SilkS")
@@
 	(segment
 		(start 162.981 92.035)
-		(end 168.656 86.36)
+		(end 156.123 92.035)
 		(width 1)
 		(layer "B.Cu")
@@
 	)
 	(segment
-		(start 142.24 94.488)
-		(end 153.67 94.488)
-		(width 1)
-		(layer "B.Cu")
-		(net "/AMPVCC")
-	)
-	(segment
-		(start 154.178 92.035)
+		(start 168.656 86.36)
 		(end 162.981 92.035)
 		(width 1)
@@
 	)
 	(segment
+		(start 154.178 93.98)
+		(end 141.732 93.98)
+		(width 1)
+		(layer "B.Cu")
+		(net "/AMPVCC")
+	)
+	(segment
+		(start 156.123 92.035)
+		(end 154.178 93.98)
+		(width 1)
+		(layer "B.Cu")
+		(net "/AMPVCC")
+	)
+	(segment
 		(start 169.418 79.248)
 		(end 168.656 80.01)
@@
 	)
 	(segment
+		(start 168.656 81.349)
+		(end 168.656 86.36)
+		(width 1)
+		(layer "B.Cu")
+		(net "/AMPVCC")
+	)
+	(segment
 		(start 181.356 80.01)
 		(end 180.594 79.248)
@@
 	)
 	(segment
-		(start 154.178 93.98)
-		(end 154.178 92.035)
-		(width 1)
-		(layer "B.Cu")
-		(net "/AMPVCC")
-	)
-	(segment
 		(start 142.24 101.172)
 		(end 142.24 94.488)
@@
 		(start 181.356 81.349)
 		(end 181.356 80.01)
-		(width 1)
-		(layer "B.Cu")
-		(net "/AMPVCC")
-	)
-	(segment
-		(start 154.178 98.298)
-		(end 153.924 98.298)
-		(width 1)
-		(layer "B.Cu")
-		(net "/AMPVCC")
-	)
-	(segment
-		(start 153.67 94.488)
-		(end 154.178 93.98)
-		(width 1)
-		(layer "B.Cu")
-		(net "/AMPVCC")
-	)
-	(segment
-		(start 168.656 86.36)
-		(end 168.656 81.349)
 		(width 1)
 		(layer "B.Cu")
@@
 	)
 	(segment
-		(start 183.965 81.28)
-		(end 183.896 81.349)
-		(width 1)
-		(layer "B.Cu")
-		(net "Net-(AMP1-OUT3)")
-	)
-	(segment
 		(start 191.193 81.349)
 		(end 191.262 81.28)
@@
 	)
 	(segment
-		(start 173.228 110.236)
-		(end 172.72 110.236)
-		(width 0.2)
-		(layer "F.Cu")
-		(net "Net-(IC1-V_OUTR)")
-	)
-	(segment
-		(start 173.355 110.236)
-		(end 173.228 110.236)
-		(width 0.2)
-		(layer "F.Cu")
-		(net "Net-(IC1-V_OUTR)")
-	)
-	(segment
 		(start 170.434 105.1)
 		(end 170.434 107.442)
@@
 	)
 	(segment
+		(start 173.134 96.906)
+		(end 187.116 96.906)
+		(width 0.4)
+		(layer "B.Cu")
+		(net "Net-(J4-Pin_1)")
+	)
+	(segment
+		(start 187.116 96.906)
+		(end 191.516 101.306)
+		(width 0.4)
+		(layer "B.Cu")
+		(net "Net-(J4-Pin_1)")
+	)
+	(segment
+		(start 197.642 107.432)
+		(end 191.516 101.306)
+		(width 0.4)
+		(layer "B.Cu")
+		(net "Net-(J4-Pin_1)")
+	)
+	(segment
+		(start 170.434 94.206)
+		(end 173.134 96.906)
+		(width 0.4)
+		(layer "B.Cu")
+		(net "Net-(J4-Pin_1)")
+	)
+	(segment
+		(start 196.342 110.704)
+		(end 197.642 109.404)
+		(width 0.4)
+		(layer "B.Cu")
+		(net "Net-(J4-Pin_1)")
+	)
+	(segment
+		(start 197.642 109.404)
+		(end 197.642 107.432)
+		(width 0.4)
+		(layer "B.Cu")
+		(net "Net-(J4-Pin_1)")
+	)
+	(segment
+		(start 170.434 86.808)
+		(end 171.196 86.046)
+		(width 0.4)
+		(layer "F.Cu")
+		(net "Net-(C23-Pad2)")
+	)
+	(segment
+		(start 170.434 90.706)
+		(end 170.434 86.808)
+		(width 0.4)
+		(layer "F.Cu")
+		(net "Net-(C23-Pad2)")
+	)
+	(segment
 		(start 193.303522 114.504)
 		(end 195.042 114.504)
@@
 	)
 	(segment
-		(start 173.134 96.906)
-		(end 187.116 96.906)
-		(width 0.4)
-		(layer "B.Cu")
-		(net "Net-(J4-Pin_1)")
-	)
-	(segment
-		(start 187.116 96.906)
-		(end 191.516 101.306)
-		(width 0.4)
-		(layer "B.Cu")
-		(net "Net-(J4-Pin_1)")
-	)
-	(segment
-		(start 197.642 107.432)
-		(end 191.516 101.306)
-		(width 0.4)
-		(layer "B.Cu")
-		(net "Net-(J4-Pin_1)")
-	)
-	(segment
-		(start 170.434 94.206)
-		(end 173.134 96.906)
-		(width 0.4)
-		(layer "B.Cu")
-		(net "Net-(J4-Pin_1)")
-	)
-	(segment
-		(start 196.342 110.704)
-		(end 197.642 109.404)
-		(width 0.4)
-		(layer "B.Cu")
-		(net "Net-(J4-Pin_1)")
-	)
-	(segment
-		(start 197.642 109.404)
-		(end 197.642 107.432)
-		(width 0.4)
-		(layer "B.Cu")
-		(net "Net-(J4-Pin_1)")
+		(start 193.842 110.704)
+		(end 192.542 109.404)
+		(width 0.4)
+		(layer "F.Cu")
+		(net "Net-(J4-Pin_3)")
+	)
+	(segment
+		(start 192.891 107.316522)
+		(end 192.891 97.681)
+		(width 0.4)
+		(layer "F.Cu")
+		(net "Net-(J4-Pin_3)")
+	)
+	(segment
+		(start 192.542 109.404)
+		(end 192.542 107.665522)
+		(width 0.4)
+		(layer "F.Cu")
+		(net "Net-(J4-Pin_3)")
+	)
+	(segment
+		(start 192.542 107.665522)
+		(end 192.891 107.316522)
+		(width 0.4)
+		(layer "F.Cu")
+		(net "Net-(J4-Pin_3)")
+	)
+	(segment
+		(start 192.891 97.681)
+		(end 191.516 96.306)
+		(width 0.4)
+		(layer "F.Cu")
+		(net "Net-(J4-Pin_3)")
+	)
+	(segment
+		(start 182.44 96.306)
+		(end 180.34 94.206)
+		(width 0.4)
+		(layer "B.Cu")
+		(net "Net-(J4-Pin_3)")
+	)
+	(segment
+		(start 191.516 96.306)
+		(end 182.44 96.306)
+		(width 0.4)
+		(layer "B.Cu")
+		(net "Net-(J4-Pin_3)")
+	)
+	(segment
+		(start 180.34 90.706)
+		(end 180.34 87.57)
+		(width 0.4)
+		(layer "F.Cu")
+		(net "Net-(C24-Pad2)")
+	)
+	(segment
+		(start 180.34 87.57)
+		(end 178.816 86.046)
+		(width 0.4)
+		(layer "F.Cu")
+		(net "Net-(C24-Pad2)")
 	)
 	(segment
@@
 		(net "Net-(C21-Pad2)")
 	)
-	(segment
-		(start 170.434 86.808)
-		(end 171.196 86.046)
-		(width 0.4)
-		(layer "F.Cu")
-		(net "Net-(C23-Pad2)")
-	)
-	(segment
-		(start 170.434 90.706)
-		(end 170.434 86.808)
-		(width 0.4)
-		(layer "F.Cu")
-		(net "Net-(C23-Pad2)")
-	)
-	(segment
-		(start 180.34 90.706)
-		(end 180.34 87.57)
-		(width 0.4)
-		(layer "F.Cu")
-		(net "Net-(C24-Pad2)")
-	)
-	(segment
-		(start 180.34 87.57)
-		(end 178.816 86.046)
-		(width 0.4)
-		(layer "F.Cu")
-		(net "Net-(C24-Pad2)")
-	)
-	(segment
-		(start 193.842 110.704)
-		(end 192.542 109.404)
-		(width 0.4)
-		(layer "F.Cu")
-		(net "Net-(J4-Pin_3)")
-	)
-	(segment
-		(start 192.891 107.316522)
-		(end 192.891 97.681)
-		(width 0.4)
-		(layer "F.Cu")
-		(net "Net-(J4-Pin_3)")
-	)
-	(segment
-		(start 192.542 109.404)
-		(end 192.542 107.665522)
-		(width 0.4)
-		(layer "F.Cu")
-		(net "Net-(J4-Pin_3)")
-	)
-	(segment
-		(start 192.542 107.665522)
-		(end 192.891 107.316522)
-		(width 0.4)
-		(layer "F.Cu")
-		(net "Net-(J4-Pin_3)")
-	)
-	(segment
-		(start 192.891 97.681)
-		(end 191.516 96.306)
-		(width 0.4)
-		(layer "F.Cu")
-		(net "Net-(J4-Pin_3)")
-	)
-	(segment
-		(start 182.44 96.306)
-		(end 180.34 94.206)
-		(width 0.4)
-		(layer "B.Cu")
-		(net "Net-(J4-Pin_3)")
-	)
-	(segment
-		(start 191.516 96.306)
-		(end 182.44 96.306)
-		(width 0.4)
-		(layer "B.Cu")
-		(net "Net-(J4-Pin_3)")
-	)
 	(zone
