File: 7377new/7377new/DiscreteClassD/DiscreteClassD.kicad_pcb (KiCad board)
At the start: 4 copper layers, 100 x 100 mm, 65 parts, among them IC1 TLV3602DGKR, J1 AUDIO IN, J14 24V INPUT, J15 SPEAKER OUT, Q5 DMN6070SY, Q6 DMN6070SY, Q7 DMN6070SY, Q8 DMN6070SY, U1 OPA1656ID, U2 UCC27301ADRCR, U3 OPA1656ID, U4 SN74LVC1G04DBVR, U5 SN74LVC2G17DBVR, U6 UCC27301ADRCR

Commit message: more
Parts:
- removed IC1: TLV3602DGKR, Package_SO:VSSOP-8_3x3mm_P0.65mm
- removed J14: 24V INPUT, Connector_Molex:Molex_KK-396_A-41791-0002_1x02_P3.96mm_Vertical
- removed TP11: PGND, TestPoint:TestPoint_Pad_D1.5mm
- removed TP9: +24V, TestPoint:TestPoint_Pad_D1.5mm
- added C101: 100nF, Capacitor_SMD:C_0805_2012Metric, F.Cu at (177.0, 134.1)
- added C102: 100nF, Capacitor_SMD:C_0805_2012Metric, F.Cu at (299.0, 128.4)
- added C103: 4.7uF, Capacitor_SMD:C_0805_2012Metric, F.Cu at (299.0, 131.4)
- added C104: 100nF, Capacitor_SMD:C_1206_3216Metric_Pad1.33x1.80mm_HandSolder, F.Cu at (283.9, 125.6)
- added C105: 1uF, Capacitor_SMD:C_1206_3216Metric_Pad1.33x1.80mm_HandSolder, F.Cu at (283.9, 128.9)
- added C106: 10uF, Capacitor_SMD:C_1206_3216Metric_Pad1.33x1.80mm_HandSolder, F.Cu at (283.9, 132.3)
- added C107: 100nF, Capacitor_SMD:C_0805_2012Metric, F.Cu at (177.0, 119.6)
- added C108: 100nF, Capacitor_SMD:C_0805_2012Metric, F.Cu at (299.0, 137.5)
- added C109: 4.7uF, Capacitor_SMD:C_0805_2012Metric, F.Cu at (299.0, 140.5)
- added C110: 100nF, Capacitor_SMD:C_1206_3216Metric_Pad1.33x1.80mm_HandSolder, F.Cu at (283.9, 135.6)
- added C111: 1uF, Capacitor_SMD:C_1206_3216Metric_Pad1.33x1.80mm_HandSolder, F.Cu at (283.9, 139.0)
- added C112: 10uF, Capacitor_SMD:C_1206_3216Metric_Pad1.33x1.80mm_HandSolder, F.Cu at (283.9, 142.3)
- added C113: 330p DNP, Capacitor_SMD:C_0805_2012Metric, F.Cu at (299.0, 143.5)
- added C114: 330p DNP, Capacitor_SMD:C_0805_2012Metric, F.Cu at (299.0, 146.5)
- added C115: 330nF, Capacitor_THT:C_Rect_L7.2mm_W3.0mm_P5.00mm_FKS2_FKP2_MKS2_MKP2, F.Cu at (194.3, 119.4)
- added C116: 100nF, Capacitor_SMD:C_1206_3216Metric_Pad1.33x1.80mm_HandSolder, F.Cu at (204.9, 110.2)
- added C118: 1nF, Capacitor_SMD:C_0805_2012Metric_Pad1.18x1.45mm_HandSolder, F.Cu at (309.4, 125.4)
- added C119: 1nF, Capacitor_SMD:C_0805_2012Metric_Pad1.18x1.45mm_HandSolder, F.Cu at (309.4, 128.4)
- added C20: 1000uF, Capacitor_THT:CP_Radial_D12.5mm_P5.00mm, F.Cu at (234.0, 52.7)
- added C21: 10u / 50V, Capacitor_SMD:C_1210_3225Metric, F.Cu at (266.8, 85.2)
- added C22: 10n C0G, Capacitor_SMD:C_0805_2012Metric, F.Cu at (252.0, 63.5)
- added C23: 10n C0G, Capacitor_SMD:C_0805_2012Metric, F.Cu at (252.0, 66.5)
- added C24: 10u / 25V, Capacitor_SMD:C_1210_3225Metric, F.Cu at (266.8, 89.4)
- added C25: 10u / 50V, Capacitor_SMD:C_1210_3225Metric, F.Cu at (266.8, 93.7)
- added C26: 10n C0G, Capacitor_SMD:C_0805_2012Metric, F.Cu at (252.0, 69.5)
- added C27: 10n C0G, Capacitor_SMD:C_0805_2012Metric, F.Cu at (252.0, 72.5)
- added C28: 10u / 25V, Capacitor_SMD:C_1210_3225Metric, F.Cu at (266.8, 97.9)
- added C29: 10u / 16V, Capacitor_SMD:C_0805_2012Metric, F.Cu at (252.0, 75.5)
- added C30: 100n / 16V, Capacitor_SMD:C_0805_2012Metric, F.Cu at (252.0, 78.5)
- added C31: 1n C0G / 1%, Capacitor_SMD:C_0805_2012Metric, F.Cu at (252.0, 81.5)
- added C32: 100nF, Capacitor_SMD:C_1206_3216Metric_Pad1.33x1.80mm_HandSolder, F.Cu at (135.2, 78.8)
- added C33: 4.7uF, Capacitor_SMD:C_0805_2012Metric, F.Cu at (256.4, 66.5)
- added C34: 100nF, Capacitor_SMD:C_1206_3216Metric_Pad1.33x1.80mm_HandSolder, F.Cu at (256.4, 69.5)
- added C35: 4.7uF, Capacitor_SMD:C_0805_2012Metric, F.Cu at (256.4, 72.5)
- added C36: 100nF, Capacitor_SMD:C_0805_2012Metric, F.Cu at (256.4, 75.5)
- added C37: 100n / 25V, Capacitor_SMD:C_0805_2012Metric, F.Cu at (256.4, 78.5)
- added C38: 100n / 25V, Capacitor_SMD:C_0805_2012Metric, F.Cu at (256.4, 81.5)
- added C39: 100n / 25V, Capacitor_SMD:C_0805_2012Metric, F.Cu at (260.9, 63.5)
- added C40: 1uF, Capacitor_THT:C_Rect_L7.2mm_W5.5mm_P5.00mm_FKS2_FKP2_MKS2_MKP2, F.Cu at (118.4, 68.8)
- added C41: 100pF, Capacitor_SMD:C_0805_2012Metric, F.Cu at (131.3, 73.0)
- added C42: 100p C0G, Capacitor_SMD:C_0805_2012Metric, F.Cu at (152.7, 76.5)
- added C43: 100p C0G, Capacitor_SMD:C_0805_2012Metric, F.Cu at (229.9, 145.7)
- added C44: 100n / 25V, Capacitor_SMD:C_0805_2012Metric, F.Cu at (260.9, 75.5)
- added C45: 1uF, Capacitor_THT:C_Rect_L7.2mm_W5.5mm_P5.00mm_FKS2_FKP2_MKS2_MKP2, F.Cu at (118.4, 86.3)
- added C46: 100pF, Capacitor_SMD:C_0805_2012Metric, F.Cu at (131.3, 84.8)
- added C47: 100p C0G, Capacitor_SMD:C_0805_2012Metric, F.Cu at (152.7, 81.5)
- added C48: 100p C0G, Capacitor_SMD:C_0805_2012Metric, F.Cu at (265.3, 63.5)
- added C49: 100n / 25V, Capacitor_SMD:C_0805_2012Metric, F.Cu at (265.3, 66.5)
- added C50: 22u / 25V, Capacitor_SMD:C_1210_3225Metric, F.Cu at (266.8, 102.2)
- added C51: 100n / 25V, Capacitor_SMD:C_0805_2012Metric, F.Cu at (265.3, 69.5)
- added D101: DNP diode, Diode_SMD:D_SOD-123, F.Cu at (304.1, 125.6)
- added D102: DNP diode, Diode_SMD:D_SOD-123, F.Cu at (304.1, 128.9)
- added D103: DNP diode, Diode_SMD:D_SOD-123, F.Cu at (304.1, 132.3)
- added D104: DNP diode, Diode_SMD:D_SOD-123, F.Cu at (304.1, 135.6)
- added D20: 1N4148W, Diode_SMD:D_SOD-123, F.Cu at (149.2, 75.4)
- added D21: 1N4148W, Diode_SMD:D_SOD-123, F.Cu at (223.7, 140.1)
- added D22: 1N4148W, Diode_SMD:D_SOD-123, F.Cu at (149.2, 82.5)
- added D23: 1N4148W, Diode_SMD:D_SOD-123, F.Cu at (158.9, 114.6)
- added J115: RIGHT SPEAKER, Connector_Molex:Molex_KK-396_A-41791-0002_1x02_P3.96mm_Vertical, F.Cu at (203.3, 118.8)
- added J16: POWER IN, Connector_Molex:Molex_KK-396_A-41791-0002_1x02_P3.96mm_Vertical, F.Cu at (143.4, 136.8)
- added L106: CSAD0660-100M, DiscreteClassD:CSAD0660-100M, F.Cu at (186.7, 116.8)
- added Q105: DMN6070SY, Package_TO_SOT_SMD:SOT-89-3, F.Cu at (174.5, 123.7)
- added Q106: DMN6070SY, Package_TO_SOT_SMD:SOT-89-3, F.Cu at (179.7, 123.7)
- added Q107: DMN6070SY, Package_TO_SOT_SMD:SOT-89-3, F.Cu at (174.5, 109.2)
- added Q108: DMN6070SY, Package_TO_SOT_SMD:SOT-89-3, F.Cu at (179.7, 109.2)
- added R101: 10R, Resistor_SMD:R_0805_2012Metric, F.Cu at (173.2, 127.5)
- added R102: 47k, Resistor_SMD:R_0805_2012Metric, F.Cu at (276.9, 116.5)
- added R103: 10R DNP, Resistor_SMD:R_0805_2012Metric, F.Cu at (276.9, 119.5)
- added R104: 10R, Resistor_SMD:R_0805_2012Metric, F.Cu at (177.3, 127.5)
- added R105: 47k, Resistor_SMD:R_0805_2012Metric, F.Cu at (281.4, 113.6)
- added R106: 10R DNP, Resistor_SMD:R_0805_2012Metric, F.Cu at (281.4, 116.5)
- added R107: 10R, Resistor_SMD:R_0805_2012Metric, F.Cu at (173.2, 113.0)
- added R108: 47k, Resistor_SMD:R_0805_2012Metric, F.Cu at (157.8, 127.4)
- added R109: 10R DNP, Resistor_SMD:R_0805_2012Metric, F.Cu at (162.2, 118.6)
- added R110: 10R, Resistor_SMD:R_0805_2012Metric, F.Cu at (177.3, 113.0)
- added R111: 47k, Resistor_SMD:R_0805_2012Metric, F.Cu at (194.6, 130.2)
- added R112: 10R DNP, Resistor_SMD:R_0805_2012Metric, F.Cu at (194.6, 133.1)
- added R113: 10R DNP, Resistor_SMD:R_1206_3216Metric, F.Cu at (309.3, 139.0)
- added R114: 10R DNP, Resistor_SMD:R_1206_3216Metric, F.Cu at (309.3, 142.3)
- added R115: 10R, Resistor_SMD:R_2512_6332Metric, F.Cu at (206.2, 124.0)
- added R20: 91k2 / 0.1%, Resistor_SMD:R_0805_2012Metric, F.Cu at (269.7, 63.5)
- added R21: 10k / 0.1%, Resistor_SMD:R_0805_2012Metric, F.Cu at (269.7, 66.4)
- added R22: 32k2 / 0.1%, Resistor_SMD:R_0805_2012Metric, F.Cu at (269.7, 69.4)
- added R23: 10k / 0.1%, Resistor_SMD:R_0805_2012Metric, F.Cu at (269.7, 72.3)
- added R24: 10k, Resistor_SMD:R_0805_2012Metric, F.Cu at (269.7, 75.3)
- added R25: 10k, Resistor_SMD:R_0805_2012Metric, F.Cu at (269.7, 78.2)
- added R26: 10k / 0.1%, Resistor_SMD:R_0805_2012Metric, F.Cu at (269.7, 81.2)
- added R27: 49k9 / 0.1%, Resistor_SMD:R_0805_2012Metric, F.Cu at (274.2, 63.5)
- added R28: 3k09 / 0.1%, Resistor_SMD:R_0805_2012Metric, F.Cu at (274.2, 66.4)
- added R29: 51K, Resistor_SMD:R_0805_2012Metric, F.Cu at (129.2, 73.0)
- added R30: 10K, Resistor_SMD:R_0805_2012Metric, F.Cu at (133.3, 73.0)
- added R31: 100R, Resistor_SMD:R_0805_2012Metric, F.Cu at (135.3, 73.0)
- added R32: 330R, Resistor_SMD:R_0805_2012Metric, F.Cu at (148.6, 73.2)
- added R33: 330R, Resistor_SMD:R_0805_2012Metric, F.Cu at (243.2, 154.4)
- added R34: 10k, Resistor_SMD:R_0805_2012Metric, F.Cu at (278.6, 63.5)
- added R35: 1k DNP, Resistor_SMD:R_0805_2012Metric, F.Cu at (278.6, 66.4)
- added R36: 51K, Resistor_SMD:R_0805_2012Metric, F.Cu at (129.2, 84.8)
- added R37: 10K, Resistor_SMD:R_0805_2012Metric, F.Cu at (133.3, 84.8)
- added R38: 100R, Resistor_SMD:R_0805_2012Metric, F.Cu at (135.3, 84.8)
- added R39: 330R, Resistor_SMD:R_0805_2012Metric, F.Cu at (148.6, 84.8)
- added R40: 330R, Resistor_SMD:R_0805_2012Metric, F.Cu at (156.5, 100.9)
- added R41: 10k, Resistor_SMD:R_0805_2012Metric, F.Cu at (283.0, 63.5)
- added R42: 1k DNP, Resistor_SMD:R_0805_2012Metric, F.Cu at (283.0, 66.4)
- added R43: 4R7, Resistor_SMD:R_0805_2012Metric, F.Cu at (283.0, 69.4)
- added TP101: SW_A, TestPoint:TestPoint_Pad_D1.5mm, F.Cu at (289.7, 113.9)
- added TP102: HO_A, TestPoint:TestPoint_Pad_D1.5mm, F.Cu at (289.7, 117.4)
- added TP103: LO_A, TestPoint:TestPoint_Pad_D1.5mm, F.Cu at (293.3, 113.9)
- added TP104: SW_B, TestPoint:TestPoint_Pad_D1.5mm, F.Cu at (293.3, 117.4)
- added TP105: HO_B, TestPoint:TestPoint_Pad_D1.5mm, F.Cu at (296.8, 113.9)
- added TP106: LO_B, TestPoint:TestPoint_Pad_D1.5mm, F.Cu at (296.8, 117.4)
- added TP107: OUT_A, TestPoint:TestPoint_Pad_D1.5mm, F.Cu at (300.4, 113.9)
- added TP108: OUT_B, TestPoint:TestPoint_Pad_D1.5mm, F.Cu at (300.4, 117.4)
- added TP20: +5V_A, TestPoint:TestPoint_Pad_D1.5mm, F.Cu at (251.5, 88.4)
- added TP21: VREF_2V5, TestPoint:TestPoint_Pad_D1.5mm, F.Cu at (251.5, 91.9)
- added TP22: OSC_SQUARE, TestPoint:TestPoint_Pad_D1.5mm, F.Cu at (251.5, 95.5)
- added TP23: TRIANGLE_400K, TestPoint:TestPoint_Pad_D1.5mm, F.Cu at (255.1, 84.8)
- added TP24: AUDIO_L, TestPoint:TestPoint_Pad_D1.5mm, F.Cu at (138.5, 72.1)
- added TP25: PWM_L, TestPoint:TestPoint_Pad_D1.5mm, F.Cu at (255.1, 91.9)
- added TP26: L_DRIVE_P, TestPoint:TestPoint_Pad_D1.5mm, F.Cu at (255.1, 95.5)
- added TP27: L_DRIVE_N, TestPoint:TestPoint_Pad_D1.5mm, F.Cu at (258.6, 84.8)
- added TP28: ENABLE_L, TestPoint:TestPoint_Pad_D1.5mm, F.Cu at (258.6, 88.4)
- added TP29: AUDIO_R, TestPoint:TestPoint_Pad_D1.5mm, F.Cu at (138.5, 85.7)
- added TP30: PWM_R, TestPoint:TestPoint_Pad_D1.5mm, F.Cu at (258.6, 95.5)
- added TP31: R_DRIVE_P, TestPoint:TestPoint_Pad_D1.5mm, F.Cu at (262.2, 84.8)
- added TP32: R_DRIVE_N, TestPoint:TestPoint_Pad_D1.5mm, F.Cu at (262.2, 88.4)
- added TP33: ENABLE_R, TestPoint:TestPoint_Pad_D1.5mm, F.Cu at (262.2, 91.9)
- added TP34: +12V_A, TestPoint:TestPoint_Pad_D1.5mm, F.Cu at (262.2, 95.5)
- added U10: SN74LVC2G17, Package_TO_SOT_SMD:SOT-23-6, F.Cu at (166.3, 81.4)
- added U102: UCC27301A, Package_SON:VSON-10-1EP_3x3mm_P0.5mm_EP1.65x2.4mm, F.Cu at (176.5, 130.8)
- added U106: UCC27301A, Package_SON:VSON-10-1EP_3x3mm_P0.5mm_EP1.65x2.4mm, F.Cu at (176.5, 116.3)
- added U11: TPS7A4901DGNR, Custom:TPS7A4901DRBR, F.Cu at (244.1, 93.3)
- added U12: TPS7A4901DGNR, Custom:TPS7A4901DRBR, F.Cu at (244.1, 99.8)
- added U7: TLV3602DGKR, Package_SO:VSSOP-8_3x3mm_P0.65mm, F.Cu at (226.8, 161.3)
- added U8: TLV3602, Package_SO:VSSOP-8_3x3mm_P0.65mm, F.Cu at (144.0, 79.0)
- added U9: SN74LVC1G04, Package_TO_SOT_SMD:SOT-23-5, F.Cu at (144.8, 83.4)
- C1, C7: value 100n / 25V -> 100nF
- C15: value 330n -> 330nF
- C16: value 100n / 100V -> 100nF
- C17: value 1000u / 35V FR -> 1000uF
- J1: value AUDIO IN -> STEREO LINE INPUT
- J15: value SPEAKER OUT -> LEFT SPEAKER
- R15: value 10R / 1W -> 10R
- U1: value OPA1656ID -> OPA1656
- U2, U6: value UCC27301ADRCR -> UCC27301A
- U4: value SN74LVC1G04DBVR -> SN74LVC1G04; footprint Package_TO_SOT_SMD:SOT-553 -> Package_TO_SOT_SMD:SOT-23-5
- U5: value SN74LVC2G17DBVR -> SN74LVC2G17
- moved U3 139.3 mm to (273.8, 106.9)
- moved U5 97.6 mm to (233.7, 137.6), turned to 90 degrees
- moved C17 82.7 mm to (267.3, 36.8), turned to 180 degrees
- moved C8 78.7 mm to (168.2, 60.7), turned to -90 degrees
- moved R8 76.9 mm to (229.1, 128.1), turned to 0 degrees
- moved C2 75.0 mm to (163.1, 71.0), turned to 90 degrees
- moved R13 53.3 mm to (269.9, 139.0)
- moved R14 53.3 mm to (269.9, 142.3)
- moved J1 44.4 mm to (120.9, 75.1), turned to -90 degrees
- moved C9 40.9 mm to (259.6, 140.5)
- moved C19 39.9 mm to (226.1, 67.9), turned to 90 degrees
- moved C18 39.0 mm to (270.0, 125.4)
- moved C13 38.8 mm to (259.6, 143.5)
- moved C14 38.8 mm to (259.6, 146.5)
- moved C3 37.4 mm to (259.6, 131.4)
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Connections:
- net /Power output stage/+12V_GD renamed +12V_GD
- net /Power output stage/+24V renamed +24V
- net /Power output stage/GH_A renamed Net-(Q5-G)
- net /Power output stage/GH_B renamed Net-(Q7-G)
- net /Power output stage/GL_A renamed Net-(Q6-G)
- net /Power output stage/GL_B renamed Net-(Q8-G)
- net /Power output stage/HB_A renamed Net-(U2-HB)
- net /Power output stage/HB_B renamed Net-(U6-HB)
- net /Power output stage/HO_A renamed Net-(D1-K)
- net /Power output stage/HO_B renamed Net-(D3-K)
- net /Power output stage/LO_A renamed Net-(D2-K)
- net /Power output stage/LO_B renamed Net-(D4-K)
- net /Power output stage/OUT_A renamed /LEFT OUTPUT/OUT_A
- net /Power output stage/OUT_B renamed /LEFT OUTPUT/OUT_B
- net /Power output stage/SW_A renamed /LEFT OUTPUT/SW_A
- net /Power output stage/SW_B renamed /LEFT OUTPUT/SW_B
- J1 pad 1: unconnected-(J1-Pin_1-Pad1) -> /LEFT_IN
- J1 pad 3: unconnected-(J1-Pin_3-Pad3) -> /RIGHT_IN
- U1 pad 1: unconnected-(U1-Pad1) -> Net-(U1A--)
- U1 pad 2: unconnected-(U1A---Pad2) -> Net-(U1A--)
- U1 pad 3: unconnected-(U1A-+-Pad3) -> Net-(U1A-+)
- U1 pad 4: unconnected-(U1C-V--Pad4) -> GND
- U1 pad 5: unconnected-(U1B-+-Pad5) -> Net-(U1B-+)
- U1 pad 6: unconnected-(U1B---Pad6) -> Net-(U1B--)
- U1 pad 7: unconnected-(U1-Pad7) -> Net-(U1B--)
- U1 pad 8: unconnected-(U1C-V+-Pad8) -> +12V_A
- U2 pad 6: /Power output stage/EN_A -> /ENABLE_L
- U2 pad 7: /Power output stage/HI_A -> /L_DRIVE_P
- U2 pad 8: /Power output stage/LI_A -> /L_DRIVE_N
- U3 pad 1: unconnected-(U3-Pad1) -> /VREF_2V5
- U3 pad 2: unconnected-(U3A---Pad2) -> /VREF_2V5
- U3 pad 3: unconnected-(U3A-+-Pad3) -> Net-(U3A-+)
- U3 pad 4: unconnected-(U3C-V--Pad4) -> GND
- U3 pad 5: unconnected-(U3B-+-Pad5) -> /VREF_2V5
- U3 pad 6: unconnected-(U3B---Pad6) -> Net-(U3B--)
- U3 pad 7: unconnected-(U3-Pad7) -> /TRIANGLE_400K
- U3 pad 8: unconnected-(U3C-V+-Pad8) -> +12V_A
- U4 pad 2: unconnected-(U4-Pad2) -> /PWM_L
- U4 pad 3: unconnected-(U4-GND-Pad3) -> GND
- U4 pad 4: unconnected-(U4-Pad4) -> Net-(D21-K)
- U4 pad 5: unconnected-(U4-VCC-Pad5) -> +5V_A
- U5 pad 1: unconnected-(U5-1A-Pad1) -> Net-(D20-A)
- U5 pad 2: unconnected-(U5-GND-Pad2) -> GND
- U5 pad 3: unconnected-(U5-2A-Pad3) -> Net-(D21-A)
- U5 pad 4: unconnected-(U5-2Y-Pad4) -> /L_DRIVE_N
- U5 pad 5: unconnected-(U5-V_{CC}-Pad5) -> +5V_A
- U5 pad 6: unconnected-(U5-1Y-Pad6) -> /L_DRIVE_P
- U6 pad 6: /Power output stage/EN_B -> /ENABLE_L
- U6 pad 7: /Power output stage/HI_B -> /L_DRIVE_N
- U6 pad 8: /Power output stage/LI_B -> /L_DRIVE_P
Routing:
- net +12V_GD: track 0.00 -> 21.7 mm, vias 0 -> 2
- net +5V_A: track 0.00 -> 19.0 mm, vias 0 -> 3
- net Net-(D101-K): track 0.00 -> 12.3 mm
- net Net-(D103-K): track 0.00 -> 12.3 mm
- net Net-(D3-K): track 0.00 -> 11.9 mm
- net /RIGHT OUTPUT/SW_B: track 0.00 -> 11.9 mm
- net /AUDIO_L: track 0.00 -> 11.6 mm
- net /AUDIO_R: track 0.00 -> 11.5 mm
- net /RIGHT OUTPUT/SW_A: track 0.00 -> 11.3 mm
- net /PWM_R: track 0.00 -> 11.1 mm
- net Net-(D1-K): track 0.00 -> 10.5 mm
- net Net-(D2-K): track 0.00 -> 9.83 mm
- net Net-(D4-K): track 0.00 -> 9.80 mm
- net /PWM_L: track 0.00 -> 9.66 mm
- net Net-(U1A-+): track 0.00 -> 7.75 mm
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- added copper zone on F.Cu, net /RIGHT OUTPUT/OUT_A
- added copper zone on F.Cu, net /RIGHT OUTPUT/OUT_B
- added copper zone on F.Cu, net /RIGHT OUTPUT/SW_A
- added copper zone on F.Cu, net /RIGHT OUTPUT/SW_B
- added copper zone on F.Cu, net Net-(C116-Pad1)
