File: 7377new/7377new/DiscreteClassD/DiscreteClassD.kicad_sch (KiCad schematic)
At the start: 1 part, among them J1 AUDIO IN

Commit message: more
Parts:
- added C17, C20: 1000uF, Capacitor_THT:CP_Radial_D12.5mm_P5.00mm, symbol Device:C_Polarized
- added C21, C25: 10u / 50V, Capacitor_SMD:C_1210_3225Metric, symbol Device:C
- added C22, C23, C26, C27: 10n C0G, Capacitor_SMD:C_0805_2012Metric, symbol Device:C
- added C24, C28: 10u / 25V, Capacitor_SMD:C_1210_3225Metric, symbol Device:C
- added C29: 10u / 16V, Capacitor_SMD:C_0805_2012Metric, symbol Device:C
- added C30: 100n / 16V, Capacitor_SMD:C_0805_2012Metric, symbol Device:C
- added C31: 1n C0G / 1%, Capacitor_SMD:C_0805_2012Metric, symbol Device:C
- added C32, C34: 100nF, Capacitor_SMD:C_1206_3216Metric_Pad1.33x1.80mm_HandSolder, symbol Device:C
- added C33, C35: 4.7uF, Capacitor_SMD:C_0805_2012Metric, symbol Device:C
- added C36: 100nF, Capacitor_SMD:C_0805_2012Metric, symbol Device:C
- added C37, C38, C39, C44, C49, C51: 100n / 25V, Capacitor_SMD:C_0805_2012Metric, symbol Device:C
- added C40, C45: 1uF, Capacitor_THT:C_Rect_L7.2mm_W5.5mm_P5.00mm_FKS2_FKP2_MKS2_MKP2, symbol Device:C
- added C41, C46: 100pF, Capacitor_SMD:C_0805_2012Metric, symbol Device:C
- added C42, C43, C47, C48: 100p C0G, Capacitor_SMD:C_0805_2012Metric, symbol Device:C
- added C50: 22u / 25V, Capacitor_SMD:C_1210_3225Metric, symbol Device:C
- added D20, D21, D22, D23: 1N4148W, Diode_SMD:D_SOD-123, symbol Device:D
- added J16: POWER IN, Connector_Molex:Molex_KK-396_A-41791-0002_1x02_P3.96mm_Vertical, symbol Connector:Conn_01x02_Socket
- added R20: 91k2 / 0.1%, Resistor_SMD:R_0805_2012Metric, symbol Device:R
- added R21, R23, R26: 10k / 0.1%, Resistor_SMD:R_0805_2012Metric, symbol Device:R
- added R22: 32k2 / 0.1%, Resistor_SMD:R_0805_2012Metric, symbol Device:R
- added R24, R25, R34, R41: 10k, Resistor_SMD:R_0805_2012Metric, symbol Device:R
- added R27: 49k9 / 0.1%, Resistor_SMD:R_0805_2012Metric, symbol Device:R
- added R28: 3k09 / 0.1%, Resistor_SMD:R_0805_2012Metric, symbol Device:R
- added R29, R36: 51K, Resistor_SMD:R_0805_2012Metric, symbol Device:R
- added R30, R37: 10K, Resistor_SMD:R_0805_2012Metric, symbol Device:R
- added R31, R38: 100R, Resistor_SMD:R_0805_2012Metric, symbol Device:R
- added R32, R33, R39, R40: 330R, Resistor_SMD:R_0805_2012Metric, symbol Device:R
- added R35, R42: 1k DNP, Resistor_SMD:R_0805_2012Metric, symbol Device:R
- added R43: 4R7, Resistor_SMD:R_0805_2012Metric, symbol Device:R
- added TP10: +12V_GD, TestPoint:TestPoint_Pad_D1.5mm, symbol Connector:TestPoint
- added TP20: +5V_A, TestPoint:TestPoint_Pad_D1.5mm, symbol Connector:TestPoint
- added TP21: VREF_2V5, TestPoint:TestPoint_Pad_D1.5mm, symbol Connector:TestPoint
- added TP22: OSC_SQUARE, TestPoint:TestPoint_Pad_D1.5mm, symbol Connector:TestPoint
- added TP23: TRIANGLE_400K, TestPoint:TestPoint_Pad_D1.5mm, symbol Connector:TestPoint
- added TP24: AUDIO_L, TestPoint:TestPoint_Pad_D1.5mm, symbol Connector:TestPoint
- added TP25: PWM_L, TestPoint:TestPoint_Pad_D1.5mm, symbol Connector:TestPoint
- added TP26: L_DRIVE_P, TestPoint:TestPoint_Pad_D1.5mm, symbol Connector:TestPoint
- added TP27: L_DRIVE_N, TestPoint:TestPoint_Pad_D1.5mm, symbol Connector:TestPoint
- added TP28: ENABLE_L, TestPoint:TestPoint_Pad_D1.5mm, symbol Connector:TestPoint
- added TP29: AUDIO_R, TestPoint:TestPoint_Pad_D1.5mm, symbol Connector:TestPoint
- added TP30: PWM_R, TestPoint:TestPoint_Pad_D1.5mm, symbol Connector:TestPoint
- added TP31: R_DRIVE_P, TestPoint:TestPoint_Pad_D1.5mm, symbol Connector:TestPoint
- added TP32: R_DRIVE_N, TestPoint:TestPoint_Pad_D1.5mm, symbol Connector:TestPoint
- added TP33: ENABLE_R, TestPoint:TestPoint_Pad_D1.5mm, symbol Connector:TestPoint
- added TP34: +12V_A, TestPoint:TestPoint_Pad_D1.5mm, symbol Connector:TestPoint
- added U1: OPA1656, Package_SO:SOIC-8_3.9x4.9mm_P1.27mm, symbol Amplifier_Operational:OPA1656ID
- added U10, U5: SN74LVC2G17, Package_TO_SOT_SMD:SOT-23-6, symbol 74xGxx:74LVC2G17
- added U11, U12: TPS7A4901DGNR, Custom:TPS7A4901DRBR, symbol DiscreteClassD:TPS7A4901DGNR
- added U3: OPA1656ID, Package_SO:SOIC-8_3.9x4.9mm_P1.27mm, symbol Amplifier_Operational:OPA1656ID
- added U4, U9: SN74LVC1G04, Package_TO_SOT_SMD:SOT-23-5, symbol 74xGxx:74LVC1G04
- added U7: TLV3602DGKR, Package_SO:VSSOP-8_3x3mm_P0.65mm, symbol DiscreteClassD:TLV3602DGKR
- added U8: TLV3602, Package_SO:VSSOP-8_3x3mm_P0.65mm, symbol DiscreteClassD:TLV3602DGKR
- J1: value AUDIO IN -> STEREO LINE INPUT
Connections:
- net GND: now also C17.2, C20.2, C21.2, C22.2, C24.2, C25.2, C26.2, C28.2, C29.2, C30.2, C32.2, C33.2, C34.2, C35.2, C36.2, C37.2, C38.2, C39.2, C42.2, C43.2, C44.2, C47.2, C48.2, C49.2, C50.2, C51.2, J16.1 (Pin_1), R21.2, R23.2, R25.2, R34.2, R41.2, U1.4 (V-), U10.2 (GND), U11.4 (GND), U11.9 (EP), U12.4 (GND), U12.9 (EP), U3.4 (V-), U4.3 (GND), U5.2 (GND), U7.4 (+), U7.5 (V-), U8.5 (V-), U9.3 (GND)
- net LEFT_IN: now reaches J1.1 (Pin_1)
- net LEFT_IN: now also C40.1
- net RIGHT_IN: now reaches J1.3 (Pin_3)
- net RIGHT_IN: now also C45.1
- new net: R26.2, R27.2, U7.1 (+)
- new net: C42.1, D20.2 (A), R32.2, U5.1
- new net: C31.1, R28.2, U3.6 (-)
- new net: C41.1, R29.2, R30.1, U1.3 (+)
- new net: D21.1 (K), R33.1, U4.4
- new net: C27.2, R22.2, R23.1, U12.2 (FB)
- new net: C26.1, U12.6 (NR/SS)
- new net: C47.1, D22.2 (A), R39.2, U10.1
- new net: C46.1, R36.2, R37.1, U1.5 (+)
- new net: C29.1, C30.1, R24.2, R25.1, U3.3 (+)
- new net: C43.1, D21.2 (A), R33.2, U5.3
- new net: C23.2, R20.2, R21.1, U11.2 (FB)
- new net: C48.1, D23.2 (A), R40.2, U10.3
- new net: D23.1 (K), R40.1, U9.4
- new net: C22.1, U11.6 (NR/SS)
- new net: C45.2, R36.1
- new net: C40.2, R29.1
- new net: R38.1, U1.6 (-), U1.7
- new net: R31.1, U1.1, U1.2 (-)
- new net +12V_A: C32.1, C33.1, C34.1, C35.1, C50.1, C51.1, R43.2, TP34.1, U1.8 (V+), U3.8 (V+)
- new net +12V_GD: C23.1, C24.1, R20.1, R43.1, TP10.1, U11.1 (OUT)
- new net +24V: C17.1, C20.1, C21.1, C25.1, J16.2 (Pin_2), U11.5 (EN), U11.8 (IN), U12.5 (EN), U12.8 (IN)
- new net +5V_A: C27.1, C28.1, C36.1, C37.1, C38.1, C39.1, C44.1, C49.1, R22.1, R24.1, R35.1, R42.1, TP20.1, U10.5 (VCC), U12.1 (OUT), U4.5 (VCC), U5.5 (VCC), U7.8 (V+), U8.8 (V+), U9.5 (VCC)
- new net AUDIO_L: R31.2, TP24.1, U8.1 (+)
- new net AUDIO_R: R38.2, TP29.1, U8.4 (+)
- new net ENABLE_L: R34.1, R35.2, TP28.1
- new net ENABLE_R: R41.1, R42.2, TP33.1
- new net L_DRIVE_N: TP27.1, U5.4
- new net L_DRIVE_P: TP26.1, U5.6
- new net OSC_SQUARE: R27.1, R28.1, TP22.1, U7.7
- new net PWM_L: D20.1 (K), R32.1, TP25.1, U4.2, U8.7
- new net PWM_R: D22.1 (K), R39.1, TP30.1, U8.6, U9.2
- new net R_DRIVE_N: TP32.1, U10.4
- new net R_DRIVE_P: TP31.1, U10.6
- new net TRIANGLE_400K: C31.2, R26.1, TP23.1, U3.7, U8.2 (-), U8.3 (-)
- new net VREF_2V5: C41.2, C46.2, R30.2, R37.2, TP21.1, U3.1, U3.2 (-), U3.5 (+), U7.2 (-), U7.3 (-)
- no-connect marks 0 -> 7
Other:
- removed sheet Power output stage
- added sheet LEFT OUTPUT (PowerOutput_L.kicad_sch)
- added sheet RIGHT OUTPUT (PowerOutput_R.kicad_sch)
- note added: "1. POWER / REGULATORS"
- note added: "10k: default disabled 1k DNP: optional auto-enable"
- note added: "2. SHARED VREF"
- note added: "3. SHARED 400 kHz OSCILLATOR"
- note added: "4. LEFT INPUT / PWM / DEAD TIME"
- note added: "5. RIGHT INPUT / PWM / DEAD TIME"
- note added: "DEAD TIME TUNE: 330R / 100pF; diode K at source, A at RC node. Delayed rise, rapid fall. Final dead time requires gate measurements."
- note added: "DGNR (DGN HVSSOP) value; DRBR footprint assigned. Custom:TPS7A4901DRBR unchanged; verify inventory. Symbol EP9 vs footprint pads 9-13 (centre 13): review. 32.2k / 10k: 5.0007 V nominal."
- note added: "DGNR (DGN HVSSOP) value; DRBR footprint assigned. Custom:TPS7A4901DRBR unchanged; verify inventory. Symbol EP9 vs footprint pads 9-13 (centre 13): review. 91.2k / 10k: 11.9922 V nominal."
- note added: "FILTERED ANALOGUE RAIL"
- note added: "IC SUPPLY PINS / LOCAL BYPASS"
- note added: "Input attenuation = 10k / (51k + 10k) = 0.163934; 2 Vrms -> 0.32787 Vrms / 0.463677 Vpk. One board-wide GND. BTL speaker terminals remain floating. OPA1656 supply: filtered +12V_A."
- note added: "Non-inverting Schmitt + inverting integrator 49.9k / 10k; 3.09k x 1nF: nominal 403.72 kHz Triangle approx. 1.999 to 3.001 V. Measure / tune."
- note added: "R43 feeds OPA1656 packages only. 22uF + 100nF at filter; retain package bypass. UCC27301A devices stay on +12V_GD."
- note added: "U8B spare: stable LOW after VREF settles."
- note removed: "Output stage is on hierarchical sheet 2. Existing control and analogue symbols remain unchanged."
- title: (none) -> 24 V stereo BTL Class-D - shared analogue / control
