File: 7377new/7377new/DiscreteClassD/PowerOutput.kicad_sch (KiCad schematic)
At the start: 63 parts, among them IC1 TLV3602DGKR, J14 24V INPUT, J15 SPEAKER OUT, Q5 DMN6070SY, Q6 DMN6070SY, Q7 DMN6070SY, Q8 DMN6070SY, U1 OPA1656ID, U2 UCC27301ADRCR, U3 OPA1656ID, U4 SN74LVC1G04DBVR, U5 SN74LVC2G17DBVR, U6 UCC27301ADRCR

Commit message: more
Parts:
- C10, C11, C12, C4, C5, C6: Layout Small local +24V / MOSFET / PGND loop -> Small local +24V / MOSFET / GND loop
- TP11: value PGND -> GND
Other:
- note added: "Place each driver against its MOSFET pair. Minimize gate loops and local 24 V ceramic loops. HS Kelvin to high-side source; VSS Kelvin to low-side source. Keep SW_A / SW_B copper compact. No ground plane under large switch-node copper. Place L6 close to bridges. Keep HI / LI away from SW copper. Keep GND distinct from analogue ground. Gate drive requires bootstrap refresh / suitable duty limits. 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"
- note added: "Speaker floats: neither terminal connects to GND. L6: 10uH per winding; verified pins 1-2 and 4-3."
- note removed: "Place each driver against its MOSFET pair. Minimize gate loops and local 24 V ceramic loops. HS Kelvin to high-side source; VSS Kelvin to low-side source. Keep SW_A / SW_B copper compact. No ground plane under large switch-node copper. Place L6 close to bridges. Keep HI / LI away from SW copper. Keep PGND distinct from analogue ground. Gate drive requires bootstrap refresh / suitable duty limits.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"
- note removed: "Speaker floats: neither terminal connects to PGND. L6: 10uH per winding; verified pins 1-2 and 4-3."
