File: 7377new/7377new/7377new.kicad_pcb (KiCad board)
At the start: 2 copper layers, 60.1 x 66.7 mm, 13 parts, among them J1 + LOW -, J2 + HI -, J3 POWER, J7 POT

Commit message: more
Parts:
- removed J7: POT, Connector_PinHeader_2.54mm:PinHeader_1x03_P2.54mm_Vertical
- added C10: 100nF, Capacitor_SMD:C_1206_3216Metric_Pad1.33x1.80mm_HandSolder, F.Cu at (81.5, 63.5)
- added C18: 10nF, Capacitor_SMD:C_0805_2012Metric_Pad1.18x1.45mm_HandSolder, F.Cu at (133.9, 103.5)
- added C27: 22uF, Capacitor_THT:CP_Radial_D5.0mm_P2.50mm, F.Cu at (101.2, 107.4)
- added C28: 100nF, Capacitor_SMD:C_1206_3216Metric_Pad1.33x1.80mm_HandSolder, F.Cu at (55.5, 89.1)
- added C29: 2.2uF, Capacitor_SMD:C_0805_2012Metric_Pad1.18x1.45mm_HandSolder, F.Cu at (60.9, 88.9)
- added C30: 2.2uF, Capacitor_SMD:C_0805_2012Metric_Pad1.18x1.45mm_HandSolder, F.Cu at (60.9, 91.9)
- added C31: 10uF, Capacitor_SMD:C_0805_2012Metric_Pad1.18x1.45mm_HandSolder, F.Cu at (60.9, 94.9)
- added C32: 100nF, Capacitor_SMD:C_1206_3216Metric_Pad1.33x1.80mm_HandSolder, F.Cu at (55.5, 92.4)
- added C33: 10uF, Capacitor_SMD:C_1206_3216Metric_Pad1.33x1.80mm_HandSolder, F.Cu at (55.5, 95.8)
- added C34: 2.7nF, Capacitor_SMD:C_0805_2012Metric_Pad1.18x1.45mm_HandSolder, F.Cu at (89.4, 79.3)
- added C35: 1uF, Capacitor_SMD:C_1206_3216Metric_Pad1.33x1.80mm_HandSolder, F.Cu at (55.5, 99.1)
- added C36: 1uF, Capacitor_SMD:C_1206_3216Metric_Pad1.33x1.80mm_HandSolder, F.Cu at (55.5, 102.5)
- added C37: 10uF, Capacitor_SMD:C_1206_3216Metric_Pad1.33x1.80mm_HandSolder, F.Cu at (134.5, 90.6)
- added C38: 2.7nF, Capacitor_SMD:C_0805_2012Metric_Pad1.18x1.45mm_HandSolder, F.Cu at (101.1, 79.2)
- added C39: 10uF, Capacitor_SMD:C_1206_3216Metric_Pad1.33x1.80mm_HandSolder, F.Cu at (134.5, 93.9)
- added C40: 10uF, Capacitor_THT:CP_Radial_D4.0mm_P1.50mm, F.Cu at (101.1, 113.4)
- added C41: 1uF, Capacitor_SMD:C_1206_3216Metric_Pad1.33x1.80mm_HandSolder, F.Cu at (134.5, 97.3)
- added C6: 10nF, Capacitor_SMD:C_0805_2012Metric_Pad1.18x1.45mm_HandSolder, F.Cu at (133.9, 100.5)
- added C66: 100nF, Capacitor_SMD:C_1206_3216Metric_Pad1.33x1.80mm_HandSolder, F.Cu at (55.5, 105.8)
- added C67: 10uF, Capacitor_SMD:C_0805_2012Metric_Pad1.18x1.45mm_HandSolder, F.Cu at (60.9, 104.0)
- added C68: 100nF, Capacitor_SMD:C_1206_3216Metric_Pad1.33x1.80mm_HandSolder, F.Cu at (55.5, 109.2)
- added C69: 10uF, Capacitor_SMD:C_0805_2012Metric_Pad1.18x1.45mm_HandSolder, F.Cu at (60.9, 107.0)
- added IC2: TPS7A4901DRBR, Custom:TPS7A4901DRBR, F.Cu at (150.5, 100.0)
- added R10: 0R*, Resistor_SMD:R_0805_2012Metric_Pad1.20x1.40mm_HandSolder, F.Cu at (154.8, 83.7)
- added R11: 100K, Resistor_SMD:R_0805_2012Metric_Pad1.20x1.40mm_HandSolder, F.Cu at (154.8, 86.6)
- added R12: 178K, Resistor_SMD:R_0805_2012Metric_Pad1.20x1.40mm_HandSolder, F.Cu at (154.8, 89.6)
- added R31: 470R, Resistor_SMD:R_0805_2012Metric_Pad1.20x1.40mm_HandSolder, F.Cu at (91.4, 83.0)
- added R32: 470R, Resistor_SMD:R_0805_2012Metric_Pad1.20x1.40mm_HandSolder, F.Cu at (99.1, 83.1)
- added R6: 100R, Resistor_SMD:R_0805_2012Metric_Pad1.20x1.40mm_HandSolder, F.Cu at (91.4, 79.3)
- added R61: 2R2, Resistor_SMD:R_0805_2012Metric_Pad1.20x1.40mm_HandSolder, F.Cu at (65.7, 106.6)
- added R7: 100R, Resistor_SMD:R_0805_2012Metric_Pad1.20x1.40mm_HandSolder, F.Cu at (99.1, 79.2)
- added R8: 47K, Resistor_SMD:R_0805_2012Metric_Pad1.20x1.40mm_HandSolder, F.Cu at (97.0, 83.1)
- added R9: 47K, Resistor_SMD:R_0805_2012Metric_Pad1.20x1.40mm_HandSolder, F.Cu at (93.5, 83.1)
- added U12: PCM5122PW, Package_SO:TSSOP-28_4.4x9.7mm_P0.65mm, F.Cu at (94.9, 98.9)
- moved C9 82.5 mm to (121.2, 135.8), turned to 0 degrees
Connections:
- net /PWRIN renamed /VCC
Routing:
- net /3V3: track 0.00 -> 16.6 mm
- net Net-(U12-OUTR): track 0.00 -> 13.5 mm
- net Net-(U12-OUTL): track 0.00 -> 13.3 mm
- net /OUT-HI-DAC: track 0.00 -> 5.89 mm
- net /OUT-LOW-DAC: track 0.00 -> 5.87 mm
- net Net-(C1-Pad1): track 2.30 -> 5.19 mm
- net /5V: track 1.44 -> 0.00 mm
- net Net-(C2-Pad1): track 4.57 -> 5.18 mm
- net GND: vias 66 -> 63
Other:
- board text removed: "5V W G"
