File: 7377new/7377new/7377new.kicad_sch (KiCad schematic)
At the start: 51 parts, among them IC1 ESP32-WROOM-32UE-N8R2, IC2 RESET, IC3 TPS7A2033, IC4 BOOT, J1 + LOW -, J2 + HI -, J3 POWER, J4 POWER IN, U1 LD1117, U12 PCM5122PW

Commit message: more
Parts:
- removed C35, C36: 1uF, Capacitor_SMD:C_1206_3216Metric_Pad1.33x1.80mm_HandSolder, symbol Device:C
- removed C40: 10uF, Capacitor_THT:CP_Radial_D4.0mm_P1.50mm, symbol Device:C_Polarized
- removed C5, C7: 100nF, Capacitor_SMD:C_1206_3216Metric_Pad1.33x1.80mm_HandSolder, symbol Device:C
- removed IC1: ESP32-WROOM-32UE-N8R2, Custom:ESP32WROOM32UEN8R2, symbol Custom:ESP32-WROOM-32UE-N8R2
- removed IC2: RESET, Custom:TS026650BK100SCRD, symbol Custom:TS02-66-50-BK-100-SCR-D
- removed IC3: TPS7A2033, Custom:SOT95P280X145-5N, symbol Custom:TPS7A2033PDBVR
- removed IC4: BOOT, Custom:TS026650BK100SCRD, symbol Custom:TS02-66-50-BK-100-SCR-D
- removed J4: POWER IN, Connector_JST:JST_XH_B2B-XH-A_1x02_P2.50mm_Vertical, symbol Connector:Conn_01x02_Socket
- removed R1, R2: 10K, Resistor_SMD:R_0603_1608Metric_Pad0.98x0.95mm_HandSolder, symbol Device:R
- removed R3, R4, R5: 22R, Resistor_SMD:R_0603_1608Metric_Pad0.98x0.95mm_HandSolder, symbol Device:R
- removed R61: 2R2, Resistor_SMD:R_0805_2012Metric_Pad1.20x1.40mm_HandSolder, symbol Device:R
- removed U1: LD1117, Package_TO_SOT_SMD:SOT-223-3_TabPin2, symbol Regulator_Linear:LD1117S33TR_SOT223
- added C18: 10nF, Capacitor_SMD:C_0805_2012Metric_Pad1.18x1.45mm_HandSolder, symbol Device:C
- added C37, C39: 10uF, Capacitor_SMD:C_1206_3216Metric_Pad1.33x1.80mm_HandSolder, symbol Device:C
- added C41: 1uF, Capacitor_SMD:C_1206_3216Metric_Pad1.33x1.80mm_HandSolder, symbol Device:C
- added IC2: TPS7A4901DRBR, Custom:TPS7A4901DRBR, symbol Custom:TPS7A4901DRBR
- added R10: 0R*, Resistor_SMD:R_0805_2012Metric_Pad1.20x1.40mm_HandSolder, symbol Device:R
- added R11: 100K, Resistor_SMD:R_0805_2012Metric_Pad1.20x1.40mm_HandSolder, symbol Device:R
- added R12: 178K, Resistor_SMD:R_0805_2012Metric_Pad1.20x1.40mm_HandSolder, symbol Device:R
- C10: value 1uF -> 100nF
- C6: value 10uF -> 10nF
Connections:
- net AVDD is gone; now on net 3V3: C27.1, C28.1, C31.1, C66.1, C67.1, C68.1, C69.1, U12.1 (CPVDD), U12.18 (MODE2/MS), U12.25 (XSMT), U12.28 (DVDD), U12.8 (AVDD)
- net PWRIN is gone; now on net VCC: AMP1.13 (VCC2), AMP1.3 (VCC1), C3.1, C4.1, C9.1, J3.1 (Pin_1), R13.2
- net 3V3: now also C18.2, C39.2, C41.2, IC2.1 (OUT), R10.2, R12.2; no longer C6.1
- net GND: now also C37.1, C39.1, C41.1, IC2.10 (EP_2), IC2.11 (EP_3), IC2.12 (EP_4), IC2.13 (EP_5), IC2.4 (GND), IC2.9 (EP_1), R11.2
- net at U12.6 (OUTL): now also R32.2; no longer R31.1
- net at U12.7 (OUTR): now also R31.1; no longer R32.2
- net EN renamed VCC
- net VCC: now also C37.2, IC2.5 (EN), IC2.8 (IN), R10.1
- new net: C18.1, IC2.2 (FB), R11.1, R12.1
- new net: C6.1, IC2.6 (NR/SS)
Other:
- moved on the sheet: AMP1, C1, C11, C17, C2, C27, C28, C29, C30, C31, C32, C33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
