File: BoostedClassD/Amplifiers.kicad_sch (KiCad schematic)
At the start: 6 parts, among them U2 TAS2320, U3 TAS2120, U4 TPS7A2018

Commit message: m0re
Parts:
- added C10, C11, C12, C9: 10uF, Capacitor_SMD:C_1206_3216Metric_Pad1.33x1.80mm_HandSolder, symbol Device:C
- added C13, C14, C17, C18: 100nF, Capacitor_SMD:C_1206_3216Metric_Pad1.33x1.80mm_HandSolder, symbol Device:C
- added C15, C16, C19, C20: 1uF, Capacitor_SMD:C_1206_3216Metric_Pad1.33x1.80mm_HandSolder, symbol Device:C
- added C21, C22, C23, C24: 2.2uF, Capacitor_SMD:C_0805_2012Metric_Pad1.18x1.45mm_HandSolder, symbol Device:C
Connections:
- net GND: now also C10.2, C11.2, C12.2, C13.2, C14.2, C15.2, C16.2, C19.2, C20.2, C21.2, C22.2, C23.2, C24.2, C9.2
- net SYS: now also L2.1, U2.14 (VBAT), U2.15 (VBAT), U3.14 (VBAT_SNS), U3.15 (VBAT), C19.1, C20.1, C9.1
- net VDD1V8: now also U2.5 (IOVDD), U3.5 (IOVDD), C21.1, C22.1, C23.1, C24.1
- net at U3.17 (GREG): now also C17.1
- net PVDD: now reaches U3.18 (VBST)
- net PVDD: now also U2.18 (VBST), C10.1, C11.1, C12.1, C13.1, C14.1, C17.2, C18.2
- net LEFT -: now reaches U3.19 (OUTN)
- net LEFT +: now reaches U3.20 (OUTP)
- net at U3.26 (DREG): now also C16.1
- net SDA: now reaches U3.3 (HW_SEL3_SDA)
- net SDA: now also U2.3 (HW_SEL3_SDA)
- net SCL: now reaches U3.4 (HW_SEL2_SCL)
- net SCL: now also U2.4 (HW_SEL2_SCL)
- net at U2.17 (GREG): now also C18.1
- net RIGHT -: now reaches U2.19 (OUTN)
- net RIGHT +: now reaches U2.20 (OUTP)
- net at U2.26 (DREG): now also C15.1

Commit message: more
Parts:
- added C28, C29, C30, C31: 1nF, Capacitor_SMD:C_0805_2012Metric_Pad1.18x1.45mm_HandSolder, symbol Device:C
- added FB1, FB2, FB3, FB4: FB, Inductor_SMD:L_0805_2012Metric_Pad1.05x1.20mm_HandSolder, symbol Device:FerriteBead
Connections:
- net GND: now also C28.2, C29.1, C30.2, C31.1
- net LEFT +: now also C30.1, FB3.2; no longer U3.20 (OUTP)
- net LEFT -: now also C31.2, FB4.2; no longer U3.19 (OUTN)
- net RIGHT +: now also C28.1, FB1.2; no longer U2.20 (OUTP)
- net RIGHT -: now also C29.2, FB2.2; no longer U2.19 (OUTN)
- new net: FB2.1, U2.19 (OUTN)
- new net: FB1.1, U2.20 (OUTP)
- new net LEFT+: FB3.1, U3.20 (OUTP)
- new net LEFT-: FB4.1, U3.19 (OUTN)

Commit message: more
Parts:
- added R22, R23: 100K, Resistor_SMD:R_0805_2012Metric_Pad1.20x1.40mm_HandSolder, symbol Device:R
- added R24, R25: 24K, Resistor_SMD:R_0805_2012Metric_Pad1.20x1.40mm_HandSolder, symbol Device:R
- C10, C11, C12: Rating (none) -> 10u / 25V X7R
- C13, C14, C17, C18: footprint Capacitor_SMD:C_1206_3216Metric_Pad1.33x1.80mm_HandSolder -> Capacitor_SMD:C_0201_0603Metric; LCSC (none) -> C307379; MPN (none) -> CL03A104KA3NNNC; Manufacturer (none) -> Samsung Electro-Mechanics; Rating (none) -> 100nF / 25V X5R
- C15, C16, C19, C20: footprint Capacitor_SMD:C_1206_3216Metric_Pad1.33x1.80mm_HandSolder -> Capacitor_SMD:C_0201_0603Metric; LCSC (none) -> C170153; MPN (none) -> CL03A105MP3NSNC; Manufacturer (none) -> Samsung Electro-Mechanics; Rating (none) -> 1uF / 10V X5R
- C21, C22, C23, C24: footprint Capacitor_SMD:C_0805_2012Metric_Pad1.18x1.45mm_HandSolder -> Capacitor_SMD:C_0201_0603Metric; LCSC (none) -> C318539; MPN (none) -> CL03A225MP3CRNC; Manufacturer (none) -> Samsung Electro-Mechanics; Rating (none) -> 2.2uF / 10V X5R
- L2: footprint Inductor_SMD:L_1008_2520Metric_Pad1.43x2.20mm_HandSolder -> Inductor_SMD:L_Vishay_IHLP-1212
- U2: symbol Custom:PTAS2120RBGR -> BoostedClassD:TAS2320
- U3: symbol Custom:TAS2320 -> BoostedClassD:TAS2120
Connections:
- net GND: now also U2.16 (HW_SEL1), U2.22 (GND), U2.23 (GND), U3.16 (HW_SEL1), U3.22 (GND), U3.23 (GND), R22.2, R23.2, R24.2
- net VDD1V8: no longer C22.1, C24.1, U2.5 (IOVDD), U3.5 (IOVDD)
- net ADDR2120: now reaches U3.2 (HW_SEL4_AD1)
- net ADDR2120: now also R24.1
- net AMP2120_SDZ: now reaches U3.7 (SD_N)
- net AMP2120_SDZ: now also R22.1
- net ADDR2320: now reaches U2.2 (HW_SEL4_AD1)
- net ADDR2320: now also R25.1
- net AMP2320_SDZ: now reaches U2.7 (SD_N)
- net AMP2320_SDZ: now also R23.1
- new net ESP3V3: C22.1, C24.1, R25.2, U2.5 (IOVDD), U3.5 (IOVDD)
- no-connect marks 0 -> 5
Other:
- note added: "C10-C12: 10u, 25 V X7R; C13/C14: 100n, 25 V X7R. C21-C24: 2u2, 6.3 V X7R. Select effective capacitance at operating bias."
- note added: "CONTROL: U3 TAS2120 = 0x49; U2 TAS2320 = 0x4A (7-bit I2C). IOVDD = 3.3 V; core VDD remains 1.8 V. SDZ defaults LOW. Firmware: release U2 secondary before U3 primary; establish clocks and observe datasheet startup delays (at least 300 us where specified)."
- note added: "L2: 1 uH value retained; exact part and saturation/thermal rating MUST be selected against programmed boost current limit before assembly. PCB footprint is unverified. PVDD capacitors: verify effective capacitance under DC bias. BTL outputs: neither is GND."
- moved on the sheet: C10, C11, C12, C13, C14, C15, C16, C17, C18, C19, C20, C21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
