File: BoostedClassD/BoostedClassD.kicad_pcb (KiCad board)
At the start: 2 copper layers, 50.5 x 53.3 mm, 26 parts, among them IC1 BQ25185, IC2 ESP32-WROOM-32UE-N8R2, IC3 RESET, IC4 BOOT, J1 SYSTEM CONNECTOR 1, J2 SYSTEM CONNECTOR 2, Q1 DMG3415U, U1 TPS631000, U2 TAS2320, U3 TAS2120, U4 TPS7A2018

Commit message: m0re
Parts:
- added C10: 10uF, Capacitor_SMD:C_1206_3216Metric_Pad1.33x1.80mm_HandSolder, F.Cu at (153.9, 138.4)
- added C11: 10uF, Capacitor_SMD:C_1206_3216Metric_Pad1.33x1.80mm_HandSolder, F.Cu at (153.9, 141.7)
- added C12: 10uF, Capacitor_SMD:C_1206_3216Metric_Pad1.33x1.80mm_HandSolder, F.Cu at (153.9, 145.1)
- added C13: 100nF, Capacitor_SMD:C_1206_3216Metric_Pad1.33x1.80mm_HandSolder, F.Cu at (159.9, 135.0)
- added C14: 100nF, Capacitor_SMD:C_1206_3216Metric_Pad1.33x1.80mm_HandSolder, F.Cu at (159.9, 138.4)
- added C15: 1uF, Capacitor_SMD:C_1206_3216Metric_Pad1.33x1.80mm_HandSolder, F.Cu at (159.9, 141.7)
- added C16: 1uF, Capacitor_SMD:C_1206_3216Metric_Pad1.33x1.80mm_HandSolder, F.Cu at (159.9, 145.1)
- added C17: 100nF, Capacitor_SMD:C_1206_3216Metric_Pad1.33x1.80mm_HandSolder, F.Cu at (165.9, 135.0)
- added C18: 100nF, Capacitor_SMD:C_1206_3216Metric_Pad1.33x1.80mm_HandSolder, F.Cu at (165.9, 138.4)
- added C19: 1uF, Capacitor_SMD:C_1206_3216Metric_Pad1.33x1.80mm_HandSolder, F.Cu at (165.9, 141.7)
- added C20: 1uF, Capacitor_SMD:C_1206_3216Metric_Pad1.33x1.80mm_HandSolder, F.Cu at (165.9, 145.1)
- added C21: 2.2uF, Capacitor_SMD:C_0805_2012Metric_Pad1.18x1.45mm_HandSolder, F.Cu at (171.3, 134.9)
- added C22: 2.2uF, Capacitor_SMD:C_0805_2012Metric_Pad1.18x1.45mm_HandSolder, F.Cu at (171.3, 137.9)
- added C23: 2.2uF, Capacitor_SMD:C_0805_2012Metric_Pad1.18x1.45mm_HandSolder, F.Cu at (171.3, 140.9)
- added C24: 2.2uF, Capacitor_SMD:C_0805_2012Metric_Pad1.18x1.45mm_HandSolder, F.Cu at (171.3, 143.9)
- added C25: 10uF, Capacitor_SMD:C_1206_3216Metric_Pad1.33x1.80mm_HandSolder, F.Cu at (189.4, 111.4)
- added C26: 1uF, Capacitor_SMD:C_1206_3216Metric_Pad1.33x1.80mm_HandSolder, F.Cu at (189.4, 114.8)
- added C27: 1uF, Capacitor_SMD:C_1206_3216Metric_Pad1.33x1.80mm_HandSolder, F.Cu at (189.4, 118.1)
- added C7: 100nF, Capacitor_SMD:C_1206_3216Metric_Pad1.33x1.80mm_HandSolder, F.Cu at (172.7, 89.2)
- added C8: 100nF, Capacitor_SMD:C_1206_3216Metric_Pad1.33x1.80mm_HandSolder, F.Cu at (201.8, 112.5)
- added C9: 10uF, Capacitor_SMD:C_1206_3216Metric_Pad1.33x1.80mm_HandSolder, F.Cu at (142.7, 106.7)
- added G***: LOGO, Custom:LOGONEW, F.Cu at (161.9, 76.8)
- added H1: ~, MountingHole:MountingHole_4.3mm_M4, F.Cu at (178.3, 75.7)
- added H2: ~, MountingHole:MountingHole_4.3mm_M4, F.Cu at (120.9, 75.7)
- added H3: ~, MountingHole:MountingHole_4.3mm_M4, F.Cu at (120.9, 120.4)
- added H4: ~, MountingHole:MountingHole_4.3mm_M4, F.Cu at (178.3, 120.4)
- added IC5: INA236, Custom:INA236BIDDFR, F.Cu at (172.3, 92.2)
- added J3: SPK OUT, Connector_JST:JST_XH_B4B-XH-A_1x04_P2.50mm_Vertical, F.Cu at (177.0, 107.3)
- added R10: 0R*2, Resistor_SMD:R_0805_2012Metric_Pad1.20x1.40mm_HandSolder, F.Cu at (164.9, 84.1)
- added R11: 0R*3, Resistor_SMD:R_0805_2012Metric_Pad1.20x1.40mm_HandSolder, F.Cu at (164.9, 86.6)
- added R12: 4K7, Resistor_SMD:R_0805_2012Metric_Pad1.20x1.40mm_HandSolder, F.Cu at (196.3, 89.3)
- added R13: 47K, Resistor_SMD:R_0805_2012Metric_Pad1.20x1.40mm_HandSolder, F.Cu at (196.3, 92.2)
- added R14: 10K, Resistor_SMD:R_0805_2012Metric_Pad1.20x1.40mm_HandSolder, F.Cu at (196.3, 95.2)
- added R15: 10K, Resistor_SMD:R_0805_2012Metric_Pad1.20x1.40mm_HandSolder, F.Cu at (196.3, 98.1)
- added R8: 4K7, Resistor_SMD:R_0805_2012Metric_Pad1.20x1.40mm_HandSolder, F.Cu at (196.3, 86.3)
- added R9: 0R02, Custom:Untitled_4, F.Cu at (176.1, 92.8)
- added TP1: TestPoint, TestPoint:TestPoint_Pad_D2.0mm, F.Cu at (187.7, 103.0)
- added U5: ATtiny412, Package_SO:SOIC-8_3.9x4.9mm_P1.27mm, F.Cu at (201.6, 116.5)
- moved C3 55.5 mm to (129.9, 76.6), turned to 180 degrees
- moved IC3 42.8 mm to (220.1, 74.8)
- moved IC4 42.8 mm to (220.1, 83.9)
- moved R1 42.8 mm to (219.9, 91.9)
- moved R2 42.8 mm to (219.9, 94.5)
- moved R3 42.8 mm to (219.9, 97.0)
- moved R4 42.8 mm to (219.9, 99.5)
- moved R5 42.8 mm to (219.9, 102.0)
- moved C4 42.8 mm to (225.1, 95.7)
- moved U1 42.3 mm to (124.3, 84.1)
- moved C1 42.3 mm to (123.6, 88.1)
- moved C2 42.3 mm to (120.5, 82.3)
- moved R6 42.3 mm to (127.7, 84.3)
- moved R7 42.3 mm to (124.4, 81.5)
- moved L1 42.3 mm to (120.8, 85.6)
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Connections:
- net /ESP32/EN renamed /ESP32-ATTINY/EN
- net /ESP32/GPIO0 renamed /ESP32-ATTINY/GPIO0
- net /ESP32/RX renamed /ESP32-ATTINY/RX
- net /ESP32/TX renamed /ESP32-ATTINY/TX
- IC1 pad 2: /BAT + -> Net-(IC1-BAT)
- IC1 pad 3: unconnected-(IC1-STAT2-Pad3) -> /CHGPOWER/STAT2
- IC1 pad 6: unconnected-(IC1-TS/MR-Pad6) -> /NTC +
- IC1 pad 9: unconnected-(IC1-STAT1-Pad9) -> /CHGPOWER/STAT1
- IC2 pad 12: unconnected-(IC2-IO27-Pad12) -> /Amplifiers/SDOUT
- IC2 pad 30: unconnected-(IC2-IO18-Pad30) -> /ENC A
- IC2 pad 31: unconnected-(IC2-IO19-Pad31) -> /ENC B
- IC2 pad 33: /ESP32/SDA -> /Amplifiers/SDA
- IC2 pad 36: /ESP32/SCL -> /Amplifiers/SCL
- IC2 pad 37: unconnected-(IC2-IO23-Pad37) -> /ESP32-ATTINY/STATUS LED
- IC2 pad 4: unconnected-(IC2-SENSOR_VP-Pad4) -> /ESP32-ATTINY/STAT1
- IC2 pad 5: unconnected-(IC2-SENSOR_VN-Pad5) -> /ESP32-ATTINY/STAT2
- IC2 pad 6: unconnected-(IC2-IO34-Pad6) -> /ESP32-ATTINY/PLAY_PAUSE
- IC2 pad 7: unconnected-(IC2-IO35-Pad7) -> /ESP32-ATTINY/POWER_OFF_REQ
- IC2 pad 8: unconnected-(IC2-IO32-Pad8) -> /ESP32-ATTINY/ALERT
- J1 pad 5: /LEFT + -> /NTC +
- J1 pad 6: /LEFT - -> GND
- J1 pad 7: /RIGHT + -> /STATUS LED +
- J1 pad 8: /RIGHT - -> /STATUS LED -
- J2 pad 8: /NC -> unconnected-(J2-Pin_8-Pad8)
- L2 pad 1: Net-(U3-VBAT) -> /Amplifiers/SYS
- Q1 pad 1: unconnected-(Q1-G-Pad1) -> Net-(Q1-G)
- R1 pad 1: /ESP32/3V3 -> /ENC 3V3
- R2 pad 1: /ESP32/3V3 -> /ENC 3V3
- U2 pad 14: unconnected-(U2-VBAT-Pad14) -> /Amplifiers/SYS
- U2 pad 15: unconnected-(U2-VBAT-Pad15) -> /Amplifiers/SYS
- U2 pad 17: unconnected-(U2-GREG-Pad17) -> Net-(U2-GREG)
- U2 pad 18: unconnected-(U2-VBST-Pad18) -> /Amplifiers/PVDD
- U2 pad 19: unconnected-(U2-OUTN-Pad19) -> /RIGHT -
- U2 pad 20: unconnected-(U2-OUTP-Pad20) -> /RIGHT +
- U2 pad 26: unconnected-(U2-DREG-Pad26) -> Net-(U2-DREG)
- U2 pad 3: unconnected-(U2-HW_SEL3_SDA-Pad3) -> /Amplifiers/SDA
- U2 pad 4: unconnected-(U2-HW_SEL2_SCL-Pad4) -> /Amplifiers/SCL
- U2 pad 5: unconnected-(U2-IOVDD-Pad5) -> /Amplifiers/VDD1V8
- U3 pad 14: Net-(U3-VBAT) -> /Amplifiers/SYS
- U3 pad 15: Net-(U3-VBAT) -> /Amplifiers/SYS
- U3 pad 17: unconnected-(U3-GREG-Pad17) -> Net-(U3-GREG)
- U3 pad 18: unconnected-(U3-VBST-Pad18) -> /Amplifiers/PVDD
- U3 pad 19: unconnected-(U3-OUTN-Pad19) -> /LEFT -
- U3 pad 20: unconnected-(U3-OUTP-Pad20) -> /LEFT +
- U3 pad 26: unconnected-(U3-DREG-Pad26) -> Net-(U3-DREG)
- U3 pad 3: unconnected-(U3-HW_SEL3_SDA-Pad3) -> /Amplifiers/SDA
- U3 pad 4: unconnected-(U3-HW_SEL2_SCL-Pad4) -> /Amplifiers/SCL
- U3 pad 5: unconnected-(U3-IOVDD-Pad5) -> /Amplifiers/VDD1V8
Routing:
- net /ENC 3V3: track 4.13 -> 9.25 mm
- net Net-(U3-SW): track 0.00 -> 3.82 mm
- net /CHGPOWER/SYS: track 4.00 -> 7.23 mm
- net /CHGPOWER/IN-: track 0.00 -> 3.00 mm
- net /CHGPOWER/IN+: track 0.00 -> 2.83 mm
- net /Amplifiers/SYS: track 5.75 -> 7.81 mm
- added copper zone on F.Cu, net GND
- added copper zone on In1.Cu, net GND
Other:
- board size 50.5 x 53.3 mm -> 66.5 x 53.3 mm
- copper layers 2 -> 4
- board text added: "3NC BTN"
- board text added: "BAT +"
- board text added: "CHG +"
- board text added: "CHG LED +"
- board text added: "CHG LED -"
- board text added: "ENC 3V3"
- board text added: "ENC A"
- board text added: "ENC B"
- board text added: "GND"
- board text added: "LEFT +"
- board text added: "LEFT -"
- board text added: "NTC +"
- board text added: "RIGHT +"
- board text added: "RIGHT -"
- board text added: "STATUS LED +"
- board text added: "STATUS LED -"
- board text added: "TAS2120 + TAS2320 1S Charger Boosted Class D Tom Watson Audio 2026"

Commit message: loads
Parts:
- added G***: LOGO, Custom:ClassDSmall, F.Cu at (164.1, 135.0)
- added J4: PROG, Connector_PinHeader_2.54mm:PinHeader_1x04_P2.54mm_Vertical, F.Cu at (179.6, 89.8)
- added R16: 100K, Resistor_SMD:R_0805_2012Metric_Pad1.20x1.40mm_HandSolder, F.Cu at (209.5, 102.8)
- added R17: 240R, Resistor_SMD:R_0805_2012Metric_Pad1.20x1.40mm_HandSolder, F.Cu at (209.5, 105.8)
- added R18: 13K7, Resistor_SMD:R_0805_2012Metric_Pad1.20x1.40mm_HandSolder, F.Cu at (209.5, 108.7)
- added R19: 2K2, Resistor_SMD:R_0805_2012Metric_Pad1.20x1.40mm_HandSolder, F.Cu at (209.5, 111.7)
- added R20: 2K2, Resistor_SMD:R_0805_2012Metric_Pad1.20x1.40mm_HandSolder, F.Cu at (209.5, 114.6)
- moved C1 88.6 mm to (211.7, 78.2), turned to 0 degrees
- moved L1 88.5 mm to (209.1, 81.0), turned to 0 degrees
- moved C2 85.3 mm to (205.8, 81.3), turned to -90 degrees
- moved U1 83.6 mm to (207.6, 77.5), turned to 90 degrees
- moved R6 80.9 mm to (207.9, 74.2), turned to 90 degrees
- moved R7 80.8 mm to (205.1, 77.5), turned to 90 degrees
- moved IC3 78.7 mm to (205.8, 152.2), turned to 180 degrees
- moved C19 73.5 mm to (132.0, 76.6), turned to 180 degrees
- moved C24 71.1 mm to (141.0, 79.6)
- moved IC4 68.5 mm to (215.2, 152.2), turned to 180 degrees
- moved C18 68.2 mm to (132.0, 79.2)
- moved C23 66.6 mm to (135.5, 84.7), turned to -90 degrees
- moved C4 65.0 mm to (198.2, 154.9)
- moved C12 64.0 mm to (132.0, 84.9), turned to 180 degrees
- moved R1 63.7 mm to (197.1, 151.3), turned to -90 degrees
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Connections:
- net Net-(Q1-G) renamed /CHGPOWER/POWER-ON-MOSFET
- C1 pad 1: /CHGPOWER/SYS -> /Amplifiers/SYS
- C25 pad 1: /CHGPOWER/SYS -> /CHGPOWER/BQ-SYS
- C8 pad 1: /CHGPOWER/SYS -> /Amplifiers/SYS
- IC1 pad 1: /CHGPOWER/SYS -> /CHGPOWER/BQ-SYS
- IC1 pad 3: /CHGPOWER/STAT2 -> Net-(IC1-STAT2)
- IC1 pad 7: unconnected-(IC1-ILIM/VSET-Pad7) -> Net-(IC1-ILIM/VSET)
- IC1 pad 8: unconnected-(IC1-ISET-Pad8) -> Net-(IC1-ISET)
- IC1 pad 9: /CHGPOWER/STAT1 -> unconnected-(IC1-STAT1-Pad9)
- IC2 pad 30: /ENC A -> /ENC B
- IC2 pad 31: /ENC B -> /ENC A
- IC2 pad 37: /ESP32-ATTINY/STATUS LED -> /STATUS LED +
- IC2 pad 4: /ESP32-ATTINY/STAT1 -> unconnected-(IC2-SENSOR_VP-Pad4)
- IC2 pad 5: /ESP32-ATTINY/STAT2 -> unconnected-(IC2-SENSOR_VN-Pad5)
- J1 pad 8: /STATUS LED - -> GND
- J2 pad 3: /ENC A -> /ENC B
- J2 pad 4: /ENC B -> /ENC A
- J2 pad 7: /CHG LED - -> GND
- J2 pad 8: unconnected-(J2-Pin_8-Pad8) -> GND
- J3 pad 1: /LEFT + -> /LEFT -
- J3 pad 2: /LEFT - -> /LEFT +
- J3 pad 3: /RIGHT + -> /RIGHT -
- J3 pad 4: /RIGHT - -> /RIGHT +
- Q1 pad 2: unconnected-(Q1-S-Pad2) -> /CHGPOWER/BQ-SYS
- Q1 pad 3: unconnected-(Q1-D-Pad3) -> /Amplifiers/SYS
- R13 pad 1: /CHGPOWER/SYS -> /Amplifiers/SYS
- U1 pad 4: /CHGPOWER/SYS -> /Amplifiers/SYS
- U1 pad 5: /CHGPOWER/SYS -> /Amplifiers/SYS
- U5 pad 1: /CHGPOWER/SYS -> /Amplifiers/SYS
Routing:
- net /Amplifiers/VDD1V8: track 2.46 -> 53.0 mm, vias 0 -> 3
- net /Amplifiers/SEL5: track 0.00 -> 29.2 mm, vias 0 -> 2
- net /Amplifiers/LRCK: track 0.00 -> 28.2 mm, vias 0 -> 2
- net /RIGHT -: track 0.00 -> 26.7 mm
- net /Amplifiers/BCK: track 0.00 -> 26.0 mm, vias 0 -> 2
- net /Amplifiers/DATA: track 0.00 -> 23.9 mm, vias 0 -> 2
- net /RIGHT +: track 0.00 -> 22.8 mm
- net /Amplifiers/SYS: track 7.81 -> 29.7 mm, vias 0 -> 2
- net /LEFT +: track 0.00 -> 21.0 mm
- net /LEFT -: track 0.00 -> 16.9 mm
- net /CHGPOWER/SYS: track 7.23 -> 0.00 mm
- net Net-(U3-GREG): track 0.00 -> 6.51 mm
- net Net-(U2-GREG): track 0.00 -> 6.47 mm
- net /ENC 3V3: track 9.25 -> 5.21 mm, vias 0 -> 1
- net /CHGPOWER/IN-: track 3.00 -> 0.00 mm
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- added copper zone on F.Cu, net /Amplifiers/PVDD
- added copper zone on In2.Cu, net /Amplifiers/PVDD
- added copper zone on F.Cu, net /Amplifiers/SYS
Other:
- board text added: "3V3"
- board text added: "ENC BTN"
- board text added: "RX"
- board text added: "TX"
- board text removed: "3NC BTN"

Commit message: more
Parts:
- removed IC3: RESET, Custom:TS026650BK100SCRD
- removed IC4: BOOT, Custom:TS026650BK100SCRD
- removed R20: 2K2, Resistor_SMD:R_0805_2012Metric_Pad1.20x1.40mm_HandSolder
- added S1: BOOT, Custom:PTS810SJM250SMTRLFS, F.Cu at (219.4, 126.6)
- added S2: EN, Custom:PTS810SJM250SMTRLFS, F.Cu at (212.0, 126.6)
- moved R8 113.4 mm to (94.2, 104.9), turned to -90 degrees
- moved IC2 102.3 mm to (211.7, 68.9)
- moved R12 99.9 mm to (103.9, 106.4), turned to -90 degrees
- moved R3 95.0 mm to (104.3, 113.8), turned to 0 degrees
- moved R4 94.8 mm to (104.3, 115.3), turned to 0 degrees
- moved U5 93.0 mm to (106.1, 92.8)
- moved R15 92.5 mm to (104.9, 83.8)
- moved R14 92.4 mm to (104.9, 81.8)
- moved R13 91.5 mm to (105.9, 78.2), turned to -90 degrees
- moved C8 85.7 mm to (105.9, 73.7), turned to 90 degrees
- moved C27 66.6 mm to (178.7, 52.4), turned to 90 degrees
- moved C26 66.2 mm to (183.3, 48.8), turned to 180 degrees
- moved G*** 65.5 mm to (132.8, 77.5)
- moved R5 61.2 mm to (207.3, 123.2)
- moved C25 60.4 mm to (183.3, 51.4)
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Routing:
- net /Amplifiers/SCL: track 0.00 -> 48.8 mm, vias 0 -> 2
- net /Amplifiers/SDA: track 0.00 -> 36.5 mm, vias 0 -> 2
- net /Amplifiers/DATA: track 23.9 -> 40.1 mm
- net /Amplifiers/BCK: track 26.0 -> 41.7 mm
- net /Amplifiers/LRCK: track 28.2 -> 43.4 mm
- net /ENC 3V3: track 5.21 -> 0.00 mm, vias 1 -> 0
- net Net-(U1-FB): track 3.85 -> 0.00 mm
- net Net-(U1-LX1): track 3.78 -> 0.00 mm
- net /Amplifiers/SYS: track 29.7 -> 26.3 mm, vias 2 -> 1
- net /Amplifiers/VDD1V8: track 53.0 -> 55.9 mm
- net Net-(U1-LX2): track 2.89 -> 0.00 mm
- net /ENC A: track 0.61 -> 0.00 mm
- net GND: vias 39 -> 38
Other:
- board size 66.5 x 53.3 mm -> 66.5 x 58.4 mm

Commit message: more
Parts:
- added C28: 1nF, Capacitor_SMD:C_0805_2012Metric_Pad1.18x1.45mm_HandSolder, F.Cu at (124.1, 91.5)
- added C29: 1nF, Capacitor_SMD:C_0805_2012Metric_Pad1.18x1.45mm_HandSolder, F.Cu at (124.1, 87.5)
- added C30: 1nF, Capacitor_SMD:C_0805_2012Metric_Pad1.18x1.45mm_HandSolder, F.Cu at (124.1, 114.3)
- added C31: 1nF, Capacitor_SMD:C_0805_2012Metric_Pad1.18x1.45mm_HandSolder, F.Cu at (124.1, 110.3)
- added F1: 3A, Fuse:Fuse_1206_3216Metric_Pad1.42x1.75mm_HandSolder, F.Cu at (172.5, 83.6)
- added F2: 3A, Fuse:Fuse_1206_3216Metric_Pad1.42x1.75mm_HandSolder, F.Cu at (163.4, 83.6)
- added FB1: FB, Inductor_SMD:L_0805_2012Metric_Pad1.05x1.20mm_HandSolder, F.Cu at (127.1, 90.4)
- added FB2: FB, Inductor_SMD:L_0805_2012Metric_Pad1.05x1.20mm_HandSolder, F.Cu at (127.1, 88.5)
- added FB3: FB, Inductor_SMD:L_0805_2012Metric_Pad1.05x1.20mm_HandSolder, F.Cu at (127.1, 113.3)
- added FB4: FB, Inductor_SMD:L_0805_2012Metric_Pad1.05x1.20mm_HandSolder, F.Cu at (127.1, 111.4)
- added J5: CC, Connector_JST:JST_XH_B2B-XH-A_1x02_P2.50mm_Vertical, F.Cu at (180.2, 76.9)
- added R20: 5K1, Resistor_SMD:R_0805_2012Metric_Pad1.20x1.40mm_HandSolder, F.Cu at (181.3, 80.8)
- added R21: 5K1, Resistor_SMD:R_0805_2012Metric_Pad1.20x1.40mm_HandSolder, F.Cu at (176.7, 80.8)
- moved R8 91.9 mm to (186.1, 101.7)
- moved R12 82.2 mm to (186.1, 106.6), turned to 90 degrees
- moved R10 68.6 mm to (273.9, 87.1)
- moved R11 68.6 mm to (275.8, 99.2)
- moved R16 68.6 mm to (275.8, 102.1)
- moved TP1 68.6 mm to (256.7, 100.3)
- moved C8 62.5 mm to (154.7, 112.8), turned to 180 degrees
- moved R4 59.0 mm to (163.2, 113.3)
- moved R3 58.9 mm to (163.2, 111.6)
- moved C3 56.1 mm to (164.0, 103.0)
- moved IC2 54.1 mm to (175.3, 108.9)
- moved U5 50.9 mm to (154.6, 108.6), turned to 180 degrees
- moved C1 50.4 mm to (179.4, 91.3), turned to -90 degrees
- moved L1 47.2 mm to (181.4, 86.4), turned to 180 degrees
- moved R6 44.1 mm to (182.5, 92.8), turned to 180 degrees
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Connections:
- C26 pad 1: /CHG + -> /USB5V +
- IC1 pad 10: /CHG + -> /USB5V +
- J1 pad 1: /BAT + -> Net-(J1-Pin_1)
- J1 pad 3: /CHG + -> Net-(J1-Pin_3)
- J1 pad 7: /STATUS LED + -> /CHG LED +
- J2 pad 6: /CHG LED + -> /STATUS LED +
- J2 pad 8: GND -> unconnected-(J2-Pin_8-Pad8)
- U2 pad 19: /RIGHT - -> Net-(U2-OUTN)
- U2 pad 20: /RIGHT + -> Net-(U2-OUTP)
- U3 pad 19: /LEFT - -> /Amplifiers/LEFT-
- U3 pad 20: /LEFT + -> /Amplifiers/LEFT+
Routing:
- net /ENC 3V3: track 0.00 -> 115.8 mm, vias 0 -> 5
- net /Amplifiers/SDA: track 36.5 -> 110.1 mm, vias 2 -> 4
- net /Amplifiers/SCL: track 48.8 -> 114.8 mm, vias 2 -> 4
- net /ESP32-ATTINY/EN: track 0.00 -> 38.6 mm, vias 0 -> 2
- net /ENC BTN: track 0.00 -> 38.4 mm, vias 0 -> 2
- net /ESP32-ATTINY/TX: track 0.00 -> 28.7 mm, vias 0 -> 1
- net /ESP32-ATTINY/RX: track 0.00 -> 27.9 mm, vias 0 -> 1
- net /Amplifiers/DATA: track 40.1 -> 66.9 mm, vias 2 -> 3
- net /USB5V +: track 0.00 -> 24.5 mm, vias 0 -> 2
- net /NTC +: track 0.00 -> 16.5 mm, vias 0 -> 1
- net /ESP32-ATTINY/POWER_OFF_REQ: track 0.00 -> 15.0 mm, vias 0 -> 2
- net Net-(IC1-STAT2): track 0.00 -> 14.8 mm, vias 0 -> 2
- net /Amplifiers/BCK: track 41.7 -> 56.1 mm, vias 2 -> 3
- net /ESP32-ATTINY/GPIO0: track 0.00 -> 13.2 mm
- net /Amplifiers/LRCK: track 43.4 -> 56.4 mm, vias 2 -> 3
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- added copper zone on F.Cu, net /ENC 3V3
- added copper zone on F.Cu, net Net-(U1-FB)
- added copper zone on F.Cu, net Net-(U1-LX1)
- added copper zone on F.Cu, net Net-(U1-LX2)
Other:
- board size 66.5 x 58.4 mm -> 82.2 x 58.4 mm
- board text added: "BAT GND"
- board text added: "CHG LED GND"
- board text added: "ENC GND"
- board text added: "NC"
- board text added: "NTC GND"
- board text added: "STATUS LED GND"
- board text added: "TAS2120 + TAS2320 1S Charger Boosted Class D © Tom Watson Audio 2026"
- board text added: "USB 5V +"
- board text added: "USB 5V GND"
- board text removed: "CHG +"
- board text removed: "CHG LED -"
- board text removed: "STATUS LED -"
- board text removed: "TAS2120 + TAS2320 1S Charger Boosted Class D Tom Watson Audio 2026"

Commit message: more
Parts:
- removed the G*** at (137.0, 78.2)
- removed R10: 0R*2, Resistor_SMD:R_0805_2012Metric_Pad1.20x1.40mm_HandSolder
- removed R11: 0R*3, Resistor_SMD:R_0805_2012Metric_Pad1.20x1.40mm_HandSolder
- removed TP1: TestPoint, TestPoint:TestPoint_Pad_D2.0mm
- added C32: 10uF, Capacitor_SMD:C_0805_2012Metric_Pad1.18x1.45mm_HandSolder, F.Cu at (160.3, 99.3)
- added J6: UPDI, Connector_PinHeader_2.54mm:PinHeader_1x03_P2.54mm_Vertical, F.Cu at (125.9, 83.0)
- added Q2: MMBT3904, Package_TO_SOT_SMD:SOT-23, F.Cu at (157.8, 104.0)
- added Q3: MMBT3904, Package_TO_SOT_SMD:SOT-23, F.Cu at (157.8, 108.5)
- added Q4: MMBT3904, Package_TO_SOT_SMD:SOT-23, F.Cu at (157.8, 118.0)
- added Q5: MMBT3906, Package_TO_SOT_SMD:SOT-23, F.Cu at (155.1, 86.0)
- added R22: 100K, Resistor_SMD:R_0805_2012Metric_Pad1.20x1.40mm_HandSolder, F.Cu at (145.9, 101.7)
- added R23: 100K, Resistor_SMD:R_0805_2012Metric_Pad1.20x1.40mm_HandSolder, F.Cu at (145.9, 88.4)
- added R24: 24K, Resistor_SMD:R_0805_2012Metric_Pad1.20x1.40mm_HandSolder, F.Cu at (145.8, 107.8)
- added R25: 24K, Resistor_SMD:R_0805_2012Metric_Pad1.20x1.40mm_HandSolder, F.Cu at (145.9, 93.0)
- added R26: 22K, Resistor_SMD:R_0805_2012Metric_Pad1.20x1.40mm_HandSolder, F.Cu at (153.9, 103.0)
- added R27: 100K, Resistor_SMD:R_0805_2012Metric_Pad1.20x1.40mm_HandSolder, F.Cu at (153.9, 105.1)
- added R28: 22K, Resistor_SMD:R_0805_2012Metric_Pad1.20x1.40mm_HandSolder, F.Cu at (153.9, 107.6)
- added R29: 100K, Resistor_SMD:R_0805_2012Metric_Pad1.20x1.40mm_HandSolder, F.Cu at (153.9, 109.5)
- added R30: 22K, Resistor_SMD:R_0805_2012Metric_Pad1.20x1.40mm_HandSolder, F.Cu at (153.9, 117.0)
- added R31: 100K, Resistor_SMD:R_0805_2012Metric_Pad1.20x1.40mm_HandSolder, F.Cu at (153.9, 119.0)
- added R32: 10K, Resistor_SMD:R_0805_2012Metric_Pad1.20x1.40mm_HandSolder, F.Cu at (160.8, 119.0)
- added R33: 4K7, Resistor_SMD:R_0805_2012Metric_Pad1.20x1.40mm_HandSolder, F.Cu at (187.0, 110.5)
- added R34: 1K, Resistor_SMD:R_0805_2012Metric_Pad1.20x1.40mm_HandSolder, F.Cu at (189.4, 102.7)
- added R35: 22K, Resistor_SMD:R_0805_2012Metric_Pad1.20x1.40mm_HandSolder, F.Cu at (153.0, 83.1)
- added R36: 100K, Resistor_SMD:R_0805_2012Metric_Pad1.20x1.40mm_HandSolder, F.Cu at (152.1, 86.0)
- C13, C14, C15, C16, C17, C18, C19, C20: footprint Capacitor_SMD:C_1206_3216Metric_Pad1.33x1.80mm_HandSolder -> Capacitor_SMD:C_0201_0603Metric
- C2: footprint Capacitor_SMD:C_0805_2012Metric_Pad1.18x1.45mm_HandSolder -> Capacitor_SMD:C_1206_3216Metric_Pad1.33x1.80mm_HandSolder
- C21, C22, C23, C24: footprint Capacitor_SMD:C_0805_2012Metric_Pad1.18x1.45mm_HandSolder -> Capacitor_SMD:C_0201_0603Metric
- C26, C27: value 1uF -> 4.7uF; footprint Capacitor_SMD:C_1206_3216Metric_Pad1.33x1.80mm_HandSolder -> Capacitor_SMD:C_0805_2012Metric_Pad1.18x1.45mm_HandSolder
- L1, L2: footprint Inductor_SMD:L_1008_2520Metric_Pad1.43x2.20mm_HandSolder -> Inductor_SMD:L_Vishay_IHLP-1212
- R17: value 240R -> 300R
- R18: value 13K7 -> 13K
- moved R16 99.3 mm to (178.1, 84.7), turned to 180 degrees
- moved R15 61.6 mm to (160.8, 109.5), turned to 90 degrees
- moved R14 60.5 mm to (160.8, 105.0), turned to 90 degrees
- moved R13 56.9 mm to (160.4, 94.6), turned to 90 degrees
- moved Q1 36.8 mm to (178.2, 87.8)
- moved U4 21.4 mm to (144.8, 119.7)
- moved C5 21.4 mm to (141.3, 118.7)
- moved C6 21.3 mm to (148.3, 118.7)
- moved C8 14.8 mm to (155.7, 98.0)
- moved U5 14.6 mm to (155.6, 94.0)
- moved C29 12.3 mm to (125.9, 99.7), turned to 90 degrees
- moved FB2 10.3 mm to (129.1, 98.7)
- moved C14 9.54 mm to (137.7, 106.2)
- moved C20 8.74 mm to (137.7, 101.2), turned to 90 degrees
- moved C16 8.50 mm to (141.7, 109.2)
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Connections:
- C2 pad 1: /ENC 3V3 -> /ESP3V3
- C22 pad 1: /Amplifiers/VDD1V8 -> /ESP3V3
- C24 pad 1: /Amplifiers/VDD1V8 -> /ESP3V3
- C25 pad 1: /CHGPOWER/BQ-SYS -> /BQ-SYS
- C3 pad 1: /ENC 3V3 -> /ESP3V3
- C7 pad 1: /ENC 3V3 -> /ESP3V3
- C8 pad 1: /Amplifiers/SYS -> /BQ-SYS
- IC1 pad 1: /CHGPOWER/BQ-SYS -> /BQ-SYS
- IC1 pad 3: Net-(IC1-STAT2) -> /CHGPOWER/STAT2_N
- IC2 pad 12: /Amplifiers/SDOUT -> /Amplifiers/AMP2320_SDZ
- IC2 pad 13: unconnected-(IC2-IO14-Pad13) -> /ESP32-ATTINY/SHUTDOWN_ACK
- IC2 pad 2: /ENC 3V3 -> /ESP3V3
- IC2 pad 37: /STATUS LED + -> Net-(IC2-IO23)
- IC2 pad 8: /ESP32-ATTINY/ALERT -> /ALERT_N
- IC2 pad 9: unconnected-(IC2-IO33-Pad9) -> /AMP2120_SDZ
- IC5 pad 4: /ENC 3V3 -> /ESP3V3
- IC5 pad 7: Net-(IC5-A0) -> GND
- IC5 pad 8: /CHGPOWER/ALERT -> /ALERT_N
- J2 pad 1: /ENC 3V3 -> /ESP3V3
- J3 pad 1: /LEFT - -> /LEFT +
- J3 pad 2: /LEFT + -> /LEFT -
- J4 pad 3: /ENC 3V3 -> /ESP3V3
- Q1 pad 2: /CHGPOWER/BQ-SYS -> /BQ-SYS
- R1 pad 1: /ENC 3V3 -> /ESP3V3
- R12 pad 1: /ENC 3V3 -> /ESP3V3
- R13 pad 1: /Amplifiers/SYS -> /BQ-SYS
- R14 pad 1: /ENC 3V3 -> /ESP3V3
- R15 pad 1: /ENC 3V3 -> /ESP3V3
- R16 pad 2: /CHGPOWER/BQ-SYS -> /BQ-SYS
- R19 pad 1: Net-(IC1-STAT2) -> Net-(Q5-C)
- R2 pad 1: /ENC 3V3 -> /ESP3V3
- R7 pad 1: /ENC 3V3 -> /ESP3V3
- R8 pad 1: /ENC 3V3 -> /ESP3V3
- U1 pad 1: /ENC 3V3 -> /ESP3V3
- U2 pad 16: unconnected-(U2-HW_SEL1-Pad16) -> GND
- U2 pad 2: unconnected-(U2-HW_SEL4_AD1-Pad2) -> /Amplifiers/ADDR2320
- U2 pad 22: unconnected-(U2-VSNSP-Pad22) -> GND
- U2 pad 23: unconnected-(U2-VSNSN-Pad23) -> GND
- U2 pad 5: /Amplifiers/VDD1V8 -> /ESP3V3
- U2 pad 7: unconnected-(U2-SD_N-Pad7) -> /Amplifiers/AMP2320_SDZ
- U3 pad 16: unconnected-(U3-HW_SEL1-Pad16) -> GND
- U3 pad 2: unconnected-(U3-HW_SEL4_AD1-Pad2) -> /Amplifiers/ADDR2120
- U3 pad 22: unconnected-(U3-VSNSP-Pad22) -> GND
- U3 pad 23: unconnected-(U3-VSNSN-Pad23) -> GND
- U3 pad 5: /Amplifiers/VDD1V8 -> /ESP3V3
- U3 pad 7: unconnected-(U3-SD_N-Pad7) -> /AMP2120_SDZ
- U5 pad 1: /Amplifiers/SYS -> /BQ-SYS
- U5 pad 4: /ESP32-ATTINY/PLAY_PAUSE -> /ESP32-ATTINY/PLAY_DRIVE
- U5 pad 5: /ESP32-ATTINY/POWER_OFF_REQ -> /ESP32-ATTINY/OFF_REQ_DRIVE
- U5 pad 7: Net-(U5-PA3) -> /ESP32-ATTINY/ACK_N
Routing:
- net /ESP3V3: track 0.00 -> 183.9 mm, vias 0 -> 10
- net /ENC 3V3: track 115.8 -> 0.00 mm, vias 5 -> 0
- net /ALERT_N: track 0.00 -> 47.4 mm, vias 0 -> 3
- net GND: track 0.00 -> 44.7 mm, vias 107 -> 125
- net /Amplifiers/SCL: track 114.8 -> 72.1 mm
- net /Amplifiers/AMP2320_SDZ: track 0.00 -> 41.5 mm, vias 0 -> 2
- net /BQ-SYS: track 0.00 -> 40.4 mm, vias 0 -> 2
- net /CHGPOWER/POWER-ON-MOSFET: track 0.00 -> 34.4 mm, vias 0 -> 2
- net /AMP2120_SDZ: track 0.00 -> 34.2 mm, vias 0 -> 2
- net /Amplifiers/SDA: track 110.1 -> 78.5 mm
- net /ESP32-ATTINY/ACK_N: track 0.00 -> 29.9 mm, vias 0 -> 2
- net /Amplifiers/PVDD: track 1.87 -> 29.6 mm
- net /USB5V +: track 24.5 -> 0.00 mm, vias 2 -> 0
- net /Amplifiers/SYS: track 28.7 -> 50.6 mm, vias 2 -> 6
- net /Amplifiers/VDD1V8: track 57.2 -> 37.2 mm, vias 3 -> 2
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- added copper zone on F.Cu, net /BQ-SYS
- added copper zone on F.Cu, net /ESP3V3
- added copper zone on F.Cu, net Net-(U3-SW)
- removed copper zone on F.Cu, net /Amplifiers/PVDD
- removed copper zone on F.Cu, net /ENC 3V3
- removed copper zone on F.Cu, net Net-(U1-FB)
Other:
- board size 82.2 x 58.4 mm -> 82.9 x 58.4 mm
- board text added: "1 - CHG LED GND 2 - CHG LED + 3 - NTC GND 4 - NTC 5 - USB 5V GND 6 - USB 5V + 7 - BAT GND 8 - BAT + 9 - USB CC 1"
- board text added: "1 2 3 4 5 6 7 8"
- board text added: "10 - USB CC 2 11 - NC 12 - STATUS LED GND 13 - STATUS LED + 14 - ENC GND 15 - ENC A 16 - ENC B 17 - ENC BTN 18 - ENC 3V3"
- board text added: "11 12 13 14 15 16 17 18"
- board text added: "9 10"
- board text added: "G P +"
