File: BoostedClassD/BoostedClassD.kicad_sch (KiCad schematic)
At the start: 3 parts, among them J1 SYSTEM CONNECTOR 1, J2 SYSTEM CONNECTOR 2, Q1 DMG3415U

Commit message: m0re
Parts:
- removed Q1: DMG3415U, Package_TO_SOT_SMD:SOT-23, symbol Transistor_FET:2N7002
- added H1, H2, H3, H4: (no value), MountingHole:MountingHole_4.3mm_M4, symbol Mechanical:MountingHole
- added J3: SPK OUT, Connector_JST:JST_XH_B4B-XH-A_1x04_P2.50mm_Vertical, symbol Connector:Conn_01x04_Socket
Connections:
- net GND: now also J1.6 (Pin_6)
- net LEFT +: now also J3.1 (Pin_1); no longer J1.5 (Pin_5)
- net LEFT -: now also J3.2 (Pin_2); no longer J1.6 (Pin_6)
- net RIGHT +: now also J3.3 (Pin_3); no longer J1.7 (Pin_7)
- net RIGHT -: now also J3.4 (Pin_4); no longer J1.8 (Pin_8)
- net NC: no longer names the net of J2.8 (Pin_8)
- new net NTC +: J1.5 (Pin_5)
- new net STATUS LED +: J1.7 (Pin_7)
- new net STATUS LED -: J1.8 (Pin_8)
Other:
- sheet ESP32 renamed ESP32-ATTINY
- sheet Amplifiers ports: added LEFT +, LEFT -, RIGHT +, RIGHT -, SCL, SDA, SDOUT; removed none
- sheet CHGPOWER ports: added ALERT, NTC +, SCL, SDA, STAT1, STAT2; removed none
- sheet ESP32-ATTINY ports: added ALERT, ENC A, ENC B, ENC BTN, SCL, SDA, SDOUT, STAT1, STAT2, STATUS LED, SYS; removed none

Commit message: loads
Connections:
- net CHG LED - is gone; now on net GND: J2.7 (Pin_7)
- net STATUS LED - is gone; now on net GND: J1.8 (Pin_8)
- net ENC A: now also J2.4 (Pin_4); no longer J2.3 (Pin_3)
- net ENC B: now also J2.3 (Pin_3); no longer J2.4 (Pin_4)
- net GND: now also J2.8 (Pin_8)
- net LEFT +: now also J3.2 (Pin_2); no longer J3.1 (Pin_1)
- net LEFT -: now also J3.1 (Pin_1); no longer J3.2 (Pin_2)
- net RIGHT +: now also J3.4 (Pin_4); no longer J3.3 (Pin_3)
- net RIGHT -: now also J3.3 (Pin_3); no longer J3.4 (Pin_4)
Other:
- sheet CHGPOWER ports: added CHG LED +, POWER-ON-MOSFET; removed STAT1, STAT2
- sheet ESP32-ATTINY ports: added POWER-ON-MOSFET; removed STAT1, STAT2

Commit message: more
Changed lines of the file:
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@@
+	(wire
+		(pts
+			(xy 97.79 43.18) (xy 118.745 43.18)
+		)
+		(stroke
+			(width 0)
+			(type default)
+		)
+	)
 	(wire
 		(pts
@@
 	(wire
 		(pts
-			(xy 119.38 43.18) (xy 118.745 43.18)
-		)
-		(stroke
-			(width 0)
-			(type default)
-		)
-	)
-	(wire
-		(pts
 			(xy 170.18 38.1) (xy 207.01 38.1)
 		)
@@
 		(pts
 			(xy 170.18 58.42) (xy 181.61 58.42)
-		)
-		(stroke
-			(width 0)
-			(type default)
-		)
-	)
-	(wire
-		(pts
-			(xy 118.745 43.18) (xy 97.79 43.18)
 		)
 		(stroke
@@
 		)
 		(stroke
+			(width 0)
+			(type default)
+		)
+	)
+	(wire
+		(pts
+			(xy 118.745 43.18) (xy 119.38 43.18)
+		)
+		(stroke

Commit message: more
Parts:
- added F1, F2: 3A, Fuse:Fuse_1206_3216Metric_Pad1.42x1.75mm_HandSolder, symbol Device:Fuse_Small
- added J5: CC, Connector_JST:JST_XH_B2B-XH-A_1x02_P2.50mm_Vertical, symbol Connector:Conn_01x02_Socket
- added R20, R21: 5K1, Resistor_SMD:R_0805_2012Metric_Pad1.20x1.40mm_HandSolder, symbol Device:R
Connections:
- net BAT +: now also F1.1; no longer J1.1 (Pin_1)
- net CHG LED +: now also J1.7 (Pin_7); no longer J2.6 (Pin_6)
- net GND: now also R20.1, R21.1; no longer J2.8 (Pin_8)
- net STATUS LED +: now also J2.6 (Pin_6); no longer J1.7 (Pin_7)
- net CHG +: no longer names the net of J1.3 (Pin_3)
- net CHG +: now also F2.2
- new net: J5.1 (Pin_1), R20.2
- new net: J5.2 (Pin_2), R21.2
- new net: F1.2, J1.1 (Pin_1)
- new net USB5V +: F2.1

Commit message: more
Connections:
- net LEFT +: now also J3.1 (Pin_1); no longer J3.2 (Pin_2)
- net LEFT -: now also J3.2 (Pin_2); no longer J3.1 (Pin_1)
- net ENC 3V3 renamed ESP3V3
- no-connect marks 0 -> 1
Other:
- sheet Amplifiers ports: added AMP2120_SDZ, AMP2320_SDZ, ESP3V3; removed SDOUT
- sheet CHGPOWER ports: added BQ-SYS; removed none
- sheet ESP32-ATTINY ports: added AMP2120_SDZ, AMP2320_SDZ, BQ-SYS; removed SDOUT, SYS
