File: BoostedClassD/CHGPOWER.kicad_sch (KiCad schematic)
At the start: 7 parts, among them IC1 BQ25185, U1 TPS631000

Commit message: m0re
Parts:
- added C25: 10uF, Capacitor_SMD:C_1206_3216Metric_Pad1.33x1.80mm_HandSolder, symbol Device:C
- added C26, C27: 1uF, Capacitor_SMD:C_1206_3216Metric_Pad1.33x1.80mm_HandSolder, symbol Device:C
- added C7: 100nF, Capacitor_SMD:C_1206_3216Metric_Pad1.33x1.80mm_HandSolder, symbol Device:C
- added IC5: INA236, Custom:INA236BIDDFR, symbol Custom:INA236BIDDFR
- added R10: 0R*2, Resistor_SMD:R_0805_2012Metric_Pad1.20x1.40mm_HandSolder, symbol Device:R
- added R11: 0R*3, Resistor_SMD:R_0805_2012Metric_Pad1.20x1.40mm_HandSolder, symbol Device:R
- added R9: 0R02, Custom:Untitled_4, symbol Device:R_Shunt
Connections:
- net BAT +: now also R9.1; no longer IC1.2 (BAT)
- net CHG +: now also C26.1
- net ESP3V3: now also C7.1, IC5.4 (VS)
- net GND: now also C25.2, C26.2, C27.2, C7.2, IC5.3 (GND), R11.2
- net SYS: now also C25.1
- net STAT2: now reaches IC1.3 (STAT2)
- net NTC +: now reaches IC1.6 (TS/MR)
- net STAT1: now reaches IC1.9 (STAT1)
- new net: IC5.7 (A0), R10.1, R11.1
- new net: C27.1, IC1.2 (BAT), R9.4
- new net 3.3V: R10.2
- new net ALERT: IC5.8 (ALERT)
- new net IN+: IC5.1 (IN+), R9.3
- new net IN-: IC5.2 (IN-), R9.2
- new net SCL: IC5.5 (SCL)
- new net SDA: IC5.6 (SDA)

Commit message: loads
Parts:
- added Q1: DMG3415U, Package_TO_SOT_SMD:SOT-23, symbol Transistor_FET:2N7002
- added R16: 100K, Resistor_SMD:R_0805_2012Metric_Pad1.20x1.40mm_HandSolder, symbol Device:R
- added R17: 240R, Resistor_SMD:R_0805_2012Metric_Pad1.20x1.40mm_HandSolder, symbol Device:R
- added R18: 13K7, Resistor_SMD:R_0805_2012Metric_Pad1.20x1.40mm_HandSolder, symbol Device:R
- added R19: 2K2, Resistor_SMD:R_0805_2012Metric_Pad1.20x1.40mm_HandSolder, symbol Device:R
Connections:
- net GND: now also R17.1, R18.1
- net SYS: now also Q1.3 (D); no longer C25.1, IC1.1 (SYS)
- net at IC1.7 (ILIM/VSET): now also R18.2
- net at IC1.8 (ISET): now also R17.2
- net STAT1: no longer names the net of IC1.9 (STAT1)
- net STAT2: no longer names the net of IC1.3 (STAT2)
- net STAT2: now also R19.1
- new net BQ-SYS: C25.1, IC1.1 (SYS), Q1.2 (S), R16.2
- new net CHG LED +: R19.2
- new net POWER-ON-MOSFET: Q1.1 (G), R16.1
Other:
- moved on the sheet: C26

Commit message: more
Parts:
- removed R10: 0R*2, Resistor_SMD:R_0805_2012Metric_Pad1.20x1.40mm_HandSolder, symbol Device:R
- removed R11: 0R*3, Resistor_SMD:R_0805_2012Metric_Pad1.20x1.40mm_HandSolder, symbol Device:R
- added Q5: MMBT3906, Package_TO_SOT_SMD:SOT-23, symbol Transistor_BJT:Q_PNP_BEC
- added R35: 22K, Resistor_SMD:R_0805_2012Metric_Pad1.20x1.40mm_HandSolder, symbol Device:R
- added R36: 100K, Resistor_SMD:R_0805_2012Metric_Pad1.20x1.40mm_HandSolder, symbol Device:R
- C2: footprint Capacitor_SMD:C_0805_2012Metric_Pad1.18x1.45mm_HandSolder -> Capacitor_SMD:C_1206_3216Metric_Pad1.33x1.80mm_HandSolder
- C26, C27: value 1uF -> 4.7uF; footprint Capacitor_SMD:C_1206_3216Metric_Pad1.33x1.80mm_HandSolder -> Capacitor_SMD:C_0805_2012Metric_Pad1.18x1.45mm_HandSolder
- IC1: symbol Custom:BQ25185DLHR -> BoostedClassD:BQ25185
- L1: footprint Inductor_SMD:L_1008_2520Metric_Pad1.43x2.20mm_HandSolder -> Inductor_SMD:L_Vishay_IHLP-1212
- R17: value 240R -> 300R
- R18: value 13K7 -> 13K
- R9: symbol Device:R_Shunt -> BoostedClassD:R_Shunt_Existing
- U1: symbol Custom:TPS631000DRLR -> BoostedClassD:TPS631000
Connections:
- net BQ-SYS: now also Q5.2 (E), R36.1
- net GND: now also IC5.7 (A0)
- net at R19.1: now also Q5.3 (C); no longer IC1.3 (STAT2)
- new net: Q5.1 (B), R35.2, R36.2
- new net STAT2_N: IC1.3 (STAT2), R35.1
- no-connect marks 0 -> 1
Other:
- note added: "BQ25185 settings retained: R17 300R => 1 A charge; R18 13k => 1.1 A input limit / 4.2 V. 7 Ah single Li-ion pouch: six-hour safety timer can prevent a full charge from deep discharge. System load and thermal regulation further reduce charging rate. Charger choice remains a design limitation. C26/C27: require at least 1 uF effective capacitance. Confirm DC-bias derating. Use protected cell/pack an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"
- note added: "L1: verify exact 1 uH part, Isat above 3.35 A with margin and adequate RMS rating. R9: verify exact 20 mOhm four-terminal shunt and footprint/Kelvin pad mapping. Neither unspecified physical part has been substituted."
- note added: "SYS is the Q1-switched supply; BQ-SYS remains alive for the ATtiny."
- moved on the sheet: R19
