File: BoostedClassD/ESP32.kicad_sch (KiCad schematic)
At the start: 10 parts, among them IC2 ESP32-WROOM-32UE-N8R2, IC3 RESET, IC4 BOOT

Commit message: m0re
Parts:
- added C8: 100nF, Capacitor_SMD:C_1206_3216Metric_Pad1.33x1.80mm_HandSolder, symbol Device:C
- added Q1: DMG3415U, Package_TO_SOT_SMD:SOT-23, symbol Transistor_FET:2N7002
- added R12, R8: 4K7, Resistor_SMD:R_0805_2012Metric_Pad1.20x1.40mm_HandSolder, symbol Device:R
- added R13: 47K, Resistor_SMD:R_0805_2012Metric_Pad1.20x1.40mm_HandSolder, symbol Device:R
- added R14, R15: 10K, Resistor_SMD:R_0805_2012Metric_Pad1.20x1.40mm_HandSolder, symbol Device:R
- added TP1: TestPoint, TestPoint:TestPoint_Pad_D2.0mm, symbol Connector:TestPoint
- added U5: ATtiny412, Package_SO:SOIC-8_3.9x4.9mm_P1.27mm, symbol MCU_Microchip_ATtiny:ATtiny412-SS
Connections:
- net 3V3 is gone; now on net ESP3V3: R1.1, R2.1
- net ESP3V3: now also R12.1, R14.1, R15.1, R8.1
- net GND: now also C8.2, U5.8 (GND)
- net SCL: now also R8.2
- net SDA: now also R12.2
- net SDOUT: now reaches IC2.12 (IO27)
- net ENC A: now reaches IC2.30 (IO18)
- net ENC B: now reaches IC2.31 (IO19)
- net STATUS LED: now reaches IC2.37 (IO23)
- net STAT1: now reaches IC2.4 (SENSOR_VP)
- net STAT2: now reaches IC2.5 (SENSOR_VN)
- net PLAY_PAUSE: now reaches IC2.6 (IO34)
- net PLAY_PAUSE: now also R14.2, U5.4 (PA1)
- net POWER_OFF_REQ: now reaches IC2.7 (IO35)
- net POWER_OFF_REQ: now also R15.2, U5.5 (PA2)
- net ALERT: now reaches IC2.8 (IO32)
- new net: TP1.1, U5.7 (PA3)
- new net: Q1.1 (G), U5.3 (PA7)
- new net ENC BTN: R13.2, U5.2 (PA6)
- new net PROG: U5.6 (~{RESET}/PA0)
- new net SYS: C8.1, R13.1, U5.1 (VCC)
Other:
- moved on the sheet: C3, IC2, R1, R2, R3, R4, R5

Commit message: loads
Parts:
- removed Q1: DMG3415U, Package_TO_SOT_SMD:SOT-23, symbol Transistor_FET:2N7002
- added J4: PROG, Connector_PinHeader_2.54mm:PinHeader_1x04_P2.54mm_Vertical, symbol Connector:Conn_01x04_Socket
Connections:
- net ENC A: now also IC2.31 (IO19); no longer IC2.30 (IO18)
- net ENC B: now also IC2.30 (IO18); no longer IC2.31 (IO19)
- net ESP3V3: now also J4.3 (Pin_3)
- net GND: now also J4.4 (Pin_4)
- net RX: now also J4.1 (Pin_1)
- net TX: now also J4.2 (Pin_2)
- net POWER-ON-MOSFET: now reaches U5.3 (PA7)
- net STAT1: no longer names the net of IC2.4 (SENSOR_VP)
- net STAT2: no longer names the net of IC2.5 (SENSOR_VN)

Commit message: more
Parts:
- removed IC3: RESET, Custom:TS026650BK100SCRD, symbol Custom:TS02-66-50-BK-100-SCR-D
- removed IC4: BOOT, Custom:TS026650BK100SCRD, symbol Custom:TS02-66-50-BK-100-SCR-D
- added S1: BOOT, Custom:PTS810SJM250SMTRLFS, symbol Custom:PTS810SJM250SMTR_LFS
- added S2: EN, Custom:PTS810SJM250SMTRLFS, symbol Custom:PTS810SJM250SMTR_LFS
Connections:
- net EN: now also S2.1 (NO_1), S2.2 (NO_2)
- net GND: now also S1.3 (COM_1), S1.4 (COM_2), S2.3 (COM_1), S2.4 (COM_2)
- net GPIO0: now also S1.1 (NO_1), S1.2 (NO_2)

Commit message: more
Parts:
- removed TP1: TestPoint, TestPoint:TestPoint_Pad_D2.0mm, symbol Connector:TestPoint
- added C32: 10uF, Capacitor_SMD:C_0805_2012Metric_Pad1.18x1.45mm_HandSolder, symbol Device:C
- added J6: UPDI, Connector_PinHeader_2.54mm:PinHeader_1x03_P2.54mm_Vertical, symbol Connector_Generic:Conn_01x03
- added Q2, Q3, Q4: MMBT3904, Package_TO_SOT_SMD:SOT-23, symbol Transistor_BJT:Q_NPN_BEC
- added R26, R28, R30: 22K, Resistor_SMD:R_0805_2012Metric_Pad1.20x1.40mm_HandSolder, symbol Device:R
- added R27, R29, R31: 100K, Resistor_SMD:R_0805_2012Metric_Pad1.20x1.40mm_HandSolder, symbol Device:R
- added R32: 10K, Resistor_SMD:R_0805_2012Metric_Pad1.20x1.40mm_HandSolder, symbol Device:R
- added R33: 4K7, Resistor_SMD:R_0805_2012Metric_Pad1.20x1.40mm_HandSolder, symbol Device:R
- added R34: 1K, Resistor_SMD:R_0805_2012Metric_Pad1.20x1.40mm_HandSolder, symbol Device:R
Connections:
- net ALERT: now also R33.2
- net ESP3V3: now also R33.1
- net GND: now also C32.2, J6.3 (Pin_3), Q2.2 (E), Q3.2 (E), Q4.2 (E), R27.2, R29.2, R31.2
- net PLAY_PAUSE: now also Q2.3 (C); no longer U5.4 (PA1)
- net POWER_OFF_REQ: now also Q3.3 (C); no longer U5.5 (PA2)
- net PROG: now also J6.2 (Pin_2)
- net STATUS LED: now also R34.2; no longer IC2.37 (IO23)
- net ACK_N: now reaches U5.7 (PA3)
- net ACK_N: now also Q4.3 (C), R32.2
- net SHUTDOWN_ACK: now reaches IC2.13 (IO14)
- net SHUTDOWN_ACK: now also R30.1
- net AMP2120_SDZ: now reaches IC2.9 (IO33)
- net SDOUT renamed AMP2320_SDZ
- net SYS renamed BQ-SYS
- net BQ-SYS: now also J6.1 (Pin_1), R32.1
- new net: IC2.37 (IO23), R34.1
- new net: Q2.1 (B), R26.2, R27.1
- new net: Q4.1 (B), R30.2, R31.1
- new net: Q3.1 (B), R28.2, R29.1
- new net OFF_REQ_DRIVE: R28.1, U5.5 (PA2)
- new net PLAY_DRIVE: R26.1, U5.4 (PA1)
- no-connect marks 0 -> 16
Other:
- note added: "J6: 1 = target VREF (BQ-SYS), 2 = UPDI, 3 = GND. Use a voltage-compatible programmer; do not back-power this rail."
- note added: "POWER CONTROL (always-on ATtiny): PA1/PA2 HIGH assert active-LOW ESP requests. ESP GPIO14 HIGH asserts ACK_N LOW at ATtiny PA3. Pull GPIO14 LOW at boot. Tiny: latch Q1 ON, request shutdown, wait for ACK_N or bounded timeout, then release Q1. ESP: mute amplifiers / SDZ LOW, finish state writes, then assert ACK. Firmware changes required; transistor interfaces invert logic and prevent rail backfeed."
- moved on the sheet: C3, C4, C8, IC2, J4, R1, R12, R13, R14, R15, R2, R3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
