File: PCM1704/PCM1704.kicad_pcb (KiCad board)
At the start: 4 copper layers, 90 x 90 mm, 122 parts, among them IC1 LT3042, IC2 LT3042, J1 AUDIO OUT, J2 POWER, J5 I2S IN, U1 PCM1704, U10 LM337, U12 LM317, U2 PCM1704, U3 DF1704, U4 OPA1611, U5 OPA1611, U6 LT3094, U7 ATtiny1614, U8 OPA1612, U9 OPA1612

Commit message: more
Parts:
- added C30: 22uF, Capacitor_SMD:C_1206_3216Metric_Pad1.33x1.80mm_HandSolder, F.Cu at (165.9, 83.9)
- added HS1: Heatsink, Custom:Tiny heatsink, F.Cu at (183.3, 98.2)
- added HS2: Heatsink, Custom:Tiny heatsink, F.Cu at (166.7, 98.2)
- added J3: PROG, Connector_JST:JST_XH_B3B-XH-A_1x03_P2.50mm_Vertical, F.Cu at (150.7, 118.2)
- C20, C21: footprint Capacitor_SMD:C_0805_2012Metric_Pad1.18x1.45mm_HandSolder -> Capacitor_SMD:C_1206_3216Metric_Pad1.33x1.80mm_HandSolder
- R3, R4: value 110R -> 240R
- R56, R74: value 590R -> 1K3
- moved REF** 84.1 mm to (169.4, 138.7)
- moved C22 37.1 mm to (188.9, 67.0), turned to 90 degrees
- moved C19 30.2 mm to (181.0, 77.5), turned to -90 degrees
- moved C90 13.6 mm to (180.1, 88.5), turned to 0 degrees
- moved C71 8.90 mm to (183.0, 94.6), turned to 90 degrees
- moved C70 8.04 mm to (196.3, 89.9), turned to 0 degrees
- moved C20 5.78 mm to (193.6, 70.0)
- moved C69 5.31 mm to (195.2, 110.4)
- moved C24 5.22 mm to (184.2, 73.5)
- moved C27 5.18 mm to (186.6, 72.8)
- moved C72 5.18 mm to (195.4, 74.5)
- moved IC1 5.18 mm to (190.0, 72.4)
- moved R57 5.18 mm to (193.3, 74.5)
- moved R3 4.73 mm to (190.0, 110.2)
- moved R56 4.73 mm to (190.0, 112.3)
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Connections:
- J1 pad 1: /OUT_L -> /OUT_R
- J1 pad 3: /OUT_R -> /OUT_L
- R62 pad 2: /OUT_L -> /OUT_R
- R63 pad 2: /OUT_R -> /OUT_L
Routing:
- net /-15V: track 123.4 -> 96.3 mm
- net /+8V: track 86.2 -> 65.7 mm
- net /+15V: track 144.9 -> 129.5 mm
- net /PROG: track 0.00 -> 11.1 mm
- net /-8V: track 28.0 -> 18.3 mm
- net GND: track 17.1 -> 22.4 mm, vias 195 -> 357
- net /+5VDF: track 160.4 -> 165.0 mm
- net Net-(U8B--): track 2.90 -> 5.77 mm
- net /PRE_N_ADJ: track 23.7 -> 26.3 mm
- net Net-(U9A--): track 1.27 -> 3.63 mm
- net Net-(U8A--): track 2.72 -> 5.07 mm
- net /+5V: track 118.1 -> 120.1 mm
- net Net-(IC1-SET): track 4.10 -> 3.27 mm
- net /DF_RST: track 34.9 -> 34.2 mm
- net /-5V: track 110.9 -> 111.5 mm
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- added copper zone on B.Cu, net /+8V
Other:
- board text added: "- G +"
- board text added: "5V P G"
- board text added: "Dual Opamps: OPA1612 / OPA1656 / OPA1642 OPA2156 / LM4562 / OPA2134"
- board text added: "PCM1704/DF1704 I2S DAC © Tom Watson Audio 2026"
- board text added: "Single Opamps: OPA1611 / OPA1655 / OPA1641 OPA827 / OPA627 / OPA171"
- board text removed: "-15V G +15V"
- board text removed: "Dual PCM1704/DF1704 I2S DAC © Tom Watson Audio 2026"
