File: PCM1704/PCM1704.kicad_pcb (KiCad board)
At the start: 4 copper layers, 90 x 90 mm, 143 parts, among them IC1 LT3042, IC2 LT3042, J1 AUDIO OUT, J2 POWER, J3 PROG, J5 I2S IN, U1 PCM1704, U10 LM337, U11 74LVC1G17, U12 LM317, U13 74LVC125APW, U14 TPS7A2033, U2 PCM1704, U3 DF1704, U4 OPA1611, U5 OPA1611, U6 LT3094, U7 ATtiny1614, U8 OPA1612, U9 OPA1612

Commit message: more work
Routing:
- net Net-(U1-WCLK): track 48.7 -> 46.6 mm
- net /-5V: track 132.1 -> 131.1 mm
