File: PCM1704/PCM1704.kicad_sch (KiCad schematic)
At the start: 0 parts

Commit message: more
Parts:
- added C1, C10, C106, C11, C12, C2, C3, C4, C41, C46, C5, C6, C69, C7, C8, C83, C84, C85, C86, C87, C88, C9: 100nF, Capacitor_SMD:C_1206_3216Metric_Pad1.33x1.80mm_HandSolder, symbol Device:C
- added C100, C101, C102, C103, C104, C72, C73, C74, C97, C98, C99: 4.7uF, Capacitor_SMD:C_0805_2012Metric_Pad1.18x1.45mm_HandSolder, symbol Device:C
- added C105, C28: 10uF, Capacitor_SMD:C_1206_3216Metric_Pad1.33x1.80mm_HandSolder, symbol Device:C
- added C13, C14, C15, C16, C19, C22: 47uF, Capacitor_THT:CP_Radial_D5.0mm_P2.50mm, symbol Device:C_Polarized
- added C17, C18: 100uF, Capacitor_THT:CP_Radial_D5.0mm_P2.50mm, symbol Device:C_Polarized
- added C20, C21, C26, C27, C70, C89: 10uF, Capacitor_SMD:C_0805_2012Metric_Pad1.18x1.45mm_HandSolder, symbol Device:C
- added C23, C24, C25, C29: 22uF, Capacitor_SMD:C_1206_3216Metric_Pad1.33x1.80mm_HandSolder, symbol Device:C
- added C44, C45: 1000uF, Capacitor_THT:CP_Radial_D12.5mm_P5.00mm, symbol Device:C_Polarized
- added C71, C90: 1uF, Capacitor_SMD:C_1206_3216Metric_Pad1.33x1.80mm_HandSolder, symbol Device:C
- added C75, C76: 47pF, Capacitor_SMD:C_0603_1608Metric_Pad1.08x0.95mm_HandSolder, symbol Device:C
- added C77, C80: 18nF, Capacitor_SMD:C_0805_2012Metric_Pad1.18x1.45mm_HandSolder, symbol Device:C
- added C78, C81: 2.2nF, Capacitor_SMD:C_0805_2012Metric_Pad1.18x1.45mm_HandSolder, symbol Device:C
- added C79, C82: 3.3nF, Capacitor_SMD:C_0805_2012Metric_Pad1.18x1.45mm_HandSolder, symbol Device:C
- added D5, D6, D7, D8: 1N4007, Diode_THT:D_DO-41_SOD81_P10.16mm_Horizontal, symbol Diode:1N4007
- added H1, H2, H3, H4: MountingHole, MountingHole:MountingHole_4mm, symbol Mechanical:MountingHole
- added IC1, IC2: LT3042, Custom:LT3042, symbol PCM1704_Support:LT3042_DFN
- added J1: AUDIO OUT, Connector_JST:JST_XH_B3B-XH-A_1x03_P2.50mm_Vertical, symbol Connector:Conn_01x03_Socket
- added J2: POWER, Connector_JST:JST_XH_B3B-XH-A_1x03_P2.50mm_Vertical, symbol Connector:Conn_01x03_Socket
- added J5: I2S IN, Connector_JST:JST_XH_B6B-XH-A_1x06_P2.50mm_Vertical, symbol Connector:Conn_01x06_Socket
- added R28, R29, R30, R31, R79, R80, R81, R82: 22R, Resistor_SMD:R_0603_1608Metric_Pad0.98x0.95mm_HandSolder, symbol Device:R
- added R3, R4: 110R, Resistor_SMD:R_0805_2012Metric_Pad1.20x1.40mm_HandSolder, symbol Device:R
- added R56, R74: 590R, Resistor_SMD:R_0805_2012Metric_Pad1.20x1.40mm_HandSolder, symbol Device:R
- added R57, R58, R59: 49K9, Resistor_SMD:R_0805_2012Metric_Pad1.20x1.40mm_HandSolder, symbol Device:R
- added R60, R61: 2K37, Resistor_SMD:R_0805_2012Metric_Pad1.20x1.40mm_HandSolder, symbol Device:R
- added R62, R63: 100R, Resistor_SMD:R_0805_2012Metric_Pad1.20x1.40mm_HandSolder, symbol Device:R
- added R66, R67, R70, R71: 768R, Resistor_SMD:R_0805_2012Metric_Pad1.20x1.40mm_HandSolder, symbol Device:R
- added R68, R72: 523R, Resistor_SMD:R_0805_2012Metric_Pad1.20x1.40mm_HandSolder, symbol Device:R
- added R69, R73: 1K21, Resistor_SMD:R_0805_2012Metric_Pad1.20x1.40mm_HandSolder, symbol Device:R
- added R75, R76: 10k, Resistor_SMD:R_0805_2012Metric_Pad1.20x1.40mm_HandSolder, symbol Device:R
- added R77, R78: 47k, Resistor_SMD:R_0805_2012Metric_Pad1.20x1.40mm_HandSolder, symbol Device:R
- added U1, U2: PCM1704, Package_SO:SO-20_5.3x12.6mm_P1.27mm, symbol PCM1704_Support:PCM1704
- added U10: LM337, Package_TO_SOT_THT:TO-220-3_Vertical, symbol Regulator_Linear:LM337_TO220
- added U12: LM317, Package_TO_SOT_THT:TO-220-3_Vertical, symbol Regulator_Linear:LM317_TO-220
- added U3: DF1704, Package_SO:SSOP-28_5.3x10.2mm_P0.65mm, symbol PCM1704_Support:DF1704
- added U4, U5: OPA1611, Package_SO:SOIC-8_3.9x4.9mm_P1.27mm, symbol Custom:OPA1611
- added U6: LT3094, Package_DFN_QFN:DFN-12-1EP_3x3mm_P0.45mm_EP1.65x2.38mm, symbol PCM1704_Support:LT3094_DFN
- added U7: ATtiny1614, Package_SO:SOIC-14_3.9x8.7mm_P1.27mm, symbol MCU_Microchip_ATtiny:ATtiny1614-SS
- added U8, U9: OPA1612, Package_SO:SOIC-8_3.9x4.9mm_P1.27mm, symbol Amplifier_Operational:OPA1612AxD
Connections:
- new net: C76.1, R61.1, U1.14 (IOUT), U4.2 (-)
- new net: C76.2, R61.2, R66.1, U4.6
- new net: C77.1, R66.2, R67.1, R68.1
- new net: C78.1, R68.2, U8.6 (-)
- new net: R79.1, U3.26 (BCKO)
- new net: R79.2, U1.2 (BCLK), U2.2 (BCLK)
- new net: C75.1, R60.1, U2.14 (IOUT), U5.2 (-)
- new net: C75.2, R60.2, R70.1, U5.6
- new net: C72.1, IC1.7 (SET), R57.1
- new net: C78.2, R67.2, R69.1, U8.7
- new net: C81.2, R71.2, R73.1, U8.1
- new net: C81.1, R72.2, U8.2 (-)
- new net: R82.2, U1.1 (DATA)
- new net: R80.2, U1.7 (WCLK), U2.7 (WCLK)
- new net: R63.1, U9.1, U9.2 (-)
- new net: C82.1, R73.2, U9.3 (+)
- new net: C79.1, R69.2, U9.5 (+)
- new net: R62.1, U9.6 (-), U9.7
- new net: C74.1, R59.1, U6.8 (SET)
- new net: C73.1, IC2.7 (SET), R58.1
- new net: J5.3 (Pin_3), R29.1
- new net: J5.4 (Pin_4), R28.1
- new net: C80.1, R70.2, R71.1, R72.1
- new net: J5.1 (Pin_1), R31.1
- new net: J5.2 (Pin_2), R30.1
- new net: R81.2, U2.1 (DATA)
- new net: R81.1, U3.24 (DOL)
- new net: R82.1, U3.23 (DOR)
- new net: R80.1, U3.25 (WCKO)
- new net +15V: C1.1, C2.1, C3.1, C41.1, C44.1, C69.1, C86.1, D6.1 (K), J2.1 (Pin_1), U12.3 (VI), U4.7 (V+), U5.7 (V+), U8.8 (V+), U9.8 (V+)
- new net +5V: C101.1, C102.1, C20.1, C4.1, C5.1, C6.1, C7.1, C97.1, C98.1, IC1.10 (OUT), IC1.9 (OUTS), U1.11 (+VCC), U1.6 (+VDD), U2.11 (+VCC), U2.6 (+VDD)
- new net +5VDF: C105.1, C106.1, C12.1, C21.1, IC2.10 (OUT), IC2.9 (OUTS), R76.1, U3.10 (MODE), U3.22 (VDD), U7.1 (VCC)
- new net +8V: C22.1, C23.1, C24.1, C26.2, C27.2, C71.1, D6.2 (A), D7.1 (K), IC1.1 (IN_1), IC1.2 (IN_2), IC1.3 (EN/UV), IC1.6 (PGFB), IC2.1 (IN_1), IC2.2 (IN_2), IC2.3 (EN/UV), IC2.6 (PGFB), R3.1, U12.2 (VO)
- new net -15V: C45.2, C46.2, C83.1, C84.1, C85.1, C87.1, C88.1, D5.2 (A), J2.3 (Pin_3), U10.2 (VI), U4.4 (V-), U5.4 (V-), U8.4 (V-), U9.4 (V-)
- new net -5V: C10.1, C100.1, C103.1, C104.1, C11.1, C13.2, C14.2, C15.2, C16.2, C29.2, C8.1, C9.1, C99.1, U1.20 (-VCC), U1.4 (-VDD), U2.20 (-VCC), U2.4 (-VDD), U6.10 (OUTS), U6.11 (OUT), U6.12 (OUT)
- new net -8V: C19.2, C25.1, C28.2, C90.1, D5.1 (K), D8.2 (A), R4.1, U10.3 (VO), U6.1 (IN), U6.13 (IN_EP), U6.2 (IN), U6.3 (EN/UV), U6.5 (PGFB)
- new net BCKIN: R30.2, U3.2 (BCKIN)
- new net DAC1_BPO: C17.1, U1.12 (BPO_DC)
- new net DAC1_REF: C15.1, U1.19 (REF_DC)
- new net DAC1_SERVO: C16.1, U1.17 (SERVO_DC)
- new net DAC2_BPO: C18.1, U2.12 (BPO_DC)
- new net DAC2_REF: C13.1, U2.19 (REF_DC)
- new net DAC2_SERVO: C14.1, U2.17 (SERVO_DC)
- new net DATAIN: R29.2, U3.1 (DIN)
- new net DF_RST: R75.1, U3.14 (RST), U7.2 (PA4)
- new net GND: C1.2, C10.2, C100.2, C101.2, C102.2, C103.2, C104.2, C105.2, C106.2, C11.2, C12.2, C17.2, C18.2, C19.1, C2.2, C20.2, C21.2, C22.2, C23.2, C24.2, C25.2, C26.1, C27.1, C28.1, C29.1, C3.2, C4.2, C41.2, C44.2, C45.1, C46.1, C5.2, C6.2, C69.2, C7.2, C70.2, C71.2, C72.2, C73.2, C74.2, C77.2, C79.2, C8.2, C80.2, C82.2, C83.2, C84.2, C85.2, C86.2, C87.2, C88.2, C89.2, C9.2, C90.2, C97.2, C98.2, C99.2, IC1.11 (GND_2), IC1.5 (ILIM), IC1.8 (GND_1), IC2.11 (GND_2), IC2.5 (ILIM), IC2.8 (GND_1), J1.2 (Pin_2), J2.2 (Pin_2), J5.5 (Pin_5), J5.6 (Pin_6), R56.2, R57.2, R58.2, R59.2, R74.2, R75.2, R77.2, R78.2, U1.10 (INVERT), U1.15 (AGND), U1.16 (AGND), U1.5 (DGND), U1.9 (20BIT), U2.10 (INVERT), U2.15 (AGND), U2.16 (AGND), U2.5 (DGND), U2.9 (20BIT), U3.15 (MUTE), U3.16 (DEM), U3.17 (SF0), U3.18 (SF1), U3.19 (OW0), U3.20 (OW1), U3.27 (SRO), U3.3 (I2S), U3.4 (IW0), U3.5 (IW1), U3.8 (VSS), U4.3 (+), U5.3 (+), U6.6 (ILIM), U6.9 (GND), U7.14 (GND), U8.3 (+), U8.5 (+)
- new net LRCKIN: R28.2, U3.28 (LRCIN)
- new net MC: R77.1, U3.12 (MC/LRIP), U7.12 (PA2)
- new net MD: R78.1, U3.11 (MD/CKO), U7.11 (PA1)
- new net ML: R76.2, U3.13 (ML/RESV), U7.13 (PA3)
- new net OUT_L: J1.1 (Pin_1), R62.2
- new net OUT_R: J1.3 (Pin_3), R63.2
- new net PRE_N_ADJ: C89.1, D8.1 (K), R4.2, R74.1, U10.1 (ADJ)
- new net PRE_P_ADJ: C70.1, D7.2 (A), R3.2, R56.1, U12.1 (ADJ)
- new net PROG: U7.10 (~{RESET}/PA0)
- new net SCKIN: R31.2, U3.6 (XTI)
- no-connect marks 0 -> 15
Other:
- note added: "2-pole MFB: unity inverting, Q = 0.9994"
- note added: "39.86 kHz RC pole + unity buffer"
- note added: "47p: initial compensation; verify settling on PCB"
- note added: "ANALOGUE OP-AMP SUPPLIES: +/-15 V"
- note added: "C107: LM337 stability capacitor. Positive terminal to GND. Place at U10 OUT."
- note added: "C20/C21: >=4.7uF EFFECTIVE at +5V. C29: >=10uF EFFECTIVE at -5V. Verify selected ceramic DC-bias curves, ESR and package before ordering. 49k9 x 100uA = +/-4.99V. CSET=4.7uF: tau~235ms; fast start disabled. EN and PGFB to IN; ILIM to GND are intentional. PG and VIOC unused."
- note added: "DAC LOCAL SUPPLY BULK: pair each 4u7 with its existing 100n at the named supply pin."
- note added: "DAC1: reference / servo / bipolar-zero decoupling"
- note added: "DAC2: reference / servo / bipolar-zero decoupling"
- note added: "DESIGN NOTES - ANALOGUE OUTPUT ONLY Nominal 3rd-order Butterworth: ~39.9 kHz; ~2.01 V RMS unloaded at 1 kHz. R60/R61 and filter resistors: thin-film 0.1%. Filter capacitors: C0G 1%, >=25 V. DC coupled: measure output offset before connecting the LM4562/PGA2310 preamp. Initial I/V compensation assumes unknown DAC/PCB capacitance; bench verification required. DAC support added separately. Hardware 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"
- note added: "External supply via J2"
- note added: "L | I/V: 2.011 V RMS nominal"
- note added: "PREREGULATORS: 110R / 590R => approximately +/-8V. Divider current ~11.4mA maintains regulation with downstream rails off. D1/D3: OUT-IN discharge protection; D2/D4: ADJ capacitor protection. TO-220 tabs differ: U12 = OUT (+8V), U10 = IN (-15V). Do not bolt bare tabs to the same heatsink or grounded metal."
- note added: "Pins 3/4/5 = GND. Hardware format inputs only; MODE=HIGH: format is programmed by MCU."
- note added: "Place each 100n at its IC supply pin; use local GND vias. Existing bulk rail capacitors retained."
- note added: "R | I/V: 2.011 V RMS nominal"
- note added: "R79-R82: 0R source links at U3 pins 26,25,24,23. Tune to 22-33R only after checking BCLK/data timing at both DACs."
- note added: "SOFTWARE MODE (MODE=+5VDF): unused strap inputs tied to GND. PA4 -> DF_RST: 10k pull-down holds reset until MCU release. Wait for stable rails and valid MCLK; release RST; wait >=1024 MCLK cycles. Then program 24-bit input/output, I2S, sharp roll-off; de-emphasis off. Mute during initialisation and clock/sample-rate changes. A fixed startup delay is not a replacement for rail/clock fault detectio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"
- note added: "U1 pin 11"
- note added: "U1 pin 20"
- note added: "U1 pin 4"
- note added: "U1 pin 6"
- note added: "U2 pin 11"
- note added: "U2 pin 20"
- note added: "U2 pin 4"
- note added: "U2 pin 6"
- note added: "U3 bulk"
- note added: "U4 local bypass"
- note added: "U5 local bypass"
- note added: "U6 exposed pad 13 = IN (-8V), never GND."

Commit message: more
Parts:
- added C30: 22uF, Capacitor_SMD:C_1206_3216Metric_Pad1.33x1.80mm_HandSolder, symbol Device:C
- added HS1, HS2: Heatsink, Custom:Tiny heatsink, symbol Mechanical:Heatsink
- added J3: PROG, Connector_JST:JST_XH_B3B-XH-A_1x03_P2.50mm_Vertical, symbol Connector:Conn_01x03_Socket
- C1, C10, C100, C101, C102, C103, C104, C105, C106, C11, C12, C13, C14, C15, C16, C17, C18, C19, C2, C22, C23, C24, C25, C26, C27, C28, C29, C3, C4, C41, C44, C45, C46, C5, C6, C69, C7, C70, C71, C72, C73, C74, C75, C76, C77, C78, C79, C8, C80, C81, C82, C83, C84, C85, C86, C87, C88, C89, C9, C90, C97, C98, C99, D5, D6, D7, D8, J1, J2, J5, R28, R29, R30, R31, R57, R58, R59, R60, R61, R62, R63, R66, R67, R68, R69, R70, R71, R72, R73, R75, R76, R77, R78, R79, R80, R81, R82, U1, U10, U12, U2, U3, U7: now left out of the parts list
- C20, C21: footprint Capacitor_SMD:C_0805_2012Metric_Pad1.18x1.45mm_HandSolder -> Capacitor_SMD:C_1206_3216Metric_Pad1.33x1.80mm_HandSolder; now left out of the parts list
- IC1, IC2: LCSC Part # (none) -> C666563
- R3, R4: value 110R -> 240R; now left out of the parts list
- R56, R74: value 590R -> 1K3; now left out of the parts list
- U4, U5: LCSC Part # (none) -> C86723
- U6: LCSC Part # (none) -> C670493
- U8, U9: LCSC Part # (none) -> C94590
Connections:
- net +5VDF: now also J3.1 (Pin_1)
- net -5V: now also C30.2
- net GND: now also C30.1, J3.3 (Pin_3)
- net OUT_L: now also J1.3 (Pin_3), R63.2; no longer J1.1 (Pin_1), R62.2
- net OUT_R: now also J1.1 (Pin_1), R62.2; no longer J1.3 (Pin_3), R63.2
- net PROG: now also J3.2 (Pin_2)

Commit message: work
Parts:
- C1, C10, C100, C101, C102, C103, C104, C105, C106, C11, C12, C13, C14, C15, C16, C17, C18, C19, C2, C20, C21, C22, C23, C24, C25, C26, C27, C28, C29, C3, C30, C4, C41, C44, C45, C46, C5, C6, C69, C7, C70, C71, C72, C73, C74, C75, C76, C77, C78, C79, C8, C80, C81, C82, C83, C84, C85, C86, C87, C88, C89, C9, C90, C97, C98, C99, D5, D6, D7, D8, H1, H2, H3, H4, HS1, HS2, J1, J2, J3, J5, R28, R29, R3, R30, R31, R4, R56, R57, R58, R59, R60, R61, R62, R63, R66, R67, R68, R69, R70, R71, R72, R73, R74, R75, R76, R77, R78, R79, R80, R81, R82, U1, U10, U12, U2, U3, U7: now in the parts list
