File: PCM1704/PCM1704.kicad_sch (KiCad schematic)
At the start: 124 parts, among them IC1 LT3042, IC2 LT3042, J1 AUDIO OUT, J2 POWER, J3 PROG, J5 I2S IN, U1 PCM1704, U10 LM337, U12 LM317, U2 PCM1704, U3 DF1704, U4 OPA1611, U5 OPA1611, U6 LT3094, U7 ATtiny1614, U8 OPA1612, U9 OPA1612

Commit message: PCM1704: snapshot before XMOS receive-buffer schematic changes
Adds DESIGN_REVIEW.md (performance review) and a manual zip backup.

Co-Authored-By: Claude Opus 5.5 <noreply@anthropic.com>
Parts:
- R75: value 10k -> 10K
Other:
- moved on the sheet: C106, HS1, HS2, R75

Commit message: PCM1704: XMOS receive buffer, GND vias, WCLK re-route, 68R DF1704 series resistors
- Add U11 (74LVC1G17) MCLK Schmitt buffer, U13 (74LVC125APW) for BCK/DATA/LRCK,
  U14 (TPS7A2033) 3V3 rail; DF1704 inputs renamed DF_*
- GND vias at new ICs and decoupling caps; fix U13 pad 10 clearance
- Re-route WCLK on B.Cu so it no longer runs under BCLK on In2
- R79-R82 22R -> 68R (DF1704 SBAS099A 50-100R guidance), note updated
- DESIGN_REVIEW.md: H3 decision, LT3094 verification, change log

Co-Authored-By: Claude Opus 5.5 <noreply@anthropic.com>
Parts:
- added C108, C109: 100nF, Capacitor_SMD:C_0603_1608Metric_Pad1.08x0.95mm_HandSolder, symbol Device:C
- added C110, C111: 4.7uF, Capacitor_SMD:C_0805_2012Metric_Pad1.18x1.45mm_HandSolder, symbol Device:C
- added C112: 47pF*, Capacitor_SMD:C_0603_1608Metric_Pad1.08x0.95mm_HandSolder, symbol Device:C
- added R83, R84, R85, R86: 51K, Resistor_SMD:R_0603_1608Metric_Pad0.98x0.95mm_HandSolder, symbol Device:R
- added R87, R88, R89, R90: 22R, Resistor_SMD:R_0603_1608Metric_Pad0.98x0.95mm_HandSolder, symbol Device:R
- added R91: 100R*, Resistor_SMD:R_0603_1608Metric_Pad0.98x0.95mm_HandSolder, symbol Device:R
- added U11: 74LVC1G17, Package_TO_SOT_SMD:SOT-23-5, symbol 74xGxx:74LVC1G17
- added U13: 74LVC125APW, Package_SO:TSSOP-14_4.4x5mm_P0.65mm, symbol 74xx:74LVC125
- added U14: TPS7A2033, Package_TO_SOT_SMD:SOT-23-5, symbol Regulator_Linear:TPS7A20xxxDBV
- R79, R80, R81, R82: value 22R -> 68R
Connections:
- net +5VDF: now also C110.1, U14.1 (IN), U14.3 (EN)
- net BCKIN: now also R84.1, U13.2; no longer U3.2 (BCKIN)
- net DATAIN: now also R85.1, U13.5; no longer U3.1 (DIN)
- net GND: now also C108.2, C109.2, C110.2, C111.2, C112.2, R83.2, R84.2, R85.2, R86.2, U11.3 (GND), U13.1, U13.10, U13.12, U13.4, U13.7 (GND), U14.2 (GND)
- net LRCKIN: now also R86.1, U13.9; no longer U3.28 (LRCIN)
- net SCKIN: now also R83.1, R91.1, U11.2; no longer U3.6 (XTI)
- new net: R88.1, U13.3
- new net: R87.1, U11.4
- new net: R89.1, U13.6
- new net: C112.1, R91.2
- new net: R90.1, U13.8
- new net +3V3: C108.1, C109.1, C111.1, U11.5 (VCC), U13.13, U13.14 (VCC), U14.5 (OUT)
- new net DF_BCK: R88.2, U3.2 (BCKIN)
- new net DF_DIN: R89.2, U3.1 (DIN)
- new net DF_LRCK: R90.2, U3.28 (LRCIN)
- new net DF_SCK: R87.2, U3.6 (XTI)
- no-connect marks 15 -> 16
Other:
- note added: "R79-R82: 68R source termination at U3 pins 26,25,24,23 (DF1704 SBAS099A: start 50-100R). TUNE 47-100R after checking BCLK/WCLK edges at both DACs."
- note added: "XMOS RX BUFFER: 3V3 rail, IOFF-rated inputs U11 Schmitt = SCK; U13 = BCK / DATA / LRCK R87-R90 22R: TUNE on scope at U3 pins R91/C112 SCK AC TERM: DNP until measured"
- note removed: "R79-R82: 0R source links at U3 pins 26,25,24,23. Tune to 22-33R only after checking BCLK/data timing at both DACs."
