File: TPA3250-SPLIT-2/MCU.kicad_sch (KiCad schematic)
At the start: 14 parts, among them J12 VOL, J6 PROG, U2 ATtiny1614, U7 TPS7A2033

Commit message: more
Parts:
- added R59: 10K, Resistor_SMD:R_0805_2012Metric_Pad1.20x1.40mm_HandSolder, symbol Device:R
Connections:
- net MCU-3V3: now also R59.2
- net TPA_FAULT: now also R59.1
Changed lines of the file:
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@@
+	)
+	(junction
+		(at 27.94 86.36)
+		(diameter 0)
+		(color 0 0 0 0)
 	)
 	(junction
@@
 	(wire
 		(pts
+			(xy 27.94 86.36) (xy 57.15 86.36)
+		)
+		(stroke
+			(width 0)
+			(type default)
+		)
+	)
+	(wire
+		(pts
 			(xy 24.13 93.98) (xy 27.94 93.98)
 		)
@@
 	(wire
 		(pts
-			(xy 50.8 86.36) (xy 57.15 86.36)
+			(xy 24.13 86.36) (xy 27.94 86.36)
 		)
 		(stroke
@@
 	(wire
 		(pts
+			(xy 27.94 64.77) (xy 27.94 72.39)
+		)
+		(stroke
+			(width 0)
+			(type default)
+		)
+	)
+	(wire
+		(pts
 			(xy 175.26 101.6) (xy 175.26 113.03)
 		)
@@
 		(pts
 			(xy 72.39 114.3) (xy 72.39 124.46)
+		)
+		(stroke
+			(width 0)
+			(type default)
+		)
+	)
+	(wire
+		(pts
+			(xy 27.94 80.01) (xy 27.94 86.36)
 		)
 		(stroke
@@
 			)
 			(justify right bottom)
+		)
+	)
+	(label "MCU-3V3"
+		(at 27.94 64.77 90)
+		(effects
+			(font
+				(size 1.27 1.27)
+			)
+			(justify left bottom)
 		)
 	)
@@
 	(hierarchical_label "TPA_FAULT"
 		(shape input)
-		(at 50.8 86.36 180)
+		(at 24.13 86.36 180)
 		(effects
 			(font
@@
 					(unit 1)
 				)
+			)
+		)
+	)
+	(symbol
+		(lib_id "Device:R")
+		(at 27.94 76.2 180)
+		(unit 1)
+		(body_style 1)
+		(exclude_from_sim no)
+		(in_bom yes)
+		(on_board yes)
+		(in_pos_files yes)
+		(dnp no)
+		(fields_autoplaced yes)
+		(property "Reference" "R59"
+			(at 30.48 74.9299 0)
+			(show_name no)
+			(do_not_autoplace no)
+			(effects
+				(font
+					(size 1.27 1.27)
+				)
+				(justify right)
+			)
+		)
+		(property "Value" "10K"
+			(at 30.48 77.4699 0)
+			(show_name no)
+			(do_not_autoplace no)
+			(effects
+				(font
+					(size 1.27 1.27)
+				)
+				(justify right)
+			)
+		)
+		(property "Footprint" "Resistor_SMD:R_0805_2012Metric_Pad1.20x1.40mm_HandSolder"
+			(at 29.718 76.2 90)
+			(hide yes)
+			(show_name no)
+			(do_not_autoplace no)
+			(effects
+				(font
+					(size 1.27 1.27)
+				)
+			)
+		)
+		(property "Datasheet" ""
+			(at 27.94 76.2 0)
+			(hide yes)
+			(show_name no)
+			(do_not_autoplace no)
+			(effects
+				(font
+					(size 1.27 1.27)
+				)
+			)
+		)
+		(property "Description" "Resistor"
+			(at 27.94 76.2 0)
+			(hide yes)
+			(show_name no)
+			(do_not_autoplace no)
+			(effects
+				(font
+					(size 1.27 1.27)
+				)
+			)
+		)
+		(pin "1"
+		)
+		(pin "2"
+		)
+		(instances
+			(project "TPA3250-SPLIT-2"
+				(path "/d0eeeeda-311a-416d-b9f7-ac3b9875c0a9/ed79208c-20ac-4652-a801-6cd46992a6c8"
+					(reference "R59")
+					(unit 1)
+				)
