File: TPA3250-SPLIT-2/TPA3250-SPLIT-2.kicad_pcb (KiCad board)
At the start: 4 copper layers, 172.1 x 99.1 mm, 224 parts, among them IC3 TPS65133, J1 L +, J10 PSU HEADER 2, J11 AUDIO IN, J12 VOL, J13 AMP HEADER 2, J14 PVDD, J15 PVDD, J16 POWER IN, J2 L -, J3 R +, J4 R -, J6 PROG, J7 PSU HEADER 1, J8 POWER SW, J9 AMP HEADER 1, K3 Relay_SPST-NO, Q1 DMP4015SK3, U1 CS3310, U10 TPA3250, U2 ATtiny1614, U3 LMR51430, U4 OPA1656/1612, U5 OPA1656/1612, U6 LM4562, U7 TPS7A2033, U8 LMR51430, U9 L7812

Commit message: more
Parts:
- added R59: 10K, Resistor_SMD:R_0805_2012Metric_Pad1.20x1.40mm_HandSolder, F.Cu at (236.4, 128.5)
Routing:
- net /MCU/MCU-3V3: track 56.4 -> 72.7 mm, vias 2 -> 3
- net /TPA_FAULT: track 44.5 -> 46.4 mm
Changed lines of the file:
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@@
 		)
 	)
+	(footprint "Resistor_SMD:R_0805_2012Metric_Pad1.20x1.40mm_HandSolder"
+		(layer "F.Cu")
+		(at 236.444 128.483)
+		(descr "Resistor SMD 0805 (2012 Metric), square (rectangular) end terminal, IPC-7351 nominal with elongated pad for handsoldering. (Body size source: IPC-SM-782 page 72, https://www.pcb-3d.com/wordpress/wp-content/uploads/ipc-sm-782a_amendment_1_and_2.pdf)")
+		(tags "resistor handsolder")
+		(property "Reference" "R59"
+			(at 0 -1.65 0)
+			(layer "F.SilkS")
+			(hide yes)
+			(effects
+				(font
+					(size 1 1)
+					(thickness 0.15)
+				)
+			)
+		)
+		(property "Value" "10K"
+			(at 0 1.311 0)
+			(layer "F.SilkS")
+			(effects
+				(font
+					(size 0.5 0.5)
+					(thickness 0.0625)
+				)
+			)
+		)
+		(property "Datasheet" ""
+			(at 0 0 0)
+			(layer "F.Fab")
+			(hide yes)
+			(effects
+				(font
+					(size 1.27 1.27)
+				)
+			)
+		)
+		(property "Description" "Resistor"
+			(at 0 0 0)
+			(layer "F.Fab")
+			(hide yes)
+			(effects
+				(font
+					(size 1.27 1.27)
+				)
+			)
+		)
+		(property "KiLib_Generator" "SMD_2terminal_chip_molded"
+			(at 0 0 0)
+			(layer "F.SilkS")
+			(hide yes)
+			(effects
+				(font
+					(size 1 1)
+					(thickness 0.15)
+				)
+			)
+		)
+		(property ki_fp_filters "R_*")
+		(sheetname "/MCU/")
+		(sheetfile "MCU.kicad_sch")
+		(units
+			(unit
+				(name "A")
+				(pins "1" "2")
+			)
+		)
+		(attr smd)
+		(duplicate_pad_numbers_are_jumpers no)
+		(fp_line
+			(start -0.227064 -0.735)
+			(end 0.227064 -0.735)
+			(stroke
+				(width 0.12)
+				(type solid)
+			)
+			(layer "F.SilkS")
+		)
+		(fp_line
+			(start -0.227064 0.735)
+			(end 0.227064 0.735)
+			(stroke
+				(width 0.12)
+				(type solid)
+			)
+			(layer "F.SilkS")
+		)
+		(fp_rect
+			(start -1.85 -0.95)
+			(end 1.85 0.95)
+			(stroke
+				(width 0.05)
+				(type solid)
+			)
+			(fill no)
+			(layer "F.CrtYd")
+		)
+		(fp_rect
+			(start -1 -0.625)
+			(end 1 0.625)
+			(stroke
+				(width 0.1)
+				(type solid)
+			)
+			(fill no)
+			(layer "F.Fab")
+		)
+		(fp_text user "${REFERENCE}"
+			(at 0 0 0)
+			(layer "F.Fab")
+			(effects
+				(font
+					(size 0.5 0.5)
+					(thickness 0.08)
+				)
+			)
+		)
+		(pad "1" smd roundrect
+			(at -1 0)
+			(size 1.2 1.4)
+			(layers "F.Cu" "F.Mask" "F.Paste")
+			(roundrect_rratio 0.208333)
+			(net "/TPA_FAULT")
+			(pintype "passive")
+		)
+		(pad "2" smd roundrect
+			(at 1 0)
+			(size 1.2 1.4)
+			(layers "F.Cu" "F.Mask" "F.Paste")
+			(roundrect_rratio 0.208333)
+			(net "/MCU/MCU-3V3")
+			(pintype "passive")
+		)
+		(embedded_fonts no)
+		(model "${KICAD10_3DMODEL_DIR}/Resistor_SMD.3dshapes/R_0805_2012Metric.step"
+			(offset
+				(xyz 0 0 0)
+			)
+			(scale
+				(xyz 1 1 1)
+			)
+			(rotate
+				(xyz 0 0 0)
+			)
+		)
+	)
 	(footprint "Connector_Molex:Molex_KK-396_A-41791-0002_1x02_P3.96mm_Vertical"
 		(layer "F.Cu")
@@
 	)
 	(segment
+		(start 236.006 129.921)
+		(end 234.188 129.921)
+		(width 0.2)
+		(layer "F.Cu")
+		(net "/MCU/MCU-3V3")
+	)
+	(segment
 		(start 224.171 111.037)
 		(end 226.9155 111.037)
@@
 	)
 	(segment
+		(start 237.444 128.483)
+		(end 236.006 129.921)
+		(width 0.2)
+		(layer "F.Cu")
+		(net "/MCU/MCU-3V3")
+	)
+	(segment
 		(start 226.722534 122.120534)
 		(end 226.722534 120.747034)
@@
 	)
 	(via
+		(at 234.188 129.921)
+		(size 0.6)
+		(drill 0.3)
+		(layers "F.Cu" "B.Cu")
+		(net "/MCU/MCU-3V3")
+	)
+	(via
 		(at 223.409 109.982)
 		(size 0.6)
@@
 	)
 	(segment
+		(start 234.188 129.921)
+		(end 232.68 129.921)
+		(width 0.2)
+		(layer "B.Cu")
+		(net "/MCU/MCU-3V3")
+	)
+	(segment
+		(start 232.68 129.921)
+		(end 224.933 122.174)
+		(width 0.2)
+		(layer "B.Cu")
+		(net "/MCU/MCU-3V3")
+	)
+	(segment
 		(start 237.325534 102.542466)
 		(end 237.325534 103.815534)
@@
 	)
 	(segment
+		(start 233.569 128.524)
+		(end 235.403 128.524)
+		(width 0.2)
+		(layer "F.Cu")
+		(net "/TPA_FAULT")
+	)
+	(segment
 		(start 203.560001 156.336501)
 		(end 204.486499 156.336501)
 		(width 0.2)
 		(layer "F.Cu")
+		(net "/TPA_FAULT")
+	)
+	(segment
+		(start 235.403 128.524)
+		(end 235.444 128.483)
+		(width 0.2)
+		(layer "F.Cu")
