File: GainClone/GainClone.kicad_sch (KiCad schematic)
At the start: 0 parts

Commit message: commit
Parts:
- added H1, H2, H3, H4: MountingHole, MountingHole:MountingHole_3.2mm_M3, symbol Mechanical:MountingHole
Other:
- sheet AMPS ports: added AMP-MUTE; removed none
