File: GainClone/AMPS.kicad_sch (KiCad schematic)
At the start: 26 parts, among them U1 LM3886, U3 LM3886

Commit message: commit
Parts:
- added C34, C35: 22uF, Capacitor_THT:CP_Radial_D5.0mm_P2.50mm, symbol Device:C_Polarized
- added R38, R43: 22K, Resistor_SMD:R_0805_2012Metric_Pad1.20x1.40mm_HandSolder, symbol Device:R
- added R47, R48: 680R, Resistor_SMD:R_0805_2012Metric_Pad1.20x1.40mm_HandSolder, symbol Device:R
- added U6, U8: VO617A-3, Package_DIP:DIP-4_W7.62mm, symbol InputSwitch:VO617A_3
Connections:
- net GND: now also C34.1, C35.1, U6.2, U8.2
- net VEE: now also U6.3, U8.3
- net L-MUTE: now reaches U1.8 (MUTE)
- net L-MUTE: now also R43.2
- net R-MUTE: now reaches U3.8 (MUTE)
- net R-MUTE: now also C34.2, R38.2
- new net: R43.1, U8.4
- new net: R47.2, U8.1
- new net: R48.2, U6.1
- new net: R38.1, U6.4
- new net AMP-MUTE: R47.1, R48.1
Other:
- moved on the sheet: C1, C10, C2, C3, C8, C9, L1, L2, R1, R10, R11, R12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

Commit message: work
Parts:
- C1, C10: footprint Capacitor_THT:C_Rect_L7.2mm_W2.5mm_P5.00mm -> Capacitor_THT:C_Rect_L7.2mm_W2.5mm_P5.00mm_FKS2_FKP2_MKS2_MKP2
Connections:
- net L-MUTE: now also C35.2
Changed lines of the file:
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@@
 	)
 	(junction
+		(at 247.65 132.08)
+		(diameter 0)
+		(color 0 0 0 0)
+	)
+	(junction
 		(at 255.27 45.72)
 		(diameter 0)
@@
 	(wire
 		(pts
-			(xy 247.65 132.08) (xy 247.65 138.43)
-		)
-		(stroke
-			(width 0)
-			(type default)
-		)
-	)
-	(wire
-		(pts
 			(xy 128.27 74.93) (xy 128.27 96.52)
 		)
@@
 	(wire
 		(pts
-			(xy 104.14 125.73) (xy 104.14 133.35)
+			(xy 104.14 120.015) (xy 104.14 133.35)
 		)
 		(stroke
@@
 	(wire
 		(pts
+			(xy 247.65 132.08) (xy 247.65 138.43)
+		)
+		(stroke
+			(width 0)
+			(type default)
+		)
+	)
+	(wire
+		(pts
 			(xy 74.93 154.94) (xy 74.93 186.69)
 		)
@@
 	(wire
 		(pts
-			(xy 101.6 36.83) (xy 101.6 44.45)
+			(xy 101.6 30.48) (xy 101.6 44.45)
 		)
 		(stroke
@@
 	(wire
 		(pts
+			(xy 247.65 132.08) (xy 261.62 132.08)
+		)
+		(stroke
+			(width 0)
+			(type default)
+		)
+	)
+	(wire
+		(pts
 			(xy 227.33 137.16) (xy 236.22 137.16)
 		)
@@
 	(wire
 		(pts
-			(xy 237.49 132.08) (xy 261.62 132.08)
+			(xy 237.49 132.08) (xy 247.65 132.08)
 		)
 		(stroke
@@
 	)
 	(label "L-MUTE"
-		(at 101.6 36.83 90)
+		(at 101.6 30.48 90)
 		(effects
 			(font
@@
 	)
 	(label "R-MUTE"
-		(at 104.14 125.73 90)
+		(at 104.14 120.015 90)
 		(effects
 			(font
@@
 			)
 		)
-		(property "Footprint" "Capacitor_THT:C_Rect_L7.2mm_W2.5mm_P5.00mm"
+		(property "Footprint" "Capacitor_THT:C_Rect_L7.2mm_W2.5mm_P5.00mm_FKS2_FKP2_MKS2_MKP2"
 			(at 131.7752 163.83 0)
 			(hide yes)
@@
 			)
 		)
-		(property "Footprint" "Capacitor_THT:C_Rect_L7.2mm_W2.5mm_P5.00mm"
+		(property "Footprint" "Capacitor_THT:C_Rect_L7.2mm_W2.5mm_P5.00mm_FKS2_FKP2_MKS2_MKP2"
 			(at 129.2352 74.93 0)
 			(hide yes)
