File: GainClone/protect.kicad_sch (KiCad schematic)
At the start: 35 parts, among them J19 OUT L, J20 OUT R, K1 Relay_DPST-NO, Q1 TIP122*, Q2 BD140, Q3 BC549, Q4 BC559, Q5 BC549

Commit message: commit
Parts:
- removed HS1: Heatsink, Custom:Tiny heatsink, symbol Mechanical:Heatsink
- removed Q3, Q5: BC549, Package_TO_SOT_THT:TO-92L_Inline_Wide, symbol Transistor_BJT:BC549
- removed Q4: BC559, Package_TO_SOT_THT:TO-92L_Inline_Wide, symbol Transistor_BJT:BC559
- added Q4, Q9: BC849, Package_TO_SOT_SMD:SOT-23, symbol Transistor_BJT:BC849
- added Q8: BC859, Package_TO_SOT_SMD:SOT-23, symbol Transistor_BJT:BC859
- D10: value ZD* -> ZD-24V
- Q1: value TIP122* -> TIP142
- R17: value 2K2* -> 2K2
Connections:
- net GND: now also Q9.2 (E)
- net at Q2.3 (B), R22.2: now also Q8.3 (C)
- net at R20.1, R21.2: now also Q8.1 (B)
- net at C13.1, Q1.3 (E), Q2.1 (E)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: now also Q8.2 (E)
- net at C14.2, D14.1 (K), D15.1 (K)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: now also Q4.1 (B)
- net at R21.1: now also Q4.3 (C)
- net at D12.2 (A), D13.2 (A), D17.2 (A): now also Q4.2 (E)
- net at R23.1: now also Q9.1 (B)
- net at R22.1: now also Q9.3 (C)

Commit message: work
Parts:
- D11: value 1N4148W* -> 1N4148W
Changed lines of the file:
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@@
+	)
+	(junction
+		(at 54.61 87.63)
+		(diameter 0)
+		(color 0 0 0 0)
+	)
+	(junction
+		(at 26.67 39.37)
+		(diameter 0)
+		(color 0 0 0 0)
 	)
 	(junction
@@
 	)
 	(junction
-		(at 54.61 87.63)
-		(diameter 0)
-		(color 0 0 0 0)
-	)
-	(junction
-		(at 26.67 39.37)
-		(diameter 0)
-		(color 0 0 0 0)
-	)
-	(junction
 		(at 100.33 100.33)
 		(diameter 0)
@@
 	)
 	(junction
+		(at 67.31 39.37)
+		(diameter 0)
+		(color 0 0 0 0)
+	)
+	(junction
 		(at 271.78 123.19)
 		(diameter 0)
 		(color 0 0 0 0)
 	)
-	(junction
-		(at 67.31 39.37)
-		(diameter 0)
-		(color 0 0 0 0)
-	)
 	(wire
 		(pts
@@
 	(wire
 		(pts
-			(xy 261.62 120.65) (xy 289.56 120.65)
+			(xy 261.62 120.65) (xy 279.4 120.65)
 		)
 		(stroke
@@
 	(wire
 		(pts
-			(xy 271.78 123.19) (xy 289.56 123.19)
+			(xy 271.78 123.19) (xy 279.4 123.19)
 		)
 		(stroke
@@
 	)
 	(label "L-IN"
-		(at 289.56 120.65 0)
+		(at 279.4 120.65 0)
 		(effects
 			(font
@@
 	)
 	(label "R-IN"
-		(at 289.56 123.19 0)
+		(at 279.4 123.19 0)
 		(effects
 			(font
@@
 			)
 		)
-		(property "Value" "1N4148W*"
+		(property "Value" "1N4148W"
 			(at 52.07 59.6899 90)
 			(show_name no)
