File: GainClone/CONTROL.kicad_sch (KiCad schematic)
At the start: 4 parts, among them J2 SYSTEM CONNECTOR, J3 PROG, U4 ATtiny1614-SS

Commit message: work
Connections:
- net +5VD: now also J2.1 (Pin_1)
Changed lines of the file:
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@@
 	(wire
 		(pts
-			(xy 148.59 93.98) (xy 161.29 93.98)
+			(xy 148.59 93.98) (xy 158.75 93.98)
 		)
 		(stroke
@@
 	(wire
 		(pts
+			(xy 198.12 92.71) (xy 198.12 93.98)
+		)
+		(stroke
+			(width 0)
+			(type default)
+		)
+	)
+	(wire
+		(pts
 			(xy 194.31 99.06) (xy 204.47 99.06)
 		)
@@
 	(wire
 		(pts
+			(xy 198.12 93.98) (xy 204.47 93.98)
+		)
+		(stroke
+			(width 0)
+			(type default)
+		)
+	)
+	(wire
+		(pts
 			(xy 198.12 109.22) (xy 204.47 109.22)
 		)
@@
 	(wire
 		(pts
-			(xy 148.59 96.52) (xy 161.29 96.52)
-		)
-		(stroke
-			(width 0)
-			(type default)
-		)
-	)
-	(wire
-		(pts
-			(xy 194.31 93.98) (xy 204.47 93.98)
+			(xy 148.59 96.52) (xy 158.75 96.52)
 		)
 		(stroke
@@
 	(wire
 		(pts
-			(xy 148.59 99.06) (xy 161.29 99.06)
+			(xy 148.59 99.06) (xy 168.91 99.06)
 		)
 		(stroke
@@
 	(wire
 		(pts
+			(xy 194.31 92.71) (xy 198.12 92.71)
+		)
+		(stroke
+			(width 0)
+			(type default)
+		)
+	)
+	(wire
+		(pts
 			(xy 204.47 104.14) (xy 198.12 104.14)
 		)
@@
 	(wire
 		(pts
-			(xy 148.59 91.44) (xy 161.29 91.44)
+			(xy 148.59 91.44) (xy 158.75 91.44)
 		)
 		(stroke
@@
 	(wire
 		(pts
-			(xy 148.59 86.36) (xy 161.29 86.36)
-		)
-		(stroke
-			(width 0)
-			(type default)
-		)
-	)
-	(wire
-		(pts
-			(xy 148.59 88.9) (xy 161.29 88.9)
+			(xy 148.59 86.36) (xy 168.91 86.36)
+		)
+		(stroke
+			(width 0)
+			(type default)
+		)
+	)
+	(wire
+		(pts
+			(xy 148.59 88.9) (xy 158.75 88.9)
 		)
 		(stroke
@@
 	)
 	(label "LED"
-		(at 161.29 99.06 0)
+		(at 168.91 99.06 0)
 		(effects
 			(font
@@
 	)
 	(label "PROG"
-		(at 161.29 86.36 0)
+		(at 168.91 86.36 0)
 		(effects
 			(font
@@
 	(hierarchical_label "CS_SCLK"
 		(shape output)
-		(at 161.29 93.98 0)
+		(at 158.75 93.98 0)
 		(effects
 			(font
@@
 	(hierarchical_label "CS_CS"
 		(shape output)
-		(at 161.29 96.52 0)
+		(at 158.75 96.52 0)
 		(effects
 			(font
@@
 	(hierarchical_label "CS_MUTE"
 		(shape output)
-		(at 161.29 91.44 0)
+		(at 158.75 91.44 0)
 		(effects
 			(font
@@
 	(hierarchical_label "CS_DATA"
 		(shape output)
-		(at 161.29 88.9 0)
+		(at 158.75 88.9 0)
 		(effects
 			(font
@@
 		)
 	)
+	(hierarchical_label "+5VD"
+		(shape output)
+		(at 194.31 92.71 180)
+		(effects
+			(font
+				(size 1.27 1.27)
+			)
+			(justify right)
+		)
+	)

Commit message: work
Parts:
- U4: value ATtiny1614-SS -> ATtiny1614
Changed lines of the file:
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@@
 			)
 		)
-		(property "Value" "ATtiny1614-SS"
+		(property "Value" "ATtiny1614"
 			(at 135.4933 78.74 0)
 			(show_name no)
