File: GainClone/GainClone.kicad_pcb (KiCad board)
At the start: 2 copper layers, 120 x 120 mm, 120 parts, among them J1 OUT L, J13 AC, J14 GND, J15 AC, J16 GND, J17 GND, J18 GND, J2 SYSTEM CONNECTOR, J3 PROG, J4 AUDIO IN, J5 OUT R, K1 Relay_DPST-NO, Q1 TIP122*, Q2 BD140, Q3 BC549, Q4 BC559, Q5 BC549, Q6 MJD31CJ, Q7 MJD32CJ, U1 LM3886, U2 OPA1656ID, U3 LM3886, U4 ATtiny1614-SS, U7 CS3310, U8 TPS7A39*

Commit message: commit
Parts:
- removed C59, C65, C70: 10nF, Capacitor_SMD:C_0805_2012Metric_Pad1.18x1.45mm_HandSolder
- removed C73, C78: 10uf 25V, Capacitor_SMD:C_1206_3216Metric_Pad1.33x1.80mm_HandSolder
- removed C79, C80: 10uF, Capacitor_SMD:C_1206_3216Metric_Pad1.33x1.80mm_HandSolder
- removed HS1: Heatsink, Custom:Tiny heatsink
- removed J1: OUT L, Spade connector:TE_62409-1
- removed JP1: Jumper, TestPoint:TestPoint_2Pads_Pitch5.08mm_Drill1.3mm
- removed Q3, Q5: BC549, Package_TO_SOT_THT:TO-92L_Inline_Wide
- removed R56: 10K, Resistor_SMD:R_0805_2012Metric_Pad1.20x1.40mm_HandSolder
- removed R57: 115K, Resistor_SMD:R_0805_2012Metric_Pad1.20x1.40mm_HandSolder
- removed R58: 127K, Resistor_SMD:R_0805_2012Metric_Pad1.20x1.40mm_HandSolder
- added C27: 10uF, Capacitor_SMD:C_1206_3216Metric_Pad1.33x1.80mm_HandSolder, F.Cu at (157.1, 101.1)
- added C28: 10uF, Capacitor_SMD:C_1206_3216Metric_Pad1.33x1.80mm_HandSolder, F.Cu at (147.3, 101.1)
- added C29: 10nF, Capacitor_SMD:C_0805_2012Metric_Pad1.18x1.45mm_HandSolder, F.Cu at (152.2, 98.2)
- added C30: 10nF, Capacitor_SMD:C_0805_2012Metric_Pad1.18x1.45mm_HandSolder, F.Cu at (154.6, 108.0)
- added C31: 10nF, Capacitor_SMD:C_0805_2012Metric_Pad1.18x1.45mm_HandSolder, F.Cu at (150.5, 108.0)
- added C32: 10uF, Capacitor_SMD:C_1206_3216Metric_Pad1.33x1.80mm_HandSolder, F.Cu at (147.3, 103.5)
- added C33: 10uF, Capacitor_SMD:C_1206_3216Metric_Pad1.33x1.80mm_HandSolder, F.Cu at (157.1, 103.5)
- added C34: 22uF, Capacitor_THT:CP_Radial_D5.0mm_P2.50mm, F.Cu at (207.9, 118.4)
- added C35: 22uF, Capacitor_THT:CP_Radial_D5.0mm_P2.50mm, F.Cu at (96.8, 87.4)
- added C36: 1uF, Capacitor_SMD:C_1206_3216Metric_Pad1.33x1.80mm_HandSolder, F.Cu at (176.1, 97.2)
- added C37: 2.2uF, Capacitor_SMD:C_0805_2012Metric_Pad1.18x1.45mm_HandSolder, F.Cu at (181.5, 97.0)
- added H1: MountingHole, MountingHole:MountingHole_3.2mm_M3, F.Cu at (209.0, 141.2)
- added H2: MountingHole, MountingHole:MountingHole_3.2mm_M3, F.Cu at (96.0, 141.1)
- added H3: MountingHole, MountingHole:MountingHole_3.2mm_M3, F.Cu at (209.0, 28.1)
- added H4: MountingHole, MountingHole:MountingHole_3.2mm_M3, F.Cu at (95.9, 28.1)
- added IC1: AP2205-50YR-13, Package_TO_SOT_SMD:SOT-89-3, F.Cu at (176.5, 92.5)
- added J19: OUT L, Spade connector:TE_62409-1, F.Cu at (294.2, 85.0)
- added J20: OUT R, Spade connector:TE_62409-1, F.Cu at (294.2, 88.7)
- added Q8: BC859, Package_TO_SOT_SMD:SOT-23, F.Cu at (297.1, 107.6)
- added Q9: BC849, Package_TO_SOT_SMD:SOT-23, F.Cu at (297.1, 112.0)
- added R34: 32K, Resistor_SMD:R_0805_2012Metric_Pad1.20x1.40mm_HandSolder, F.Cu at (154.5, 105.9)
- added R35: 10K, Resistor_SMD:R_0805_2012Metric_Pad1.20x1.40mm_HandSolder, F.Cu at (154.6, 110.0)
- added R36: 10K, Resistor_SMD:R_0805_2012Metric_Pad1.20x1.40mm_HandSolder, F.Cu at (150.5, 110.0)
- added R37: 42K, Resistor_SMD:R_0805_2012Metric_Pad1.20x1.40mm_HandSolder, F.Cu at (150.6, 105.9)
- added R38: 22K, Resistor_SMD:R_0805_2012Metric_Pad1.20x1.40mm_HandSolder, F.Cu at (203.7, 116.9)
- added R47: 680R, Resistor_SMD:R_0805_2012Metric_Pad1.20x1.40mm_HandSolder, F.Cu at (113.9, 47.7)
- added R48: 680R, Resistor_SMD:R_0805_2012Metric_Pad1.20x1.40mm_HandSolder, F.Cu at (113.9, 44.7)
- added U5: TPS7A39*, Package_SON:Texas_S-PVSON-N10_ThermalVias, F.Cu at (152.2, 102.5)
- added U6: VO617A-3, Package_DIP:DIP-4_W7.62mm, F.Cu at (203.7, 129.9)
- C3, C8: footprint Capacitor_THT:C_Rect_L7.2mm_W7.2mm_P5.00mm -> Capacitor_THT:C_Rect_L7.2mm_W7.2mm_P5.00mm_FKS2_FKP2_MKS2_MKP2
- D10: value ZD* -> ZD-24V
- Q1: value TIP122* -> TIP142
- Q4: value BC559 -> BC849; footprint Package_TO_SOT_THT:TO-92L_Inline_Wide -> Package_TO_SOT_SMD:SOT-23
- R17: value 2K2* -> 2K2
- R43: value 10K -> 22K
- R7, R8: footprint Resistor_THT:R_Axial_DIN0207_L6.3mm_D2.5mm_P10.16mm_Horizontal -> Resistor_SMD:R_0805_2012Metric_Pad1.20x1.40mm_HandSolder
- U8: value TPS7A39* -> VO617A-3; footprint Package_SON:Texas_S-PVSON-N10_ThermalVias -> Package_DIP:DIP-4_W7.62mm
- moved R43 279.6 mm to (101.0, 88.8), turned to -90 degrees
- moved C1 272.2 mm to (108.1, 121.2), turned to 180 degrees
- moved C3 269.9 mm to (110.3, 87.9), turned to 180 degrees
- moved R39 266.0 mm to (318.6, 90.6)
- moved R44 266.0 mm to (323.3, 87.6)
- moved R45 266.0 mm to (323.3, 90.6)
- moved R46 266.0 mm to (323.3, 93.5)
- moved R2 257.3 mm to (108.1, 117.9), turned to 90 degrees
- moved R1 254.3 mm to (105.9, 98.6)
- moved C2 254.3 mm to (110.6, 100.7)
- moved R4 254.2 mm to (105.9, 93.4), turned to 180 degrees
- moved R3 254.2 mm to (105.9, 96.1), turned to 180 degrees
- moved R5 254.2 mm to (105.9, 101.3), turned to 180 degrees
- moved R6 252.1 mm to (112.9, 117.9), turned to 90 degrees
- moved C22 106.9 mm to (147.3, 120.7), turned to 180 degrees
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Connections:
- C13 pad 1: Net-(JP1-B) -> Net-(Q1-E)
- C16 pad 2: /POWER/VEE -> /AMPS/VEE
- C20 pad 1: /CONTROL/5V_DIG -> /CONTROL/+5VD
- C4 pad 1: /POWER/VCC -> /AMPS/VCC
- D2 pad 1: /POWER/VEE -> /AMPS/VEE
- D2 pad 4: /POWER/VCC -> /AMPS/VCC
- J3 pad 1: /CONTROL/5V_DIG -> /CONTROL/+5VD
- Q1 pad 2: /PROTECT/DC -> /AMPS/VCC
- Q1 pad 3: Net-(JP1-B) -> Net-(Q1-E)
- Q2 pad 1: Net-(JP1-B) -> Net-(Q1-E)
- Q4 pad 1: Net-(Q2-B) -> Net-(D14-K)
- Q4 pad 2: Net-(Q4-B) -> Net-(D12-A)
- Q4 pad 3: Net-(JP1-B) -> Net-(Q4-C)
- Q6 pad 2: /POWER/VCC -> /AMPS/VCC
- Q6 pad 3: Net-(Q6-E) -> Net-(IC1-VIN)
- Q7 pad 2: /POWER/VEE -> /AMPS/VEE
- R14 pad 1: Net-(J5-P1-Pad1) -> /PROTECT/R-IN
- R17 pad 1: /PROTECT/DC -> /AMPS/VCC
- R18 pad 2: Net-(JP1-B) -> Net-(Q1-E)
- R20 pad 1: Net-(Q4-B) -> Net-(Q8-B)
- R20 pad 2: Net-(JP1-B) -> Net-(Q1-E)
- R21 pad 1: Net-(Q3-C) -> Net-(Q4-C)
- R21 pad 2: Net-(Q4-B) -> Net-(Q8-B)
- R25 pad 2: /PROTECT/AC -> /POWER/AC
- R26 pad 1: /POWER/VCC -> /AMPS/VCC
- R27 pad 1: /POWER/VEE -> /AMPS/VEE
- R39 pad 1: /INPUTVOL/CS-CS -> /CS_CS
- R43 pad 1: Net-(U8-BUF) -> Net-(R43-Pad1)
- R43 pad 2: Net-(U8-FBN) -> /AMPS/L-MUTE
- R44 pad 1: /INPUTVOL/CS-SDI -> /CS_DATA
- R45 pad 1: /INPUTVOL/CD-SCLK -> /CS_SCLK
- R46 pad 2: /INPUTVOL/CS-MUTE -> /CS_MUTE
- R6 pad 1: Net-(J1-P1-Pad1) -> /PROTECT/L-IN
- U1 pad 8: unconnected-(U1-MUTE-Pad8) -> /AMPS/L-MUTE
- U3 pad 8: unconnected-(U3-MUTE-Pad8) -> /AMPS/R-MUTE
- U4 pad 1: /CONTROL/5V_DIG -> /CONTROL/+5VD
- U4 pad 11: /CONTROL/CS_DATA -> /CS_DATA
- U4 pad 12: unconnected-(U4-PA2-Pad12) -> /CS_MUTE
- U4 pad 13: /CONTROL/CS_SCLK -> /CS_SCLK
- U4 pad 2: /CONTROL/CS_CS -> /CS_CS
- U4 pad 6: /CONTROL/AMP_MUTE -> /AMPS/AMP-MUTE
- U7 pad 1: /INPUTVOL/+5VD -> /CONTROL/+5VD
- U7 pad 11: /INPUTVOL/LM-IN-R -> /AMPS/LM-IN-R
- U7 pad 14: /INPUTVOL/LM-IN-L -> /AMPS/LM-IN-L
- U7 pad 4: /INPUTVOL/+5VD -> /CONTROL/+5VD
- U8 pad 1: Net-(Q6-E) -> Net-(R47-Pad2)
- U8 pad 2: Net-(Q6-E) -> GND
- U8 pad 3: Net-(U8-NR/SS) -> /AMPS/VEE
- U8 pad 4: GND -> Net-(R43-Pad1)
Routing:
- net /AMPS/VEE: track 10.2 -> 45.9 mm
- net Net-(L1-Pad1): track 0.00 -> 21.3 mm
- net Net-(Q6-E): track 19.1 -> 0.00 mm, vias 2 -> 0
- net Net-(IC1-VIN): track 0.00 -> 18.4 mm, vias 0 -> 2
- net /AMPS/R-MUTE: track 0.00 -> 15.0 mm
- net Net-(U2A-+): track 0.00 -> 14.5 mm
- net Net-(U2B-+): track 0.00 -> 13.3 mm
- net Net-(J4-Pin_1): track 0.00 -> 9.84 mm
- net Net-(J4-Pin_3): track 0.00 -> 9.79 mm
- net Net-(C3-Pad2): track 0.00 -> 9.13 mm
- net Net-(U1-+): track 0.00 -> 7.93 mm
- net Net-(L2-Pad1): track 13.4 -> 21.3 mm
- net /POWER/-15V: track 0.00 -> 7.33 mm
- net /POWER/+15V: track 0.00 -> 7.02 mm
- net Net-(C22-Pad2): track 0.00 -> 7.01 mm
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- added copper zone on B.Cu, net /AMPS/VCC
- added copper zone on F.Cu, net /AMPS/VCC
- added copper zone on B.Cu, net /AMPS/VEE
- added copper zone on F.Cu, net /AMPS/VEE
- removed copper zone on B.Cu, net /POWER/VCC
- removed copper zone on F.Cu, net /POWER/VCC
- removed copper zone on B.Cu, net /POWER/VEE
- removed copper zone on F.Cu, net /POWER/VEE
Other:
- board text added: "R G L"

Commit message: work
Parts:
- added G***: LOGO, Custom:LOGONEW, F.Cu at (203.1, 33.5)
- C1, C10: footprint Capacitor_THT:C_Rect_L7.2mm_W2.5mm_P5.00mm -> Capacitor_THT:C_Rect_L7.2mm_W2.5mm_P5.00mm_FKS2_FKP2_MKS2_MKP2
- moved R45 206.6 mm to (121.3, 134.0)
- moved R44 206.5 mm to (121.3, 130.2)
- moved R46 206.5 mm to (121.3, 136.0), turned to 180 degrees
- moved R39 200.8 mm to (121.3, 128.1)
- moved U4 71.6 mm to (113.0, 132.0), turned to 0 degrees
- moved J2 27.1 mm to (150.3, 139.1)
- moved C21 25.8 mm to (173.1, 131.2)
- moved C22 25.8 mm to (173.1, 121.5)
- moved C23 25.8 mm to (164.5, 122.3)
- moved C24 25.8 mm to (164.5, 131.9)
- moved C7 25.8 mm to (160.3, 126.4)
- moved J4 25.8 mm to (179.8, 128.8)
- moved R30 25.8 mm to (164.5, 120.2)
- moved R31 25.8 mm to (164.5, 129.9)
- moved R32 25.8 mm to (164.5, 118.2)
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Routing:
- net /AMPS/VCC: track 29.0 -> 18.7 mm
- net /CONTROL/+5VD: track 0.00 -> 6.87 mm
- net Net-(U7-~{CS}): track 0.00 -> 3.33 mm
- net Net-(U7-~{MUTE}): track 0.00 -> 3.25 mm
- net Net-(U7-SDATAI): track 0.00 -> 3.03 mm
- net Net-(U7-SCLK): track 0.00 -> 3.03 mm
- net Net-(U2A-+): track 14.5 -> 13.1 mm
- net Net-(L1-Pad1): track 21.3 -> 20.4 mm
- net Net-(L2-Pad1): track 21.3 -> 20.4 mm
- added copper zone on B.Cu, net GND
Other:
- board text added: "GainClone - Stereo LM3886 CS3310 - Tom Watson Audio Power Supply ±25V - ±35V 2026"

Commit message: work
Parts:
- removed J5: OUT R, Spade connector:TE_62409-1
- added C38: 100nF, Capacitor_SMD:C_1206_3216Metric_Pad1.33x1.80mm_HandSolder, F.Cu at (80.8, 165.2)
- D11: value 1N4148W* -> 1N4148W
- IC1: value AP2205-50YR-13 -> AP2205
- U2: value OPA1656ID -> OPA1656
- U4: value ATtiny1614-SS -> ATtiny1614
- U5: value TPS7A39* -> TPS7A39
- moved Q9 148.8 mm to (149.5, 131.1)
- moved D18 145.4 mm to (134.2, 134.2)
- moved D11 142.1 mm to (141.2, 125.7)
- moved Q4 141.1 mm to (157.7, 125.0), turned to 180 degrees
- moved Q8 139.6 mm to (157.9, 117.6), turned to -90 degrees
- moved J19 139.0 mm to (166.4, 139.7)
- moved R21 131.6 mm to (153.4, 125.0), turned to 180 degrees
- moved Q2 131.2 mm to (162.7, 114.8), turned to -90 degrees
- moved D17 124.5 mm to (154.1, 122.7)
- moved C11 123.9 mm to (169.2, 134.6), turned to 90 degrees
- moved R24 122.7 mm to (167.1, 115.3), turned to -90 degrees
- moved R23 121.0 mm to (184.1, 150.8)
- moved C13 121.0 mm to (179.3, 167.4)
- moved C14 121.0 mm to (179.3, 173.9)
- moved C15 121.0 mm to (179.3, 180.5)
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Connections:
- C30 pad 1: /POWER/+15V -> /INPUTVOL/+5VA
- C31 pad 2: /POWER/-15V -> /INPUTVOL/-5VA
- C32 pad 1: /POWER/-15V -> /INPUTVOL/-5VA
- C33 pad 1: /POWER/+15V -> /INPUTVOL/+5VA
- J2 pad 1: unconnected-(J2-Pin_1-Pad1) -> /CONTROL/+5VD
- R34 pad 1: /POWER/+15V -> /INPUTVOL/+5VA
- R37 pad 2: /POWER/-15V -> /INPUTVOL/-5VA
- U5 pad 10: /POWER/+15V -> /INPUTVOL/+5VA
- U5 pad 6: /POWER/-15V -> /INPUTVOL/-5VA
Routing:
- net /PROTECT/L-IN: track 0.00 -> 93.2 mm
- net /PROTECT/R-IN: track 0.00 -> 64.6 mm
- net Net-(D1-K): track 0.00 -> 21.6 mm
- net Net-(IC1-VIN): track 18.4 -> 38.6 mm, vias 2 -> 3
- net Net-(D12-A): track 0.00 -> 13.8 mm
- net Net-(D14-K): track 0.00 -> 12.8 mm
- net Net-(J20-P1-Pad1): track 0.00 -> 12.6 mm
- net Net-(J19-P1-Pad1): track 0.00 -> 11.7 mm
- net Net-(D12-K): track 0.00 -> 10.6 mm
- net Net-(D13-K): track 0.00 -> 10.6 mm
- net /CONTROL/+5VD: track 6.87 -> 14.9 mm
- net /POWER/-15V: track 7.33 -> 0.00 mm
- net /INPUTVOL/-5VA: track 4.58 -> 11.9 mm
- net /INPUTVOL/+5VA: track 4.62 -> 11.6 mm
- net /POWER/+15V: track 7.02 -> 0.00 mm
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