File: InputSwitch/Power.kicad_sch (KiCad schematic)
At the start: 14 parts, among them J7 12V POWER, U1 R-78K5.0-2.0

Commit message: commit
Parts:
- added C11: 22uF, Capacitor_SMD:C_1206_3216Metric_Pad1.33x1.80mm_HandSolder, symbol Device:C
- added L1: 4.7uH, Inductor_SMD:L_1008_2520Metric, symbol Device:L
- C2: value 10uF -> 22uF; MPN (none) -> CL31A226KAHNNNE
Connections:
- net +12V: now also L1.1; no longer U1.1 (VIN)
- net GND: now also C11.2
- new net BUCK_VIN_FILTERED: C11.1, L1.2, U1.1 (VIN)
Other:
- note added: "RECOM single-stage input EMI filter (nominal Class-A reference values). L1: Murata 1239AS-H-4R7M=P2; C2/C11: Samsung CL31A226KAHNNNE. Keep C11 directly at U1 VIN/GND; short loop. C1 retained upstream. MLCC DC bias, startup/ringing and system EMC remain unqualified. Filter feeds U1 only; relay/trigger +12V stays upstream."
