File: InputSwitch/Control.kicad_sch (KiCad schematic)
At the start: 27 parts, among them J10 POWER RLY, J11 Marantz LED, J12 PreAmp LED, J13 SUB TRIGGER 12V, J8 UPDI / +5V / GND, J9 PRE / COM / MTZ, K1 G6K-2P-Y DC5, K2 G6K-2P-Y DC5, K3 G6K-2P-Y DC5, K4 G6K-2P-Y DC5, U2 ATtiny412, U3 ULN2003A, U4 ULN2003A, U9 SN74LVC1G04

Commit message: more work
Parts:
- K1, K2, K3: footprint Relay_THT:Relay_DPDT_Omron_G6K-2P-Y -> InputSwitch:Relay_DPDT_Omron_G6K-2P-Y_Datasheet
Changed lines of the file:
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@@
 			)
 		)
-		(property "Footprint" "Relay_THT:Relay_DPDT_Omron_G6K-2P-Y"
+		(property "Footprint" "InputSwitch:Relay_DPDT_Omron_G6K-2P-Y_Datasheet"
 			(at 182.88 190.5 0)
 			(hide yes)
@@
 			)
 		)
-		(property "Footprint" "Relay_THT:Relay_DPDT_Omron_G6K-2P-Y"
+		(property "Footprint" "InputSwitch:Relay_DPDT_Omron_G6K-2P-Y_Datasheet"
 			(at 199.39 190.5 0)
 			(hide yes)
@@
 			)
 		)
-		(property "Footprint" "Relay_THT:Relay_DPDT_Omron_G6K-2P-Y"
+		(property "Footprint" "InputSwitch:Relay_DPDT_Omron_G6K-2P-Y_Datasheet"
 			(at 214.63 190.5 0)
 			(hide yes)
