File: InputSwitch/InputSwitch.kicad_pcb (KiCad board)
At the start: 4 copper layers, 100 x 100 mm, 107 parts, among them J1 PREAMP L, J10 POWER RLY, J11 Marantz LED, J12 PreAmp LED, J13 SUB TRIGGER 12V, J2 MARANTZ L, J3 PREAMP R, J4 MARANTZ R, J5 OUT L, J6 OUT R, J7 12V POWER, J8 UPDI / +5V / GND, J9 PRE / COM / MTZ, K1 G6K-2P-Y DC5, K2 G6K-2P-Y DC5, K3 G6K-2P-Y DC5, K4 G6K-2P-Y DC5, Q2 BC549, Q3 BC549, U1 R-78K5.0-2.0, U10 SPU03L-05, U11 SPU03L-05, U2 ATtiny412, U3 ULN2003A, U4 ULN2003A, U5 LM358N, U6 VO617A-3, U7 LM358N, U8 VO617A-3, U9 SN74LVC1G04

Commit message: commit
Parts:
- added C11: 22uF, Capacitor_SMD:C_1206_3216Metric_Pad1.33x1.80mm_HandSolder, F.Cu at (70.5, 125.6)
- added L1: 4.7uH, Inductor_SMD:L_1008_2520Metric, F.Cu at (78.1, 130.6)
- C2: value 10uF -> 22uF
- U5, U7: footprint Package_DIP:DIP-8_W7.62mm -> Package_DIP:DIP-8_W7.62mm_Socket
- moved C2 12.7 mm to (82.7, 130.2), turned to 0 degrees
- moved D1 3.17 mm to (76.1, 134.5)
- moved D2 2.69 mm to (83.8, 134.0)
- moved G*** 2.45 mm to (151.1, 112.9)
Connections:
- U1 pad 1: +12V -> /12V input and 5V buck supply/BUCK_VIN_FILTERED
Routing:
- net /12V input and 5V buck supply/BUCK_VIN_FILTERED: track 0.00 -> 15.8 mm
- net +12V: track 73.0 -> 88.7 mm, vias 2 -> 7
- net GND: vias 125 -> 131
- removed copper zone on F.Cu, net +12V
Other:
- board text added: "Reference"
- board text added: "Series"

Commit message: more
Parts:
- moved J9 0.11 mm to (67.1, 115.0)
Routing:
- net K4_LOW: track 39.0 -> 38.3 mm
Other:
- board text removed: "G 12V"
Changed lines of the file:
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@@
 	(footprint "Connector_JST:JST_XH_B3B-XH-A_1x03_P2.50mm_Vertical"
 		(layer "F.Cu")
-		(at 66.946 114.959 -90)
+		(at 67.056 114.959 -90)
 		(descr "JST XH series connector, B3B-XH-A (http://www.jst-mfg.com/product/pdf/eng/eXH.pdf)")
 		(tags "connector JST XH vertical")
@@
 		)
 		(property "Value" "PRE / COM / MTZ"
-			(at 2.5 4.6 90)
+			(at 2.516 4.572 90)
 			(layer "F.SilkS")
 			(effects
@@
 		)
 	)
-	(gr_text "G   12V"
+	(gr_text "-    +"
 		(at 81.788 77.724 0)
 		(layer "F.SilkS")
@@
 	)
 	(segment
-		(start 83.742213 98.815787)
+		(start 82.866774 99.691226)
 		(end 82.3135 100.2445)
 		(width 0.4)
@@
 	)
 	(segment
-		(start 84.328 84.648427)
-		(end 84.328 97.401573)
+		(start 84.328 85.975104)
+		(end 84.328 96.163514)
 		(width 0.4)
 		(layer "F.Cu")
 		(net "/ATtiny412 and relay drivers/SUB_TRIGGER_12V")
 	)
-	(segment
+	(arc
+		(start 84.200759 97.281942)
+		(mid 83.703199 98.580374)
+		(end 82.866774 99.691226)
+		(width 0.4)
+		(layer "F.Cu")
+		(net "/ATtiny412 and relay drivers/SUB_TRIGGER_12V")
+	)
+	(arc
 		(start 82.804 82.296)
-		(end 83.742214 83.234214)
+		(mid 83.683333 83.466595)
+		(end 84.201805 84.835807)
 		(width 0.4)
 		(layer "F.Cu")
@@
 	)
 	(arc
-		(start 84.328 84.648427)
-		(mid 84.175759 83.88306)
-		(end 83.742214 83.234214)
+		(start 84.201805 84.835807)
+		(mid 84.296409 85.401968)
+		(end 84.328 85.975104)
 		(width 0.4)
 		(layer "F.Cu")
@@
 	)
 	(arc
-		(start 84.328 97.401573)
-		(mid 84.175759 98.16694)
-		(end 83.742213 98.815787)
+		(start 84.328 96.163514)
+		(mid 84.296148 96.726349)
+		(end 84.200759 97.281942)
 		(width 0.4)
 		(layer "F.Cu")
@@
 	)
 	(segment
-		(start 112.342576 106.961981)
-		(end 111.737735 106.35714)
+		(start 112.358051 106.977631)
+		(end 112.394352 107.014342)
 		(width 0.4)
 		(layer "F.Cu")
@@
 	)
 	(segment
-		(start 97.568576 104.599781)
-		(end 95.042756 102.073961)
+		(start 113.221256 109.081359)
+		(end 113.221256 109.607461)
 		(width 0.4)
 		(layer "F.Cu")
@@
 	)
 	(segment
-		(start 109.616415 105.478461)
-		(end 99.689897 105.478461)
+		(start 112.342576 106.961981)
+		(end 112.358051 106.977631)
+		(width 0.4)
+		(layer "F.Cu")
+		(net "K1_LOW")
+	)
+	(segment
+		(start 99.689897 105.478461)
+		(end 108.76107 105.478461)
 		(width 0.4)
 		(layer "F.Cu")
@@
 	)
 	(segment
-		(start 113.221256 109.607461)
-		(end 113.221256 109.083302)
+		(start 95.042756 102.073961)
+		(end 97.568576 104.599781)
 		(width 0.4)
 		(layer "F.Cu")
@@
 	)
 	(arc
-		(start 109.616415 105.478461)
-		(mid 110.764465 105.706822)
-		(end 111.737735 106.35714)
+		(start 110.516423 105.792866)
+		(mid 111.492656 106.278728)
+		(end 112.342576 106.961981)
 		(width 0.4)
 		(layer "F.Cu")
@@
 	)
 	(arc
-		(start 99.689897 105.478461)
+		(start 97.568576 104.599781)
 		(mid 98.541846 105.250099)
-		(end 97.568576 104.599781)
+		(end 99.689897 105.478461)
 		(width 0.4)
 		(layer "F.Cu")
@@
 	)
 	(arc
-		(start 113.221256 109.083302)
-		(mid 112.992894 107.935251)
-		(end 112.342576 106.961981)
+		(start 108.76107 105.478461)
+		(mid 109.652757 105.557563)
+		(end 110.516423 105.792866)
+		(width 0.4)
+		(layer "F.Cu")
+		(net "K1_LOW")
+	)
+	(arc
+		(start 112.394352 107.014342)
+		(mid 113.006862 107.968218)
+		(end 113.221256 109.081359)
 		(width 0.4)
 		(layer "F.Cu")
@@
 	)
 	(segment
-		(start 82.55 141.13525)
-		(end 82.56175 141.1235)
-		(width 0.4)
-		(layer "F.Cu")
-		(net "UPDI")
-	)
-	(segment
-		(start 69.168 96.6)
-		(end 70.485 97.917)
+		(start 67.305535 96.6)
+		(end 67.056 96.6)
 		(width 0.4)
 		(layer "F.Cu")
@@
 	)
 	(segment
-		(start 67.056 96.6)
-		(end 69.168 96.6)
+		(start 82.55 141.13525)
+		(end 82.56175 141.1235)
 		(width 0.4)
 		(layer "F.Cu")
@@
 		(net "UPDI")
 	)
+	(arc
+		(start 70.485 97.917)
+		(mid 69.862353 97.39771)
+		(end 69.156489 96.998865)
+		(width 0.4)
+		(layer "F.Cu")
+		(net "UPDI")
+	)
+	(arc
+		(start 69.156489 96.998865)
+		(mid 68.252236 96.700988)
+		(end 67.305535 96.6)
+		(width 0.4)
+		(layer "F.Cu")
+		(net "UPDI")
+	)
 	(segment
 		(start 82.55 142.834528)
@@
 	)
 	(segment
+		(start 90.269026 97.720026)
+		(end 87.3935 94.8445)
+		(width 0.4)
+		(layer "F.Cu")
+		(net "K4_LOW")
+	)
+	(segment
+		(start 117.031256 110.58246)
+		(end 116.693502 110.920214)
+		(width 0.4)
+		(layer "F.Cu")
+		(net "K4_LOW")
+	)
+	(segment
 		(start 115.279289 111.506)
-		(end 102.174427 111.506)
+		(end 108.800253 111.506)
 		(width 0.4)
 		(layer "F.Cu")
@@
 	)
 	(segment
-		(start 91.44 100.393402)
-		(end 91.439549 100.308059)
+		(start 91.088571 98.844928)
+		(end 91.088271 98.844344)
 		(width 0.4)
 		(layer "F.Cu")
@@
 	)
 	(segment
-		(start 90.377641 97.828641)
-		(end 87.3935 94.8445)
+		(start 91.73267 101.656653)
+		(end 91.729037 101.64852)
 		(width 0.4)
 		(layer "F.Cu")
@@
 	)
 	(segment
-		(start 117.031256 110.58246)
-		(end 116.693502 110.920214)
+		(start 96.075047 106.235047)
+		(end 92.293148 102.453148)
 		(width 0.4)
 		(layer "F.Cu")
@@
 	)
 	(segment
-		(start 100.760213 110.920213)
-		(end 92.293148 102.453148)
+		(start 91.976902 102.079435)
+		(end 91.898564 101.963361)
+		(width 0.4)
+		(layer "F.Cu")
+		(net "K4_LOW")
+	)
+	(segment
+		(start 91.267318 99.285828)
+		(end 91.214845 99.134639)
+		(width 0.4)
+		(layer "F.Cu")
+		(net "K4_LOW")
+	)
+	(segment
+		(start 91.439549 100.308059)
+		(end 91.437037 100.221405)
 		(width 0.4)
 		(layer "F.Cu")
@@
 	)
 	(arc
-		(start 92.293148 102.453148)
-		(mid 92.061066 102.191352)
-		(end 91.861893 101.903712)
+		(start 91.729037 101.64852)
+		(mid 91.514537 100.993354)
+		(end 91.439549 100.308059)
 		(width 0.4)
 		(layer "F.Cu")
@@
 	)
 	(arc
-		(start 91.861893 101.903712)
-		(mid 91.547321 101.177492)
-		(end 91.44 100.393402)
+		(start 91.898564 101.963361)
+		(mid 91.811434 101.812277)
+		(end 91.73267 101.656653)
 		(width 0.4)
 		(layer "F.Cu")
@@
 	)
 	(arc
-		(start 91.439549 100.308059)
-		(mid 91.368212 99.672759)
-		(end 91.185647 99.060137)
+		(start 91.437037 100.221405)
+		(mid 91.434365 100.171652)
+		(end 91.429947 100.12202)
+		(width 0.4)
+		(layer "F.Cu")
+		(net "K4_LOW")
+	)
+	(arc
+		(start 91.214845 99.134639)
+		(mid 91.154281 98.988671)
+		(end 91.088571 98.844928)
 		(width 0.4)
 		(layer "F.Cu")
@@
 	)
 	(arc
-		(start 91.185647 99.060137)
-		(mid 90.844662 98.403066)
-		(end 90.377641 97.828641)
+		(start 90.82157 98.391777)
+		(mid 90.561632 98.042465)
+		(end 90.269026 97.720026)
 		(width 0.4)
 		(layer "F.Cu")
@@
 	)
 	(arc
-		(start 102.174427 111.506)
-		(mid 101.40906 111.353759)
-		(end 100.760213 110.920213)
+		(start 91.088271 98.844344)
+		(mid 90.961533 98.614164)
+		(end 90.82157 98.391777)
+		(width 0.4)
+		(layer "F.Cu")
+		(net "K4_LOW")
+	)
+	(arc
+		(start 108.800253 111.506)
+		(mid 105.593291 111.217951)
+		(end 102.489148 110.362607)
+		(width 0.4)
+		(layer "F.Cu")
+		(net "K4_LOW")
+	)
+	(arc
+		(start 102.489148 110.362607)
+		(mid 99.061047 108.642377)
+		(end 96.075047 106.235047)
+		(width 0.4)
+		(layer "F.Cu")
+		(net "K4_LOW")
+	)
+	(arc
+		(start 91.429947 100.12202)
+		(mid 91.372995 99.699219)
+		(end 91.267318 99.285828)
 		(width 0.4)
 		(layer "F.Cu")
 		(net "K4_LOW")
 	)
+	(arc
+		(start 92.293148 102.453148)
+		(mid 92.127372 102.272781)
+		(end 91.976902 102.079435)
+		(width 0.4)
+		(layer "F.Cu")
+		(net "K4_LOW")
+	)
+	(segment
+		(start 119.315221 105.478461)
+		(end 131.641115 105.478461)
+		(width 0.4)
+		(layer "F.Cu")
+		(net "K2_LOW")
+	)
+	(segment
+		(start 117.193977 106.35714)
+		(end 117.194049 106.357068)
+		(width 0.4)
+		(layer "F.Cu")
+		(net "K2_LOW")
+	)
 	(segment
-		(start 116.639936 106.911181)
+		(start 117.046493 106.504624)
 		(end 117.193977 106.35714)
 		(width 0.4)
@@
 	)
 	(segment
-		(start 119.315297 105.478461)
-		(end 131.641115 105.478461)
+		(start 117.194154 106.356963)
+		(end 117.193977 106.35714)
 		(width 0.4)
 		(layer "F.Cu")
 		(net "K2_LOW")
 	)
-	(segment
+	(arc
+		(start 131.641115 105.478461)
+		(mid 132.789166 105.2501)
+		(end 133.762436 104.599781)
+		(width 0.4)
+		(layer "F.Cu")
+		(net "K2_LOW")
+	)
+	(arc
 		(start 115.761256 109.607461)
-		(end 115.761256 109.032502)
+		(mid 116.05075 108.040075)
+		(end 116.881187 106.679654)
 		(width 0.4)
 		(layer "F.Cu")
@@
 	)
 	(arc
-		(start 115.761256 109.032502)
-		(mid 115.989618 107.884451)
-		(end 116.639936 106.911181)
+		(start 117.194049 106.357068)
+		(mid 117.820075 105.877626)
+		(end 118.549531 105.578353)
 		(width 0.4)
 		(layer "F.Cu")
@@
 	)
 	(arc
-		(start 133.762436 104.599781)
-		(mid 132.789166 105.2501)
-		(end 131.641115 105.478461)
+		(start 116.881187 106.679654)
+		(mid 116.962738 106.591101)
+		(end 117.046493 106.504624)
 		(width 0.4)
 		(layer "F.Cu")
@@
 	)
 	(arc
-		(start 117.193977 106.35714)
-		(mid 118.167247 105.706822)
-		(end 119.315297 105.478461)
+		(start 118.549531 105.578353)
+		(mid 118.929165 105.503923)
+		(end 119.315221 105.478461)
 		(width 0.4)
 		(layer "F.Cu")
@@
 		(polygon
 			(pts
-				(xy 106.1974 158.845927) (xy 106.1974 167.227927) (xy 86.8172 167.227927) (xy 86.8172 170.942) (xy 110.7694 170.942)
+				(xy 106.1974 158.845927) (xy 106.1974 167.227927) (xy 86.614 167.227927) (xy 86.614 171.069) (xy 110.7694 171.069)
 				(xy 110.7694 158.845927)
 			)
@@
 		(polygon
 			(pts
-				(xy 137.948238 154.500462) (xy 137.948238 167.200461) (xy 121.565238 167.200461) (xy 121.565238 171.264461)
+				(xy 137.948238 154.500462) (xy 137.948238 167.200461) (xy 121.438238 167.200461) (xy 121.438238 171.264461)
 				(xy 142.520238 171.264461) (xy 142.520238 154.500462)
 			)

Commit message: more work
Parts:
- K1, K2, K3: footprint Relay_THT:Relay_DPDT_Omron_G6K-2P-Y -> InputSwitch:Relay_DPDT_Omron_G6K-2P-Y_Datasheet
- moved K3 0.14 mm to (120.9, 102.2)
- moved Q3 0.09 mm to (146.6, 149.4)
Routing:
- net +5V: track 319.2 -> 324.5 mm
- net +12V: track 88.7 -> 88.0 mm
- net /12V input and 5V buck supply/BUCK_VIN_FILTERED: track 15.8 -> 16.3 mm
