File: InputSwitch/InputSwitch.kicad_sch (KiCad schematic)
At the start: 13 parts, among them J1 PREAMP L, J2 MARANTZ L, J3 PREAMP R, J4 MARANTZ R, J5 OUT L, J6 OUT R, K1 G6K-2P-Y DC5, K2 G6K-2P-Y DC5, K3 G6K-2P-Y DC5

Commit message: more work
Parts:
- K1, K2, K3: footprint Relay_THT:Relay_DPDT_Omron_G6K-2P-Y -> InputSwitch:Relay_DPDT_Omron_G6K-2P-Y_Datasheet
Changed lines of the file:
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@@
 			)
 		)
-		(property "Footprint" "Relay_THT:Relay_DPDT_Omron_G6K-2P-Y"
+		(property "Footprint" "InputSwitch:Relay_DPDT_Omron_G6K-2P-Y_Datasheet"
 			(at 119.38 167.64 0)
 			(hide yes)
@@
 			)
 		)
-		(property "Footprint" "Relay_THT:Relay_DPDT_Omron_G6K-2P-Y"
+		(property "Footprint" "InputSwitch:Relay_DPDT_Omron_G6K-2P-Y_Datasheet"
 			(at 119.38 109.22 0)
 			(hide yes)
@@
 			)
 		)
-		(property "Footprint" "Relay_THT:Relay_DPDT_Omron_G6K-2P-Y"
+		(property "Footprint" "InputSwitch:Relay_DPDT_Omron_G6K-2P-Y_Datasheet"
 			(at 279.4 76.2 0)
 			(hide yes)
@@
 			)
 		)
-		(property "Footprint" "Relay_THT:Relay_DPDT_Omron_G6K-2P-Y"
+		(property "Footprint" "InputSwitch:Relay_DPDT_Omron_G6K-2P-Y_Datasheet"
 			(at 119.38 200.66 0)
 			(hide yes)
@@
 			)
 		)
-		(property "Footprint" "Relay_THT:Relay_DPDT_Omron_G6K-2P-Y"
+		(property "Footprint" "InputSwitch:Relay_DPDT_Omron_G6K-2P-Y_Datasheet"
 			(at 279.4 167.64 0)
 			(hide yes)
@@
 			)
 		)
-		(property "Footprint" "Relay_THT:Relay_DPDT_Omron_G6K-2P-Y"
+		(property "Footprint" "InputSwitch:Relay_DPDT_Omron_G6K-2P-Y_Datasheet"
 			(at 119.38 76.2 0)
 			(hide yes)
