File: TWALib.kicad_blocks/TPS7A39.kicad_block/TPS7A39.kicad_sch (KiCad schematic)
At the start: 12 parts, among them U8 TPS7A39*

Commit message: commit
Parts:
- removed U8: TPS7A39*, Package_SON:Texas_S-PVSON-N10_ThermalVias, symbol Regulator_Linear:TPS7A39
- added U7: TPS7A39*, Package_SON:Texas_S-PVSON-N10_ThermalVias, symbol Regulator_Linear:TPS7A39
- C59, C65, C70: value 10nF -> 10nF*
- C73, C78: value 10uf 25V -> 10uf 25V*
- C79, C80: value 10uF -> 10uf 50V*
- R43, R56: value 10K -> 10K*
- R57: value 115K -> 115K*
- R58: value 127K -> 127K*
Connections:
- net GND: now also U7.11 (GND), U7.4 (GND)
- net at C65.1, R43.2, R58.1: now also U7.7 (FBN)
- net VEE: now reaches C80.1
- net VEE: now also U7.5 (INN)
- net at C59.2, R56.1, R57.2: now also U7.9 (FBP)
- net at C70.1: now also U7.3 (NR/SS)
- net at R43.1: now also U7.8 (BUF)
- net VCC: now reaches C79.1
- net VCC: now also U7.1 (INP), U7.2 (EN)
- net +5VA renamed +15V
- net +15V: now also U7.10 (OUTP)
- net -5VA renamed -15V
- net -15V: now also U7.6 (OUTN)
