File: StreamerIsolater/StreamerIsolater.kicad_sch (KiCad schematic)
At the start: 30 parts, among them IC2 USBLC6, J1 USB-A1HSW6, J16 POWER IN, J17 PI POWER, J2 SYSTEM CONNECTOR, J3 USB-B CONNECTOR, Q1 2N7002, U1 ISOUSB211, U10 SPU03L-05, U2 ATtiny412, U3 TPS7A2050, U4 TPS22975NDSGR, U5 TPS7A2033, U6 TPS7A2033, U7 TPS7A2033

Commit message: more
Parts:
- added C14, C17, C33, C34: 10uF, Capacitor_SMD:C_1206_3216Metric_Pad1.33x1.80mm_HandSolder, symbol Device:C
- added C15, C18, C20, C23, C26, C29, C35: 100nF, Capacitor_SMD:C_0603_1608Metric_Pad1.08x0.95mm_HandSolder, symbol Device:C
- added C16: 47uF, Capacitor_THT:CP_Radial_D5.0mm_P2.00mm, symbol Device:C_Polarized
- added C19, C22, C25, C28: 2.2uF, Capacitor_SMD:C_0805_2012Metric_Pad1.18x1.45mm_HandSolder, symbol Device:C
- added C21, C24, C27, C30: 10nF, Capacitor_SMD:C_0805_2012Metric_Pad1.18x1.45mm_HandSolder, symbol Device:C
- added C31: 1nF, Capacitor_SMD:C_0805_2012Metric_Pad1.18x1.45mm_HandSolder, symbol Device:C
- added C32: 220uF, Capacitor_THT:CP_Radial_D6.3mm_P2.50mm, symbol Device:C_Polarized
- added C36, C37: 1uF, Capacitor_SMD:C_0805_2012Metric_Pad1.18x1.45mm_HandSolder, symbol Device:C
- added D1, D2: LED, LED_SMD:LED_0805_2012Metric_Pad1.15x1.40mm_HandSolder, symbol Device:LED
- added F1: T4A, Fuse:Fuse_Littelfuse_395Series, symbol Device:Fuse
- added H1, H2, H3, H4: MountingHole, MountingHole:MountingHole_3.2mm_M3, symbol Mechanical:MountingHole
- added J4: UPDI, Connector_PinHeader_2.54mm:PinHeader_1x03_P2.54mm_Vertical, symbol Connector_Generic:Conn_01x03
- added R3: 100K, Resistor_SMD:R_0805_2012Metric_Pad1.20x1.40mm_HandSolder, symbol Device:R
- added R4: 1K, Resistor_SMD:R_0805_2012Metric_Pad1.20x1.40mm_HandSolder, symbol Device:R
- added R5, R7: 10K, Resistor_SMD:R_0805_2012Metric_Pad1.20x1.40mm_HandSolder, symbol Device:R
- added R6: 390R, Resistor_SMD:R_0805_2012Metric_Pad1.20x1.40mm_HandSolder, symbol Device:R
- added R8, R9: 680R, Resistor_SMD:R_0805_2012Metric_Pad1.20x1.40mm_HandSolder, symbol Device:R
- C1, C12, C13, C2, C3, C5, C6, C7, C8, C9: footprint Capacitor_SMD:C_1206_3216Metric_Pad1.33x1.80mm_HandSolder -> Capacitor_SMD:C_0805_2012Metric_Pad1.18x1.45mm_HandSolder; DigiKey Part Number (none) -> 1276-6469-1-ND; Manufacturer_Name (none) -> Samsung Electro-Mechanics; Manufacturer_Part_Number (none) -> CL21B105KAFNNNG
- C10, C11, C4: footprint Capacitor_SMD:C_1206_3216Metric_Pad1.33x1.80mm_HandSolder -> Capacitor_SMD:C_0603_1608Metric_Pad1.08x0.95mm_HandSolder; DigiKey Part Number (none) -> 399-C0603C104M5RACTUCT-ND; Manufacturer_Name (none) -> KEMET; Manufacturer_Part_Number (none) -> C0603C104M5RACTU
- J16: value POWER IN -> POWER IN 5V
- J17: value PI POWER -> PI POWER OUT 5V
- U4: value TPS22975NDSGR -> TPS22975; footprint DSG0008B -> Custom:DSG0008B
Connections:
- net 3V3-CLEAN: now also U1.16 (CDPEN2_N), C37.1
- net 3V3-DIRTY: now also U1.13 (CDPEN1_N), C36.1
- net 3V3-TINY: now also J4.1 (Pin_1), R5.1
- net 5V_SWITCHED: now also C5.1, U10.1 (VIN+), U5.1 (IN), U5.3 (EN), C14.1, C15.1, C34.1
- net GND: now also U1.19 (EQ21), U1.20 (EQ20), C16.2, C17.2, C18.2, C25.2, C26.2, C27.2, C28.2, C29.2, C30.2, C37.2, D2.1 (K); no longer C12.2, C13.2, C3.2, C4.2, C5.2, C6.2, U5.2 (GND), U7.2 (GND)
- net GNDD: now also C12.2, C13.2, C3.2, C4.2, C5.2, C6.2, J3.5 (Shield), U1.10 (EQ11), U1.9 (EQ10), U5.2 (GND), U7.2 (GND), C14.2, C15.2, C19.2, C20.2, C21.2, C22.2, C23.2, C24.2, C31.2, C32.2, C33.2, C34.2, C35.2, C36.2, D1.1 (K), J4.3 (Pin_3), R3.2
- net PI_SAFE_TO_OFF: now also R7.1; no longer R2.1, U2.7 (PA3)
- net POWER-IN: now also C32.1, C33.1, F1.2; no longer J16.2 (Pin_2)
- net POWER_BUTTON: now also C35.1, R4.2, R5.2; no longer J2.4 (Pin_4)
- net PROG: now also J4.2 (Pin_2)
- net STATUS_LED: now also R6.1; no longer J2.2 (Pin_2)
- net UNREG-CLEAN: now also C16.1
- net XMOS-VBUS: now also C17.1, C18.1
- net at Q1.1 (G), U2.5 (PA2): now also R3.1
- net PI_BUTTON2: now reaches J2.8 (Pin_8)
- net at U4.6 (CT): now also C31.1
- net 1V8_ISO1: now reaches U1.11 (V1P8V1)
- net 1V8_ISO1: now also U1.4 (V1P8V1), C19.1, C20.1, C21.1, C22.1, C23.1, C24.1
- net 1V8_ISO2: now reaches U1.18 (V1P8V2)
- net 1V8_ISO2: now also U1.25 (V1P8V2), C25.1, C26.1, C27.1, C28.1, C29.1, C30.1
- net V1OK: now reaches U1.23 (V1OK)
- net V1OK: now also R9.1
- net V2OK: now reaches U1.6 (V2OK)
- net V2OK: now also R8.1
- net USB_XMOS_N1 renamed USB_XMOS1_N
- net USB_XMOS1_N: now also IC2.1 (I/O1_1); no longer IC2.3 (I/O2_1)
- net USB_XMOS_N2 renamed USB_XMOS2_N
- net USB_XMOS2_N: now also IC2.6 (I/O1_2); no longer IC2.4 (I/O2_2)
- net USB_XMOS_P1 renamed USB_XMOS1_P
- net USB_XMOS1_P: now also IC2.3 (I/O2_1); no longer IC2.1 (I/O1_1)
- net USB_XMOS_P2 renamed USB_XMOS2_P
- net USB_XMOS2_P: now also IC2.4 (I/O2_2); no longer IC2.6 (I/O1_2)
- new net: D1.2 (A), R8.2
- new net: D2.2 (A), R9.2
- new net FP_POWER_BTN: J2.4 (Pin_4), R4.1
- new net FP_STATUS_LED: J2.2 (Pin_2), R6.2
- new net SAFE_TO_OFF_IN: R2.1, R7.2, U2.7 (PA3)
- new net VIN_RAW: F1.1, J16.2 (Pin_2)
- no-connect marks 0 -> 3
Other:
- note added: "C36 at U1 pin 5 VCC1 -> pin 3 GND1; C37 at U1 pin 24 VCC2 -> pin 26 GND2 (per ISOUSB211DPEVM C22/C31). Smallest loop, no vias."
- note added: "F1: T4A time-lag TE5 (Littelfuse 39214000000, DigiKey F5505CT-ND), at J16 ahead of U4/U7. Supply RS-25-5 (5 A, hiccup at 110-180 %). F1 clears sustained faults above TPS22975 6 A rating. Keep RS-25 at 5.1 V."
- note added: "Front-panel / Pi GPIO interface (all GNDD)"
- note added: "ISOLATION: GNDD (Pi side) and GND (isolated USB side) must never join. Only U1 and U10 straddle the barrier. J1 shell is not connected (NPTH pegs only): J1 must not contact an earthed / GNDD-bonded panel."
- note added: "ISOUSB211 internal 1.8 V LDO outputs (VCCx = 3.3 V). Per TI SLLSFC5D sec. 8.3: one 2.2u + 100n + 10n set at EACH V1P8V pin, smallest value closest, no vias between cap and pin/GND pin. Join pin 4 to 11 (and 18 to 25) AFTER the caps, on an inner/bottom layer. Side 1 = GNDD (Pi), side 2 = GND (isolated)."
- note added: "ISOUSB211 power-good LEDs: D1 = side 2 up (Pi side, GNDD), D2 = side 1 up (isolated, GND). V*OK VOH = V3P3Vx-0.2 V @ 3 mA, abs max 10 mA. Use 570 nm GaP green (Vf ~2.1 V): 680R gives ~1.5 mA. Do NOT fit an InGaN green (Vf ~3 V)."
- note added: "Pi config.txt (verify on target): dtoverlay=gpio-shutdown,gpio_pin=23,active_low=1,gpio_pull=up dtoverlay=gpio-poweroff,gpiopin=22,active_low=0 GPIO23 (PI_SHUTDOWN_REQ): Q1 open drain, Pi internal pull-up. Pulse LOW >= 500 ms. GPIO22 (PI_SAFE_TO_OFF): LOW at reset (BCM pull-down + R2) and while running; driven HIGH only by gpio-poweroff after halt. Keep EEPROM POWER_OFF_ON_HALT=0 so 3V3 stays up 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"
- note added: "Place 220u at J16; 10u at U4 VIN/VBIAS; 10u at U4 VOUT"
- note added: "Place at J1 / IC2 VBUS pin"
- note added: "UPDI: 1 VTG 2 UPDI 3 GND"
- note added: "pins 11/12"
- note added: "pins 18/17"
- note added: "pins 25/26"
- note added: "pins 4/3"
- note removed: "NC"
