File: StreamerIsolater/StreamerIsolater.kicad_pcb (KiCad board)
At the start: 4 copper layers, 77 x 60 mm, 32 parts, among them IC2 USBLC6, J1 USB-A1HSW6, J16 POWER IN, J17 PI POWER, J2 POWER IN, J2 SYSTEM CONNECTOR, J3 USB-B CONNECTOR, Q1 2N7002, U1 ISOUSB211, U10 SPU03L-05, U2 ATtiny412, U3 TPS7A2050, U4 TPS22975NDSGR, U5 TPS7A2033, U6 TPS7A2033, U7 TPS7A2033

Commit message: more
Parts:
- removed the J2 at (245.7, 119.2)
- removed the J2 at (117.1, 69.9)
- added C14: 10uF, Capacitor_SMD:C_1206_3216Metric_Pad1.33x1.80mm_HandSolder, F.Cu at (167.4, 106.6)
- added C15: 100nF, Capacitor_SMD:C_0603_1608Metric_Pad1.08x0.95mm_HandSolder, F.Cu at (171.6, 108.7)
- added C16: 47uF, Capacitor_THT:CP_Radial_D5.0mm_P2.00mm, F.Cu at (194.8, 104.1)
- added C17: 10uF, Capacitor_SMD:C_1206_3216Metric_Pad1.33x1.80mm_HandSolder, F.Cu at (195.3, 130.8)
- added C18: 100nF, Capacitor_SMD:C_0603_1608Metric_Pad1.08x0.95mm_HandSolder, F.Cu at (196.0, 128.1)
- added C19: 2.2uF, Capacitor_SMD:C_0805_2012Metric_Pad1.18x1.45mm_HandSolder, F.Cu at (168.9, 127.6)
- added C20: 100nF, Capacitor_SMD:C_0603_1608Metric_Pad1.08x0.95mm_HandSolder, F.Cu at (170.8, 127.4)
- added C21: 10nF, Capacitor_SMD:C_0805_2012Metric_Pad1.18x1.45mm_HandSolder, F.Cu at (172.6, 121.0)
- added C22: 2.2uF, Capacitor_SMD:C_0805_2012Metric_Pad1.18x1.45mm_HandSolder, F.Cu at (168.8, 120.9)
- added C23: 100nF, Capacitor_SMD:C_0603_1608Metric_Pad1.08x0.95mm_HandSolder, F.Cu at (170.7, 121.2)
- added C24: 10nF, Capacitor_SMD:C_0805_2012Metric_Pad1.18x1.45mm_HandSolder, F.Cu at (172.7, 127.6)
- added C25: 2.2uF, Capacitor_SMD:C_0805_2012Metric_Pad1.18x1.45mm_HandSolder, F.Cu at (190.2, 127.7)
- added C26: 100nF, Capacitor_SMD:C_0603_1608Metric_Pad1.08x0.95mm_HandSolder, F.Cu at (188.5, 121.2)
- added C27: 10nF, Capacitor_SMD:C_0805_2012Metric_Pad1.18x1.45mm_HandSolder, F.Cu at (186.6, 121.0)
- added C28: 2.2uF, Capacitor_SMD:C_0805_2012Metric_Pad1.18x1.45mm_HandSolder, F.Cu at (190.4, 120.9)
- added C29: 100nF, Capacitor_SMD:C_0603_1608Metric_Pad1.08x0.95mm_HandSolder, F.Cu at (188.3, 127.4)
- added C30: 10nF, Capacitor_SMD:C_0805_2012Metric_Pad1.18x1.45mm_HandSolder, F.Cu at (186.4, 127.6)
- added C31: 1nF, Capacitor_SMD:C_0805_2012Metric_Pad1.18x1.45mm_HandSolder, F.Cu at (159.8, 95.1)
- added C32: 220uF, Capacitor_THT:CP_Radial_D6.3mm_P2.50mm, F.Cu at (151.5, 100.5)
- added C33: 10uF, Capacitor_SMD:C_1206_3216Metric_Pad1.33x1.80mm_HandSolder, F.Cu at (160.9, 99.8)
- added C34: 10uF, Capacitor_SMD:C_1206_3216Metric_Pad1.33x1.80mm_HandSolder, F.Cu at (154.4, 93.2)
- added C35: 100nF, Capacitor_SMD:C_0603_1608Metric_Pad1.08x0.95mm_HandSolder, F.Cu at (166.0, 95.8)
- added C36: 1uF, Capacitor_SMD:C_0805_2012Metric_Pad1.18x1.45mm_HandSolder, F.Cu at (176.4, 131.7)
- added C37: 1uF, Capacitor_SMD:C_0805_2012Metric_Pad1.18x1.45mm_HandSolder, F.Cu at (182.8, 131.7)
- added D1: LED, LED_SMD:LED_0805_2012Metric_Pad1.15x1.40mm_HandSolder, F.Cu at (164.6, 120.9)
- added D2: LED, LED_SMD:LED_0805_2012Metric_Pad1.15x1.40mm_HandSolder, F.Cu at (194.6, 120.8)
- added F1: T4A, Fuse:Fuse_Littelfuse_395Series, F.Cu at (140.7, 100.5)
- added H1: MountingHole, MountingHole:MountingHole_3.2mm_M3, F.Cu at (140.7, 131.1)
- added H2: MountingHole, MountingHole:MountingHole_3.2mm_M3, F.Cu at (210.8, 131.1)
- added H3: MountingHole, MountingHole:MountingHole_3.2mm_M3, F.Cu at (140.6, 85.2)
- added H4: MountingHole, MountingHole:MountingHole_3.2mm_M3, F.Cu at (210.8, 85.1)
- added J2: SYSTEM CONNECTOR, Connector_JST:JST_XH_B8B-XH-A_1x08_P2.50mm_Vertical, F.Cu at (157.3, 85.3)
- added J4: UPDI, Connector_PinHeader_2.54mm:PinHeader_1x03_P2.54mm_Vertical, F.Cu at (164.1, 131.2)
- added R3: 100K, Resistor_SMD:R_0805_2012Metric_Pad1.20x1.40mm_HandSolder, F.Cu at (174.0, 96.0)
- added R4: 1K, Resistor_SMD:R_0805_2012Metric_Pad1.20x1.40mm_HandSolder, F.Cu at (164.8, 92.3)
- added R5: 10K, Resistor_SMD:R_0805_2012Metric_Pad1.20x1.40mm_HandSolder, F.Cu at (167.0, 92.3)
- added R6: 390R, Resistor_SMD:R_0805_2012Metric_Pad1.20x1.40mm_HandSolder, F.Cu at (160.8, 91.3)
- added R7: 10K, Resistor_SMD:R_0805_2012Metric_Pad1.20x1.40mm_HandSolder, F.Cu at (169.8, 92.3)
- added R8: 680R, Resistor_SMD:R_0805_2012Metric_Pad1.20x1.40mm_HandSolder, F.Cu at (166.8, 120.9)
- added R9: 680R, Resistor_SMD:R_0805_2012Metric_Pad1.20x1.40mm_HandSolder, F.Cu at (192.5, 120.9)
- C1, C12, C13, C2, C3, C5, C6, C7, C8, C9: footprint Capacitor_SMD:C_1206_3216Metric_Pad1.33x1.80mm_HandSolder -> Capacitor_SMD:C_0805_2012Metric_Pad1.18x1.45mm_HandSolder
- C10, C11, C4: footprint Capacitor_SMD:C_1206_3216Metric_Pad1.33x1.80mm_HandSolder -> Capacitor_SMD:C_0603_1608Metric_Pad1.08x0.95mm_HandSolder
- J16: value POWER IN -> POWER IN 5V
- J17: value PI POWER -> PI POWER OUT 5V
- U4: value TPS22975NDSGR -> TPS22975
- moved C5 70.7 mm to (168.7, 112.7), turned to 90 degrees
- moved C6 64.6 mm to (175.0, 112.7), turned to -90 degrees
- moved C4 64.6 mm to (174.8, 117.8), turned to 90 degrees
- moved C3 62.7 mm to (176.8, 117.0), turned to 90 degrees
- moved U6 60.7 mm to (188.5, 112.5)
- moved C9 58.4 mm to (182.4, 117.0), turned to 90 degrees
- moved C10 57.1 mm to (184.3, 118.0), turned to 90 degrees
- moved C7 52.8 mm to (188.3, 109.3), turned to 180 degrees
- moved C8 51.9 mm to (188.6, 115.7), turned to 180 degrees
- moved C13 49.1 mm to (168.3, 102.7), turned to -90 degrees
- moved C12 45.6 mm to (164.8, 99.1)
- moved R2 40.8 mm to (162.3, 116.3), turned to -90 degrees
- moved J16 40.2 mm to (144.3, 109.6), turned to 90 degrees
- moved U7 40.1 mm to (164.9, 102.1)
- moved U5 34.8 mm to (171.8, 113.1)
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Connections:
- net /PI_SAFE_TO_OFF renamed /SAFE_TO_OFF_IN
- C12 pad 2: GND -> GNDD
- C13 pad 2: GND -> GNDD
- C3 pad 2: GND -> GNDD
- C4 pad 2: GND -> GNDD
- C5 pad 1: Net-(U5-EN) -> /5V_SWITCHED
- C5 pad 2: GND -> GNDD
- C6 pad 2: GND -> GNDD
- IC2 pad 1: /USB_XMOS_P1 -> /USB_XMOS1_N
- IC2 pad 3: /USB_XMOS_N1 -> /USB_XMOS1_P
- IC2 pad 4: /USB_XMOS_N2 -> /USB_XMOS2_P
- IC2 pad 6: /USB_XMOS_P2 -> /USB_XMOS2_N
- J1 pad 2: /USB_XMOS_N2 -> /USB_XMOS2_N
- J1 pad 3: /USB_XMOS_P2 -> /USB_XMOS2_P
- J16 pad 2: /POWER-IN -> /VIN_RAW
- J3 pad 5: unconnected-(J3-Shield-Pad5) -> GNDD
- U1 pad 10: unconnected-(U1-EQ11-Pad10) -> GNDD
- U1 pad 11: unconnected-(U1-V1P8V1-Pad11) -> /1V8_ISO1
- U1 pad 13: unconnected-(U1-CDPEN1_N-Pad13) -> /3V3-DIRTY
- U1 pad 16: unconnected-(U1-CDPEN2_N-Pad16) -> /3V3-CLEAN
- U1 pad 18: unconnected-(U1-V1P8V2-Pad18) -> /1V8_ISO2
- U1 pad 19: unconnected-(U1-EQ21-Pad19) -> GND
- U1 pad 20: unconnected-(U1-EQ20-Pad20) -> GND
- U1 pad 21: /USB_XMOS_P1 -> /USB_XMOS1_P
- U1 pad 22: /USB_XMOS_N1 -> /USB_XMOS1_N
- U1 pad 23: unconnected-(U1-V1OK-Pad23) -> /V1OK
- U1 pad 25: unconnected-(U1-V1P8V2-Pad25) -> /1V8_ISO2
- U1 pad 4: unconnected-(U1-V1P8V1-Pad4) -> /1V8_ISO1
- U1 pad 6: unconnected-(U1-V2OK-Pad6) -> /V2OK
- U1 pad 9: unconnected-(U1-EQ10-Pad9) -> GNDD
- U10 pad 1: unconnected-(U10-VIN+-Pad1) -> /5V_SWITCHED
- U4 pad 6: unconnected-(U4-CT-Pad6) -> Net-(U4-CT)
- U4 pad V: (no net) -> GNDD
- U5 pad 1: Net-(U5-EN) -> /5V_SWITCHED
- U5 pad 2: GND -> GNDD
- U5 pad 3: Net-(U5-EN) -> /5V_SWITCHED
- U7 pad 2: GND -> GNDD
Routing:
- net /3V3-TINY: track 0.00 -> 55.7 mm, vias 0 -> 3
- net /5V_SWITCHED: track 0.00 -> 53.0 mm
- net /XMOS-VBUS: track 3.24 -> 45.0 mm, vias 0 -> 1
- net /3V3-DIRTY: track 0.00 -> 39.6 mm
- net /3V3-CLEAN: track 0.00 -> 34.8 mm
- net Net-(Q1-G): track 0.00 -> 27.9 mm, vias 0 -> 2
- net /SAFE_TO_OFF_IN: track 0.00 -> 25.0 mm, vias 0 -> 2
- net /UNREG-CLEAN: track 14.9 -> 36.3 mm
- net /POWER_BUTTON: track 0.00 -> 21.3 mm, vias 0 -> 2
- net /1V8_ISO1: track 0.00 -> 21.1 mm, vias 0 -> 2
- net /1V8_ISO2: track 0.00 -> 20.9 mm, vias 0 -> 2
- net /PROG: track 0.00 -> 18.5 mm, vias 0 -> 1
- net /STATUS_LED: track 0.00 -> 16.8 mm, vias 0 -> 2
- net /USB_XMOS2_P: track 0.00 -> 10.4 mm
- net /USB_XMOS1_N: track 0.00 -> 10.3 mm
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- added copper zone on F.Cu, net /5V_SWITCHED
- added copper zone on F.Cu, net /POWER-IN
- added copper zone on B.Cu, net /VIN_RAW
- added copper zone on In2.Cu, net /VIN_RAW
Other:
- board size 77 x 60 mm -> 77 x 52.8 mm
- board text added: "- +"
- board text added: "1"
- board text added: "1 - STATUS LED - 2 - STATUS LED + 3 - POWER BTN 1 4 - POWER BTN 2 5 - PI GND 6 - PI SAFE TO OFF 7 - PI SHUTDOWN REQ 8 - NC"
- board text added: "G P 3V3"
- board text added: "USB IN"
- board text added: "USB Isolator & Pi Control Tom Watson Audio 2026"
- board text added: "USB OUT"
- board text removed: "USB Isolator Tom Watson Audio 2026"

Commit message: more work
Parts:
- moved C29 0.05 mm to (188.3, 127.4)
Routing:
- net /3V3-DIRTY: track 39.6 -> 38.6 mm
- net GNDD: vias 62 -> 117
- net GND: vias 32 -> 81
