File: SubProcessorDigital/PROTECT.kicad_sch (KiCad schematic)
At the start: 5 parts, among them U7 TPS3850G12QDRCRQ1

Commit message: more
Parts:
- added C118, C120, C121, C122, C123: 100nF, Capacitor_SMD:C_0603_1608Metric_Pad1.08x0.95mm_HandSolder, symbol Device:C
- added C119: 10nF, Capacitor_SMD:C_0805_2012Metric_Pad1.18x1.45mm_HandSolder, symbol Device:C
- added D5: 1N4148W, Diode_SMD:D_SOD-123, symbol Diode:1N4148W
- added R48: 22K, Resistor_SMD:R_0805_2012Metric_Pad1.20x1.40mm_HandSolder, symbol Device:R
- added R49: 3K3, Resistor_SMD:R_0805_2012Metric_Pad1.20x1.40mm_HandSolder, symbol Device:R
- added R50, R53: 100K, Resistor_SMD:R_0805_2012Metric_Pad1.20x1.40mm_HandSolder, symbol Device:R
- added R51: 270K, Resistor_SMD:R_0805_2012Metric_Pad1.20x1.40mm_HandSolder, symbol Device:R
- added R52: 10K, Resistor_SMD:R_0805_2012Metric_Pad1.20x1.40mm_HandSolder, symbol Device:R
- added TP18: FAULT_N, TestPoint:TestPoint_Pad_D1.5mm, symbol Connector:TestPoint
- added TP19: SUP_RST_N, TestPoint:TestPoint_Pad_D1.5mm, symbol Connector:TestPoint
- added TP20: RLY_EN_LATCH, TestPoint:TestPoint_Pad_D1.5mm, symbol Connector:TestPoint
- added TP21: AUDIO_READY, TestPoint:TestPoint_Pad_D1.5mm, symbol Connector:TestPoint
- added TP22: WDI, TestPoint:TestPoint_Pad_D1.5mm, symbol Connector:TestPoint
- added U10, U11, U12: TPS3808G33DBVR, Package_TO_SOT_SMD:SOT-23-6, symbol SPD:TPS3808DBV_OD
- added U13: SN74AUP1G74DCUR, Package_SO:VSSOP-8_2.3x2mm_P0.5mm, symbol 74xGxx:74AUP1G74
- added U9: TPS3808G01DBVR, Package_TO_SOT_SMD:SOT-23-6, symbol SPD:TPS3808DBV_OD
- C8: footprint Capacitor_SMD:C_1206_3216Metric_Pad1.33x1.80mm_HandSolder -> Capacitor_SMD:C_0603_1608Metric_Pad1.08x0.95mm_HandSolder; MPN (none) -> Multicomp Pro MC0603B104K500CT (100nF 50V X7R 10% 1608); Notes (none) -> At U7 VDD
- R10, R11: MPN (none) -> KOA RK73B2ATTD103J (inventory)
- R9: MPN (none) -> 10k 0.1% thin film 2012 (inventory); Notes (none) -> CWD to VDD (9-11k): factory timing
- U7: value TPS3850G12QDRCRQ1 -> TPS3850H01DRCR; footprint DRC0010R -> Package_SON:VSON-10-1EP_3x3mm_P0.5mm_EP1.65x2.4mm; symbol Custom:TPS3850G12QDRCRQ1 -> SPD:TPS3850_DRC; MPN (none) -> TPS3850H01DRCR; Manufacturer (none) -> Texas Instruments; Manufacturer_Part_Number (none) -> TPS3850H01DRCR; Notes (none) -> Adjustable (0.4 V) UV-only variant. G12 = 1.2 V window: wou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
Connections:
- net GND: now also C118.2, C119.2, C120.2, C121.2, C122.2, C123.2, R49.2, R50.2, R52.2, R53.2, U10.2 (GND), U11.2 (GND), U12.2 (GND), U13.4 (GND), U9.2 (GND)
- net WATCHDOG_HEARTBEAT: now also R50.1, TP22.1
- net +3V3_ESP: now reaches R11.1
- net +3V3_ESP: now also C8.1, R10.1, R9.1, U7.1 (VDD), U7.6 (SET1), C118.1, C120.1, C121.1, C122.1, C123.1, R48.1, U10.6 (VDD), U11.6 (VDD), U12.6 (VDD), U13.2 (D), U13.7 (~{PRE}), U13.8 (VCC), U9.6 (VDD); no longer U7.8 (WDO_N)
- net SUP_RST_N: now reaches U7.9 (RESET_N)
- net SUP_RST_N: now also R10.2, D5.1 (K), TP19.1; no longer R10.1
- removed net 3V3_ESP: C8.1, R10.2, R11.2, R9.1, U7.1 (VDD), U7.10 (SENSE), U7.6 (SET1)
- new net: C119.1, R51.2, R52.1, U9.5 (SENSE)
- new net: R48.2, R49.1, U7.10 (SENSE)
- new net +15V: R51.1
- new net +3V3_A_ADC: U11.5 (SENSE)
- new net +3V3_DAC: U10.5 (SENSE)
- new net +3V3_D_ADC: U12.5 (SENSE)
- new net AUDIO_READY: R53.1, TP21.1, U13.1 (C)
- new net FAULT_N: D5.2 (A), R11.2, TP18.1, U10.1 (~{RESET}), U11.1 (~{RESET}), U12.1 (~{RESET}), U13.6 (~{CLR}), U7.8 (WDO_N), U9.1 (~{RESET})
- new net RLY_EN_LATCH: TP20.1, U13.5 (Q)
- no-connect marks 1 -> 10
Other:
- note added: "+15V falling < 0.405 x (1 + 270/10) = 11.3 V: early power-fail warning."
- note added: "A GPIO stuck high produces no new edge: after any fault the relay stays open until firmware"
- note added: "All RESET outputs are open-drain, wired-OR on FAULT_N (R11 pull-up). CT open = 20 ms release delay."
- note added: "C6 (1000 uF) then holds 5 V for ~18 ms at full load: relay is open well before any rail sags."
- note added: "ESP32 SUPERVISOR + WINDOW WATCHDOG"
- note added: "FAULT AND RESET NETS"
- note added: "FAULT_N low (any of: TPS3850 RESET via D5, TPS3850 WDO, U9 +15V, U10 DAC, U11 ADC-A, U12 ADC-D) -> Q = 0."
- note added: "Firmware arm sequence: kick WDI >= 3 windows -> read FAULT_N = 1 -> AUDIO_READY 0->1 ->"
- note added: "LATCH OPERATION"
- note added: "OUTPUT-RELAY FAULT LATCH (SN74AUP1G74, Schmitt inputs)"
- note added: "Power loss: +15V monitor trips first; latch, Q1/Q4 and coil all fail to the de-energised state."
- note added: "Q = 1 only on a RISING edge of AUDIO_READY while FAULT_N is high (D = 1)."
- note added: "RAIL SUPERVISORS (TPS3808, SENSE independent of VDD: a dead rail is still reported)"
- note added: "RESET -> ESP32 EN (via 470R). WDO -> FAULT_N only (not EN): ESP32 boot time exceeds any useful window."
- note added: "Relay coil current needs BOTH Q (Q1) and AUDIO_READY level (Q4) - see ADCESPDAC sheet."
- note added: "SENSE trip = 0.4 V x (1 + R48/R49) = 0.4 x (1 + 22/3.3) = 3.07 V falling (ESP32-S3 min 3.0 V; TS1117B min 3.235 V)."
- note added: "SET0 = 0, SET1 = 1, CWD = 10k: window 10.35 ms (max lower) .. 165.8 ms (min upper). Kick WDI every ~50 ms"
- note added: "TPS3850H01 (TI SBVS301B), DRC0010J VSON-10"
- note added: "check OUT_RLY_SENSE (IO3) low within 10 ms -> wait 20 ms -> DAC XSMT high -> ramp volume."
- note added: "drops AUDIO_READY and raises it again (after re-verifying clocks, ADC data and FAULT_N on IO42)."
- note added: "from the audio task only while audio is verified healthy. CRST open: tRST = 200 ms (RESET and WDO pulse)."
- note added: "trips if +3V3_A_ADC < 3.07 V"
- note added: "trips if +3V3_DAC < 3.07 V"
- note added: "trips if +3V3_D_ADC < 3.07 V"
- company: (none) -> P68 Subwoofer DSP Controller
- title: (none) -> Protection: supervisors, watchdog, output-relay fault latch
- moved on the sheet: C8, R10, R11, R9, U7
