File: SubProcessorDigital/ADCESPDAC.kicad_sch (KiCad schematic)
At the start: 52 parts, among them IC1 ESP32-S3-WROOM-1U-N16R8, IC2 PCM1863QDBTRQ1, IC3 USBLC6, IC4 RESET, IC5 BOOT, J3 USB PROGRAMMING, J5 OUT, J6 SYSTEM CONNECTOR, K1 AGN2004H, Q1 BC546, U2 PCM5102A

Commit message: more
Parts:
- removed C26: 2.7nF, Capacitor_SMD:C_0805_2012Metric_Pad1.18x1.45mm_HandSolder, symbol Device:C
- removed C73: 1uF, Capacitor_SMD:C_1206_3216Metric_Pad1.33x1.80mm_HandSolder, symbol Device:C
- removed IC3: USBLC6, Package_TO_SOT_SMD:SOT-23-6_Handsoldering, symbol Custom:USBLC6-2SC6
- removed J6: SYSTEM CONNECTOR, Connector_IDC:IDC-Header_2x10_P2.54mm_Vertical, symbol Connector:DIN41612_02x10_AB
- removed K1: AGN2004H, Custom:Relay_DPDT_Panasonic_AGN2004H, symbol SubController:AGN2004H
- removed R14: 470R, Resistor_SMD:R_0805_2012Metric_Pad1.20x1.40mm_HandSolder, symbol Device:R
- added C114: 100nF, Capacitor_SMD:C_0603_1608Metric_Pad1.08x0.95mm_HandSolder, symbol Device:C
- added C115, C116: 10uF, Capacitor_SMD:C_0805_2012Metric_Pad1.18x1.45mm_HandSolder, symbol Device:C
- added C117: 4.7nF, Capacitor_SMD:C_0805_2012Metric_Pad1.18x1.45mm_HandSolder, symbol Device:C
- added D4: 1N4148W, Diode_SMD:D_SOD-123, symbol Diode:1N4148W
- added IC3: USBLC6, Package_TO_SOT_SMD:SOT-23-6, symbol SPD:USBLC6-2SC6
- added K1: AGN2004H, SPD:Relay_DPDT_Panasonic_AGN2004H, symbol SPD:AGN2004H
- added Q4: BC546, Package_TO_SOT_THT:TO-92_Wide, symbol Transistor_BJT:BC546
- added R32: 22R DNP, Resistor_SMD:R_0805_2012Metric_Pad1.20x1.40mm_HandSolder, symbol Device:R
- added R33, R40, R42: 100K, Resistor_SMD:R_0805_2012Metric_Pad1.20x1.40mm_HandSolder, symbol Device:R
- added R34, R35, R36, R37: 22R, Resistor_SMD:R_0805_2012Metric_Pad1.20x1.40mm_HandSolder, symbol Device:R
- added R38: 2K, Resistor_SMD:R_0805_2012Metric_Pad1.20x1.40mm_HandSolder, symbol Device:R
- added R39: 6K8, Resistor_SMD:R_0805_2012Metric_Pad1.20x1.40mm_HandSolder, symbol Device:R
- added R41: 10K, Resistor_SMD:R_0805_2012Metric_Pad1.20x1.40mm_HandSolder, symbol Device:R
- added R43: 1K, Resistor_SMD:R_0805_2012Metric_Pad1.20x1.40mm_HandSolder, symbol Device:R
- added R44: 470R, Resistor_SMD:R_0805_2012Metric_Pad1.20x1.40mm_HandSolder, symbol Device:R
- added R45: 1M, Resistor_SMD:R_0805_2012Metric_Pad1.20x1.40mm_HandSolder, symbol Device:R
- added R46, R47: 0R, Resistor_SMD:R_0805_2012Metric_Pad1.20x1.40mm_HandSolder, symbol Device:R
- added TP11: I2S_BCK, TestPoint:TestPoint_Pad_D1.5mm, symbol Connector:TestPoint
- added TP12: I2S_LRCK, TestPoint:TestPoint_Pad_D1.5mm, symbol Connector:TestPoint
- added TP13: I2S_DIN, TestPoint:TestPoint_Pad_D1.5mm, symbol Connector:TestPoint
- added TP14: I2S_DOUT, TestPoint:TestPoint_Pad_D1.5mm, symbol Connector:TestPoint
- added TP15: DAC_XSMT, TestPoint:TestPoint_Pad_D1.5mm, symbol Connector:TestPoint
- added TP16: DAC_OUT, TestPoint:TestPoint_Pad_D1.5mm, symbol Connector:TestPoint
- added TP17: AMP_OUT, TestPoint:TestPoint_Pad_D1.5mm, symbol Connector:TestPoint
- added TP24: ESP_EN, TestPoint:TestPoint_Pad_D1.5mm, symbol Connector:TestPoint
- C1: value 10uF -> 10uF NP; MPN (none) -> Nichicon UES1H100MPM bipolar (inventory); Notes (none) -> AC coupling; ADC input biased at AVDD/2
- C18, C20: MPN (none) -> Samsung CL21B225KPFNNNE X7R (inventory)
- C19: value 2.2uF -> 1uF; footprint Capacitor_SMD:C_0805_2012Metric_Pad1.18x1.45mm_HandSolder -> Capacitor_SMD:C_1206_3216Metric_Pad1.33x1.80mm_HandSolder; MPN (none) -> Samsung CL31B105KBHNFNE (inventory); Notes (none) -> VREF: 1 uF per SLAS831D
- C2: value 10uF -> 10uF NP; MPN (none) -> Nichicon UES1H100MPM bipolar (inventory)
- C21: value 2.2uF -> 10uF; MPN (none) -> Samsung CL21A106KOQNNNF (inventory)
- C23, C66, C67, C68, C70, C71, C74, C75: footprint Capacitor_SMD:C_1206_3216Metric_Pad1.33x1.80mm_HandSolder -> Capacitor_SMD:C_0603_1608Metric_Pad1.08x0.95mm_HandSolder; MPN (none) -> Multicomp Pro MC0603B104K500CT (100nF 50V X7R 10% 1608)
- C24: MPN (none) -> Samsung CL31B105KBHNFNE (inventory)
- C25: MPN (none) -> Walsin 0805N272J500CT C0G (inventory); Notes (none) -> fc = 125 kHz with R13
- C3, C4: MPN (none) -> Walsin 0805N103J500CT C0G (inventory)
- C5: value 1uF -> 100nF; footprint Capacitor_SMD:C_1206_3216Metric_Pad1.33x1.80mm_HandSolder -> Capacitor_SMD:C_0603_1608Metric_Pad1.08x0.95mm_HandSolder; MPN (none) -> Multicomp Pro MC0603B104K500CT (100nF 50V X7R 10% 1608); Notes (none) -> Reduced from 1uF: supervisor provides reset timing
- C69: MPN (none) -> Samsung CL21A106KOQNNNF X5R 16V (inventory)
- C72, C76: value 1uF -> 10uF; footprint Capacitor_SMD:C_1206_3216Metric_Pad1.33x1.80mm_HandSolder -> Capacitor_SMD:C_0805_2012Metric_Pad1.18x1.45mm_HandSolder; MPN (none) -> Samsung CL21A106KOQNNNF X5R 16V (inventory)
- C77: value 10uF -> 22uF; footprint Capacitor_SMD:C_0805_2012Metric_Pad1.18x1.45mm_HandSolder -> Capacitor_SMD:C_1206_3216Metric_Pad1.33x1.80mm_HandSolder; MPN (none) -> Samsung CL31A226KAHNNNE X5R 25V (inventory)
- IC1: value ESP32-S3-WROOM-1U-N16R8 -> ESP32-S3-WROOM-1U-N8; footprint ESP32S3WROOM1UN16R8 -> SPD:ESP32S3WROOM1UN16R8; symbol Custom:ESP32-S3-WROOM-1U-N16R8 -> SPD:ESP32-S3-WROOM-1U; Description_1 WiFi Modules - 802.11 [Engineering Samples] SMD Module, ESP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 -> ESP32-S3 module, 8 MB quad flash, no PSRAM, U.FL antenna co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; Height 3.35 -> (none); MPN (none) -> ESP32-S3-WROOM-1U-N8; Manufacturer (none) -> Espressif; Manufacturer_Name Espressif Systems -> (none); Manufacturer_Part_Number ESP32-S3-WROOM-1U-N16R8 -> ESP32-S3-WROOM-1U-N8; Mouser Part Number 356-ESP32S3WM1UN16R8 -> (none); Mouser Price/Stock https://www.mouser.co.uk/ProductDetail/Espressif-Systems/ES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 -> (none); Notes (none) -> Inventory. Footprint common to all WROOM-1U variants. No an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
- IC2: footprint SOP50P640X120-30N -> SPD:SOP50P640X120-30N; symbol Custom:PCM1863QDBTRQ1 -> SPD:PCM1863QDBTRQ1; Description_1 Automotive 110dB 2-Channel Software-Controlled Audio ADC Wi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 -> (none); Height 1.2 -> (none); MPN (none) -> PCM1863QDBTRQ1 (or PCM1863DBTR); Manufacturer (none) -> Texas Instruments; Manufacturer_Name Texas Instruments -> (none); Manufacturer_Part_Number PCM1863QDBTRQ1 -> (none); Mouser Price/Stock https://www.mouser.co.uk/ProductDetail/Texas-Instruments/PC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 -> (none)
- IC4, IC5: footprint Custom:TS026650BK100SCRD -> SPD:TS026650BK100SCRD; symbol Custom:TS02-66-50-BK-100-SCR-D -> SPD:TS02-66-50-BK-100-SCR-D; Height 5.2 -> (none); MPN (none) -> Same Sky TS02-66-50-BK-100-SCR-D (inventory); Manufacturer_Name Same Sky -> (none); Manufacturer_Part_Number TS02-66-50-BK-100-SCR-D -> (none); Mouser Part Number 179-TS026650BK100SCR -> (none); Mouser Price/Stock https://www.mouser.co.uk/ProductDetail/Same-Sky/TS02-66-50-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 -> (none)
- J3: value USB PROGRAMMING -> USB-B; footprint Custom:USBC -> Connector_USB:USB_B_OST_USB-B1HSxx_Horizontal; MPN (none) -> On Shore USB-B1HSW6 (check vs. stocked USB-B part)
- J5: value OUT -> + OUT -; MPN (none) -> JST B2B-XH-A; Notes (none) -> 1 = signal, 2 = GND
- Q1: MPN (none) -> STMicroelectronics BC546 (inventory); Notes (none) -> Upper switch: latch Q
- R1, R2: MPN (none) -> Stackpole RMCF0805FT4K70 (inventory)
- R13: MPN (none) -> Susumu RR1220P-471-D thin film (inventory); Notes (none) -> TI recommended output RC
- R15: value 10K -> 100K; MPN (none) -> Thick film 2012 (inventory); Notes (none) -> 100k/100k limits back-feed into unpowered ESP32
- R16: value 10K -> 100K; MPN (none) -> Thick film 2012 (inventory)
- R19: MPN (none) -> Thick film 2012 (inventory); Notes (none) -> Mute shunt: P68 input held at GND when relay released
- R20: MPN (none) -> Thick film 2012 (inventory); Notes (none) -> Keeps P68 input referenced during relay transfer
- R21: MPN (none) -> Thick film 2012 (inventory)
- R22: MPN (none) -> Stackpole RMCF0805FT16R0 (inventory)
- R3: MPN (none) -> 100R thin film 2012 (inventory); Notes (none) -> TI SLAS831D Fig 61
- R4: MPN (none) -> 100R thin film 2012 (inventory)
- R5, R6: footprint Resistor_SMD:R_0603_1608Metric_Pad0.98x0.95mm_HandSolder -> Resistor_SMD:R_0805_2012Metric_Pad1.20x1.40mm_HandSolder; MPN (none) -> KOA RK73B2ATTD103J (inventory)
- R7, R8: MPN (none) -> 100k thin film 2012 (inventory); Notes (none) -> Bleed: holds relay COM side at 0 V
- U2: MPN (none) -> PCM5102APWR; Manufacturer (none) -> Texas Instruments; Notes (none) -> Inventory lists "PCM5102" - confirm marking is PCM5102A (sa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
Connections:
- net 3V3_DAC is gone; now on net +3V3_DAC: U2.1 (CPVDD), U2.11 (FLT), U2.20 (DVDD), U2.8 (AVDD)
- net 3V3_ESP is gone; now on net +3V3_ESP: C75.1, C77.1, IC1.2 (3V3), R5.1, R6.1
- net INTC is gone; now on net ADC_INT: IC2.19 (GPIO3/INTC)
- net GND: now also IC2.10 (XI), R16.2, R19.1, R7.2, R8.2, C114.2, C115.2, C116.2, C117.2, IC3.2 (GND), K1.6 (COM), Q4.3 (E), R33.2, R39.2, R40.2, R42.2, R45.2; no longer Q1.3 (E), R16.1, R19.2, R7.1, R8.1
- net I2S_BCK: now also R34.2, TP11.1; no longer IC1.18 (IO10)
- net I2S_DIN: now also R37.2, TP13.1; no longer IC2.18 (DOUT)
- net I2S_DOUT: now also R36.2, TP14.1; no longer IC1.31 (IO38)
- net I2S_LRCK: now also R35.2, TP12.1; no longer IC1.19 (IO11)
- net I2S_MCLK: now also R32.1
- net IN-LEFT: now also R8.1; no longer R8.2
- net IN-RIGHT: now also R7.1; no longer R7.2
- net at J5.1 (Pin_1), R20.1: now also K1.3 (COM), TP17.1
- net at Q1.1 (C): now also D4.2 (A), K1.8 (COIL-)
- net at Q1.2 (B), R21.2: now also R42.1
- net ADC_VREF: now reaches C19.1, IC2.6 (VREF)
- net at J3.2 (D-): now also IC3.1 (I/O1_1)
- net at J3.3 (D+): now also IC3.3 (I/O2_1)
- net at C25.1, R13.2: now also R38.1
- net +5V: now reaches R22.1
- net ADC_LDO: now reaches C21.1, IC2.11 (LDO)
- net ADC_LDO: now also C114.1
- net ENC2_B: now reaches IC1.11 (IO18)
- net ENC2_SW: now reaches IC1.12 (IO8)
- net OUT_RLY_SENSE: now reaches IC1.15 (IO3)
- net OUT_RLY_SENSE: now also K1.5 (NO), R41.2
- net STATUS_LED: now reaches IC1.16 (IO46)
- net UI_SDA: now reaches IC1.22 (IO14)
- net UI_SCL: now reaches IC1.23 (IO21)
- net MODE_TRIG_N: now reaches IC1.24 (IO47)
- net ADC_INT: now reaches IC1.25 (IO48)
- net INPUT_SEL: now reaches IC1.26 (IO45)
- net ENC3_A: now reaches IC1.32 (IO39)
- net ENC3_B: now reaches IC1.33 (IO40)
- net ENC3_SW: now reaches IC1.34 (IO41)
- net FAULT_N: now reaches IC1.35 (IO42)
- net ENC1_A: now reaches IC1.4 (IO4)
- net ENC1_B: now reaches IC1.5 (IO5)
- net ENC1_SW: now reaches IC1.6 (IO6)
- net ENC2_A: now reaches IC1.8 (IO15)
- net 3V3-DAC renamed +3V3_DAC
- net +3V3_DAC: now also C115.1, C116.1
- net 3V3-ESP renamed +3V3_ESP
- net +3V3_ESP: now also R41.1
- net 3V3_A_ADC renamed +3V3_A_ADC
- net 3V3_D_ADC renamed +3V3_D_ADC
- net 5V: no longer names the net of R22.2
- net 5V: now also D4.1 (K), K1.1 (COIL+)
- net AMP_ENABLE renamed RLY_EN_LATCH
- net AUDIO-READY renamed AUDIO_READY
- net AUDIO_READY: now also R43.1
- net EN renamed ESP_EN
- net ESP_EN: now also R44.1, TP24.1
- net I2S_SCLK renamed ADC_SCKI
- net ADC_SCKI: now also R32.2, R33.1
- net RX renamed DBG_RX
- net TX renamed DBG_TX
- net USB-D+ renamed USB_DP
- net USB_DP: now also R46.2
- net USB-D- renamed USB_DM
- net USB_DM: now also R47.2
- net USB-VBUS renamed USB_VBUS
- net USB_VBUS: now also R15.1, IC3.5 (VBUS); no longer R15.2
- removed net USB-VBUS-SENSE: IC1.10 (IO17), R15.1, R16.2
- net XSMT renamed DAC_XSMT
- net DAC_XSMT: now also R40.1, TP15.1
- new net: Q4.2 (B), R43.2
- new net: IC3.4 (I/O2_2), R46.1
- new net: IC3.6 (I/O1_2), R47.1
- new net: Q1.3 (E), Q4.1 (C)
- new net: K1.2 (NC), R19.2
- new net: C117.1, J3.SH (Shield), R45.1
- new net: K1.4 (NO), R38.2, R39.1, TP16.1
- new net: IC2.18 (DOUT), R37.1
- new net I2S_BCK_ESP: IC1.18 (IO10), R34.1
- new net I2S_DOUT_ESP: IC1.31 (IO38), R36.1
- new net I2S_LRCK_ESP: IC1.19 (IO11), R35.1
- new net SUP_RST_N: R44.2
- new net USB_VBUS_SENSE: IC1.10 (IO17), R15.2, R16.1
- no-connect marks 13 -> 16
Other:
- note added: "3V3 pin 2: 22u + 100n (Espressif)"
- note added: "ADC CLOCK OPTION / I2C0 PULL-UPS"
- note added: "ADC DECOUPLING (place at pins)"
- note added: "ADC PCM1863 (I2C 0x4A, I2S slave, BCK-PLL)"
- note added: "AVDD pin 8"
- note added: "CPVDD pin 1"
- note added: "Coil 145R +/-10 %: ~4.3 V across coil via R22 (96 % nom.), must-operate 75 %. D4 clamps turn-off."
- note added: "DAC DECOUPLING (place at pins)"
- note added: "DAC PCM5102A"
- note added: "DVDD pin 13"
- note added: "DVDD pin 20"
- note added: "ESP32 SUPPLY / RESET / BOOT"
- note added: "ESP32-S3-WROOM-1U-N8"
- note added: "GPIO map: root sheet notes. IO45/IO46/IO0 are strapping pins (low/high-Z at reset)."
- note added: "Hardware mode: I2S, low-latency filter, de-emphasis off, BCK-PLL (SCK = GND)."
- note added: "I2S SOURCE TERMINATION (place R34-R36 within 5 mm of ESP32 pins)"
- note added: "I2S0 full duplex, ESP32 master: BCK 3.072 MHz (64fs), LRCK 48 kHz. MCLK (IO9) optional."
- note added: "IOVDD pin 14"
- note added: "Input FS 2.1 Vrms single-ended per pin; Zin 10k; TI filter: 10 uF + 100R + 10 nF film/C0G at pin."
- note added: "K1 de-energised (no power / fault / not armed): P68 input = GND via R19 1k + R20 100k."
- note added: "K1 pole B = relay-state feedback to ESP32 IO3 (low = closed)."
- note added: "LDO pin 11"
- note added: "MD0 = 0: I2C control. MS/AD = 0: address 0x4A. Low-latency IIR decimation = 10 samples."
- note added: "Mute sequence: XSMT low (104-sample soft mute) -> wait 5 ms -> drop AUDIO_READY (relay opens)."
- note added: "No PSRAM (85 degC rating). IO35-37 left free, so the N8R8 also fits."
- note added: "OUTPUT RELAY DRIVER (two series switches = hardware AND)"
- note added: "Relay energises only if: latch Q (PROTECT) = 1 AND AUDIO_READY = 1 AND +5V present."
- note added: "SCKI held low by R33 = BCK-PLL slave mode (Table 15). Fit R32 to use ESP32 MCLK instead."
- note added: "Shield: 1M || 4n7 to GND (bleed + RF path, no hard DC bond). Ground-loop note: USB GND = board GND;"
- note added: "TEST POINTS"
- note added: "USB (native ESP32-S3 USB-Serial/JTAG; self-powered, VBUS only sensed)"
- note added: "Unmute: AUDIO_READY rising edge arms latch -> relay closes (DAC muted, 0 V) -> wait 20 ms -> XSMT high."
- note added: "VREF"
- note added: "XI tied to DGND: XI and SCKI clocks are OR-ed internally (SLAS831D 9.3.9)."
- note added: "XSMT pull-down"
- note added: "for listening sessions with a Mac attached, use an isolated USB hub/isolator (ADuM4160-based)."
- note removed: "ADC"
- note removed: "DAC"
- note removed: "ESP32-S3"
- note removed: "I2C pull-ups"
- note removed: "USB header for config"
- note removed: "VBUS SENSE"
- company: (none) -> P68 Subwoofer DSP Controller
- title: (none) -> ADC / ESP32-S3 DSP / DAC / output relay
- moved on the sheet: C1, C18, C19, C2, C20, C21, C23, C24, C25, C3, C4, C5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

Commit message: more work
Parts:
- added J11: ESP, Connector_PinSocket_2.54mm:PinSocket_1x04_P2.54mm_Vertical, symbol Connector:Conn_01x04_Socket
- C1, C2, C3, C4, R3, R4, R7, R8: Config (none) -> LOW-LEVEL build only
- IC2: value PCM1863QDBTRQ1 -> PCM1863
- J3: value USB-B -> USB PROGRAMMING
- Q1, Q4: value BC546 -> BC849C; footprint Package_TO_SOT_THT:TO-92_Wide -> Package_TO_SOT_SMD:SOT-23; symbol Transistor_BJT:BC546 -> Transistor_BJT:BC849; MPN STMicroelectronics BC546 (inventory) -> Nexperia BC849C,215 (purchase)
Connections:
- net +3V3_ESP: now also J11.4 (Pin_4)
- net DBG_RX: now also J11.2 (Pin_2)
- net DBG_TX: now also J11.1 (Pin_1)
- net GND: now also Q4.2 (E), J11.3 (Pin_3); no longer Q4.3 (E)
- net at R43.2: now also Q4.1 (B); no longer Q4.2 (B)
- net at D4.2 (A), K1.8 (COIL-): now also Q1.3 (C); no longer Q1.1 (C)
- net at R21.2, R42.1: now also Q1.1 (B); no longer Q1.2 (B)
- net HL-LEFT: now reaches IC2.29 (VINL3/VIN4P)
- net HL-RIGHT: now reaches IC2.30 (VINR3/VIN3P)
- new net: Q1.2 (E), Q4.3 (C)
- no-connect marks 16 -> 14
Other:
- note added: "DEBUG UART0 (115200 8N1, 3.3 V)"
- note added: "J8-1 = ESP32 TXD0 (out), J8-2 = ESP32 RXD0 (in)"
