File: SubProcessorDigital/AUDIO-IN.kicad_sch (KiCad schematic)
At the start: 2 parts, among them J1 PreAmp In, J2 LFE In

Commit message: more
Parts:
- added D2, D3: 1N4148W, Diode_SMD:D_SOD-123, symbol Diode:1N4148W
- added K2, K3: AGN2004H, SPD:Relay_DPDT_Panasonic_AGN2004H, symbol SPD:AGN2004H
- added Q2, Q3: BC546, Package_TO_SOT_THT:TO-92_Wide, symbol Transistor_BJT:BC546
- added R25, R26: 4K7, Resistor_SMD:R_0805_2012Metric_Pad1.20x1.40mm_HandSolder, symbol Device:R
- added R27, R29: 16R, Resistor_SMD:R_0805_2012Metric_Pad1.20x1.40mm_HandSolder, symbol Device:R
- added R28, R30: 1K, Resistor_SMD:R_0805_2012Metric_Pad1.20x1.40mm_HandSolder, symbol Device:R
- added R31: 100K, Resistor_SMD:R_0805_2012Metric_Pad1.20x1.40mm_HandSolder, symbol Device:R
- added TP10: INPUT_SEL, TestPoint:TestPoint_Pad_D1.5mm, symbol Connector:TestPoint
- J1: value PreAmp In -> PREAMP IN; MPN (none) -> JST B3B-XH-A; Notes (none) -> 1 = L, 2 = preamp GND, 3 = R
- J2: value LFE In -> MARANTZ LFE IN; MPN (none) -> JST B2B-XH-A; Notes (none) -> 1 = LFE, 2 = Marantz GND
Connections:
- net IN-LEFT: now also R25.2
- net IN-RIGHT: now also R26.2
- net LFE: now reaches J2.1 (Pin_1)
- net LFE: now also K2.4 (NO), K2.5 (NO)
- net LFE_GND: now reaches J2.2 (Pin_2)
- net LFE_GND: now also K3.4 (NO), K3.5 (NO)
- net PRE_L: now reaches J1.1 (Pin_1)
- net PRE_L: now also K2.2 (NC)
- net PRE_GND: now reaches J1.2 (Pin_2)
- net PRE_GND: now also K3.2 (NC), K3.7 (NC)
- net PRE_R: now reaches J1.3 (Pin_3)
- net PRE_R: now also K2.7 (NC)
- new net: D3.1 (K), K3.1 (COIL+), R29.2
- new net: D3.2 (A), K3.8 (COIL-), Q3.1 (C)
- new net: D2.1 (K), K2.1 (COIL+), R27.2
- new net: D2.2 (A), K2.8 (COIL-), Q2.1 (C)
- new net: K2.3 (COM), R25.1
- new net: Q2.2 (B), R28.2
- new net: Q3.2 (B), R30.2
- new net: K2.6 (COM), R26.1
- new net +5V: R27.1, R29.1
- new net GND: K3.3 (COM), K3.6 (COM), Q2.3 (E), Q3.3 (E), R31.2
- new net INPUT_SEL: R28.1, R30.1, R31.1, TP10.1
Other:
- note added: "Bleed resistors (100k) are on the ADC side of R25/R26 (ADCESPDAC sheet), referenced to board GND,"
- note added: "Coil: 145 ohm +/-10 %, 31 mA. 5 V - Vce(sat) via 16R gives ~4.3 V (96 % nom.); must-operate <= 75 % (3.38 V)."
- note added: "Contacts shown de-energised = PREAMP (stereo) selected."
- note added: "Energised (INPUT_SEL high) = MARANTZ LFE on both ADC channels; the preamp is then fully disconnected."
- note added: "K2: signal poles. K3: source-ground poles (both poles paralleled)."
- note added: "PRE_GND and LFE_GND are NOT connected to board GND"
- note added: "Polarised GN coil: pin 1 (+) to supply. 1N4148W clamps turn-off spike (release <= ~4 ms + diode delay)."
- note added: "R25/R26 4k7: input attenuation/protection. 0R = 2.1 Vrms FS, 4k7 = 3.1 Vrms, 10k = 4.2 Vrms."
- note added: "R31 holds INPUT_SEL low during ESP32 reset (GPIO45 strap must be low at boot)."
- note added: "RELAY DRIVERS"
- note added: "SOURCE CONNECTORS"
- note added: "SOURCE SELECT RELAYS"
- note added: "except through the selected K3 contacts."
- note added: "so no resistor bridges an unselected source to board GND."
- company: (none) -> P68 Subwoofer DSP Controller
- title: (none) -> Audio input selection
- moved on the sheet: J1, J2

Commit message: more work
Parts:
- added C137, C138, C141, C142: 4.7nF, Capacitor_SMD:C_0805_2012Metric_Pad1.18x1.45mm_HandSolder, symbol Device:C
- added C139, C143: 10uF NP, Capacitor_THT:C_Radial_D8.0mm_H11.5mm_P3.50mm, symbol Device:C
- added C140, C144: 10nF, Capacitor_SMD:C_0805_2012Metric_Pad1.18x1.45mm_HandSolder, symbol Device:C
- added C145, C146: 100nF, Capacitor_SMD:C_0603_1608Metric_Pad1.08x0.95mm_HandSolder, symbol Device:C
- added C147, C148: 10uF, Capacitor_SMD:C_1206_3216Metric_Pad1.33x1.80mm_HandSolder, symbol Device:C
- added J10: HIGH LEVEL IN, Connector_JST:JST_XH_B4B-XH-A_1x04_P2.50mm_Vertical, symbol Connector:Conn_01x04_Socket
- added R81, R82, R86, R87: 100K, Resistor_SMD:R_0805_2012Metric_Pad1.20x1.40mm_HandSolder, symbol Device:R
- added R83, R84, R88, R89: 10K, Resistor_SMD:R_0805_2012Metric_Pad1.20x1.40mm_HandSolder, symbol Device:R
- added R85, R90: 1K, Resistor_SMD:R_0805_2012Metric_Pad1.20x1.40mm_HandSolder, symbol Device:R
- added U16: RC4580, Package_SO:SOIC-8_3.9x4.9mm_P1.27mm, symbol Amplifier_Operational:RC4580
- D2, D3, J1, J2, K2, K3, R25, R26, R27, R28, R29, R30: Config (none) -> LOW-LEVEL build only
- Q2, Q3: value BC546 -> BC849C; footprint Package_TO_SOT_THT:TO-92_Wide -> Package_TO_SOT_SMD:SOT-23; symbol Transistor_BJT:BC546 -> Transistor_BJT:BC849; Config (none) -> LOW-LEVEL build only; MPN STMicroelectronics BC546 (inventory) -> Nexperia BC849C,215 (purchase)
Connections:
- net GND: now also Q2.2 (E), Q3.2 (E), C137.2, C140.2, C141.2, C144.2, C145.1, C146.2, C147.2, C148.1, R83.2, R88.2; no longer Q2.3 (E), Q3.3 (E)
- net at D3.2 (A), K3.8 (COIL-): now also Q3.3 (C); no longer Q3.1 (C)
- net at D2.2 (A), K2.8 (COIL-): now also Q2.3 (C); no longer Q2.1 (C)
- net at R28.2: now also Q2.1 (B); no longer Q2.2 (B)
- net at R30.2: now also Q3.1 (B); no longer Q3.2 (B)
- new net: C139.2, R85.1
- new net: C141.1, R86.2, R88.1, U16.5 (+)
- new net: C142.1, R87.2, R89.1, U16.6 (-)
- new net: C142.2, C143.1, R89.2, U16.7
- new net: C137.1, R81.2, R83.1, U16.3 (+)
- new net: C138.1, R82.2, R84.1, U16.2 (-)
- new net: C143.2, R90.1
- new net: C138.2, C139.1, R84.2, U16.1
- new net +15V: C146.1, C147.1, U16.8 (V+)
- new net -15V: C145.2, C148.2, U16.4 (V-)
- new net HL-LEFT: C140.1, R85.2
- new net HL-RIGHT: C144.1, R90.2
- new net SPK_L+: J10.1 (Pin_1), R81.1
- new net SPK_L-: J10.2 (Pin_2), R82.1
- new net SPK_R+: J10.4 (Pin_4), R86.1
- new net SPK_R-: J10.3 (Pin_3), R87.1
Other:
- note added: "Assembly option: fit EITHER this block (HIGH-LEVEL build) OR J1/J2/K2/K3 + drivers (LOW-LEVEL build). See Config field."
- note added: "C146 at U16 pin 8, C145 at U16 pin 4."
- note added: "Common mode: matched 100K/10K pairs; worst-case CMRR ~35 dB with 0.5 % 100K (0.1 % 100K -> ~49 dB). Cf/Cg remove Class-D residue."
- note added: "Difference amplifier on +/-15 V: Vout = (Rf/Rin)(SPK+ - SPK-), referenced to GND. Zin = 200k differential, 110k each leg to GND."
- note added: "Feeds PCM1863 VINL3/VINR3; firmware selects ADC input VIN3 and sums L+R to mono. No relays."
- note added: "Fitted for <= 50 W: 20 Vrms (8R) / 14 Vrms (4R)."
- note added: "HIGH-LEVEL (SPEAKER) INPUT"
- note added: "Higher-power amps: change Rf = Rg (and Cf = Cg) together: 6K8/6.8nF for 100 W, 4K7/10nF for 200 W into 8R. Rin stays 100K."
- note added: "Speaker terminals: neither side is ground."
