File: SubProcessorDigital/CONTROL.kicad_sch (KiCad schematic)
At the start: 49 parts, among them J6 FRONT PANEL CONNECTOR, J7 + 12V TRIG -, J8 UART0, J9 + 12V TRIG -, U14 VO617A-3

Commit message: more work
Parts:
- removed J8: UART0, Connector_PinHeader_2.54mm:PinHeader_1x03_P2.54mm_Vertical, symbol Connector_Generic:Conn_01x03
Other:
- note removed: "DEBUG UART0 (115200 8N1, 3.3 V)"
- note removed: "J8-1 = ESP32 TXD0 (out), J8-2 = ESP32 RXD0 (in)"
Changed lines of the file:
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@@
 		)
 	)
-	(text "J8-1 = ESP32 TXD0 (out), J8-2 = ESP32 RXD0 (in)"
-		(exclude_from_sim no)
-		(at 172.72 213.36 0)
-		(effects
-			(font
-				(size 1.27 1.27)
-			)
-			(justify left)
-		)
-	)
 	(text "DAUGHTERBOARD HEADER J6 (2x10 shrouded IDC, short ribbon)"
 		(exclude_from_sim no)
@@
 		)
 	)
-	(text "DEBUG UART0 (115200 8N1, 3.3 V)"
-		(exclude_from_sim no)
-		(at 172.72 182.88 0)
-		(effects
-			(font
-				(size 1.6 1.6)
-				(bold yes)
-			)
-			(justify left)
-		)
-	)
 	(text "Inputs read by ESP32 PCNT (quadrature) + GPIO; firmware debounce on switches.  tau = 100 us."
 		(exclude_from_sim no)
@@
 	(wire
 		(pts
-			(xy 190.5 205.74) (xy 187.96 205.74)
-		)
-		(stroke
-			(width 0)
-			(type default)
-		)
-	)
-	(wire
-		(pts
 			(xy 281.94 66.04) (xy 281.94 68.58)
 		)
@@
 	(wire
 		(pts
-			(xy 190.5 200.66) (xy 187.96 200.66)
-		)
-		(stroke
-			(width 0)
-			(type default)
-		)
-	)
-	(wire
-		(pts
 			(xy 279.4 86.36) (xy 281.94 86.36)
 		)
@@
 	(wire
 		(pts
-			(xy 190.5 203.2) (xy 187.96 203.2)
-		)
-		(stroke
-			(width 0)
-			(type default)
-		)
-	)
-	(wire
-		(pts
 			(xy 30.48 154.94) (xy 34.29 154.94)
 		)
@@
 		)
 	)
-	(hierarchical_label "DBG_TX"
-		(shape input)
-		(at 187.96 200.66 180)
-		(effects
-			(font
-				(size 1.27 1.27)
-			)
-			(justify right)
-		)
-	)
 	(hierarchical_label "ENC2_SW"
 		(shape output)
@@
 		)
 	)
-	(hierarchical_label "DBG_RX"
-		(shape output)
-		(at 187.96 203.2 180)
-		(effects
-			(font
-				(size 1.27 1.27)
-			)
-			(justify right)
-		)
-	)
 	(hierarchical_label "ENC1_SW"
 		(shape output)
@@
 	)
 	(symbol
-		(lib_id "power:GND")
-		(at 187.96 205.74 270)
-		(unit 1)
-		(body_style 1)
-		(exclude_from_sim no)
-		(in_bom yes)
-		(on_board yes)
-		(in_pos_files yes)
-		(dnp no)
-		(property "Reference" "#PWRCON031"
-			(at 180.34 205.74 90)
-			(hide yes)
-			(show_name no)
-			(do_not_autoplace no)
-			(effects
-				(font
-					(size 1.27 1.27)
-				)
-			)
-		)
-		(property "Value" "GND"
-			(at 182.88 205.74 90)
-			(show_name no)
-			(do_not_autoplace no)
-			(effects
-				(font
-					(size 1.27 1.27)
-				)
-				(justify right)
-			)
-		)
-		(property "Footprint" ""
-			(at 187.96 205.74 90)
-			(hide yes)
-			(show_name no)
-			(do_not_autoplace no)
-			(effects
-				(font
-					(size 1.27 1.27)
-				)
-			)
-		)
-		(property "Datasheet" ""
-			(at 187.96 205.74 90)
-			(hide yes)
-			(show_name no)
-			(do_not_autoplace no)
-			(effects
-				(font
-					(size 1.27 1.27)
-				)
-			)
-		)
-		(property "Description" "Power symbol creates a global label with name \"GND\" , ground"
-			(at 187.96 205.74 90)
-			(hide yes)
-			(show_name no)
-			(do_not_autoplace no)
-			(effects
-				(font
-					(size 1.27 1.27)
-				)
-			)
-		)
-		(pin "1"
-		)
-		(instances
-			(project "SubProcessorDigital"
-				(path "/d270386e-be0f-4547-84de-01e193634fe2/6c1e2f3a-7b4d-4e5f-9a0b-1c2d3e4f5a6b"
-					(reference "#PWRCON031")
-					(unit 1)
-				)
-			)
-		)
-	)
-	(symbol
 		(lib_id "Device:R")
 		(at 52.07 81.28 90)
@@
 					(unit 1)
 				)
-			)
-		)
-	)
-	(symbol
-		(lib_id "Connector_Generic:Conn_01x03")
-		(at 195.58 203.2 0)
-		(unit 1)
-		(body_style 1)
-		(exclude_from_sim no)
-		(in_bom yes)
-		(on_board yes)
-		(in_pos_files yes)
-		(dnp no)
-		(property "Reference" "J8"
-			(at 193.04 196.85 0)
-			(show_name no)
-			(do_not_autoplace no)
-			(effects
-				(font
-					(size 1.27 1.27)
-				)
-				(justify left)
-			)
-		)
-		(property "Value" "UART0"
-			(at 193.04 209.55 0)
-			(show_name no)
-			(do_not_autoplace no)
-			(effects
-				(font
-					(size 1.27 1.27)
-				)
-				(justify left)
-			)
-		)
-		(property "Footprint" "Connector_PinHeader_2.54mm:PinHeader_1x03_P2.54mm_Vertical"
-			(at 195.58 203.2 0)
-			(hide yes)
-			(show_name no)
-			(do_not_autoplace no)
-			(effects
-				(font
-					(size 1.27 1.27)
-				)
-			)
-		)
-		(property "Datasheet" ""
-			(at 195.58 203.2 0)
-			(hide yes)
-			(show_name no)
-			(do_not_autoplace no)
-			(effects
-				(font
-					(size 1.27 1.27)
-				)
-			)
-		)
-		(property "Description" "Generic connector, single row, 01x03, script generated (kicad-library-utils/schlib/autogen/connector/)"
-			(at 195.58 203.2 0)
-			(hide yes)
-			(show_name no)
-			(do_not_autoplace no)
-			(effects
-				(font
-					(size 1.27 1.27)
-				)
-			)
-		)
-		(property "MPN" "2.54 mm 1x3 pin header"
-			(at 195.58 203.2 0)
-			(hide yes)
-			(show_name no)
-			(do_not_autoplace no)
-			(effects
-				(font
-					(size 1.27 1.27)
-				)
-			)
-		)
-		(pin "1"
-		)
-		(pin "2"
-		)
-		(pin "3"
-		)
-		(instances
-			(project "SubProcessorDigital"
-				(path "/d270386e-be0f-4547-84de-01e193634fe2/6c1e2f3a-7b4d-4e5f-9a0b-1c2d3e4f5a6b"
-					(reference "J8")
-					(unit 1)
-				)
