File: SubProcessorDigital/POWER.kicad_sch (KiCad schematic)
At the start: 23 parts, among them J4 POWER, U1 TPS7A2033, U3 LMR51430, U4 TPS7A2033, U5 TPS7A2033, U6 AMS1117-3.3

Commit message: more
Parts:
- added C109: 100nF, Capacitor_SMD:C_0603_1608Metric_Pad1.08x0.95mm_HandSolder, symbol Device:C
- added C110, C111: 22uF, Capacitor_SMD:C_1206_3216Metric_Pad1.33x1.80mm_HandSolder, symbol Device:C
- added C112, C134, C135: 1uF, Capacitor_SMD:C_1206_3216Metric_Pad1.33x1.80mm_HandSolder, symbol Device:C
- added C113, C136: 10uF, Capacitor_SMD:C_0805_2012Metric_Pad1.18x1.45mm_HandSolder, symbol Device:C
- added D1: 1N5819, Diode_THT:D_DO-41_SOD81_P10.16mm_Horizontal, symbol Diode:1N5819
- added F1: 3A fast, Fuse:Fuse_1206_3216Metric_Pad1.42x1.75mm_HandSolder, symbol Device:Fuse
- added R23, R24: 4R7, Resistor_SMD:R_0805_2012Metric_Pad1.20x1.40mm_HandSolder, symbol Device:R
- added TP1: +15V, TestPoint:TestPoint_Pad_D1.5mm, symbol Connector:TestPoint
- added TP2: +5V, TestPoint:TestPoint_Pad_D1.5mm, symbol Connector:TestPoint
- added TP26: +5V_UI, TestPoint:TestPoint_Pad_D1.5mm, symbol Connector:TestPoint
- added TP3: +3V3_ESP, TestPoint:TestPoint_Pad_D1.5mm, symbol Connector:TestPoint
- added TP4: +3V3_DAC, TestPoint:TestPoint_Pad_D1.5mm, symbol Connector:TestPoint
- added TP5: +3V3_A_ADC, TestPoint:TestPoint_Pad_D1.5mm, symbol Connector:TestPoint
- added TP6: +3V3_D_ADC, TestPoint:TestPoint_Pad_D1.5mm, symbol Connector:TestPoint
- added TP7: +3V3_UI, TestPoint:TestPoint_Pad_D1.5mm, symbol Connector:TestPoint
- added TP9: GND, TestPoint:TestPoint_THTPad_2.0x2.0mm_Drill1.0mm, symbol Connector:TestPoint
- added U15: AP2205-50Y-13, Package_TO_SOT_SMD:SOT-89-3, symbol SPD:AP2205-50Y
- added U8: TPS7A2033, Package_TO_SOT_SMD:SOT-23-5, symbol Regulator_Linear:TPS7A20xxxDBV
- C100, C99: value 1uF -> 10uF; MPN (none) -> Samsung CL31A106KBHNNNE (inventory)
- C101, C102, C103, C104, C105, C106: MPN (none) -> Samsung CL31B105KBHNFNE
- C107, C108: MPN (none) -> Taiyo Yuden TMK316B7106KL-TD
- C32: footprint Capacitor_SMD:C_1206_3216Metric_Pad1.33x1.80mm_HandSolder -> Capacitor_SMD:C_0603_1608Metric_Pad1.08x0.95mm_HandSolder; MPN (none) -> Multicomp Pro MC0603B104K500CT (100nF 50V X7R 10% 1608)
- C33, C34: MPN (none) -> Samsung CL31A226KAHNNNE X5R 25V 3216 (inventory)
- C6: MPN (none) -> Panasonic EEUFR1V102 (FR); Notes (none) -> Inventory
- J4: value POWER -> POWER IN; MPN (none) -> JST B3B-XH-A; Notes (none) -> Pin3 +15V, Pin2 GND, Pin1 -15V (unused)
- L3: footprint Custom:SRP6030WA-6R8M -> SPD:SRP6030WA-6R8M; MPN (none) -> Bourns SRP6030WA-6R8M (inventory); Notes (none) -> Isat 6.1 A, Irms 5.2 A, DCR 42 mohm
- R17: MPN (none) -> 100k thin film 0.5% 2012 (inventory)
- R18: MPN (none) -> 13k7 thick film 1% 2012 (inventory)
- U1, U4, U5: MPN (none) -> TPS7A2033PDBVR; Manufacturer (none) -> Texas Instruments; Notes (none) -> Inventory
- U3: value LMR51430 -> LMR51430XFDDCR; MPN (none) -> LMR51430XFDDCR; Manufacturer (none) -> Texas Instruments; Notes (none) -> 500 kHz FPWM; inventory
- U6: value AMS1117-3.3 -> TS1117BCW33; MPN (none) -> Taiwan Semiconductor TS1117BCW33 RPG; Notes (none) -> Pin-compatible with AMS1117 symbol; inventory
Connections:
- net GND: now also C109.2, C110.2, C111.2, C112.2, C113.2, C134.2, C135.2, C136.2, TP9.1, U15.2 (GND), U8.2 (GND)
- net 3V3_A_ADC renamed +3V3_A_ADC
- net +3V3_A_ADC: now also TP5.1
- net 3V3_DAC renamed +3V3_DAC
- net +3V3_DAC: now also TP4.1
- net 3V3_D_ADC renamed +3V3_D_ADC
- net +3V3_D_ADC: now also TP6.1
- net 3V3_ESP renamed +3V3_ESP
- net +3V3_ESP: now also TP3.1
- net 5V renamed +5V
- net +5V: now also C112.1, R23.1, R24.1, TP2.1, U8.1 (IN), U8.3 (EN); no longer C101.1, C103.1, U1.1 (IN), U1.3 (EN), U4.1 (IN), U4.3 (EN)
- net VCC renamed +15V
- net +15V: now also C109.1, C134.1, D1.1 (K), TP1.1, U15.1 (IN); no longer J4.3 (Pin_3)
- new net: C101.1, C110.1, R23.2, U1.1 (IN), U1.3 (EN)
- new net: C103.1, C111.1, R24.2, U4.1 (IN), U4.3 (EN)
- new net: F1.1, J4.3 (Pin_3)
- new net: D1.2 (A), F1.2
- new net +3V3_UI: C113.1, TP7.1, U8.5 (OUT)
- new net +5V_UI: C135.1, C136.1, TP26.1, U15.3 (OUT)
- no-connect marks 0 -> 5
Other:
- note added: "+15 V INPUT, PROTECTION AND 5 V BUCK"
- note added: "-15 V (not used)"
- note added: "5 V DISPLAY SUPPLY (+5V_UI, J6 pin 20)"
- note added: "ADC ANALOGUE SUPPLY (+3V3_A_ADC)"
- note added: "ADC DIGITAL SUPPLY (+3V3_D_ADC)"
- note added: "CIN >= 4.7 uF X7R 50 V + 100 nF at VIN/GND pins (TI 9.2.2.6); C109 closest to U3."
- note added: "D1: reverse-polarity protection against a -15 V/+15 V harness swap."
- note added: "DAC SUPPLY (+3V3_DAC)"
- note added: "ESP32 SUPPLY (+3V3_ESP)"
- note added: "F1: wiring/harness fault protection only (3 A fast, inventory)."
- note added: "LINEAR REGULATORS (all fed from +5V)"
- note added: "LMR51430XFDDCR (TI SLUSEF4A): 500 kHz forced-PWM, no PFM bursts at light load."
- note added: "Layout: keep SW node (U3.2-L3-C32) compact; FB divider away from L3; C33/C34 GND to U3 GND."
- note added: "RC pre-filter R23/C110: fc = 1.5 kHz"
- note added: "RC pre-filter R24/C111: fc = 1.5 kHz"
- note added: "Separate LDO: a ribbon-cable fault cannot pull down +3V3_ESP (current-limited 160 mA)."
- note added: "Separate from the buck +5V: no switching ripple or relay steps on the display, and a ribbon fault"
- note added: "TEST POINTS"
- note added: "TP8 near U3/C33 (power ground); TP9 near the ADC (quiet ground)."
- note added: "TS1117B: 10 uF MLCC in/out required (TSC datasheet I2405). Pd ~ 1.7 V x 0.15 A = 0.26 W typ;"
- note added: "UI / DAUGHTERBOARD SUPPLY (+3V3_UI)"
- note added: "VOUT = 0.6 V x (1 + R17/R18) = 4.98 V. L/COUT per TI Table 9-1 (6.8 uH, 2 x 22 uF/25 V)."
- note added: "cannot pull down the main rail. Pd = 10 V x I: keep display <= 50 mA (0.5 W, give the tab copper)."
- note added: "give SOT-223 tab >= 2 cm2 copper. 22 uF + 100 nF also at module 3V3 pin (ADCESPDAC sheet)."
- note removed: "5V PreReg Buck"
- note removed: "ADC Analog Power"
- note removed: "ADC Digital Power"
- note removed: "DAC Power"
- note removed: "ESP Power"
- company: (none) -> P68 Subwoofer DSP Controller
- title: (none) -> Power supply
- moved on the sheet: C100, C101, C102, C103, C104, C105, C106, C107, C108, C32, C33, C34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

Commit message: more work
Parts:
- added D8: 1N4148W, Diode_SMD:D_SOD-123, symbol Diode:1N4148W
- added F2: 3A fast, Fuse:Fuse_1206_3216Metric_Pad1.42x1.75mm_HandSolder, symbol Device:Fuse
- added TP8: -15V, TestPoint:TestPoint_Pad_D1.5mm, symbol Connector:TestPoint
- J4: Notes Pin3 +15V, Pin2 GND, Pin1 -15V (unused) -> Pin3 +15V, Pin2 GND, Pin1 -15V (used by HIGH-LEVEL input op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
- U15: value AP2205-50Y-13 -> AP2205-50Y
- U3: value LMR51430XFDDCR -> LMR51430XF
- U6: value TS1117BCW33 -> TS1117-33
Connections:
- net at J4.1 (Pin_1): now also F2.1
- new net: D8.1 (K), F2.2
- new net -15V: D8.2 (A), TP8.1
- no-connect marks 5 -> 4
Other:
- note added: "-15V: HIGH-LEVEL build only (U16). D8 blocks a swapped harness."
- note removed: "-15 V (not used)"
