File: SubProcessorDigital/SubProcessorDigital.kicad_pcb (KiCad board)
At the start: 2 copper layers, 100 x 100 mm, 82 parts, among them IC1 ESP32-S3-WROOM-1U-N16R8, IC2 PCM1863QDBTRQ1, IC3 USBLC6, IC4 RESET, IC5 BOOT, J1 PreAmp In, J2 LFE In, J3 USB PROGRAMMING, J4 POWER, J5 OUT, J6 SYSTEM CONNECTOR, K1 AGN2004H, Q1 BC546, U1 TPS7A2033, U2 PCM5102A, U3 LMR51430, U4 TPS7A2033, U5 TPS7A2033, U6 AMS1117-3.3, U7 TPS3850G12QDRCRQ1

Commit message: more
Parts:
- removed C26: 2.7nF, Capacitor_SMD:C_0805_2012Metric_Pad1.18x1.45mm_HandSolder
- removed C73: 1uF, Capacitor_SMD:C_1206_3216Metric_Pad1.33x1.80mm_HandSolder
- removed R14: 470R, Resistor_SMD:R_0805_2012Metric_Pad1.20x1.40mm_HandSolder
- added C109: 100nF, Capacitor_SMD:C_0603_1608Metric_Pad1.08x0.95mm_HandSolder, F.Cu at (195.7, 91.2)
- added C110: 22uF, Capacitor_SMD:C_1206_3216Metric_Pad1.33x1.80mm_HandSolder, F.Cu at (198.3, 111.9)
- added C111: 22uF, Capacitor_SMD:C_1206_3216Metric_Pad1.33x1.80mm_HandSolder, F.Cu at (198.3, 118.0)
- added C112: 1uF, Capacitor_SMD:C_1206_3216Metric_Pad1.33x1.80mm_HandSolder, F.Cu at (200.8, 130.2)
- added C113: 10uF, Capacitor_SMD:C_0805_2012Metric_Pad1.18x1.45mm_HandSolder, F.Cu at (207.7, 129.8)
- added C114: 100nF, Capacitor_SMD:C_0603_1608Metric_Pad1.08x0.95mm_HandSolder, F.Cu at (164.1, 107.4)
- added C115: 10uF, Capacitor_SMD:C_0805_2012Metric_Pad1.18x1.45mm_HandSolder, F.Cu at (54.6, 103.5)
- added C116: 10uF, Capacitor_SMD:C_0805_2012Metric_Pad1.18x1.45mm_HandSolder, F.Cu at (54.6, 106.5)
- added C117: 4.7nF, Capacitor_SMD:C_0805_2012Metric_Pad1.18x1.45mm_HandSolder, F.Cu at (138.4, 72.1)
- added C118: 100nF, Capacitor_SMD:C_0603_1608Metric_Pad1.08x0.95mm_HandSolder, F.Cu at (186.0, 100.1)
- added C119: 10nF, Capacitor_SMD:C_0805_2012Metric_Pad1.18x1.45mm_HandSolder, F.Cu at (190.6, 99.9)
- added C120: 100nF, Capacitor_SMD:C_0603_1608Metric_Pad1.08x0.95mm_HandSolder, F.Cu at (191.1, 110.5)
- added C121: 100nF, Capacitor_SMD:C_0603_1608Metric_Pad1.08x0.95mm_HandSolder, F.Cu at (191.2, 116.5)
- added C122: 100nF, Capacitor_SMD:C_0603_1608Metric_Pad1.08x0.95mm_HandSolder, F.Cu at (191.2, 122.5)
- added C123: 100nF, Capacitor_SMD:C_0603_1608Metric_Pad1.08x0.95mm_HandSolder, F.Cu at (48.0, 138.5)
- added C124: 10nF, Capacitor_SMD:C_0805_2012Metric_Pad1.18x1.45mm_HandSolder, F.Cu at (184.4, 135.1)
- added C125: 10nF, Capacitor_SMD:C_0805_2012Metric_Pad1.18x1.45mm_HandSolder, F.Cu at (184.4, 141.4)
- added C126: 10nF, Capacitor_SMD:C_0805_2012Metric_Pad1.18x1.45mm_HandSolder, F.Cu at (184.4, 147.7)
- added C127: 10nF, Capacitor_SMD:C_0805_2012Metric_Pad1.18x1.45mm_HandSolder, F.Cu at (189.0, 135.1)
- added C128: 10nF, Capacitor_SMD:C_0805_2012Metric_Pad1.18x1.45mm_HandSolder, F.Cu at (189.0, 141.4)
- added C129: 10nF, Capacitor_SMD:C_0805_2012Metric_Pad1.18x1.45mm_HandSolder, F.Cu at (189.0, 147.7)
- added C130: 10nF, Capacitor_SMD:C_0805_2012Metric_Pad1.18x1.45mm_HandSolder, F.Cu at (193.6, 135.1)
- added C131: 10nF, Capacitor_SMD:C_0805_2012Metric_Pad1.18x1.45mm_HandSolder, F.Cu at (193.6, 141.4)
- added C132: 10nF, Capacitor_SMD:C_0805_2012Metric_Pad1.18x1.45mm_HandSolder, F.Cu at (193.6, 147.7)
- added C133: 10nF, Capacitor_SMD:C_0805_2012Metric_Pad1.18x1.45mm_HandSolder, F.Cu at (236.5, 94.6)
- added C134: 1uF, Capacitor_SMD:C_1206_3216Metric_Pad1.33x1.80mm_HandSolder, F.Cu at (207.7, 135.5)
- added C135: 1uF, Capacitor_SMD:C_1206_3216Metric_Pad1.33x1.80mm_HandSolder, F.Cu at (207.7, 143.3)
- added C136: 10uF, Capacitor_SMD:C_0805_2012Metric_Pad1.18x1.45mm_HandSolder, F.Cu at (207.1, 145.6)
- added D1: 1N5819, Diode_THT:D_DO-41_SOD81_P10.16mm_Horizontal, F.Cu at (195.4, 73.5)
- added D2: 1N4148W, Diode_SMD:D_SOD-123, F.Cu at (174.1, 86.9)
- added D3: 1N4148W, Diode_SMD:D_SOD-123, F.Cu at (163.9, 86.8)
- added D4: 1N4148W, Diode_SMD:D_SOD-123, F.Cu at (166.6, 138.8)
- added D5: 1N4148W, Diode_SMD:D_SOD-123, F.Cu at (177.2, 126.8)
- added D6: RED, LED_SMD:LED_0805_2012Metric_Pad1.15x1.40mm_HandSolder, F.Cu at (105.0, 82.8)
- added D7: 1N4148W, Diode_SMD:D_SOD-123, F.Cu at (124.5, 146.2)
- added F1: 3A fast, Fuse:Fuse_1206_3216Metric_Pad1.42x1.75mm_HandSolder, F.Cu at (205.5, 67.5)
- added G***: LOGO, Custom:cuteyeyes, F.Cu at (246.9, 118.8)
- added G***: LOGO, Custom:LOGONEW, F.Cu at (148.6, 67.0)
- added H1: M3, MountingHole:MountingHole_3.2mm_M3, F.Cu at (117.6, 65.5)
- added H2: M3, MountingHole:MountingHole_3.2mm_M3, F.Cu at (210.8, 65.5)
- added H3: M3, MountingHole:MountingHole_3.2mm_M3, F.Cu at (117.6, 158.6)
- added H4: M3, MountingHole:MountingHole_3.2mm_M3, F.Cu at (210.7, 158.6)
- added J7: + 12V TRIG -, Connector_JST:JST_XH_B2B-XH-A_1x02_P2.50mm_Vertical, F.Cu at (118.3, 145.7)
- added J8: UART0, Connector_PinHeader_2.54mm:PinHeader_1x03_P2.54mm_Vertical, F.Cu at (138.9, 130.2)
- added J9: + 12V TRIG -, Connector_JST:JST_XH_B2B-XH-A_1x02_P2.50mm_Vertical, F.Cu at (118.3, 135.0)
- added K2: AGN2004H, SPD:Relay_DPDT_Panasonic_AGN2004H, F.Cu at (177.6, 83.6)
- added K3: AGN2004H, SPD:Relay_DPDT_Panasonic_AGN2004H, F.Cu at (167.2, 83.5)
- added Q2: BC546, Package_TO_SOT_THT:TO-92_Wide, F.Cu at (158.5, 74.2)
- added Q3: BC546, Package_TO_SOT_THT:TO-92_Wide, F.Cu at (158.5, 81.3)
- added Q4: BC546, Package_TO_SOT_THT:TO-92_Wide, F.Cu at (158.7, 131.9)
- added R23: 4R7, Resistor_SMD:R_0805_2012Metric_Pad1.20x1.40mm_HandSolder, F.Cu at (196.0, 111.4)
- added R24: 4R7, Resistor_SMD:R_0805_2012Metric_Pad1.20x1.40mm_HandSolder, F.Cu at (196.0, 117.4)
- added R25: 4K7, Resistor_SMD:R_0805_2012Metric_Pad1.20x1.40mm_HandSolder, F.Cu at (180.4, 79.2)
- added R26: 4K7, Resistor_SMD:R_0805_2012Metric_Pad1.20x1.40mm_HandSolder, F.Cu at (171.6, 79.2)
- added R27: 16R, Resistor_SMD:R_0805_2012Metric_Pad1.20x1.40mm_HandSolder, F.Cu at (178.5, 86.7)
- added R28: 1K, Resistor_SMD:R_0805_2012Metric_Pad1.20x1.40mm_HandSolder, F.Cu at (151.1, 77.7)
- added R29: 16R, Resistor_SMD:R_0805_2012Metric_Pad1.20x1.40mm_HandSolder, F.Cu at (168.2, 86.6)
- added R30: 1K, Resistor_SMD:R_0805_2012Metric_Pad1.20x1.40mm_HandSolder, F.Cu at (151.1, 82.8)
- added R31: 100K, Resistor_SMD:R_0805_2012Metric_Pad1.20x1.40mm_HandSolder, F.Cu at (14.8, 139.3)
- added R32: 22R DNP, Resistor_SMD:R_0805_2012Metric_Pad1.20x1.40mm_HandSolder, F.Cu at (19.6, 82.7)
- added R33: 100K, Resistor_SMD:R_0805_2012Metric_Pad1.20x1.40mm_HandSolder, F.Cu at (159.4, 101.2)
- added R34: 22R, Resistor_SMD:R_0805_2012Metric_Pad1.20x1.40mm_HandSolder, F.Cu at (124.9, 107.3)
- added R35: 22R, Resistor_SMD:R_0805_2012Metric_Pad1.20x1.40mm_HandSolder, F.Cu at (124.9, 109.2)
- added R36: 22R, Resistor_SMD:R_0805_2012Metric_Pad1.20x1.40mm_HandSolder, F.Cu at (135.4, 123.4)
- added R37: 22R, Resistor_SMD:R_0805_2012Metric_Pad1.20x1.40mm_HandSolder, F.Cu at (139.2, 97.4)
- added R38: 2K, Resistor_SMD:R_0805_2012Metric_Pad1.20x1.40mm_HandSolder, F.Cu at (158.1, 150.8)
- added R39: 6K8, Resistor_SMD:R_0805_2012Metric_Pad1.20x1.40mm_HandSolder, F.Cu at (160.2, 150.8)
- added R40: 100K, Resistor_SMD:R_0805_2012Metric_Pad1.20x1.40mm_HandSolder, F.Cu at (24.3, 82.7)
- added R41: 10K, Resistor_SMD:R_0805_2012Metric_Pad1.20x1.40mm_HandSolder, F.Cu at (170.0, 149.7)
- added R42: 100K, Resistor_SMD:R_0805_2012Metric_Pad1.20x1.40mm_HandSolder, F.Cu at (150.5, 140.8)
- added R43: 1K, Resistor_SMD:R_0805_2012Metric_Pad1.20x1.40mm_HandSolder, F.Cu at (150.5, 134.5)
- added R44: 470R, Resistor_SMD:R_0805_2012Metric_Pad1.20x1.40mm_HandSolder, F.Cu at (151.8, 99.1)
- added R45: 1M, Resistor_SMD:R_0805_2012Metric_Pad1.20x1.40mm_HandSolder, F.Cu at (140.5, 72.2)
- added R46: 0R, Resistor_SMD:R_0805_2012Metric_Pad1.20x1.40mm_HandSolder, F.Cu at (127.0, 81.7)
- added R47: 0R, Resistor_SMD:R_0805_2012Metric_Pad1.20x1.40mm_HandSolder, F.Cu at (133.3, 81.8)
- added R48: 22K, Resistor_SMD:R_0805_2012Metric_Pad1.20x1.40mm_HandSolder, F.Cu at (173.3, 128.4)
- added R49: 3K3, Resistor_SMD:R_0805_2012Metric_Pad1.20x1.40mm_HandSolder, F.Cu at (173.3, 126.4)
- added R50: 100K, Resistor_SMD:R_0805_2012Metric_Pad1.20x1.40mm_HandSolder, F.Cu at (178.7, 132.3)
- added R51: 270K, Resistor_SMD:R_0805_2012Metric_Pad1.20x1.40mm_HandSolder, F.Cu at (188.5, 99.9)
- added R52: 10K, Resistor_SMD:R_0805_2012Metric_Pad1.20x1.40mm_HandSolder, F.Cu at (189.5, 102.9)
- added R53: 100K, Resistor_SMD:R_0805_2012Metric_Pad1.20x1.40mm_HandSolder, F.Cu at (42.6, 145.2)
- added R54: 100R, Resistor_SMD:R_0805_2012Metric_Pad1.20x1.40mm_HandSolder, F.Cu at (124.6, 112.7)
- added R55: 100R, Resistor_SMD:R_0805_2012Metric_Pad1.20x1.40mm_HandSolder, F.Cu at (124.6, 114.7)
- added R56: 4K7, Resistor_SMD:R_0805_2012Metric_Pad1.20x1.40mm_HandSolder, F.Cu at (229.8, 129.4)
- added R57: 4K7, Resistor_SMD:R_0805_2012Metric_Pad1.20x1.40mm_HandSolder, F.Cu at (229.8, 132.3)
- added R58: 10K, Resistor_SMD:R_0805_2012Metric_Pad1.20x1.40mm_HandSolder, F.Cu at (184.4, 130.9)
- added R59: 10K, Resistor_SMD:R_0805_2012Metric_Pad1.20x1.40mm_HandSolder, F.Cu at (184.4, 133.0)
- added R60: 10K, Resistor_SMD:R_0805_2012Metric_Pad1.20x1.40mm_HandSolder, F.Cu at (184.4, 137.2)
- added R61: 10K, Resistor_SMD:R_0805_2012Metric_Pad1.20x1.40mm_HandSolder, F.Cu at (184.4, 139.3)
- added R62: 10K, Resistor_SMD:R_0805_2012Metric_Pad1.20x1.40mm_HandSolder, F.Cu at (184.4, 143.5)
- added R63: 10K, Resistor_SMD:R_0805_2012Metric_Pad1.20x1.40mm_HandSolder, F.Cu at (184.4, 145.6)
- added R64: 10K, Resistor_SMD:R_0805_2012Metric_Pad1.20x1.40mm_HandSolder, F.Cu at (189.0, 130.9)
- added R65: 10K, Resistor_SMD:R_0805_2012Metric_Pad1.20x1.40mm_HandSolder, F.Cu at (189.0, 133.0)
- added R66: 10K, Resistor_SMD:R_0805_2012Metric_Pad1.20x1.40mm_HandSolder, F.Cu at (189.0, 137.2)
- added R67: 10K, Resistor_SMD:R_0805_2012Metric_Pad1.20x1.40mm_HandSolder, F.Cu at (189.0, 139.3)
- added R68: 10K, Resistor_SMD:R_0805_2012Metric_Pad1.20x1.40mm_HandSolder, F.Cu at (189.0, 143.5)
- added R69: 10K, Resistor_SMD:R_0805_2012Metric_Pad1.20x1.40mm_HandSolder, F.Cu at (189.0, 145.6)
- added R70: 10K, Resistor_SMD:R_0805_2012Metric_Pad1.20x1.40mm_HandSolder, F.Cu at (193.6, 130.9)
- added R71: 10K, Resistor_SMD:R_0805_2012Metric_Pad1.20x1.40mm_HandSolder, F.Cu at (193.6, 133.0)
- added R72: 10K, Resistor_SMD:R_0805_2012Metric_Pad1.20x1.40mm_HandSolder, F.Cu at (193.6, 137.2)
- added R73: 10K, Resistor_SMD:R_0805_2012Metric_Pad1.20x1.40mm_HandSolder, F.Cu at (193.6, 139.3)
- added R74: 10K, Resistor_SMD:R_0805_2012Metric_Pad1.20x1.40mm_HandSolder, F.Cu at (193.6, 143.5)
- added R75: 10K, Resistor_SMD:R_0805_2012Metric_Pad1.20x1.40mm_HandSolder, F.Cu at (193.6, 145.6)
- added R76: 1K, Resistor_SMD:R_0805_2012Metric_Pad1.20x1.40mm_HandSolder, F.Cu at (105.0, 65.0)
- added R77: 680R, Resistor_SMD:R_0805_2012Metric_Pad1.20x1.40mm_HandSolder, F.Cu at (105.0, 68.0)
- added R78: 4K7, Resistor_SMD:R_0805_2012Metric_Pad1.20x1.40mm_HandSolder, F.Cu at (119.3, 150.0)
- added R79: 10K, Resistor_SMD:R_0805_2012Metric_Pad1.20x1.40mm_HandSolder, F.Cu at (127.6, 146.3)
- added R80: 10K, Resistor_SMD:R_0805_2012Metric_Pad1.20x1.40mm_HandSolder, F.Cu at (235.3, 86.2)
- added TP1: +15V, TestPoint:TestPoint_Pad_D1.5mm, F.Cu at (196.8, 80.9)
- added TP10: INPUT_SEL, TestPoint:TestPoint_Pad_D1.5mm, F.Cu at (34.2, 128.6)
- added TP11: I2S_BCK, TestPoint:TestPoint_Pad_D1.5mm, F.Cu at (44.3, 112.8)
- added TP12: I2S_LRCK, TestPoint:TestPoint_Pad_D1.5mm, F.Cu at (44.3, 116.3)
- added TP13: I2S_DIN, TestPoint:TestPoint_Pad_D1.5mm, F.Cu at (47.9, 112.8)
- added TP14: I2S_DOUT, TestPoint:TestPoint_Pad_D1.5mm, F.Cu at (138.0, 151.8)
- added TP15: DAC_XSMT, TestPoint:TestPoint_Pad_D1.5mm, F.Cu at (51.4, 112.8)
- added TP16: DAC_OUT, TestPoint:TestPoint_Pad_D1.5mm, F.Cu at (156.1, 145.0)
- added TP17: AMP_OUT, TestPoint:TestPoint_Pad_D1.5mm, F.Cu at (156.2, 157.7)
- added TP18: FAULT_N, TestPoint:TestPoint_Pad_D1.5mm, F.Cu at (174.3, 119.6)
- added TP19: SUP_RST_N, TestPoint:TestPoint_Pad_D1.5mm, F.Cu at (182.2, 125.9)
- added TP2: +5V, TestPoint:TestPoint_Pad_D1.5mm, F.Cu at (210.6, 89.8)
- added TP20: RLY_EN_LATCH, TestPoint:TestPoint_Pad_D1.5mm, F.Cu at (57.9, 129.0)
- added TP21: AUDIO_READY, TestPoint:TestPoint_Pad_D1.5mm, F.Cu at (57.9, 132.5)
- added TP22: WDI, TestPoint:TestPoint_Pad_D1.5mm, F.Cu at (165.1, 127.3)
- added TP23: MODE_TRIG_N, TestPoint:TestPoint_Pad_D1.5mm, F.Cu at (184.0, 54.7)
- added TP24: ESP_EN, TestPoint:TestPoint_Pad_D1.5mm, F.Cu at (55.0, 116.3)
- added TP26: +5V_UI, TestPoint:TestPoint_Pad_D1.5mm, F.Cu at (210.3, 150.1)
- added TP3: +3V3_ESP, TestPoint:TestPoint_Pad_D1.5mm, F.Cu at (186.6, 105.5)
- added TP4: +3V3_DAC, TestPoint:TestPoint_Pad_D1.5mm, F.Cu at (210.9, 107.1)
- added TP5: +3V3_A_ADC, TestPoint:TestPoint_Pad_D1.5mm, F.Cu at (211.1, 116.2)
- added TP6: +3V3_D_ADC, TestPoint:TestPoint_Pad_D1.5mm, F.Cu at (211.2, 122.3)
- added TP7: +3V3_UI, TestPoint:TestPoint_Pad_D1.5mm, F.Cu at (211.5, 129.7)
- added TP9: GND, TestPoint:TestPoint_THTPad_2.0x2.0mm_Drill1.0mm, F.Cu at (172.9, 144.1)
- added U10: TPS3808G33DBVR, Package_TO_SOT_SMD:SOT-23-6, F.Cu at (188.1, 110.5)
- added U11: TPS3808G33DBVR, Package_TO_SOT_SMD:SOT-23-6, F.Cu at (188.1, 116.6)
- added U12: TPS3808G33DBVR, Package_TO_SOT_SMD:SOT-23-6, F.Cu at (188.1, 122.6)
- added U13: SN74AUP1G74DCUR, Package_SO:VSSOP-8_2.3x2mm_P0.5mm, F.Cu at (53.8, 143.9)
- added U14: VO617A-3, Package_DIP:DIP-4_W7.62mm, F.Cu at (124.5, 139.1)
- added U15: AP2205-50Y-13, Package_TO_SOT_SMD:SOT-89-3, F.Cu at (208.0, 139.4)
- added U8: TPS7A2033, Package_TO_SOT_SMD:SOT-23-5, F.Cu at (204.4, 129.6)
- added U9: TPS3808G01DBVR, Package_TO_SOT_SMD:SOT-23-6, F.Cu at (183.0, 100.2)
- C1, C2: value 10uF -> 10uF NP
- C100, C99: value 1uF -> 10uF
- C19: value 2.2uF -> 1uF; footprint Capacitor_SMD:C_0805_2012Metric_Pad1.18x1.45mm_HandSolder -> Capacitor_SMD:C_1206_3216Metric_Pad1.33x1.80mm_HandSolder
- C21: value 2.2uF -> 10uF
- C23, C32, C66, C67, C68, C70, C71, C74, C75, C8: footprint Capacitor_SMD:C_1206_3216Metric_Pad1.33x1.80mm_HandSolder -> Capacitor_SMD:C_0603_1608Metric_Pad1.08x0.95mm_HandSolder
- C5: value 1uF -> 100nF; footprint Capacitor_SMD:C_1206_3216Metric_Pad1.33x1.80mm_HandSolder -> Capacitor_SMD:C_0603_1608Metric_Pad1.08x0.95mm_HandSolder
- C72, C76: value 1uF -> 10uF; footprint Capacitor_SMD:C_1206_3216Metric_Pad1.33x1.80mm_HandSolder -> Capacitor_SMD:C_0805_2012Metric_Pad1.18x1.45mm_HandSolder
- C77: value 10uF -> 22uF; footprint Capacitor_SMD:C_0805_2012Metric_Pad1.18x1.45mm_HandSolder -> Capacitor_SMD:C_1206_3216Metric_Pad1.33x1.80mm_HandSolder
- IC1: value ESP32-S3-WROOM-1U-N16R8 -> ESP32-S3-WROOM-1U-N8; footprint Custom:ESP32S3WROOM1UN16R8 -> SPD:ESP32S3WROOM1UN16R8
- IC2: footprint Custom:SOP50P640X120-30N -> SPD:SOP50P640X120-30N
- IC3: footprint Package_TO_SOT_SMD:SOT-23-6_Handsoldering -> Package_TO_SOT_SMD:SOT-23-6
- IC4, IC5: footprint Custom:TS026650BK100SCRD -> SPD:TS026650BK100SCRD
- J1: value PreAmp In -> PREAMP IN
- J2: value LFE In -> MARANTZ LFE IN
- J3: value USB PROGRAMMING -> USB-B; footprint Custom:USBC -> Connector_USB:USB_B_OST_USB-B1HSxx_Horizontal
- J4: value POWER -> POWER IN
- J5: value OUT -> + OUT -
- J6: value SYSTEM CONNECTOR -> FRONT PANEL CONNECTOR
- K1: footprint Custom:Relay_DPDT_Panasonic_AGN2004H -> SPD:Relay_DPDT_Panasonic_AGN2004H
- L3: footprint Custom:SRP6030WA-6R8M -> SPD:SRP6030WA-6R8M
- R15, R16: value 10K -> 100K
- R5, R6: footprint Resistor_SMD:R_0603_1608Metric_Pad0.98x0.95mm_HandSolder -> Resistor_SMD:R_0805_2012Metric_Pad1.20x1.40mm_HandSolder
- U3: value LMR51430 -> LMR51430XFDDCR
- U6: value AMS1117-3.3 -> TS1117BCW33
- U7: value TPS3850G12QDRCRQ1 -> TPS3850H01DRCR; footprint Custom:DRC0010R -> Package_SON:VSON-10-1EP_3x3mm_P0.5mm_EP1.65x2.4mm
- moved R21 249.8 mm to (19.6, 76.8)
- moved C77 223.6 mm to (21.5, 102.6)
- moved C5 203.8 mm to (15.5, 85.9)
- moved C75 198.3 mm to (21.5, 99.3)
- moved C23 150.2 mm to (15.5, 92.6)
- moved C24 150.2 mm to (15.5, 95.9)
- moved C66 150.2 mm to (15.5, 99.3)
- moved C70 145.9 mm to (21.5, 85.9)
- moved C71 145.9 mm to (21.5, 89.2)
- moved C33 145.6 mm to (210.7, 95.4), turned to -90 degrees
- moved U5 143.8 mm to (204.3, 123.5)
- moved U4 143.8 mm to (204.3, 117.4)
- moved U1 143.7 mm to (204.2, 111.3)
- moved C34 143.7 mm to (208.3, 95.4), turned to -90 degrees
- moved L3 138.7 mm to (202.4, 93.9)
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Connections:
- net /ADCESPDAC/3V3_A_ADC renamed +3V3_A_ADC
- net /ADCESPDAC/3V3_D_ADC renamed +3V3_D_ADC
- net /ADCESPDAC/EN renamed /ADCESPDAC/ESP_EN
- net /ADCESPDAC/XSMT renamed /ADCESPDAC/DAC_XSMT
- net Net-(IC2-LDO) renamed /ADCESPDAC/ADC_LDO
- net Net-(IC2-VREF) renamed /ADCESPDAC/ADC_VREF
- C1 pad 1: /ADCESPDAC/IN-LEFT -> /IN-LEFT
- C100 pad 1: /POWER/VCC -> +15V
- C101 pad 1: /POWER/5V-PRE -> Net-(U1-EN)
- C102 pad 1: /ADCESPDAC/3V3_DAC -> +3V3_DAC
- C103 pad 1: /POWER/5V-PRE -> Net-(U4-EN)
- C105 pad 1: /POWER/5V-PRE -> +5V
- C107 pad 1: /POWER/5V-PRE -> +5V
- C108 pad 1: /ADCESPDAC/3V3_ESP -> +3V3_ESP
- C2 pad 1: /ADCESPDAC/IN-RIGHT -> /IN-RIGHT
- C25 pad 1: Net-(K1A-NO) -> Net-(C25-Pad1)
- C33 pad 1: /POWER/5V-PRE -> +5V
- C34 pad 1: /POWER/5V-PRE -> +5V
- C6 pad 1: /POWER/VCC -> +15V
- C66 pad 1: /ADCESPDAC/3V3-DAC -> +3V3_DAC
- C69 pad 1: /ADCESPDAC/3V3-DAC -> +3V3_DAC
- C70 pad 1: /ADCESPDAC/3V3-DAC -> +3V3_DAC
- C71 pad 1: /ADCESPDAC/3V3-DAC -> +3V3_DAC
- C75 pad 1: /ADCESPDAC/3V3_ESP -> +3V3_ESP
- C77 pad 1: /ADCESPDAC/3V3_ESP -> +3V3_ESP
- C8 pad 1: /PROTECT/3V3_ESP -> +3V3_ESP
- C99 pad 1: /POWER/VCC -> +15V
- IC1 pad 10: /ADCESPDAC/USB-VBUS-SENSE -> /ADCESPDAC/USB_VBUS_SENSE
- IC1 pad 11: unconnected-(IC1-IO18-Pad11) -> /ENC2_B
- IC1 pad 12: unconnected-(IC1-IO8-Pad12) -> /ENC2_SW
- IC1 pad 13: /ADCESPDAC/USB-D- -> /ADCESPDAC/USB_DM
- IC1 pad 14: /ADCESPDAC/USB-D+ -> /ADCESPDAC/USB_DP
- IC1 pad 15: unconnected-(IC1-IO3-Pad15) -> /ADCESPDAC/OUT_RLY_SENSE
- IC1 pad 16: unconnected-(IC1-IO46-Pad16) -> /STATUS_LED
- IC1 pad 18: /ADCESPDAC/I2S_BCK -> /ADCESPDAC/I2S_BCK_ESP
- IC1 pad 19: /ADCESPDAC/I2S_LRCK -> /ADCESPDAC/I2S_LRCK_ESP
- IC1 pad 2: /ADCESPDAC/3V3_ESP -> +3V3_ESP
- IC1 pad 22: unconnected-(IC1-IO14-Pad22) -> /UI_SDA
- IC1 pad 23: unconnected-(IC1-IO21-Pad23) -> /UI_SCL
- IC1 pad 24: unconnected-(IC1-IO47-Pad24) -> /MODE_TRIG_N
- IC1 pad 25: unconnected-(IC1-IO48-Pad25) -> /ADCESPDAC/ADC_INT
- IC1 pad 26: unconnected-(IC1-IO45-Pad26) -> /INPUT_SEL
- IC1 pad 31: /ADCESPDAC/I2S_DOUT -> /ADCESPDAC/I2S_DOUT_ESP
- IC1 pad 32: unconnected-(IC1-IO39-Pad32) -> /ENC3_A
- IC1 pad 33: unconnected-(IC1-IO40-Pad33) -> /ENC3_B
- IC1 pad 34: unconnected-(IC1-IO41-Pad34) -> /ENC3_SW
- IC1 pad 35: unconnected-(IC1-IO42-Pad35) -> /FAULT_N
- IC1 pad 36: /ADCESPDAC/RX -> /DBG_RX
- IC1 pad 37: /ADCESPDAC/TX -> /DBG_TX
- IC1 pad 38: /ADCESPDAC/WATCHDOG_HEARTBEAT -> /WATCHDOG_HEARTBEAT
- IC1 pad 4: unconnected-(IC1-IO4-Pad4) -> /ENC1_A
- IC1 pad 5: unconnected-(IC1-IO5-Pad5) -> /ENC1_B
- IC1 pad 6: unconnected-(IC1-IO6-Pad6) -> /ENC1_SW
- IC1 pad 8: unconnected-(IC1-IO15-Pad8) -> /ENC2_A
- IC1 pad 9: /ADCESPDAC/AUDIO-READY -> /AUDIO_READY
- IC2 pad 10: unconnected-(IC2-XI-Pad10) -> GND
- IC2 pad 15: /ADCESPDAC/I2S_SCLK -> /ADCESPDAC/ADC_SCKI
- IC2 pad 18: /ADCESPDAC/I2S_DIN -> Net-(IC2-DOUT)
- IC2 pad 19: /ADCESPDAC/INTC -> /ADCESPDAC/ADC_INT
- IC3 pad 1: /ADCESPDAC/USB-D- -> Net-(IC3-I/O1_1)
- IC3 pad 3: /ADCESPDAC/USB-D+ -> Net-(IC3-I/O2_1)
- IC3 pad 5: /ADCESPDAC/USB-VBUS -> /ADCESPDAC/USB_VBUS
- J1 pad 1: unconnected-(J1-Pin_1-Pad1) -> /AUDIO-IN/PRE_L
- J1 pad 2: unconnected-(J1-Pin_2-Pad2) -> /AUDIO-IN/PRE_GND
- J1 pad 3: unconnected-(J1-Pin_3-Pad3) -> /AUDIO-IN/PRE_R
- J2 pad 1: unconnected-(J2-Pin_1-Pad1) -> /AUDIO-IN/LFE
- J2 pad 2: unconnected-(J2-Pin_2-Pad2) -> /AUDIO-IN/LFE_GND
- J3 pad 1: /ADCESPDAC/USB-VBUS -> /ADCESPDAC/USB_VBUS
- J3 pad 2: Net-(IC3-I/O1_2) -> Net-(IC3-I/O1_1)
- J3 pad 3: Net-(IC3-I/O2_2) -> Net-(IC3-I/O2_1)
- J4 pad 3: /POWER/VCC -> Net-(J4-Pin_3)
- J6 pad 1: (no net) -> +3V3_UI
- J6 pad 10: (no net) -> GND
- J6 pad 11: (no net) -> /CONTROL/ENC2_A_C
- J6 pad 12: (no net) -> /CONTROL/ENC2_B_C
- J6 pad 13: (no net) -> /CONTROL/ENC2_SW_C
- J6 pad 14: (no net) -> GND
- J6 pad 15: (no net) -> /CONTROL/ENC3_A_C
- J6 pad 16: (no net) -> /CONTROL/ENC3_B_C
- J6 pad 17: (no net) -> /CONTROL/ENC3_SW_C
- J6 pad 18: (no net) -> GND
- J6 pad 19: (no net) -> /CONTROL/UI_LED_C
- J6 pad 2: (no net) -> GND
- J6 pad 20: (no net) -> +5V_UI
- J6 pad 3: (no net) -> /CONTROL/UI_SDA_C
- J6 pad 4: (no net) -> GND
- J6 pad 5: (no net) -> /CONTROL/UI_SCL_C
- J6 pad 6: (no net) -> GND
- J6 pad 7: (no net) -> /CONTROL/ENC1_A_C
- J6 pad 8: (no net) -> /CONTROL/ENC1_B_C
- J6 pad 9: (no net) -> /CONTROL/ENC1_SW_C
- K1 pad 1: Net-(K1C-COIL+) -> Net-(D4-K)
- K1 pad 5: (no net) -> /ADCESPDAC/OUT_RLY_SENSE
- K1 pad 6: (no net) -> GND
- K1 pad 7: (no net) -> unconnected-(K1B-NC-Pad7)
- L3 pad 2: /POWER/5V-PRE -> +5V
- Q1 pad 3: GND -> Net-(Q1-E)
- R1 pad 1: /ADCESPDAC/3V3-ESP -> +3V3_ESP
- R10 pad 1: Net-(U7-RESET_N) -> +3V3_ESP
- R10 pad 2: /PROTECT/3V3_ESP -> /SUP_RST_N
- R11 pad 1: Net-(U7-WDO_N) -> +3V3_ESP
- R11 pad 2: /PROTECT/3V3_ESP -> /FAULT_N
- R13 pad 2: Net-(K1A-NO) -> Net-(C25-Pad1)
- R15 pad 1: /ADCESPDAC/USB-VBUS-SENSE -> /ADCESPDAC/USB_VBUS
- R15 pad 2: /ADCESPDAC/USB-VBUS -> /ADCESPDAC/USB_VBUS_SENSE
- R16 pad 1: GND -> /ADCESPDAC/USB_VBUS_SENSE
- R16 pad 2: /ADCESPDAC/USB-VBUS-SENSE -> GND
- R17 pad 1: /POWER/5V-PRE -> +5V
- R19 pad 1: Net-(K1A-NC) -> GND
- R19 pad 2: GND -> Net-(K1A-NC)
- R2 pad 1: /ADCESPDAC/3V3-ESP -> +3V3_ESP
- R21 pad 1: /ADCESPDAC/AMP_ENABLE -> /RLY_EN_LATCH
- R22 pad 1: Net-(K1C-COIL+) -> +5V
- R22 pad 2: /POWER/5V-PRE -> Net-(D4-K)
- R5 pad 1: /ADCESPDAC/3V3_ESP -> +3V3_ESP
- R6 pad 1: /ADCESPDAC/3V3_ESP -> +3V3_ESP
- R7 pad 1: GND -> /IN-RIGHT
- R7 pad 2: /ADCESPDAC/IN-RIGHT -> GND
- R8 pad 1: GND -> /IN-LEFT
- R8 pad 2: /ADCESPDAC/IN-LEFT -> GND
- R9 pad 1: /PROTECT/3V3_ESP -> +3V3_ESP
- U1 pad 1: /POWER/5V-PRE -> Net-(U1-EN)
- U1 pad 3: /POWER/5V-PRE -> Net-(U1-EN)
- U1 pad 5: /ADCESPDAC/3V3_DAC -> +3V3_DAC
- U2 pad 1: /ADCESPDAC/3V3_DAC -> +3V3_DAC
- U2 pad 11: /ADCESPDAC/3V3_DAC -> +3V3_DAC
- U2 pad 20: /ADCESPDAC/3V3_DAC -> +3V3_DAC
- U2 pad 7: Net-(U2-OUTR) -> unconnected-(U2-OUTR-Pad7)
- U2 pad 8: /ADCESPDAC/3V3_DAC -> +3V3_DAC
- U3 pad 3: /POWER/VCC -> +15V
- U3 pad 5: /POWER/VCC -> +15V
- U4 pad 1: /POWER/5V-PRE -> Net-(U4-EN)
- U4 pad 3: /POWER/5V-PRE -> Net-(U4-EN)
- U5 pad 1: /POWER/5V-PRE -> +5V
- U5 pad 3: /POWER/5V-PRE -> +5V
- U6 pad 2: /ADCESPDAC/3V3_ESP -> +3V3_ESP
- U6 pad 3: /POWER/5V-PRE -> +5V
- U7 pad 1: /PROTECT/3V3_ESP -> +3V3_ESP
- U7 pad 10: /PROTECT/3V3_ESP -> Net-(U7-SENSE)
- U7 pad 6: /PROTECT/3V3_ESP -> +3V3_ESP
- U7 pad 7: /PROTECT/WATCHDOG_HEARTBEAT -> /WATCHDOG_HEARTBEAT
- U7 pad 8: Net-(U7-WDO_N) -> /FAULT_N
- U7 pad 9: Net-(U7-RESET_N) -> /SUP_RST_N
Routing:
- net +3V3_ESP: track 0.00 -> 280.1 mm, vias 0 -> 27
- net +5V: track 0.00 -> 181.3 mm, vias 0 -> 26
- net +3V3_DAC: track 0.00 -> 153.6 mm, vias 0 -> 4
- net +15V: track 0.00 -> 137.7 mm, vias 0 -> 4
- net /ADCESPDAC/I2S_BCK: track 0.00 -> 99.8 mm, vias 0 -> 4
- net /ADCESPDAC/I2S_LRCK: track 0.00 -> 98.1 mm, vias 0 -> 3
- net /FAULT_N: track 0.00 -> 94.9 mm, vias 0 -> 7
- net +3V3_D_ADC: track 0.00 -> 69.7 mm, vias 0 -> 3
- net +3V3_UI: track 0.00 -> 67.7 mm, vias 0 -> 1
- net +3V3_A_ADC: track 0.00 -> 61.4 mm, vias 0 -> 3
- net /SUP_RST_N: track 0.00 -> 56.4 mm
- net /INPUT_SEL: track 0.00 -> 53.4 mm, vias 0 -> 2
- net /WATCHDOG_HEARTBEAT: track 0.00 -> 52.5 mm, vias 0 -> 2
- net /ADCESPDAC/I2C_SCL: track 0.00 -> 43.4 mm, vias 0 -> 2
- net /ADCESPDAC/I2C_SDA: track 0.00 -> 41.8 mm, vias 0 -> 2
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- added copper zone on F.Cu, net GND
- added copper zone on In1.Cu, net GND
Other:
- copper layers 2 -> 4
- board text added: "- +"
- board text added: "Digital Subwoofer Controller Tom Watson Audio - 2026"
- board text added: "NC G +"
- board text added: "R G L"

Commit message: more work
Parts:
- removed J8: UART0, Connector_PinHeader_2.54mm:PinHeader_1x03_P2.54mm_Vertical
- added C137: 4.7nF, Capacitor_SMD:C_0805_2012Metric_Pad1.18x1.45mm_HandSolder, F.Cu at (154.9, 74.1)
- added C138: 4.7nF, Capacitor_SMD:C_0805_2012Metric_Pad1.18x1.45mm_HandSolder, F.Cu at (156.1, 81.4)
- added C139: 10uF NP, Capacitor_THT:C_Radial_D8.0mm_H11.5mm_P3.50mm, F.Cu at (151.2, 88.6)
- added C140: 10nF, Capacitor_SMD:C_0805_2012Metric_Pad1.18x1.45mm_HandSolder, F.Cu at (160.4, 89.7)
- added C141: 4.7nF, Capacitor_SMD:C_0805_2012Metric_Pad1.18x1.45mm_HandSolder, F.Cu at (143.3, 74.1)
- added C142: 4.7nF, Capacitor_SMD:C_0805_2012Metric_Pad1.18x1.45mm_HandSolder, F.Cu at (142.1, 79.6)
- added C143: 10uF NP, Capacitor_THT:C_Radial_D8.0mm_H11.5mm_P3.50mm, F.Cu at (145.9, 88.6)
- added C144: 10nF, Capacitor_SMD:C_0805_2012Metric_Pad1.18x1.45mm_HandSolder, F.Cu at (136.7, 89.6)
- added C145: 100nF, Capacitor_SMD:C_0603_1608Metric_Pad1.08x0.95mm_HandSolder, F.Cu at (154.8, 78.4)
- added C146: 100nF, Capacitor_SMD:C_0603_1608Metric_Pad1.08x0.95mm_HandSolder, F.Cu at (143.4, 82.7)
- added C147: 10uF, Capacitor_SMD:C_1206_3216Metric_Pad1.33x1.80mm_HandSolder, F.Cu at (139.8, 79.0)
- added C148: 10uF, Capacitor_SMD:C_1206_3216Metric_Pad1.33x1.80mm_HandSolder, F.Cu at (158.4, 80.8)
- added D8: 1N4148W, Diode_SMD:D_SOD-123, F.Cu at (188.3, 68.1)
- added F2: 3A fast, Fuse:Fuse_1206_3216Metric_Pad1.42x1.75mm_HandSolder, F.Cu at (191.5, 68.1)
- added J10: HIGH LEVEL IN, Connector_JST:JST_XH_B4B-XH-A_1x04_P2.50mm_Vertical, F.Cu at (152.9, 67.6)
- added J11: ESP, Connector_PinSocket_2.54mm:PinSocket_1x04_P2.54mm_Vertical, F.Cu at (146.7, 126.5)
- added R81: 100K, Resistor_SMD:R_0805_2012Metric_Pad1.20x1.40mm_HandSolder, F.Cu at (152.9, 74.0)
- added R82: 100K, Resistor_SMD:R_0805_2012Metric_Pad1.20x1.40mm_HandSolder, F.Cu at (150.4, 74.1)
- added R83: 10K, Resistor_SMD:R_0805_2012Metric_Pad1.20x1.40mm_HandSolder, F.Cu at (157.0, 74.0)
- added R84: 10K, Resistor_SMD:R_0805_2012Metric_Pad1.20x1.40mm_HandSolder, F.Cu at (154.1, 81.4)
- added R85: 1K, Resistor_SMD:R_0805_2012Metric_Pad1.20x1.40mm_HandSolder, F.Cu at (158.4, 89.7)
- added R86: 100K, Resistor_SMD:R_0805_2012Metric_Pad1.20x1.40mm_HandSolder, F.Cu at (145.3, 74.0)
- added R87: 100K, Resistor_SMD:R_0805_2012Metric_Pad1.20x1.40mm_HandSolder, F.Cu at (147.8, 74.1)
- added R88: 10K, Resistor_SMD:R_0805_2012Metric_Pad1.20x1.40mm_HandSolder, F.Cu at (141.2, 74.1)
- added R89: 10K, Resistor_SMD:R_0805_2012Metric_Pad1.20x1.40mm_HandSolder, F.Cu at (144.1, 79.6)
- added R90: 1K, Resistor_SMD:R_0805_2012Metric_Pad1.20x1.40mm_HandSolder, F.Cu at (138.7, 89.7)
- added TP8: -15V, TestPoint:TestPoint_Pad_D1.5mm, F.Cu at (185.5, 71.5)
- added U16: RC4580, Package_SO:SOIC-8_3.9x4.9mm_P1.27mm, F.Cu at (149.1, 80.5)
- IC2: value PCM1863QDBTRQ1 -> PCM1863
- J3: value USB-B -> USB PROGRAMMING
- Q1, Q2, Q3, Q4: value BC546 -> BC849C; footprint Package_TO_SOT_THT:TO-92_Wide -> Package_TO_SOT_SMD:SOT-23
- U15: value AP2205-50Y-13 -> AP2205-50Y
- U3: value LMR51430XFDDCR -> LMR51430XF
- U6: value TS1117BCW33 -> TS1117-33
- moved R21 145.1 mm to (148.0, 144.4), turned to -90 degrees
- moved C70 141.4 mm to (143.7, 157.1), turned to 180 degrees
- moved C66 140.3 mm to (146.2, 150.2), turned to 90 degrees
- moved C71 135.8 mm to (138.6, 157.9), turned to -90 degrees
- moved C23 135.5 mm to (135.7, 154.9), turned to 180 degrees
- moved C24 134.2 mm to (134.9, 157.0), turned to 180 degrees
- moved R40 131.7 mm to (135.6, 153.2), turned to 180 degrees
- moved C77 127.6 mm to (149.0, 99.3)
- moved C75 124.1 mm to (145.6, 98.8), turned to 90 degrees
- moved R80 117.2 mm to (130.8, 139.3)
- moved C133 114.0 mm to (130.8, 137.3)
- moved C115 104.7 mm to (143.5, 158.9), turned to 180 degrees
- moved C69 103.7 mm to (145.0, 147.5), turned to 180 degrees
- moved C116 96.6 mm to (135.5, 159.3), turned to 180 degrees
- moved U13 89.3 mm to (143.0, 138.3)
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Connections:
- IC2 pad 29: unconnected-(IC2-VINL3/VIN4P-Pad29) -> /HL-LEFT
- IC2 pad 30: unconnected-(IC2-VINR3/VIN3P-Pad30) -> /HL-RIGHT
- J4 pad 1: unconnected-(J4-Pin_1-Pad1) -> Net-(J4-Pin_1)
- Q1 pad 1: Net-(D4-A) -> Net-(Q1-B)
- Q1 pad 2: Net-(Q1-B) -> Net-(Q1-E)
- Q1 pad 3: Net-(Q1-E) -> Net-(D4-A)
- Q2 pad 1: Net-(D2-A) -> Net-(Q2-B)
- Q2 pad 2: Net-(Q2-B) -> GND
- Q2 pad 3: GND -> Net-(D2-A)
- Q3 pad 1: Net-(D3-A) -> Net-(Q3-B)
- Q3 pad 2: Net-(Q3-B) -> GND
- Q3 pad 3: GND -> Net-(D3-A)
- Q4 pad 1: Net-(Q1-E) -> Net-(Q4-B)
- Q4 pad 2: Net-(Q4-B) -> GND
- Q4 pad 3: GND -> Net-(Q1-E)
Routing:
- net +3V3_DAC: track 153.6 -> 48.4 mm
- net /FAULT_N: track 94.9 -> 0.00 mm, vias 7 -> 0
- net /ENC2_B: track 2.93 -> 83.4 mm, vias 0 -> 2
- net /ENC2_SW: track 2.93 -> 80.9 mm, vias 0 -> 2
- net /ENC3_SW: track 2.93 -> 71.9 mm, vias 0 -> 2
- net /ENC2_A: track 2.94 -> 69.3 mm, vias 0 -> 3
- net /ENC1_SW: track 2.93 -> 69.0 mm, vias 0 -> 2
- net /ENC3_B: track 2.93 -> 68.5 mm, vias 0 -> 4
- net /ENC3_A: track 2.93 -> 66.6 mm, vias 0 -> 4
- net /ENC1_B: track 2.94 -> 66.0 mm, vias 0 -> 2
- net +3V3_UI: track 67.7 -> 5.72 mm, vias 1 -> 0
- net /ENC1_A: track 2.94 -> 62.8 mm, vias 0 -> 2
- net -15V: track 0.00 -> 57.4 mm, vias 0 -> 2
- net /SUP_RST_N: track 56.4 -> 0.00 mm
- net +3V3_D_ADC: track 69.7 -> 15.2 mm, vias 3 -> 0
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Other:
- board text added: "- G +"
- board text added: "DNP if high level not needed"
- board text added: "Isolated trigger input and passthrough"
- board text added: "R+ R- L- L+"
- board text removed: "NC G +"
