File: SubProcessorDigital/SubProcessorDigital.kicad_sch (KiCad schematic)
At the start: 0 parts

Commit message: more
Other:
- added sheet CONTROL (CONTROL.kicad_sch)
- sheet ADCESPDAC ports: added AUDIO_READY, DBG_RX, DBG_TX, ENC1_A, ENC1_B, ENC1_SW, ENC2_A, ENC2_B, ENC2_SW, ENC3_A, ENC3_B, ENC3_SW, FAULT_N, INPUT_SEL, MODE_TRIG_N, RLY_EN_LATCH, STATUS_LED, SUP_RST_N, UI_SCL, UI_SDA, WATCHDOG_HEARTBEAT; removed 3V3_A_ADC, 3V3_DAC, 3V3_D_ADC, 3V3_ESP, 5V, AUDIO-TO-AMP, VCC
- sheet AUDIO-IN ports: added INPUT_SEL; removed none
- sheet POWER ports: added none; removed 3V3_A_ADC, 3V3_DAC, 3V3_D_ADC, 3V3_ESP, 5V, VCC
- sheet PROTECT ports: added AUDIO_READY, FAULT_N, RLY_EN_LATCH, SUP_RST_N, WATCHDOG_HEARTBEAT; removed none
- note added: "1-2 blocks + DAC low-latency 3.5/fs. With 32-frame blocks at 48 kHz ~ 2.3-3.0 ms; 16-frame ~ 1.3-1.6 ms. MEASURE."
- note added: "Clocks: ESP32-S3 I2S0 master, full duplex: BCK 3.072 MHz, LRCK 48 kHz. PCM1863 and PCM5102A both use internal BCK-PLLs."
- note added: "DESIGN NOTES (full engineering report: SubProcessorDigital/DESIGN_REVIEW.md)"
- note added: "GPIO: IO1 XSMT, IO2 WDI, IO3 RLY_SENSE, IO4/5/6 ENC1 A/B/SW, IO7 I2S DIN, IO8 ENC2 SW, IO9 MCLK(opt), IO10 BCK, IO11 LRCK,"
- note added: "IO12/13 I2C0 SDA/SCL (ADC), IO14/21 I2C1 SDA/SCL (UI), IO15/18 ENC2 A/B, IO16 AUDIO_READY, IO17 VBUS sense, IO19/20 USB,"
- note added: "IO38 I2S DOUT, IO39/40/41 ENC3 A/B/SW, IO42 FAULT_N in, IO43/44 UART0, IO45 INPUT_SEL, IO46 STATUS_LED, IO47 MODE_TRIG_N,"
- note added: "IO48 ADC_INT. IO35/36/37 unused (PSRAM on N8R8). IO0 BOOT. Wi-Fi/BT unused (U.FL left open)."
- note added: "Latency (fixed, excl. filter group delay): ADC low-latency IIR 10/fs + DMA in 1 block + processing 1 block + DMA out"
- note added: "Power: +15 V -> 1N5819 -> LMR51430 (500 kHz FPWM) -> +5 V -> TPS7A2033 x4 (DAC, ADC-A, ADC-D, UI) + TS1117B (ESP32)."
- note added: "Protection: K1 energises only with latch Q (cleared by any supervisor/watchdog/power fault) AND AUDIO_READY level."
- note added: "Signal: preamp L/R or Marantz LFE -> K2/K3 relays (signal AND source-ground switched) -> 4k7 -> 10u NP -> 100R/10n -> PCM1863."
- company: (none) -> SubProcessorDigital
- title: (none) -> P68 Subwoofer DSP Controller

Commit message: more work
Other:
- sheet ADCESPDAC ports: added HL-LEFT, HL-RIGHT; removed none
- sheet AUDIO-IN ports: added HL-LEFT, HL-RIGHT; removed none
Changed lines of the file:
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@@
+	(wire
+		(pts
+			(xy 127 53.34) (xy 121.92 53.34)
+		)
+		(stroke
+			(width 0)
+			(type default)
+		)
+	)
+	(wire
+		(pts
+			(xy 76.2 88.9) (xy 81.28 88.9)
+		)
+		(stroke
+			(width 0)
+			(type default)
+		)
+	)
 	(wire
 		(pts
@@
 	(wire
 		(pts
+			(xy 127 50.8) (xy 121.92 50.8)
+		)
+		(stroke
+			(width 0)
+			(type default)
+		)
+	)
+	(wire
+		(pts
 			(xy 76.2 83.82) (xy 81.28 83.82)
 		)
@@
 		(pts
 			(xy 187.96 66.04) (xy 193.04 66.04)
+		)
+		(stroke
+			(width 0)
+			(type default)
+		)
+	)
+	(wire
+		(pts
+			(xy 76.2 91.44) (xy 81.28 91.44)
 		)
 		(stroke
@@
 		)
 	)
+	(label "HL-RIGHT"
+		(at 121.92 53.34 180)
+		(effects
+			(font
+				(size 1.27 1.27)
+			)
+			(justify right)
+		)
+	)
 	(label "IN-LEFT"
 		(at 121.92 43.18 180)
@@
 		)
 	)
+	(label "HL-RIGHT"
+		(at 81.28 91.44 0)
+		(effects
+			(font
+				(size 1.27 1.27)
+			)
+			(justify left)
+		)
+	)
 	(label "ENC3_B"
 		(at 193.04 73.66 0)
@@
 		)
 	)
+	(label "HL-LEFT"
+		(at 81.28 88.9 0)
+		(effects
+			(font
+				(size 1.27 1.27)
+			)
+			(justify left)
+		)
+	)
 	(label "WATCHDOG_HEARTBEAT"
 		(at 193.04 45.72 0)
@@
 	(label "SUP_RST_N"
 		(at 259.08 50.8 180)
+		(effects
+			(font
+				(size 1.27 1.27)
+			)
+			(justify right)
+		)
+	)
+	(label "HL-LEFT"
+		(at 121.92 50.8 180)
 		(effects
 			(font
@@
 			)
 		)
+		(pin "HL-LEFT" input
+			(at 127 50.8 180)
+			(effects
+				(font
+					(size 1.27 1.27)
+				)
+				(justify left)
+			)
+		)
+		(pin "HL-RIGHT" input
+			(at 127 53.34 180)
+			(effects
+				(font
+					(size 1.27 1.27)
+				)
+				(justify left)
+			)
+		)
 		(instances
 			(project "SubProcessorDigital"
@@
 			(effects
 				(font
+					(size 1.27 1.27)
+				)
+				(justify right)
+			)
+		)
+		(pin "HL-LEFT" output
+			(at 76.2 88.9 0)
+			(effects
+				(font
+					(size 1.27 1.27)
+				)
+				(justify right)
+			)
+		)
+		(pin "HL-RIGHT" output
+			(at 76.2 91.44 0)
+			(effects
+				(font
