File: TPA3220/Amp.kicad_sch (KiCad schematic)
At the start: 33 parts, among them J16 OUT L, J17 OUT R, U1 TPA3220DDWR

Commit message: more
Parts:
- added C55, C56: 1000uF, Capacitor_THT:CP_Radial_D12.5mm_P5.00mm, symbol Device:C_Polarized
- added C57: 100n, Capacitor_SMD:C_0603_1608Metric_Pad1.08x0.95mm_HandSolder, symbol Device:C
- added C58, C59: 1u, Capacitor_SMD:C_1206_3216Metric_Pad1.33x1.80mm_HandSolder, symbol Device:C
- added C60: 33nF, Capacitor_SMD:C_0805_2012Metric_Pad1.18x1.45mm_HandSolder, symbol Device:C
- added R33: 3R3, Resistor_SMD:R_2512_6332Metric_Pad1.40x3.35mm_HandSolder, symbol Device:R
- added R34: 5K6, Resistor_SMD:R_0805_2012Metric_Pad1.20x1.40mm_HandSolder, symbol Device:R
- added R35: 49K9, Resistor_SMD:R_0805_2012Metric_Pad1.20x1.40mm_HandSolder, symbol Device:R
- added R36: 4k7, Resistor_SMD:R_0805_2012Metric_Pad1.20x1.40mm_HandSolder, symbol Device:R
- C40, C41, C42, C43: footprint Capacitor_SMD:C_1206_3216Metric_Pad1.33x1.80mm_HandSolder -> Capacitor_SMD:C_0603_1608Metric_Pad1.08x0.95mm_HandSolder
- J16: value OUT L -> - OUT R +
- J17: value OUT R -> - OUT L +
- U1: value TPA3220DDWR -> TPA3220
Connections:
- net GND: now also U1.11 (HEAD), C55.2, C56.2, C57.1, C58.2, C59.2, C60.2, R34.1, R35.2, R36.2
- net IN1-M: now also C6.1; no longer C2.1
- net IN1-P: now also C5.1; no longer C1.1
- net IN2-M: now also C2.1; no longer C6.1
- net IN2-P: now also C1.1; no longer C5.1
- net PVDD: now also U1.1 (VDD), C55.1, C56.1, C57.2
- net AMP_RESET_N: now reaches U1.10 (RESET_N)
- net AMP_RESET_N: now also R36.1
- net at U1.14 (FREQ_ADJ): now also R35.1
- net at U1.17 (CMUTE_N): now also C60.1
- net at U1.2 (GAIN_SLV): now also R34.2
- net AMP_AVDD: now reaches U1.21 (AVDD)
- net AMP_AVDD: now also C58.1, R33.1
- net AMP_GVDD: now reaches U1.22 (GVDD)
- net AMP_GVDD: now also C59.1, R33.2
- net AMP_OTW_N: now reaches U1.3 (OTW_CLIP_N)
- net AMP_FAULT_N: now reaches U1.4 (FAULT_N)
- no-connect marks 0 -> 2
Other:
- note added: "L6/L7 CODACA CSAD0660-100M: winding 1-2 and 4-3. Codaca does not publish dot polarity; the KiCad L_Coupled symbol dots are generic. VERIFY on a sample before layout: short pins 2-3, measure L(1-4). ~2x L(1-2) = uncoupled, >2x = aiding (OK), <<2x = opposing (re-wire)."
- note added: "PVDD BULK: C55 at pins 29-31, C56 at pins 36-38"
- note added: "Stereo BTL, AD modulation (HEAD = 0), master (OSCM/OSCP open), gain 18 dB (GAIN/SLV 5.6k to GND, latched on RESET rising edge), fPWM 600 kHz nominal (FREQ_ADJ 49.9k). Input impedance 48k: 1 uF coupling -> 3.3 Hz HPF. Single-ended: INx_M is AC-grounded at the top level - route its GND end back to the DAC output ground. Supplies: VDD = PVDD, internal LDO -> AVDD (1 uF), GVDD via 3R3/1 uF. AVDD must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"
- note added: "TPA3220 AVDD / GVDD (internal LDO, VDD = PVDD)"
- note added: "TPA3220 CONFIGURATION"
