File: TPA3220/DAC.kicad_sch (KiCad schematic)
At the start: 21 parts, among them IC4 TPS7A2033, U2 PCM5122PW

Commit message: more
Parts:
- added R32: 10k, Resistor_SMD:R_0603_1608Metric_Pad0.98x0.95mm_HandSolder, symbol Device:R
Connections:
- net AVDD: no longer U2.25 (XSMT)
- net GND: now also U2.10 (VCOM/DEMP), R32.2
- net DOUT renamed DATA
- net ESP5V renamed 5V
- new net DAC_XSMT: R32.1, U2.25 (XSMT)
- no-connect marks 0 -> 4
Other:
- note added: "I2C mode: MODE1 = 0, MODE2 = 1. Address ADR2 = ADR1 = 0 -> 0x4C (7-bit). SCK tied to GND: 3-wire I2S, PLL referenced to BCK. Firmware must set P0-R13 SRCREF = BCK (0x10) and use BCK = 64 fs (32-bit slots) or 32 fs. Volume: P0-R61/R62 digital volume over I2C (master volume). OUTL -> amp CH1 (woofer), OUTR -> amp CH2 (tweeter); 2.1 Vrms FS, ground-centred. 470R + 2.7 nF output filter = 125 kHz (TI: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"
- note added: "PCM5122 CONFIGURATION"
