File: TPA3220/ESP32.kicad_sch (KiCad schematic)
At the start: 13 parts, among them IC1 ESP32-WROOM-32UE-N8R2, IC2 RESET, IC3 BOOT, J4 PROG

Commit message: more
Parts:
- added C54: 22u, Capacitor_SMD:C_1206_3216Metric_Pad1.33x1.80mm_HandSolder, symbol Device:C
- added R29, R30: 10k, Resistor_SMD:R_0603_1608Metric_Pad0.98x0.95mm_HandSolder, symbol Device:R
- added R31: 10k, Resistor_SMD:R_0603_1608Metric_Pad0.98x0.95mm_HandSolder, symbol Device:R_Small
Connections:
- net 3V3-ESP: now also C3.2, C54.2, R29.1, R30.2, R31.2; no longer C3.1
- net GND: now also C3.1, C54.1
- net at IC1.27 (IO16): now also R31.1
- net VIN_SENSE: now reaches IC1.4 (SENSOR_VP)
- net AMP_OTW_N: now reaches IC1.7 (IO35)
- net AMP_OTW_N: now also R30.1
- net DAC_XSMT: now reaches IC1.9 (IO33)
- net FAULT renamed AMP_FAULT_N
- net AMP_FAULT_N: now also R29.2
- net SDZ renamed AMP_RESET_N
- no-connect marks 0 -> 19
Other:
- note added: "ESP32 I/O MAP"
- note added: "IO25 LRCK, IO26 BCK, IO13 DATA (22R source terminations) -> PCM5122. IO21 SDA, IO22 SCL (4k7 to 3V3) -> PCM5122 @ 0x4C. IO27 AMP_RESET_N -> TPA3220 RESET (4k7 pull-down at amp: reset until driven high). IO33 DAC_XSMT -> PCM5122 XSMT (10k pull-down at DAC: muted until driven high). IO34 AMP_FAULT_N <- TPA3220 FAULT (input-only pin, R29 pull-up). IO35 AMP_OTW_N <- TPA3220 OTW_CLIP: OTW level + ~500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"
- moved on the sheet: C3
