File: TPA3220/TPA3220.kicad_pcb (KiCad board)
At the start: 4 copper layers, 100 x 100 mm, 73 parts, among them IC1 ESP32-WROOM-32UE-N8R2, IC2 RESET, IC3 BOOT, IC4 TPS7A2033, J1 LINE IN, J16 OUT L, J17 OUT R, J4 PROG, U1 TPA3220DDWR, U2 PCM5122PW

Commit message: more
Parts:
- removed C21: 220pF*, Capacitor_SMD:C_0805_2012Metric_Pad1.18x1.45mm_HandSolder
- added C45: 10u/50V, Capacitor_SMD:C_1210_3225Metric_Pad1.33x2.70mm_HandSolder, F.Cu at (38.3, 120.4)
- added C46: 100n, Capacitor_SMD:C_0603_1608Metric_Pad1.08x0.95mm_HandSolder, F.Cu at (43.8, 102.9)
- added C48: 100n, Capacitor_SMD:C_0603_1608Metric_Pad1.08x0.95mm_HandSolder, F.Cu at (43.8, 105.4)
- added C49: 22u/25V, Capacitor_SMD:C_1206_3216Metric_Pad1.33x1.80mm_HandSolder, F.Cu at (38.3, 107.2)
- added C50: 22u/25V, Capacitor_SMD:C_1206_3216Metric_Pad1.33x1.80mm_HandSolder, F.Cu at (38.3, 110.6)
- added C51: 10u, Capacitor_SMD:C_0805_2012Metric_Pad1.18x1.45mm_HandSolder, F.Cu at (37.7, 113.7)
- added C52: 10u, Capacitor_SMD:C_0805_2012Metric_Pad1.18x1.45mm_HandSolder, F.Cu at (37.7, 116.8)
- added C53: 100n, Capacitor_SMD:C_0603_1608Metric_Pad1.08x0.95mm_HandSolder, F.Cu at (43.8, 107.9)
- added C54: 22u, Capacitor_SMD:C_1206_3216Metric_Pad1.33x1.80mm_HandSolder, F.Cu at (71.2, 120.3)
- added C55: 1000uF, Capacitor_THT:CP_Radial_D12.5mm_P5.00mm, F.Cu at (161.2, 137.9)
- added C56: 1000uF, Capacitor_THT:CP_Radial_D12.5mm_P5.00mm, F.Cu at (161.3, 102.1)
- added C57: 100n, Capacitor_SMD:C_0603_1608Metric_Pad1.08x0.95mm_HandSolder, F.Cu at (77.8, 94.7)
- added C58: 1u, Capacitor_SMD:C_1206_3216Metric_Pad1.33x1.80mm_HandSolder, F.Cu at (78.0, 110.0)
- added C59: 1u, Capacitor_SMD:C_1206_3216Metric_Pad1.33x1.80mm_HandSolder, F.Cu at (78.0, 113.1)
- added C60: 33nF, Capacitor_SMD:C_0805_2012Metric_Pad1.18x1.45mm_HandSolder, F.Cu at (145.9, 125.0)
- added D1: 10V, Diode_THT:D_DO-41_SOD81_P10.16mm_Horizontal, F.Cu at (168.8, 82.2)
- added D2: SMAJ18A, Diode_SMD:D_SMA, F.Cu at (174.8, 86.7)
- added F2: T3.15A, Fuse:Fuse_Littelfuse_395Series, F.Cu at (178.7, 66.8)
- added G***: LOGO, Custom:LOGONEW, F.Cu at (213.9, 100.8)
- added G***: LOGO, Custom:ClassDSmall, F.Cu at (170.2, 120.3)
- added L1: 6.8uH, Custom:SRP6030WA-6R8M, F.Cu at (159.8, 69.0)
- added Q1: DMP4015SK3, Package_TO_SOT_SMD:TO-252-2, F.Cu at (177.5, 79.9)
- added R22: 10K, Resistor_SMD:R_0603_1608Metric_Pad0.98x0.95mm_HandSolder, F.Cu at (172.5, 73.9)
- added R23: 100k, Resistor_SMD:R_0603_1608Metric_Pad0.98x0.95mm_HandSolder, F.Cu at (43.8, 113.0)
- added R24: 13k7, Resistor_SMD:R_0603_1608Metric_Pad0.98x0.95mm_HandSolder, F.Cu at (43.8, 115.5)
- added R27: 100k, Resistor_SMD:R_0603_1608Metric_Pad0.98x0.95mm_HandSolder, F.Cu at (43.8, 118.0)
- added R28: 10k, Resistor_SMD:R_0603_1608Metric_Pad0.98x0.95mm_HandSolder, F.Cu at (43.8, 120.5)
- added R29: 10k, Resistor_SMD:R_0603_1608Metric_Pad0.98x0.95mm_HandSolder, F.Cu at (66.0, 119.8)
- added R30: 10k, Resistor_SMD:R_0603_1608Metric_Pad0.98x0.95mm_HandSolder, F.Cu at (66.0, 122.3)
- added R31: 10k, Resistor_SMD:R_0603_1608Metric_Pad0.98x0.95mm_HandSolder, F.Cu at (66.0, 124.9)
- added R32: 10k, Resistor_SMD:R_0603_1608Metric_Pad0.98x0.95mm_HandSolder, F.Cu at (33.9, 126.3)
- added R33: 3R3, Resistor_SMD:R_2512_6332Metric_Pad1.40x3.35mm_HandSolder, F.Cu at (85.9, 101.6)
- added R34: 5K6, Resistor_SMD:R_0805_2012Metric_Pad1.20x1.40mm_HandSolder, F.Cu at (145.4, 113.8)
- added R35: 49K9, Resistor_SMD:R_0805_2012Metric_Pad1.20x1.40mm_HandSolder, F.Cu at (145.4, 120.5)
- added R36: 4k7, Resistor_SMD:R_0805_2012Metric_Pad1.20x1.40mm_HandSolder, F.Cu at (77.8, 107.3)
- added TP1: PVDD, TestPoint:TestPoint_Pad_D1.5mm, F.Cu at (33.5, 107.3)
- added TP2: 5V, TestPoint:TestPoint_Pad_D1.5mm, F.Cu at (33.5, 110.9)
- added TP3: 3V3, TestPoint:TestPoint_Pad_D1.5mm, F.Cu at (33.5, 114.4)
- added TP4: GND, TestPoint:TestPoint_Pad_D1.5mm, F.Cu at (33.5, 118.0)
- added U3: LMR51430XFDDCR, Package_TO_SOT_SMD:TSOT-23-6, F.Cu at (152.9, 69.0)
- added U4: TLV1117LV33DCYR, Package_TO_SOT_SMD:SOT-223-3_TabPin2, F.Cu at (50.9, 114.2)
- C40, C41, C42, C43: footprint Capacitor_SMD:C_1206_3216Metric_Pad1.33x1.80mm_HandSolder -> Capacitor_SMD:C_0603_1608Metric_Pad1.08x0.95mm_HandSolder
- J1: value LINE IN -> DC IN 12-16V; footprint Connector_JST:JST_XH_B2B-XH-A_1x02_P2.50mm_Vertical -> Connector_Molex:Molex_KK-396_A-41791-0002_1x02_P3.96mm_Vertical
- J16: value OUT L -> - OUT R +
- J17: value OUT R -> - OUT L +
- U1: value TPA3220DDWR -> TPA3220
- moved IC1 129.3 mm to (126.9, 75.0)
- moved C7 116.0 mm to (113.5, 109.6), turned to -90 degrees
- moved C2 112.9 mm to (133.8, 115.7)
- moved C6 112.9 mm to (133.8, 130.2)
- moved C1 112.9 mm to (133.8, 109.6)
- moved C5 112.9 mm to (133.8, 124.1)
- moved C23 111.4 mm to (112.1, 119.3), turned to 180 degrees
- moved IC4 110.7 mm to (120.6, 109.7)
- moved C20 110.1 mm to (111.9, 127.8), turned to -90 degrees
- moved U2 109.2 mm to (119.4, 121.4), turned to 180 degrees
- moved C17 102.3 mm to (114.2, 127.2), turned to -90 degrees
- moved C10 100.5 mm to (128.1, 109.0), turned to -90 degrees
- moved C15 99.9 mm to (116.6, 129.9), turned to -90 degrees
- moved C8 99.5 mm to (117.2, 110.4), turned to -90 degrees
- moved C13 98.0 mm to (124.3, 129.9), turned to -90 degrees
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Connections:
- C1 pad 1: /AMP/IN1-P -> /AMP/IN2-P
- C16 pad 1: /DAC/OUT-L-DAC -> /AMP/IN1-P
- C19 pad 1: /DAC/OUT-R-DAC -> /AMP/IN2-P
- C2 pad 1: /AMP/IN1-M -> GND
- C3 pad 1: /ESP32/3V3-ESP -> GND
- C3 pad 2: unconnected-(C3-Pad2) -> /ESP32/3V3-ESP
- C5 pad 1: /AMP/IN2-P -> /AMP/IN1-P
- C6 pad 1: /AMP/IN2-M -> GND
- IC1 pad 12: /ESP32/SDZ -> /AMP_RESET_N
- IC1 pad 27: unconnected-(IC1-IO16-Pad27) -> Net-(IC1-IO16)
- IC1 pad 33: /ESP32/SDA -> /DAC/SDA
- IC1 pad 36: /ESP32/SCL -> /DAC/SCL
- IC1 pad 4: unconnected-(IC1-SENSOR_VP-Pad4) -> /ESP32/VIN_SENSE
- IC1 pad 6: /ESP32/FAULT -> /AMP_FAULT_N
- IC1 pad 7: unconnected-(IC1-IO35-Pad7) -> /AMP_OTW_N
- IC1 pad 9: unconnected-(IC1-IO33-Pad9) -> /DAC/DAC_XSMT
- R1 pad 1: /DAC/ESP5V -> /DAC/5V
- R10 pad 1: /ESP32/BCK -> /DAC/BCK
- R11 pad 1: /ESP32/DATA -> /DAC/DATA
- R2 pad 2: /DAC/OUT-L-DAC -> /AMP/IN1-P
- R3 pad 1: /DAC/OUT-R-DAC -> /AMP/IN2-P
- R6 pad 2: /ESP32/SCL -> /DAC/SCL
- R7 pad 2: /ESP32/SDA -> /DAC/SDA
- R9 pad 1: /ESP32/LRCK -> /DAC/LRCK
- U1 pad 1: unconnected-(U1-VDD-Pad1) -> /AMP/PVDD
- U1 pad 10: unconnected-(U1-RESET_N-Pad10) -> /AMP_RESET_N
- U1 pad 11: unconnected-(U1-HEAD-Pad11) -> GND
- U1 pad 14: unconnected-(U1-FREQ_ADJ-Pad14) -> Net-(U1-FREQ_ADJ)
- U1 pad 17: unconnected-(U1-CMUTE_N-Pad17) -> Net-(U1-CMUTE_N)
- U1 pad 2: unconnected-(U1-GAIN_SLV-Pad2) -> Net-(U1-GAIN_SLV)
- U1 pad 21: unconnected-(U1-AVDD-Pad21) -> /AMP/AMP_AVDD
- U1 pad 22: unconnected-(U1-GVDD-Pad22) -> /AMP/AMP_GVDD
- U1 pad 3: unconnected-(U1-OTW_CLIP_N-Pad3) -> /AMP_OTW_N
- U1 pad 4: unconnected-(U1-FAULT_N-Pad4) -> /AMP_FAULT_N
- U2 pad 10: unconnected-(U2-VCOM/DEMP-Pad10) -> GND
- U2 pad 22: /DAC/DOUT -> /DAC/DATA
- U2 pad 25: /DAC/AVDD -> /DAC/DAC_XSMT
Routing:
- net /DAC/AVDD: track 0.00 -> 64.4 mm, vias 0 -> 4
- net /AMP/IN2-P: track 0.00 -> 17.3 mm
- net Net-(U1-IN1_P): track 0.00 -> 14.5 mm
- net Net-(U1-IN2_M): track 0.00 -> 13.9 mm
- net Net-(U1-OUT1_M): track 0.00 -> 12.4 mm, vias 0 -> 2
- net Net-(U1-OUT2_P): track 0.00 -> 12.0 mm, vias 0 -> 2
- net Net-(U1-IN1_M): track 0.00 -> 11.0 mm
- net Net-(U1-IN2_P): track 0.00 -> 10.8 mm
- net Net-(IC4-EN): track 0.00 -> 9.63 mm
- net Net-(D1-A): track 0.00 -> 9.27 mm
- net /AMP/IN1-P: track 0.00 -> 8.43 mm
- net Net-(U2-LDOO): track 0.00 -> 8.40 mm
- net Net-(U2-VNEG): track 0.00 -> 7.61 mm
- net Net-(U1-BST1_M): track 0.00 -> 5.83 mm
- net Net-(U1-BST2_P): track 0.00 -> 5.80 mm
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- added copper zone on F.Cu, net /AMP/PVDD
- added copper zone on In2.Cu, net /AMP/PVDD
- added copper zone on F.Cu, net Net-(C24-Pad2)
- added copper zone on F.Cu, net Net-(C27-Pad2)
- added copper zone on F.Cu, net Net-(J1-Pin_1)
- added copper zone on F.Cu, net Net-(J16-Pin_1)
- added copper zone on F.Cu, net Net-(J16-Pin_2)
- added copper zone on F.Cu, net Net-(J17-Pin_1)
- added copper zone on F.Cu, net Net-(J17-Pin_2)
- added copper zone on F.Cu, net Net-(Q1-D)
- added copper zone on F.Cu, net Net-(U1-OUT1_M)
- added copper zone on F.Cu, net Net-(U1-OUT2_P)
Other:
- board size 100 x 100 mm -> 92.8 x 86.4 mm
- board text added: "+ -"
- board text added: "ESP32 / PCM5122 / TDA3220 Portable Amp Tom Watson Audio 2026"
