File: TPA3220/TPA3220.kicad_sch (KiCad schematic)
At the start: 4 parts

Commit message: more
Other:
- added sheet POWER (Power.kicad_sch)
- sheet AMP ports: added AMP_FAULT_N, AMP_OTW_N, AMP_RESET_N, IN1-M, IN1-P, IN2-M, IN2-P, PVDD; removed none
- sheet DAC ports: added 5V, DAC_XSMT, OUT-L-DAC, OUT-R-DAC, SCL, SDA; removed none
- sheet ESP32 ports: added 3V3-ESP, AMP_FAULT_N, AMP_OTW_N, AMP_RESET_N, DAC_XSMT, VIN_SENSE; removed FAULT, SDZ
- note added: "POWER TREE (12-16 V DC in, J1 on POWER sheet) VIN -> F1 5 A T -> Q1 reverse-polarity P-FET -> D2 TVS -> PVDD PVDD -> TPA3220 PVDD + VDD (internal 5 V LDO for AVDD/GVDD) ... up to ~3.5 A peak PVDD -> U3 LMR51430XF buck 5.0 V / 500 kHz FPWM .................... ~0.35 A max 5V -> U4 TLV1117LV33 -> 3V3-ESP (ESP32, pull-ups) ............ 0.15-0.25 A avg, 0.5 A peak 5V -> R1 2R2 -> IC4 TPS7A2033 -> DAC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"
- note added: "TPA3220 ACTIVE SPEAKER - ESP32 / PCM5122 / TPA3220"
