File: DarlingtonAmpDual/DarlingtonAmpDual.kicad_pcb (KiCad board)
At the start: 2 copper layers, 81.2 x 98.9 mm, 54 parts, among them J2 IN, J4 OUT, J5 VEE, J6 VCC, J7 GND, Q1 2SC2240, Q10 2SC4793, Q11 2SD2390, Q12 2SB1560, Q13 2SD2390, Q14 2SB1560, Q2 2SC2240, Q3 2SA970, Q4 2SA970, Q5 2SC2240, Q6 2SC2240, Q7 2SC2240, Q8 2SA1837, Q9 BD139

Commit message: work
Routing:
- net /DRIVE_P: track 101.8 -> 98.2 mm
- net /DRIVE_N: track 86.7 -> 84.5 mm
- added copper zone on F.Cu, net /+35V
- added copper zone on B.Cu, net Net-(Q11-E)
- added copper zone on B.Cu, net Net-(Q12-E)
- added copper zone on B.Cu, net Net-(Q13-E)
- added copper zone on B.Cu, net Net-(Q14-E)
- removed copper zone on B.Cu, net /+35V
- removed copper zone on F.Cu, net /AMP_OUT
- removed copper zone on F.Cu, net Net-(Q11-E)
- removed copper zone on F.Cu, net Net-(Q12-E)
- removed copper zone on F.Cu, net Net-(Q13-E)
- removed copper zone on F.Cu, net Net-(Q14-E)

Commit message: more
Parts:
- moved J5 1.32 mm to (191.8, 82.2)

Commit message: more work
Other:
- board text added: "Darlington Transistor Discrete Amplifier ±35V - Tom Watson Audio - 2026"
- board text removed: "Darlington Discrete Amplifier ±35V - Tom Watson Audio - 2026"
Changed lines of the file:
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@@
 		)
 	)
-	(gr_text "Darlington Discrete Amplifier\n±35V - Tom Watson Audio - 2026"
+	(gr_text "Darlington Transistor Discrete Amplifier\n±35V - Tom Watson Audio - 2026"
 		(at 201.295 113.411 0)
 		(layer "F.SilkS")
