File: SubAmp/SubAmp.kicad_pcb (KiCad board)
At the start: 2 copper layers, 187.3 x 64.8 mm, 41 parts, among them J1 OUT, J2 VCC, J3 VEE, J6 IN, Q1 MPSA42, Q10 2SA1943, Q11 2SC5200, Q12 2SA1943, Q2 MPSA42, Q3 MPSA42, Q4 MJE15033, Q5 MJE15032, Q6 MJE15033, Q7 2SA1943, Q8 2SC5200, Q9 2SC5200

Commit message: more
Parts:
- added C10: 100nF, Capacitor_THT:C_Rect_L7.0mm_W2.5mm_P5.00mm, F.Cu at (16.8, 85.6)
- added C11: 100nF, Capacitor_THT:C_Rect_L7.0mm_W2.5mm_P5.00mm, F.Cu at (56.1, 107.7)
- added C12: 100uF, Capacitor_THT:CP_Radial_D8.0mm_P2.50mm, F.Cu at (144.8, 97.7)
- added C13: 100uF, Capacitor_THT:CP_Radial_D8.0mm_P2.50mm, F.Cu at (144.8, 126.9)
- added C2: 220pF, Capacitor_SMD:C_0805_2012Metric_Pad1.18x1.45mm_HandSolder, F.Cu at (22.4, 123.7)
- added C3: 220pF, Capacitor_SMD:C_0805_2012Metric_Pad1.18x1.45mm_HandSolder, F.Cu at (55.6, 125.5)
- added C6: 220pF, Capacitor_SMD:C_0805_2012Metric_Pad1.18x1.45mm_HandSolder, F.Cu at (55.6, 87.9)
- added C8: 100nF, Capacitor_SMD:C_1206_3216Metric_Pad1.33x1.80mm_HandSolder, F.Cu at (180.3, 121.2)
- added C9: 100nF, Capacitor_SMD:C_1206_3216Metric_Pad1.33x1.80mm_HandSolder, F.Cu at (180.3, 101.3)
- added G***: LOGO, Custom:LOGONEW, F.Cu at (135.9, 110.5)
- added J4: GND, Spade connector:TE_62409-1, F.Cu at (180.3, 111.3)
- added R2: 22K, Resistor_THT:R_Axial_DIN0207_L6.3mm_D2.5mm_P10.16mm_Horizontal, F.Cu at (18.8, 89.9)
- added R23: 10R, Resistor_THT:R_Axial_DIN0614_L14.3mm_D5.7mm_P15.24mm_Horizontal, F.Cu at (32.5, 80.0)
- added R8: 22K, Resistor_THT:R_Axial_DIN0207_L6.3mm_D2.5mm_P10.16mm_Horizontal, F.Cu at (20.3, 112.8)
- C1: value 2.2uF -> 10uF; footprint Capacitor_THT:C_Rect_L7.5mm_W6.5mm_P5.00mm -> Capacitor_THT:C_Radial_D8.0mm_H11.5mm_P3.50mm
- R16, R17: value 3R3 -> 3R9
- moved D1 302.4 mm to (25.1, 94.2), turned to -90 degrees
- moved C1 298.9 mm to (28.2, 137.2), turned to 180 degrees
- moved J6 293.4 mm to (36.1, 137.2)
- moved D2 275.1 mm to (51.1, 106.7), turned to -90 degrees
- moved D3 274.6 mm to (51.1, 93.5), turned to -90 degrees
- moved Q2 270.4 mm to (25.9, 115.3), turned to 90 degrees
- moved Q1 270.4 mm to (25.9, 107.7), turned to 90 degrees
- moved C4 267.6 mm to (38.9, 84.6)
- moved Q5 267.5 mm to (51.1, 139.3), turned to 90 degrees
- moved Q4 266.6 mm to (51.1, 127.0), turned to 90 degrees
- moved Q6 264.9 mm to (51.1, 88.9), turned to 90 degrees
- moved Q3 262.8 mm to (33.3, 115.3), turned to 90 degrees
- moved C5 238.6 mm to (67.8, 111.3), turned to 180 degrees
- moved R1 229.4 mm to (26.9, 128.5), turned to 90 degrees
- moved R3 225.5 mm to (30.2, 128.5), turned to 90 degrees
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Connections:
- net Net-(D1-K) renamed /VEE
- net Net-(Q11-C) renamed /VCC
- J6 pad 1: unconnected-(J6-Pin_1-Pad1) -> SGND
- R9 pad 2: GND -> SGND
Routing:
- net Net-(Q10-B): track 0.00 -> 135.1 mm
- net Net-(Q11-B): track 0.00 -> 134.8 mm
- net /VEE: track 0.00 -> 133.2 mm
- net /VCC: track 0.00 -> 121.8 mm
- net Net-(Q6-C): track 0.00 -> 58.2 mm
- net Net-(Q5-C): track 0.00 -> 51.1 mm
- net Net-(D2-A): track 0.00 -> 48.4 mm
- net Net-(C2-Pad1): track 0.00 -> 41.7 mm
- net Net-(D3-K): track 0.00 -> 36.7 mm
- net Net-(Q3-B): track 0.00 -> 36.5 mm
- net Net-(Q2-C): track 0.00 -> 36.3 mm
- net Net-(C5-Pad2): track 0.00 -> 36.2 mm
- net Net-(C5-Pad1): track 0.00 -> 33.6 mm
- net Net-(Q1-C): track 0.00 -> 21.0 mm
- net Net-(J6-Pin_2): track 0.00 -> 14.6 mm
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- added copper zone on F.Cu, net GND
- added copper zone on F.Cu, net SGND
Other:
- board size 187.3 x 64.8 mm -> 170.4 x 67 mm
- board text added: "- +"
- board text added: "300W Subwoofer Amplifier ±56V Max"

Commit message: commit
Changed lines of the file:
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@@
 		(polygon
 			(pts
-				(xy 129.2098 133.7056) (xy 130.3782 132.4356) (xy 131.953 133.8834) (xy 147.291778 134.1882) (xy 149.86 136.2202)
-				(xy 161.544 136.2202) (xy 161.544 134.1882) (xy 183.642 134.1882) (xy 183.642 129.6162) (xy 161.544 129.6162)
+				(xy 129.2098 133.7056) (xy 130.3782 132.4356) (xy 131.953 133.8834) (xy 147.291778 134.1882) (xy 149.86 139.065)
+				(xy 161.544 139.065) (xy 161.544 134.1882) (xy 183.642 134.1882) (xy 183.642 129.6162) (xy 161.544 129.6162)
 				(xy 161.544 125.8062) (xy 140.716 125.8062) (xy 140.716 130.3274) (xy 131.064 130.3274) (xy 130.302 130.6322)
 				(xy 127.4826 131.2164)
@@
 		(polygon
 			(pts
-				(xy 132.1308 90.1446) (xy 130.937 91.186) (xy 131.1148 91.9226) (xy 149.900956 92.118904) (xy 149.900956 94.150904)
-				(xy 161.584956 94.150904) (xy 161.584956 92.118904) (xy 183.682956 92.118904) (xy 183.682956 87.546904)
+				(xy 132.1308 90.1446) (xy 130.937 91.186) (xy 131.1148 91.9226) (xy 149.900956 92.118904) (xy 149.900956 96.52)
+				(xy 161.584956 96.52) (xy 161.584956 92.118904) (xy 183.682956 92.118904) (xy 183.682956 87.546904)
 				(xy 161.584956 87.546904) (xy 161.584956 79.622104) (xy 140.756956 79.622104) (xy 140.756956 88.258104)
 				(xy 131.104956 88.4174) (xy 131.1402 88.4428) (xy 129.9972 88.4936)

Commit message: more
Parts:
- moved J3 1.08 mm to (142.8, 84.3)
- moved J1 0.56 mm to (141.2, 111.0)
- moved J2 0.51 mm to (143.0, 134.6)
- moved J4 0.25 mm to (180.1, 111.3)
Routing:
- net Net-(C7-Pad1): track 3.09 -> 0.00 mm
- added copper zone on F.Cu, net Net-(C7-Pad1)

Commit message: more work
Changed lines of the file:
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@@
 		(polygon
 			(pts
-				(xy 183.515 82.804) (xy 171.196 82.804) (xy 171.196 108.204) (xy 175.006 108.204) (xy 175.006 86.106)
+				(xy 183.515 82.804) (xy 171.196 82.804) (xy 171.196 107.1372) (xy 175.006 107.1372) (xy 175.006 86.106)
 				(xy 183.515 86.106)
 			)
@@
 		(polygon
 			(pts
-				(xy 183.515 128.016) (xy 171.196 128.016) (xy 171.196 114.046) (xy 175.006 114.046) (xy 175.006 124.714)
+				(xy 183.515 128.016) (xy 171.196 128.016) (xy 171.196 115.062) (xy 175.006 115.062) (xy 175.006 124.714)
 				(xy 183.515 124.714)
 			)
@@
 		(polygon
 			(pts
-				(xy 163.83 108.966) (xy 163.83 113.284) (xy 175.514 113.284) (xy 175.514 120.65) (xy 184.404 120.65)
-				(xy 184.404 101.854) (xy 175.514 101.854) (xy 175.514 108.966)
-			)
-		)
+				(xy 163.83 107.8992) (xy 163.83 114.3) (xy 175.514 114.3) (xy 175.514 120.65) (xy 184.404 120.65)
+				(xy 184.404 101.854) (xy 175.514 101.854) (xy 175.514 107.8992)
+			)
+		)
