File: SubAmp/SubAmp.kicad_sch (KiCad schematic)
At the start: 41 parts, among them J1 OUT, J2 VCC, J3 VEE, J6 IN, Q1 MPSA42, Q10 2SA1943, Q11 2SC5200, Q12 2SA1943, Q2 MPSA42, Q3 MPSA42, Q4 MJE15033, Q5 MJE15032, Q6 MJE15033, Q7 2SA1943, Q8 2SC5200, Q9 2SC5200

Commit message: more
Parts:
- added C10, C11: 100nF, Capacitor_THT:C_Rect_L7.0mm_W2.5mm_P5.00mm, symbol Device:C
- added C12, C13: 100uF, Capacitor_THT:CP_Radial_D8.0mm_P2.50mm, symbol Device:C_Polarized
- added C2, C3, C6: 220pF, Capacitor_SMD:C_0805_2012Metric_Pad1.18x1.45mm_HandSolder, symbol Device:C
- added C8, C9: 100nF, Capacitor_SMD:C_1206_3216Metric_Pad1.33x1.80mm_HandSolder, symbol Device:C
- added J4: GND, Spade connector:TE_62409-1, symbol Spade connector:62409-1
- added R2, R8: 22K, Resistor_THT:R_Axial_DIN0207_L6.3mm_D2.5mm_P10.16mm_Horizontal, symbol Device:R
- added R23: 10R, Resistor_THT:R_Axial_DIN0614_L14.3mm_D5.7mm_P15.24mm_Horizontal, symbol Device:R
- C1: value 2.2uF -> 10uF; footprint Capacitor_THT:C_Rect_L7.5mm_W6.5mm_P5.00mm -> Capacitor_THT:C_Radial_D8.0mm_H11.5mm_P3.50mm
- R16, R17: value 3R3 -> 3R9
Connections:
- net GND: now also C10.2, C12.1, C13.2, C8.2, C9.2, J4.1 (P1), J4.2 (P1), R23.1; no longer R9.2
- net VCC: now reaches J2.1 (P1), J2.2 (P1), Q11.2 (C), Q4.3 (E), Q7.3 (E), Q9.2 (C), R13.1, R5.1, R6.1
- net VCC: now also C13.1, C8.1
- net VEE: now reaches D1.1 (K), J3.1 (P1), J3.2 (P1), Q10.2 (C), Q12.2 (C), Q8.3 (E), R11.2, R14.2, R7.2
- net VEE: now also C12.2, C9.1
- net at D1.2 (A), Q1.2 (B): now also R8.2
- net SGND: now reaches J6.1 (Pin_1)
- net SGND: now also R9.2, C10.1, C2.2, R2.1, R23.2, R8.1
- net at D2.2 (A), Q4.2 (C), Q5.1 (B): now also C11.1, C3.2
- net at R1.2, R3.1: now also C2.1, R2.2
- net at Q2.3 (C), Q4.1 (B), R5.2: now also C3.1
- net at Q6.2 (C), Q8.1 (B), R14.1: now also C6.2
- net at D3.1 (K), Q6.1 (B), R10.1: now also C11.2, C6.1

Commit message: more work
Other:
- moved on the sheet: C1, C10, C11, C12, C13, C2, C3, C4, C5, C6, C7, C8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
